File: Register/Registersatz.sch (KiCad schematic (older format))
At the start: 1 part

Commit message: Wiring of Registers to MUX
Connections:
- net labels added: R020, R021, R022, R023, R024, R025, R026, R027
- wire segments 18 -> 88
Other:
- moved on the sheet: REG1
