File: 16-2MUX.sch (KiCad schematic (older format))
At the start: 4 parts

Commit message: SPICE capacitance and ground symbols
Parts:
- removed C? (x2): 100n, symbol C_Small
- added C? (x2): 100nF, symbol C
Connections:
- net labels added: 0
- net labels removed: GND
- wire segments 70 -> 80
Changed lines of the file:
@@
 EESchema Schematic File Version 2
-LIBS:power
-LIBS:device
-LIBS:transistors
-LIBS:conn
-LIBS:linear
-LIBS:regul
-LIBS:74xx
-LIBS:cmos4000
-LIBS:adc-dac
-LIBS:memory
-LIBS:xilinx
-LIBS:microcontrollers
-LIBS:dsp
-LIBS:microchip
-LIBS:analog_switches
-LIBS:motorola
-LIBS:texas
-LIBS:intel
-LIBS:audio
-LIBS:interface
-LIBS:digital-audio
-LIBS:philips
-LIBS:display
-LIBS:cypress
-LIBS:siliconi
-LIBS:opto
-LIBS:atmel
-LIBS:contrib
-LIBS:valves
+LIBS:spice
+LIBS:pspice
 LIBS:myCpu-cache
 EELAYER 25 0
@@
 Comment4 ""
 $EndDescr
-$Comp
-L C_Small C?
-U 1 1 5AE9E181
-P 1400 5175
-F 0 "C?" H 1410 5245 50  0000 L CNN
-F 1 "100n" H 1410 5095 50  0000 L CNN
-F 2 "" H 1400 5175 50  0000 C CNN
-F 3 "" H 1400 5175 50  0000 C CNN
-	1    1400 5175
-	1    0    0    -1
-$EndComp
-$Comp
-L C_Small C?
-U 1 1 5AE9E21C
-P 5225 5150
-F 0 "C?" H 5235 5220 50  0000 L CNN
-F 1 "100n" H 5235 5070 50  0000 L CNN
-F 2 "" H 5225 5150 50  0000 C CNN
-F 3 "" H 5225 5150 50  0000 C CNN
-	1    5225 5150
-	1    0    0    -1
-$EndComp
 $Comp
 L 74LS151 U?
@@
 	4250 6750 4250 5975
 $Comp
-L GND #PWR?
-U 1 1 5AE9E85C
-P 5225 4775
-F 0 "#PWR?" H 5225 4525 50  0001 C CNN
-F 1 "GND" H 5225 4625 50  0000 C CNN
-F 2 "" H 5225 4775 50  0000 C CNN
-F 3 "" H 5225 4775 50  0000 C CNN
-	1    5225 4775
-	1    0    0    -1
-$EndComp
-$Comp
-L GND #PWR?
-U 1 1 5AE9E87C
-P 1600 4825
-F 0 "#PWR?" H 1600 4575 50  0001 C CNN
-F 1 "GND" H 1600 4675 50  0000 C CNN
-F 2 "" H 1600 4825 50  0000 C CNN
-F 3 "" H 1600 4825 50  0000 C CNN
-	1    1600 4825
-	1    0    0    -1
-$EndComp
-$Comp
 L VCC #PWR?
 U 1 1 5AE9E89C
-P 1425 5475
-F 0 "#PWR?" H 1425 5325 50  0001 C CNN
-F 1 "VCC" H 1425 5625 50  0000 C CNN
-F 2 "" H 1425 5475 50  0000 C CNN
-F 3 "" H 1425 5475 50  0000 C CNN
-	1    1425 5475
+P 1200 5675
+F 0 "#PWR?" H 1200 5525 50  0001 C CNN
+F 1 "VCC" H 1200 5825 50  0000 C CNN
+F 2 "" H 1200 5675 50  0000 C CNN
+F 3 "" H 1200 5675 50  0000 C CNN
+	1    1200 5675
 	1    0    0    -1
 $EndComp
@@
 Wire Wire Line
 	5100 5250 5225 5250
-Wire Wire Line
-	5225 4775 5225 5050
-Wire Wire Line
-	1425 5475 1425 5275
-Wire Wire Line
-	1425 5275 1400 5275
-Wire Wire Line
-	1400 5075 1600 5075
-Wire Wire Line
-	1600 4825 1600 5325
 Text HLabel 2775 7375 3    60   Input ~ 0
 S1
@@
 S3
 Wire Wire Line
-	2875 5925 2875 7175
+	2875 5925 2875 7125
+Wire Wire Line
+	2875 7125 2875 7175
 Wire Wire Line
 	2875 7175 2775 7175
@@
 	2875 7375 2875 7275
 Wire Wire Line
-	2875 7275 2975 7275
+	2875 7275 2950 7275
+Wire Wire Line
+	2950 7275 2975 7275
 Wire Wire Line
 	2975 7275 2975 5925
@@
 Wire Wire Line
 	5000 5025 5225 5025
+Wire Wire Line
+	5225 5025 5525 5025
 Connection ~ 5225 5025
 Wire Wire Line
@@
 Wire Wire Line
 	3275 5325 1600 5325
-Connection ~ 1600 5075
 Text HLabel 2150 3700 1    60   Output ~ 0
 Z0
@@
 Wire Wire Line
 	3700 3700 3700 4575
+$Comp
+L C C?
+U 1 1 5AEB02AD
+P 5725 5150
+F 0 "C?" V 5575 5150 60  0000 C CNN
+F 1 "100nF" V 5875 5150 60  0000 C CNN
+F 2 "" H 5725 5150 60  0000 C CNN
+F 3 "" H 5725 5150 60  0000 C CNN
+	1    5725 5150
+	1    0    0    -1
+$EndComp
+$Comp
+L 0 #GND?
+U 1 1 5AEB030E
+P 5525 4775
+F 0 "#GND?" H 5525 4675 60  0001 C CNN
+F 1 "0" H 5525 4705 60  0000 C CNN
+F 2 "" H 5525 4775 60  0000 C CNN
+F 3 "" H 5525 4775 60  0000 C CNN
+	1    5525 4775
+	1    0    0    -1
+$EndComp
+Wire Wire Line
+	5225 5250 5225 5425
+Wire Wire Line
+	5225 5425 5725 5425
+Wire Wire Line
+	5725 5425 5725 5400
+Wire Wire Line
+	5525 5025 5525 4775
+Wire Wire Line
+	5525 4775 5725 4775
+Wire Wire Line
+	5725 4775 5725 4900
+$Comp
+L C C?
+U 1 1 5AEB04DC
+P 1225 5250
+F 0 "C?" V 1075 5250 60  0000 C CNN
+F 1 "100nF" V 1375 5250 60  0000 C CNN
+F 2 "" H 1225 5250 60  0000 C CNN
+F 3 "" H 1225 5250 60  0000 C CNN
+	1    1225 5250
+	1    0    0    -1
+$EndComp
+$Comp
+L 0 #GND?
+U 1 1 5AEB056F
+P 1400 5025
+F 0 "#GND?" H 1400 4925 60  0001 C CNN
+F 1 "0" H 1400 4955 60  0000 C CNN
+F 2 "" H 1400 5025 60  0000 C CNN
+F 3 "" H 1400 5025 60  0000 C CNN
+	1    1400 5025
+	1    0    0    -1
+$EndComp
+Wire Wire Line
+	1225 5000 1400 5000
+Wire Wire Line
+	1400 5000 1400 5025
+Wire Wire Line
+	1600 5325 1600 5025
+Wire Wire Line
+	1600 5025 1400 5025
+Wire Wire Line
+	1225 5500 1425 5500
+Wire Wire Line
+	1425 5500 1200 5675
 $EndSCHEMATC

Commit message: fixed duplicate names
Parts:
- gave numbers to parts that had none: 4
Connections:
- wire segments 80 -> 77
Changed lines of the file:
@@
 $EndDescr
 $Comp
-L 74LS151 U?
+L 74LS151 U19
 U 1 1 5AE9E2A5
 P 2625 5225
-F 0 "U?" H 2625 5225 50  0000 C CNN
+AR Path="/5AE62FB7/5AE9DF6E/5AE9E178/5AE9E2A5" Ref="U19"  Part="1"
+AR Path="/5AE62FB7/5AE9DF6E/5AEA87F7/5AE9E2A5" Ref="U21"  Part="1"
+AR Path="/5AE62FB7/5AE9DF6E/5AEB0026/5AE9E2A5" Ref="U23"  Part="1"
+AR Path="/5AE62FB7/5AE9DF6E/5AEB003D/5AE9E2A5" Ref="U25"  Part="1"
+AR Path="/5AE62FB7/5AE9DF6E/5AEC7274/5AE9E2A5" Ref="U27"  Part="1"
+AR Path="/5AE62FB7/5AE9DF6E/5AEC728B/5AE9E2A5" Ref="U29"  Part="1"
+AR Path="/5AE62FB7/5AE9DF6E/5AEC72A2/5AE9E2A5" Ref="U31"  Part="1"
+AR Path="/5AE62FB7/5AE9DF6E/5AEC72B9/5AE9E2A5" Ref="U33"  Part="1"
+F 0 "U33" H 2625 5225 50  0000 C CNN
 F 1 "74LS151" H 2625 5075 50  0000 C CNN
 F 2 "" H 2625 5225 50  0000 C CNN
@@
 $EndComp
 $Comp
-L 74LS151 U?
+L 74LS151 U20
 U 1 1 5AE9E4A8
 P 4200 5275
-F 0 "U?" H 4200 5275 50  0000 C CNN
+AR Path="/5AE62FB7/5AE9DF6E/5AE9E178/5AE9E4A8" Ref="U20"  Part="1"
+AR Path="/5AE62FB7/5AE9DF6E/5AEA87F7/5AE9E4A8" Ref="U22"  Part="1"
+AR Path="/5AE62FB7/5AE9DF6E/5AEB0026/5AE9E4A8" Ref="U24"  Part="1"
+AR Path="/5AE62FB7/5AE9DF6E/5AEB003D/5AE9E4A8" Ref="U26"  Part="1"
+AR Path="/5AE62FB7/5AE9DF6E/5AEC7274/5AE9E4A8" Ref="U28"  Part="1"
+AR Path="/5AE62FB7/5AE9DF6E/5AEC728B/5AE9E4A8" Ref="U30"  Part="1"
+AR Path="/5AE62FB7/5AE9DF6E/5AEC72A2/5AE9E4A8" Ref="U32"  Part="1"
+AR Path="/5AE62FB7/5AE9DF6E/5AEC72B9/5AE9E4A8" Ref="U34"  Part="1"
+F 0 "U34" H 4200 5275 50  0000 C CNN
 F 1 "74LS151" H 4200 5125 50  0000 C CNN
 F 2 "" H 4200 5275 50  0000 C CNN
@@
 	4250 6750 4250 5975
 $Comp
-L VCC #PWR?
+L VCC #PWR019
 U 1 1 5AE9E89C
 P 1200 5675
-F 0 "#PWR?" H 1200 5525 50  0001 C CNN
+AR Path="/5AE62FB7/5AE9DF6E/5AE9E178/5AE9E89C" Ref="#PWR019"  Part="1"
+AR Path="/5AE62FB7/5AE9DF6E/5AEA87F7/5AE9E89C" Ref="#PWR021"  Part="1"
+AR Path="/5AE62FB7/5AE9DF6E/5AEB0026/5AE9E89C" Ref="#PWR023"  Part="1"
+AR Path="/5AE62FB7/5AE9DF6E/5AEB003D/5AE9E89C" Ref="#PWR025"  Part="1"
+AR Path="/5AE62FB7/5AE9DF6E/5AEC7274/5AE9E89C" Ref="#PWR027"  Part="1"
+AR Path="/5AE62FB7/5AE9DF6E/5AEC728B/5AE9E89C" Ref="#PWR029"  Part="1"
+AR Path="/5AE62FB7/5AE9DF6E/5AEC72A2/5AE9E89C" Ref="#PWR031"  Part="1"
+AR Path="/5AE62FB7/5AE9DF6E/5AEC72B9/5AE9E89C" Ref="#PWR033"  Part="1"
+F 0 "#PWR033" H 1200 5525 50  0001 C CNN
 F 1 "VCC" H 1200 5825 50  0000 C CNN
 F 2 "" H 1200 5675 50  0000 C CNN
@@
 $EndComp
 $Comp
-L VCC #PWR?
+L VCC #PWR020
 U 1 1 5AE9E8B8
 P 5275 5850
-F 0 "#PWR?" H 5275 5700 50  0001 C CNN
+AR Path="/5AE62FB7/5AE9DF6E/5AE9E178/5AE9E8B8" Ref="#PWR020"  Part="1"
+AR Path="/5AE62FB7/5AE9DF6E/5AEA87F7/5AE9E8B8" Ref="#PWR022"  Part="1"
+AR Path="/5AE62FB7/5AE9DF6E/5AEB0026/5AE9E8B8" Ref="#PWR024"  Part="1"
+AR Path="/5AE62FB7/5AE9DF6E/5AEB003D/5AE9E8B8" Ref="#PWR026"  Part="1"
+AR Path="/5AE62FB7/5AE9DF6E/5AEC7274/5AE9E8B8" Ref="#PWR028"  Part="1"
+AR Path="/5AE62FB7/5AE9DF6E/5AEC728B/5AE9E8B8" Ref="#PWR030"  Part="1"
+AR Path="/5AE62FB7/5AE9DF6E/5AEC72A2/5AE9E8B8" Ref="#PWR032"  Part="1"
+AR Path="/5AE62FB7/5AE9DF6E/5AEC72B9/5AE9E8B8" Ref="#PWR034"  Part="1"
+F 0 "#PWR034" H 5275 5700 50  0001 C CNN
 F 1 "VCC" H 5275 6000 50  0000 C CNN
 F 2 "" H 5275 5850 50  0000 C CNN
@@
 S3
 Wire Wire Line
-	2875 5925 2875 7125
-Wire Wire Line
-	2875 7125 2875 7175
+	2875 5925 2875 7175
 Wire Wire Line
 	2875 7175 2775 7175
@@
 	2875 7375 2875 7275
 Wire Wire Line
-	2875 7275 2950 7275
-Wire Wire Line
-	2950 7275 2975 7275
+	2875 7275 2975 7275
 Wire Wire Line
 	2975 7275 2975 5925
@@
 	5000 5975 5000 5025
 Wire Wire Line
-	5000 5025 5225 5025
-Wire Wire Line
-	5225 5025 5525 5025
+	5000 5025 5525 5025
 Connection ~ 5225 5025
 Wire Wire Line
@@
 	3700 3700 3700 4575
 $Comp
-L C C?
+L C C18
 U 1 1 5AEB02AD
 P 5725 5150
-F 0 "C?" V 5575 5150 60  0000 C CNN
+AR Path="/5AE62FB7/5AE9DF6E/5AE9E178/5AEB02AD" Ref="C18"  Part="1"
+AR Path="/5AE62FB7/5AE9DF6E/5AEA87F7/5AEB02AD" Ref="C20"  Part="1"
+AR Path="/5AE62FB7/5AE9DF6E/5AEB0026/5AEB02AD" Ref="C22"  Part="1"
+AR Path="/5AE62FB7/5AE9DF6E/5AEB003D/5AEB02AD" Ref="C24"  Part="1"
+AR Path="/5AE62FB7/5AE9DF6E/5AEC7274/5AEB02AD" Ref="C26"  Part="1"
+AR Path="/5AE62FB7/5AE9DF6E/5AEC728B/5AEB02AD" Ref="C28"  Part="1"
+AR Path="/5AE62FB7/5AE9DF6E/5AEC72A2/5AEB02AD" Ref="C30"  Part="1"
+AR Path="/5AE62FB7/5AE9DF6E/5AEC72B9/5AEB02AD" Ref="C32"  Part="1"
+F 0 "C32" V 5575 5150 60  0000 C CNN
 F 1 "100nF" V 5875 5150 60  0000 C CNN
 F 2 "" H 5725 5150 60  0000 C CNN
@@
 $EndComp
 $Comp
-L 0 #GND?
+L 0 #GND20
 U 1 1 5AEB030E
 P 5525 4775
-F 0 "#GND?" H 5525 4675 60  0001 C CNN
+AR Path="/5AE62FB7/5AE9DF6E/5AE9E178/5AEB030E" Ref="#GND20"  Part="1"
+AR Path="/5AE62FB7/5AE9DF6E/5AEA87F7/5AEB030E" Ref="#GND22"  Part="1"
+AR Path="/5AE62FB7/5AE9DF6E/5AEB0026/5AEB030E" Ref="#GND24"  Part="1"
+AR Path="/5AE62FB7/5AE9DF6E/5AEB003D/5AEB030E" Ref="#GND26"  Part="1"
+AR Path="/5AE62FB7/5AE9DF6E/5AEC7274/5AEB030E" Ref="#GND28"  Part="1"
+AR Path="/5AE62FB7/5AE9DF6E/5AEC728B/5AEB030E" Ref="#GND30"  Part="1"
+AR Path="/5AE62FB7/5AE9DF6E/5AEC72A2/5AEB030E" Ref="#GND32"  Part="1"
+AR Path="/5AE62FB7/5AE9DF6E/5AEC72B9/5AEB030E" Ref="#GND34"  Part="1"
+F 0 "#GND34" H 5525 4675 60  0001 C CNN
 F 1 "0" H 5525 4705 60  0000 C CNN
 F 2 "" H 5525 4775 60  0000 C CNN
@@
 	5725 4775 5725 4900
 $Comp
-L C C?
+L C C17
 U 1 1 5AEB04DC
 P 1225 5250
-F 0 "C?" V 1075 5250 60  0000 C CNN
+AR Path="/5AE62FB7/5AE9DF6E/5AE9E178/5AEB04DC" Ref="C17"  Part="1"
+AR Path="/5AE62FB7/5AE9DF6E/5AEA87F7/5AEB04DC" Ref="C19"  Part="1"
+AR Path="/5AE62FB7/5AE9DF6E/5AEB0026/5AEB04DC" Ref="C21"  Part="1"
+AR Path="/5AE62FB7/5AE9DF6E/5AEB003D/5AEB04DC" Ref="C23"  Part="1"
+AR Path="/5AE62FB7/5AE9DF6E/5AEC7274/5AEB04DC" Ref="C25"  Part="1"
+AR Path="/5AE62FB7/5AE9DF6E/5AEC728B/5AEB04DC" Ref="C27"  Part="1"
+AR Path="/5AE62FB7/5AE9DF6E/5AEC72A2/5AEB04DC" Ref="C29"  Part="1"
+AR Path="/5AE62FB7/5AE9DF6E/5AEC72B9/5AEB04DC" Ref="C31"  Part="1"
+F 0 "C31" V 1075 5250 60  0000 C CNN
 F 1 "100nF" V 1375 5250 60  0000 C CNN
 F 2 "" H 1225 5250 60  0000 C CNN
@@
 $EndComp
 $Comp
-L 0 #GND?
+L 0 #GND19
 U 1 1 5AEB056F
 P 1400 5025
-F 0 "#GND?" H 1400 4925 60  0001 C CNN
+AR Path="/5AE62FB7/5AE9DF6E/5AE9E178/5AEB056F" Ref="#GND19"  Part="1"
+AR Path="/5AE62FB7/5AE9DF6E/5AEA87F7/5AEB056F" Ref="#GND21"  Part="1"
+AR Path="/5AE62FB7/5AE9DF6E/5AEB0026/5AEB056F" Ref="#GND23"  Part="1"
+AR Path="/5AE62FB7/5AE9DF6E/5AEB003D/5AEB056F" Ref="#GND25"  Part="1"
+AR Path="/5AE62FB7/5AE9DF6E/5AEC7274/5AEB056F" Ref="#GND27"  Part="1"
+AR Path="/5AE62FB7/5AE9DF6E/5AEC728B/5AEB056F" Ref="#GND29"  Part="1"
+AR Path="/5AE62FB7/5AE9DF6E/5AEC72A2/5AEB056F" Ref="#GND31"  Part="1"
+AR Path="/5AE62FB7/5AE9DF6E/5AEC72B9/5AEB056F" Ref="#GND33"  Part="1"
+F 0 "#GND33" H 1400 4925 60  0001 C CNN
 F 1 "0" H 1400 4955 60  0000 C CNN
 F 2 "" H 1400 5025 60  0000 C CNN

Commit message: NC-symbols
Connections:
- no-connect marks 0 -> 2
Changed lines of the file:
@@
 $Descr A4 11693 8268
 encoding utf-8
-Sheet 12 21
+Sheet 13 21
 Title ""
 Date ""
@@
 AR Path="/5AE62FB7/5AE9DF6E/5AEC72A2/5AE9E2A5" Ref="U31"  Part="1"
 AR Path="/5AE62FB7/5AE9DF6E/5AEC72B9/5AE9E2A5" Ref="U33"  Part="1"
-F 0 "U33" H 2625 5225 50  0000 C CNN
+F 0 "U21" H 2625 5225 50  0000 C CNN
 F 1 "74LS151" H 2625 5075 50  0000 C CNN
 F 2 "" H 2625 5225 50  0000 C CNN
@@
 AR Path="/5AE62FB7/5AE9DF6E/5AEC72A2/5AE9E4A8" Ref="U32"  Part="1"
 AR Path="/5AE62FB7/5AE9DF6E/5AEC72B9/5AE9E4A8" Ref="U34"  Part="1"
-F 0 "U34" H 4200 5275 50  0000 C CNN
+F 0 "U22" H 4200 5275 50  0000 C CNN
 F 1 "74LS151" H 4200 5125 50  0000 C CNN
 F 2 "" H 4200 5275 50  0000 C CNN
@@
 AR Path="/5AE62FB7/5AE9DF6E/5AEC72A2/5AE9E89C" Ref="#PWR031"  Part="1"
 AR Path="/5AE62FB7/5AE9DF6E/5AEC72B9/5AE9E89C" Ref="#PWR033"  Part="1"
-F 0 "#PWR033" H 1200 5525 50  0001 C CNN
+F 0 "#PWR021" H 1200 5525 50  0001 C CNN
 F 1 "VCC" H 1200 5825 50  0000 C CNN
 F 2 "" H 1200 5675 50  0000 C CNN
@@
 AR Path="/5AE62FB7/5AE9DF6E/5AEC72A2/5AE9E8B8" Ref="#PWR032"  Part="1"
 AR Path="/5AE62FB7/5AE9DF6E/5AEC72B9/5AE9E8B8" Ref="#PWR034"  Part="1"
-F 0 "#PWR034" H 5275 5700 50  0001 C CNN
+F 0 "#PWR022" H 5275 5700 50  0001 C CNN
 F 1 "VCC" H 5275 6000 50  0000 C CNN
 F 2 "" H 5275 5850 50  0000 C CNN
@@
 AR Path="/5AE62FB7/5AE9DF6E/5AEC72A2/5AEB02AD" Ref="C30"  Part="1"
 AR Path="/5AE62FB7/5AE9DF6E/5AEC72B9/5AEB02AD" Ref="C32"  Part="1"
-F 0 "C32" V 5575 5150 60  0000 C CNN
+F 0 "C20" V 5575 5150 60  0000 C CNN
 F 1 "100nF" V 5875 5150 60  0000 C CNN
 F 2 "" H 5725 5150 60  0000 C CNN
@@
 AR Path="/5AE62FB7/5AE9DF6E/5AEC72A2/5AEB030E" Ref="#GND32"  Part="1"
 AR Path="/5AE62FB7/5AE9DF6E/5AEC72B9/5AEB030E" Ref="#GND34"  Part="1"
-F 0 "#GND34" H 5525 4675 60  0001 C CNN
+F 0 "#GND22" H 5525 4675 60  0001 C CNN
 F 1 "0" H 5525 4705 60  0000 C CNN
 F 2 "" H 5525 4775 60  0000 C CNN
@@
 AR Path="/5AE62FB7/5AE9DF6E/5AEC72A2/5AEB04DC" Ref="C29"  Part="1"
 AR Path="/5AE62FB7/5AE9DF6E/5AEC72B9/5AEB04DC" Ref="C31"  Part="1"
-F 0 "C31" V 1075 5250 60  0000 C CNN
+F 0 "C19" V 1075 5250 60  0000 C CNN
 F 1 "100nF" V 1375 5250 60  0000 C CNN
 F 2 "" H 1225 5250 60  0000 C CNN
@@
 AR Path="/5AE62FB7/5AE9DF6E/5AEC72A2/5AEB056F" Ref="#GND31"  Part="1"
 AR Path="/5AE62FB7/5AE9DF6E/5AEC72B9/5AEB056F" Ref="#GND33"  Part="1"
-F 0 "#GND33" H 1400 4925 60  0001 C CNN
+F 0 "#GND21" H 1400 4925 60  0001 C CNN
 F 1 "0" H 1400 4955 60  0000 C CNN
 F 2 "" H 1400 5025 60  0000 C CNN
@@
 Wire Wire Line
 	1425 5500 1200 5675
+NoConn ~ 2225 4525
+NoConn ~ 3800 4575
 $EndSCHEMATC

Commit message: spice libs from the internet, opened with new kicad 5.0.0, added spice models to components
Parts:
- C17, C18: symbol C -> spice:C
- U19, U20: symbol 74LS151 -> myCpu-rescue:74LS151; Spice_Lib_File (none) -> 74hc.lib; Spice_Model (none) -> 74HC151; Spice_Netlist_Enabled (none) -> Y; Spice_Primitive (none) -> X
Changed lines of the file:
@@
-EESchema Schematic File Version 2
-LIBS:spice
-LIBS:pspice
+EESchema Schematic File Version 4
 LIBS:myCpu-cache
-EELAYER 25 0
+EELAYER 26 0
 EELAYER END
 $Descr A4 11693 8268
@@
 $EndDescr
 $Comp
-L 74LS151 U19
+L myCpu-rescue:74LS151 U19
 U 1 1 5AE9E2A5
 P 2625 5225
@@
 F 2 "" H 2625 5225 50  0000 C CNN
 F 3 "" H 2625 5225 50  0000 C CNN
+F 4 "X" H 2625 5225 50  0001 C CNN "Spice_Primitive"
+F 5 "74HC151" H 2625 5225 50  0001 C CNN "Spice_Model"
+F 6 "Y" H 2625 5225 50  0001 C CNN "Spice_Netlist_Enabled"
+F 7 "74hc.lib" H 2625 5225 50  0001 C CNN "Spice_Lib_File"
 	1    2625 5225
 	0    -1   -1   0
 $EndComp
 $Comp
-L 74LS151 U20
+L myCpu-rescue:74LS151 U20
 U 1 1 5AE9E4A8
 P 4200 5275
@@
 F 2 "" H 4200 5275 50  0000 C CNN
 F 3 "" H 4200 5275 50  0000 C CNN
+F 4 "X" H 4200 5275 50  0001 C CNN "Spice_Primitive"
+F 5 "74HC151" H 4200 5275 50  0001 C CNN "Spice_Model"
+F 6 "Y" H 4200 5275 50  0001 C CNN "Spice_Netlist_Enabled"
+F 7 "74hc.lib" H 4200 5275 50  0001 C CNN "Spice_Lib_File"
 	1    4200 5275
 	0    -1   -1   0
@@
 	4250 6750 4250 5975
 $Comp
-L VCC #PWR019
+L myCpu-rescue:VCC #PWR019
 U 1 1 5AE9E89C
 P 1200 5675
@@
 $EndComp
 $Comp
-L VCC #PWR020
+L myCpu-rescue:VCC #PWR020
 U 1 1 5AE9E8B8
 P 5275 5850
@@
 S3
 Wire Wire Line
-	2875 5925 2875 7175
+	2875 5925 2875 7125
 Wire Wire Line
 	2875 7175 2775 7175
@@
 Wire Wire Line
 	2875 7375 2875 7275
-Wire Wire Line
-	2875 7275 2975 7275
 Wire Wire Line
 	2975 7275 2975 5925
@@
 Wire Wire Line
 	4550 5975 4550 7275
-Wire Wire Line
-	4550 7275 2950 7275
 Connection ~ 2950 7275
-Connection ~ 3075 7375
 Wire Wire Line
 	4650 5975 4650 7375
 Wire Wire Line
 	4650 7375 4625 7375
-Connection ~ 4625 7375
 Wire Wire Line
 	4850 5975 5000 5975
 Wire Wire Line
 	5000 5975 5000 5025
-Wire Wire Line
-	5000 5025 5525 5025
-Connection ~ 5225 5025
 Wire Wire Line
 	3275 5925 3275 5325
@@
 	3700 3700 3700 4575
 $Comp
-L C C18
+L spice:C C18
 U 1 1 5AEB02AD
 P 5725 5150
@@
 $EndComp
 $Comp
-L 0 #GND20
+L spice:0 #GND20
 U 1 1 5AEB030E
 P 5525 4775
@@
 	5725 4775 5725 4900
 $Comp
-L C C17
+L spice:C C17
 U 1 1 5AEB04DC
 P 1225 5250
@@
 $EndComp
 $Comp
-L 0 #GND19
+L spice:0 #GND19
 U 1 1 5AEB056F
 P 1400 5025
@@
 NoConn ~ 2225 4525
 NoConn ~ 3800 4575
+Wire Wire Line
+	2875 7125 2875 7175
+Wire Wire Line
+	5000 5025 5525 5025
+Wire Wire Line
+	2875 7275 4550 7275
 $EndSCHEMATC

Commit message: lots of work done
Parts:
- renumbered C17 to C18, C18 to C19, U19 to U20, U20 to U21

Commit message: b
Parts:
- renumbered C18 to C20, C19 to C21, U20 to U22, U21 to U23
