File: 16-2MUX.sch (KiCad schematic (older format))
At the start: 4 parts, among them U22 74LS151, U23 74LS151

Commit message: tst
Connections:
- wire segments 77 -> 79
Changed lines of the file:
@@
 AR Path="/5B1119BA/5C00E21C/5AEC72A2/5AE9E2A5" Ref="U145"  Part="1"
 AR Path="/5B1119BA/5C00E21C/5AEC72B9/5AE9E2A5" Ref="U147"  Part="1"
-F 0 "U147" H 2625 5225 50  0000 C CNN
+F 0 "U22" H 2625 5225 50  0000 C CNN
 F 1 "74LS151" H 2625 5075 50  0000 C CNN
 F 2 "" H 2625 5225 50  0000 C CNN
@@
 AR Path="/5B1119BA/5C00E21C/5AEC72A2/5AE9E4A8" Ref="U146"  Part="1"
 AR Path="/5B1119BA/5C00E21C/5AEC72B9/5AE9E4A8" Ref="U148"  Part="1"
-F 0 "U148" H 4200 5275 50  0000 C CNN
+F 0 "U23" H 4200 5275 50  0000 C CNN
 F 1 "74LS151" H 4200 5125 50  0000 C CNN
 F 2 "" H 4200 5275 50  0000 C CNN
@@
 	2675 5925 2775 5925
 Wire Wire Line
-	2775 5925 2775 6750
-Wire Wire Line
 	3550 5975 3550 6450
 Wire Wire Line
@@
 AR Path="/5B1119BA/5C00E21C/5AEC72A2/5AE9E89C" Ref="#PWR0346"  Part="1"
 AR Path="/5B1119BA/5C00E21C/5AEC72B9/5AE9E89C" Ref="#PWR0348"  Part="1"
-F 0 "#PWR0348" H 1200 5525 50  0001 C CNN
+F 0 "#PWR030" H 1200 5525 50  0001 C CNN
 F 1 "VCC" H 1200 5825 50  0000 C CNN
 F 2 "" H 1200 5675 50  0000 C CNN
@@
 AR Path="/5B1119BA/5C00E21C/5AEC72A2/5AE9E8B8" Ref="#PWR0347"  Part="1"
 AR Path="/5B1119BA/5C00E21C/5AEC72B9/5AE9E8B8" Ref="#PWR0349"  Part="1"
-F 0 "#PWR0349" H 5275 5700 50  0001 C CNN
+F 0 "#PWR031" H 5275 5700 50  0001 C CNN
 F 1 "VCC" H 5275 6000 50  0000 C CNN
 F 2 "" H 5275 5850 50  0000 C CNN
@@
 	2875 7375 2875 7275
 Wire Wire Line
-	2975 7275 2975 5925
-Wire Wire Line
 	3075 5925 3075 7375
 Wire Wire Line
@@
 Wire Wire Line
 	4650 5975 4650 7375
-Wire Wire Line
-	4650 7375 4625 7375
 Wire Wire Line
 	4850 5975 5000 5975
@@
 AR Path="/5B1119BA/5C00E21C/5AEC72A2/5AEB02AD" Ref="C205"  Part="1"
 AR Path="/5B1119BA/5C00E21C/5AEC72B9/5AEB02AD" Ref="C207"  Part="1"
-F 0 "C207" V 5575 5150 60  0000 C CNN
+F 0 "C21" V 5575 5150 60  0000 C CNN
 F 1 "100nF" V 5875 5150 60  0000 C CNN
 F 2 "" H 5725 5150 60  0000 C CNN
@@
 AR Path="/5B1119BA/5C00E21C/5AEC72A2/5AEB030E" Ref="#GND77"  Part="1"
 AR Path="/5B1119BA/5C00E21C/5AEC72B9/5AEB030E" Ref="#GND79"  Part="1"
-F 0 "#GND79" H 5525 4675 60  0001 C CNN
+F 0 "#GND22" H 5525 4675 60  0001 C CNN
 F 1 "0" H 5525 4705 60  0000 C CNN
 F 2 "" H 5525 4775 60  0000 C CNN
@@
 AR Path="/5B1119BA/5C00E21C/5AEC72A2/5AEB04DC" Ref="C204"  Part="1"
 AR Path="/5B1119BA/5C00E21C/5AEC72B9/5AEB04DC" Ref="C206"  Part="1"
-F 0 "C206" V 1075 5250 60  0000 C CNN
+F 0 "C20" V 1075 5250 60  0000 C CNN
 F 1 "100nF" V 1375 5250 60  0000 C CNN
 F 2 "" H 1225 5250 60  0000 C CNN
@@
 AR Path="/5B1119BA/5C00E21C/5AEC72A2/5AEB056F" Ref="#GND76"  Part="1"
 AR Path="/5B1119BA/5C00E21C/5AEC72B9/5AEB056F" Ref="#GND78"  Part="1"
-F 0 "#GND78" H 1400 4925 60  0001 C CNN
+F 0 "#GND21" H 1400 4925 60  0001 C CNN
 F 1 "0" H 1400 4955 60  0000 C CNN
 F 2 "" H 1400 5025 60  0000 C CNN
@@
 	5000 5025 5525 5025
 Wire Wire Line
-	2875 7275 4550 7275
+	2975 7375 3075 7375
+Wire Wire Line
+	3075 7375 4650 7375
+Connection ~ 3075 7375
+Wire Wire Line
+	2975 5925 2975 7275
+Wire Wire Line
+	2875 7275 2975 7275
+Connection ~ 2975 7275
+Wire Wire Line
+	2975 7275 4550 7275
+Wire Wire Line
+	2775 5925 2775 6725
 $EndSCHEMATC

Commit message: fixed errors
Connections:
- wire segments 79 -> 80
Changed lines of the file:
@@
 $Descr A4 11693 8268
 encoding utf-8
-Sheet 41 92
+Sheet 14 92
 Title ""
 Date ""
@@
 AR Path="/5B1119BA/5C00E21C/5AEC72A2/5AE9E2A5" Ref="U145"  Part="1"
 AR Path="/5B1119BA/5C00E21C/5AEC72B9/5AE9E2A5" Ref="U147"  Part="1"
-F 0 "U22" H 2625 5225 50  0000 C CNN
+F 0 "U26" H 2625 5225 50  0000 C CNN
 F 1 "74LS151" H 2625 5075 50  0000 C CNN
 F 2 "" H 2625 5225 50  0000 C CNN
@@
 AR Path="/5B1119BA/5C00E21C/5AEC72A2/5AE9E4A8" Ref="U146"  Part="1"
 AR Path="/5B1119BA/5C00E21C/5AEC72B9/5AE9E4A8" Ref="U148"  Part="1"
-F 0 "U23" H 4200 5275 50  0000 C CNN
+F 0 "U27" H 4200 5275 50  0000 C CNN
 F 1 "74LS151" H 4200 5125 50  0000 C CNN
 F 2 "" H 4200 5275 50  0000 C CNN
@@
 	2350 5925 2350 6500
 Wire Wire Line
-	2375 5925 2375 6425
-Wire Wire Line
-	2375 6425 2575 6425
+	2375 5925 2375 6350
 Wire Wire Line
 	2475 6425 2475 5925
@@
 AR Path="/5B1119BA/5C00E21C/5AEC72A2/5AEB02AD" Ref="C205"  Part="1"
 AR Path="/5B1119BA/5C00E21C/5AEC72B9/5AEB02AD" Ref="C207"  Part="1"
-F 0 "C21" V 5575 5150 60  0000 C CNN
+F 0 "C25" V 5575 5150 60  0000 C CNN
 F 1 "100nF" V 5875 5150 60  0000 C CNN
 F 2 "" H 5725 5150 60  0000 C CNN
@@
 AR Path="/5B1119BA/5C00E21C/5AEC72A2/5AEB030E" Ref="#GND77"  Part="1"
 AR Path="/5B1119BA/5C00E21C/5AEC72B9/5AEB030E" Ref="#GND79"  Part="1"
-F 0 "#GND22" H 5525 4675 60  0001 C CNN
+F 0 "#GND26" H 5525 4675 60  0001 C CNN
 F 1 "0" H 5525 4705 60  0000 C CNN
 F 2 "" H 5525 4775 60  0000 C CNN
@@
 AR Path="/5B1119BA/5C00E21C/5AEC72A2/5AEB04DC" Ref="C204"  Part="1"
 AR Path="/5B1119BA/5C00E21C/5AEC72B9/5AEB04DC" Ref="C206"  Part="1"
-F 0 "C20" V 1075 5250 60  0000 C CNN
+F 0 "C24" V 1075 5250 60  0000 C CNN
 F 1 "100nF" V 1375 5250 60  0000 C CNN
 F 2 "" H 1225 5250 60  0000 C CNN
@@
 AR Path="/5B1119BA/5C00E21C/5AEC72A2/5AEB056F" Ref="#GND76"  Part="1"
 AR Path="/5B1119BA/5C00E21C/5AEC72B9/5AEB056F" Ref="#GND78"  Part="1"
-F 0 "#GND21" H 1400 4925 60  0001 C CNN
+F 0 "#GND25" H 1400 4925 60  0001 C CNN
 F 1 "0" H 1400 4955 60  0000 C CNN
 F 2 "" H 1400 5025 60  0000 C CNN
@@
 Wire Wire Line
 	2775 5925 2775 6725
+Wire Wire Line
+	2575 6425 2575 6350
+Wire Wire Line
+	2575 6350 2375 6350
 $EndSCHEMATC

Commit message: message
Parts:
- renumbered U22 to U35, U23 to U36

Commit message: .
Connections:
- wire segments 80 -> 81
