File: ADD.sch (KiCad schematic (older format))
At the start: 4 parts

Commit message: SPICE capacitance and ground symbols
Parts:
- removed C? (x2): 100n, symbol C_Small
- added C? (x2): 100nF, symbol C
Connections:
- net labels added: 0
- net labels removed: GND
- wire segments 80 -> 81
Changed lines of the file:
@@
 EESchema Schematic File Version 2
-LIBS:power
-LIBS:device
-LIBS:transistors
-LIBS:conn
-LIBS:linear
-LIBS:regul
-LIBS:74xx
-LIBS:cmos4000
-LIBS:adc-dac
-LIBS:memory
-LIBS:xilinx
-LIBS:microcontrollers
-LIBS:dsp
-LIBS:microchip
-LIBS:analog_switches
-LIBS:motorola
-LIBS:texas
-LIBS:intel
-LIBS:audio
-LIBS:interface
-LIBS:digital-audio
-LIBS:philips
-LIBS:display
-LIBS:cypress
-LIBS:siliconi
-LIBS:opto
-LIBS:atmel
-LIBS:contrib
-LIBS:valves
+LIBS:spice
+LIBS:pspice
 LIBS:myCpu-cache
 EELAYER 25 0
@@
 $Descr A4 11693 8268
 encoding utf-8
-Sheet 9 21
+Sheet 10 21
 Title ""
 Date ""
@@
 	5225 3850 5225 3800
 $Comp
-L C_Small C?
-U 1 1 5AE8D2BA
-P 2125 4450
-F 0 "C?" H 2135 4520 50  0000 L CNN
-F 1 "100n" H 2135 4370 50  0000 L CNN
-F 2 "" H 2125 4450 50  0000 C CNN
-F 3 "" H 2125 4450 50  0000 C CNN
-	1    2125 4450
-	1    0    0    -1
-$EndComp
-$Comp
-L C_Small C?
-U 1 1 5AE8D35A
-P 5375 4600
-F 0 "C?" H 5385 4670 50  0000 L CNN
-F 1 "100n" H 5385 4520 50  0000 L CNN
-F 2 "" H 5375 4600 50  0000 C CNN
-F 3 "" H 5375 4600 50  0000 C CNN
-	1    5375 4600
-	1    0    0    -1
-$EndComp
-$Comp
 L VCC #PWR?
 U 1 1 5AE8D3DE
@@
 	1    0    0    -1
 $EndComp
-$Comp
-L GND #PWR?
-U 1 1 5AE8D416
-P 2125 4000
-F 0 "#PWR?" H 2125 3750 50  0001 C CNN
-F 1 "GND" H 2125 3850 50  0000 C CNN
-F 2 "" H 2125 4000 50  0000 C CNN
-F 3 "" H 2125 4000 50  0000 C CNN
-	1    2125 4000
-	1    0    0    -1
-$EndComp
-$Comp
-L GND #PWR?
-U 1 1 5AE8D432
-P 5325 4275
-F 0 "#PWR?" H 5325 4025 50  0001 C CNN
-F 1 "GND" H 5325 4125 50  0000 C CNN
-F 2 "" H 5325 4275 50  0000 C CNN
-F 3 "" H 5325 4275 50  0000 C CNN
-	1    5325 4275
-	1    0    0    -1
-$EndComp
-Wire Wire Line
-	2050 4825 2050 4550
-Wire Wire Line
-	2050 4550 2125 4550
-Wire Wire Line
-	2125 4350 2125 4000
-Wire Wire Line
-	5300 4275 5375 4275
-Wire Wire Line
-	5375 4275 5375 4500
-Wire Wire Line
-	5275 4925 5375 4925
-Wire Wire Line
-	5375 4925 5375 4700
+Wire Wire Line
+	5275 4925 5600 4925
+$Comp
+L C C?
+U 1 1 5AEB4A12
+P 5600 4450
+F 0 "C?" V 5450 4450 60  0000 C CNN
+F 1 "100nF" V 5750 4450 60  0000 C CNN
+F 2 "" H 5600 4450 60  0000 C CNN
+F 3 "" H 5600 4450 60  0000 C CNN
+	1    5600 4450
+	1    0    0    -1
+$EndComp
+$Comp
+L C C?
+U 1 1 5AEB4A63
+P 2200 4450
+F 0 "C?" V 2050 4450 60  0000 C CNN
+F 1 "100nF" V 2350 4450 60  0000 C CNN
+F 2 "" H 2200 4450 60  0000 C CNN
+F 3 "" H 2200 4450 60  0000 C CNN
+	1    2200 4450
+	1    0    0    -1
+$EndComp
+$Comp
+L 0 #GND?
+U 1 1 5AEB4A84
+P 5850 4125
+F 0 "#GND?" H 5850 4025 60  0001 C CNN
+F 1 "0" H 5850 4055 60  0000 C CNN
+F 2 "" H 5850 4125 60  0000 C CNN
+F 3 "" H 5850 4125 60  0000 C CNN
+	1    5850 4125
+	1    0    0    -1
+$EndComp
+$Comp
+L 0 #GND?
+U 1 1 5AEB4AA0
+P 2300 4000
+F 0 "#GND?" H 2300 3900 60  0001 C CNN
+F 1 "0" H 2300 3930 60  0000 C CNN
+F 2 "" H 2300 4000 60  0000 C CNN
+F 3 "" H 2300 4000 60  0000 C CNN
+	1    2300 4000
+	1    0    0    -1
+$EndComp
+Wire Wire Line
+	2050 4825 2200 4825
+Wire Wire Line
+	2200 4825 2200 4700
+Wire Wire Line
+	2200 4200 2200 4000
+Wire Wire Line
+	2200 4000 2300 4000
+Wire Wire Line
+	5850 4125 5600 4125
+Wire Wire Line
+	5600 4125 5600 4200
+Wire Wire Line
+	5600 4925 5600 4700
 $EndSCHEMATC

Commit message: fixed duplicate names
Parts:
- gave numbers to parts that had none: 4
Changed lines of the file:
@@
 $Descr A4 11693 8268
 encoding utf-8
-Sheet 10 21
+Sheet 9 21
 Title ""
 Date ""
@@
 Z7
 $Comp
-L 74LS283 U?
+L 74LS283 U13
 U 1 1 5AEA474F
 P 3075 4500
-F 0 "U?" H 3075 4500 50  0000 C CNN
+AR Path="/5AE62FB7/5AEA44C6/5AEA474F" Ref="U13"  Part="1"
+AR Path="/5AE62FB7/5AE93FA0/5AEA474F" Ref="U15"  Part="1"
+F 0 "U15" H 3075 4500 50  0000 C CNN
 F 1 "74LS283" H 3125 4150 50  0000 C CNN
 F 2 "" H 3075 4500 50  0000 C CNN
@@
 $EndComp
 $Comp
-L 74LS283 U?
+L 74LS283 U14
 U 1 1 5AEA4880
 P 4525 4550
-F 0 "U?" H 4525 4550 50  0000 C CNN
+AR Path="/5AE62FB7/5AEA44C6/5AEA4880" Ref="U14"  Part="1"
+AR Path="/5AE62FB7/5AE93FA0/5AEA4880" Ref="U16"  Part="1"
+F 0 "U16" H 4525 4550 50  0000 C CNN
 F 1 "74LS283" H 4575 4200 50  0000 C CNN
 F 2 "" H 4525 4550 50  0000 C CNN
@@
 	5225 3850 5225 3800
 $Comp
-L VCC #PWR?
+L VCC #PWR013
 U 1 1 5AE8D3DE
 P 2050 4825
-F 0 "#PWR?" H 2050 4675 50  0001 C CNN
+AR Path="/5AE62FB7/5AEA44C6/5AE8D3DE" Ref="#PWR013"  Part="1"
+AR Path="/5AE62FB7/5AE93FA0/5AE8D3DE" Ref="#PWR015"  Part="1"
+F 0 "#PWR015" H 2050 4675 50  0001 C CNN
 F 1 "VCC" H 2050 4975 50  0000 C CNN
 F 2 "" H 2050 4825 50  0000 C CNN
@@
 $EndComp
 $Comp
-L VCC #PWR?
+L VCC #PWR014
 U 1 1 5AE8D3FA
 P 5275 4925
-F 0 "#PWR?" H 5275 4775 50  0001 C CNN
+AR Path="/5AE62FB7/5AEA44C6/5AE8D3FA" Ref="#PWR014"  Part="1"
+AR Path="/5AE62FB7/5AE93FA0/5AE8D3FA" Ref="#PWR016"  Part="1"
+F 0 "#PWR016" H 5275 4775 50  0001 C CNN
 F 1 "VCC" H 5275 5075 50  0000 C CNN
 F 2 "" H 5275 4925 50  0000 C CNN
@@
 	5275 4925 5600 4925
 $Comp
-L C C?
+L C C12
 U 1 1 5AEB4A12
 P 5600 4450
-F 0 "C?" V 5450 4450 60  0000 C CNN
+AR Path="/5AE62FB7/5AEA44C6/5AEB4A12" Ref="C12"  Part="1"
+AR Path="/5AE62FB7/5AE93FA0/5AEB4A12" Ref="C14"  Part="1"
+F 0 "C14" V 5450 4450 60  0000 C CNN
 F 1 "100nF" V 5750 4450 60  0000 C CNN
 F 2 "" H 5600 4450 60  0000 C CNN
@@
 $EndComp
 $Comp
-L C C?
+L C C11
 U 1 1 5AEB4A63
 P 2200 4450
-F 0 "C?" V 2050 4450 60  0000 C CNN
+AR Path="/5AE62FB7/5AEA44C6/5AEB4A63" Ref="C11"  Part="1"
+AR Path="/5AE62FB7/5AE93FA0/5AEB4A63" Ref="C13"  Part="1"
+F 0 "C13" V 2050 4450 60  0000 C CNN
 F 1 "100nF" V 2350 4450 60  0000 C CNN
 F 2 "" H 2200 4450 60  0000 C CNN
@@
 $EndComp
 $Comp
-L 0 #GND?
+L 0 #GND14
 U 1 1 5AEB4A84
 P 5850 4125
-F 0 "#GND?" H 5850 4025 60  0001 C CNN
+AR Path="/5AE62FB7/5AEA44C6/5AEB4A84" Ref="#GND14"  Part="1"
+AR Path="/5AE62FB7/5AE93FA0/5AEB4A84" Ref="#GND16"  Part="1"
+F 0 "#GND16" H 5850 4025 60  0001 C CNN
 F 1 "0" H 5850 4055 60  0000 C CNN
 F 2 "" H 5850 4125 60  0000 C CNN
@@
 $EndComp
 $Comp
-L 0 #GND?
+L 0 #GND13
 U 1 1 5AEB4AA0
 P 2300 4000
-F 0 "#GND?" H 2300 3900 60  0001 C CNN
+AR Path="/5AE62FB7/5AEA44C6/5AEB4AA0" Ref="#GND13"  Part="1"
+AR Path="/5AE62FB7/5AE93FA0/5AEB4AA0" Ref="#GND15"  Part="1"
+F 0 "#GND15" H 2300 3900 60  0001 C CNN
 F 1 "0" H 2300 3930 60  0000 C CNN
 F 2 "" H 2300 4000 60  0000 C CNN

Commit message: NC-symbols
Changed lines of the file:
@@
 AR Path="/5AE62FB7/5AEA44C6/5AEA474F" Ref="U13"  Part="1"
 AR Path="/5AE62FB7/5AE93FA0/5AEA474F" Ref="U15"  Part="1"
-F 0 "U15" H 3075 4500 50  0000 C CNN
+F 0 "U13" H 3075 4500 50  0000 C CNN
 F 1 "74LS283" H 3125 4150 50  0000 C CNN
 F 2 "" H 3075 4500 50  0000 C CNN
@@
 AR Path="/5AE62FB7/5AEA44C6/5AEA4880" Ref="U14"  Part="1"
 AR Path="/5AE62FB7/5AE93FA0/5AEA4880" Ref="U16"  Part="1"
-F 0 "U16" H 4525 4550 50  0000 C CNN
+F 0 "U14" H 4525 4550 50  0000 C CNN
 F 1 "74LS283" H 4575 4200 50  0000 C CNN
 F 2 "" H 4525 4550 50  0000 C CNN
@@
 AR Path="/5AE62FB7/5AEA44C6/5AE8D3DE" Ref="#PWR013"  Part="1"
 AR Path="/5AE62FB7/5AE93FA0/5AE8D3DE" Ref="#PWR015"  Part="1"
-F 0 "#PWR015" H 2050 4675 50  0001 C CNN
+F 0 "#PWR013" H 2050 4675 50  0001 C CNN
 F 1 "VCC" H 2050 4975 50  0000 C CNN
 F 2 "" H 2050 4825 50  0000 C CNN
@@
 AR Path="/5AE62FB7/5AEA44C6/5AE8D3FA" Ref="#PWR014"  Part="1"
 AR Path="/5AE62FB7/5AE93FA0/5AE8D3FA" Ref="#PWR016"  Part="1"
-F 0 "#PWR016" H 5275 4775 50  0001 C CNN
+F 0 "#PWR014" H 5275 4775 50  0001 C CNN
 F 1 "VCC" H 5275 5075 50  0000 C CNN
 F 2 "" H 5275 4925 50  0000 C CNN
@@
 AR Path="/5AE62FB7/5AEA44C6/5AEB4A12" Ref="C12"  Part="1"
 AR Path="/5AE62FB7/5AE93FA0/5AEB4A12" Ref="C14"  Part="1"
-F 0 "C14" V 5450 4450 60  0000 C CNN
+F 0 "C12" V 5450 4450 60  0000 C CNN
 F 1 "100nF" V 5750 4450 60  0000 C CNN
 F 2 "" H 5600 4450 60  0000 C CNN
@@
 AR Path="/5AE62FB7/5AEA44C6/5AEB4A63" Ref="C11"  Part="1"
 AR Path="/5AE62FB7/5AE93FA0/5AEB4A63" Ref="C13"  Part="1"
-F 0 "C13" V 2050 4450 60  0000 C CNN
+F 0 "C11" V 2050 4450 60  0000 C CNN
 F 1 "100nF" V 2350 4450 60  0000 C CNN
 F 2 "" H 2200 4450 60  0000 C CNN
@@
 AR Path="/5AE62FB7/5AEA44C6/5AEB4A84" Ref="#GND14"  Part="1"
 AR Path="/5AE62FB7/5AE93FA0/5AEB4A84" Ref="#GND16"  Part="1"
-F 0 "#GND16" H 5850 4025 60  0001 C CNN
+F 0 "#GND14" H 5850 4025 60  0001 C CNN
 F 1 "0" H 5850 4055 60  0000 C CNN
 F 2 "" H 5850 4125 60  0000 C CNN
@@
 AR Path="/5AE62FB7/5AEA44C6/5AEB4AA0" Ref="#GND13"  Part="1"
 AR Path="/5AE62FB7/5AE93FA0/5AEB4AA0" Ref="#GND15"  Part="1"
-F 0 "#GND15" H 2300 3900 60  0001 C CNN
+F 0 "#GND13" H 2300 3900 60  0001 C CNN
 F 1 "0" H 2300 3930 60  0000 C CNN
 F 2 "" H 2300 4000 60  0000 C CNN

Commit message: spice libs from the internet, opened with new kicad 5.0.0, added spice models to components
Parts:
- C11, C12: symbol C -> spice:C
- U13, U14: symbol 74LS283 -> myCpu-rescue:74LS283; Spice_Lib_File (none) -> 74hc.lib; Spice_Model (none) -> 74HC283; Spice_Netlist_Enabled (none) -> Y; Spice_Primitive (none) -> X
Changed lines of the file:
@@
-EESchema Schematic File Version 2
-LIBS:spice
-LIBS:pspice
+EESchema Schematic File Version 4
 LIBS:myCpu-cache
-EELAYER 25 0
+EELAYER 26 0
 EELAYER END
 $Descr A4 11693 8268
 encoding utf-8
-Sheet 9 21
+Sheet 10 21
 Title ""
 Date ""
@@
 Z7
 $Comp
-L 74LS283 U13
+L myCpu-rescue:74LS283 U13
 U 1 1 5AEA474F
 P 3075 4500
 AR Path="/5AE62FB7/5AEA44C6/5AEA474F" Ref="U13"  Part="1"
 AR Path="/5AE62FB7/5AE93FA0/5AEA474F" Ref="U15"  Part="1"
-F 0 "U13" H 3075 4500 50  0000 C CNN
+F 0 "U15" H 3075 4500 50  0000 C CNN
 F 1 "74LS283" H 3125 4150 50  0000 C CNN
 F 2 "" H 3075 4500 50  0000 C CNN
 F 3 "" H 3075 4500 50  0000 C CNN
+F 4 "X" H 3075 4500 50  0001 C CNN "Spice_Primitive"
+F 5 "74HC283" H 3075 4500 50  0001 C CNN "Spice_Model"
+F 6 "Y" H 3075 4500 50  0001 C CNN "Spice_Netlist_Enabled"
+F 7 "74hc.lib" H 3075 4500 50  0001 C CNN "Spice_Lib_File"
 	1    3075 4500
 	0    -1   -1   0
 $EndComp
 $Comp
-L 74LS283 U14
+L myCpu-rescue:74LS283 U14
 U 1 1 5AEA4880
 P 4525 4550
 AR Path="/5AE62FB7/5AEA44C6/5AEA4880" Ref="U14"  Part="1"
 AR Path="/5AE62FB7/5AE93FA0/5AEA4880" Ref="U16"  Part="1"
-F 0 "U14" H 4525 4550 50  0000 C CNN
+F 0 "U16" H 4525 4550 50  0000 C CNN
 F 1 "74LS283" H 4575 4200 50  0000 C CNN
 F 2 "" H 4525 4550 50  0000 C CNN
 F 3 "" H 4525 4550 50  0000 C CNN
+F 4 "X" H 4525 4550 50  0001 C CNN "Spice_Primitive"
+F 5 "74HC283" H 4525 4550 50  0001 C CNN "Spice_Model"
+F 6 "Y" H 4525 4550 50  0001 C CNN "Spice_Netlist_Enabled"
+F 7 "74hc.lib" H 4525 4550 50  0001 C CNN "Spice_Lib_File"
 	1    4525 4550
 	0    -1   -1   0
@@
 	5225 3850 5225 3800
 $Comp
-L VCC #PWR013
+L myCpu-rescue:VCC #PWR013
 U 1 1 5AE8D3DE
 P 2050 4825
 AR Path="/5AE62FB7/5AEA44C6/5AE8D3DE" Ref="#PWR013"  Part="1"
 AR Path="/5AE62FB7/5AE93FA0/5AE8D3DE" Ref="#PWR015"  Part="1"
-F 0 "#PWR013" H 2050 4675 50  0001 C CNN
+F 0 "#PWR015" H 2050 4675 50  0001 C CNN
 F 1 "VCC" H 2050 4975 50  0000 C CNN
 F 2 "" H 2050 4825 50  0000 C CNN
@@
 $EndComp
 $Comp
-L VCC #PWR014
+L myCpu-rescue:VCC #PWR014
 U 1 1 5AE8D3FA
 P 5275 4925
 AR Path="/5AE62FB7/5AEA44C6/5AE8D3FA" Ref="#PWR014"  Part="1"
 AR Path="/5AE62FB7/5AE93FA0/5AE8D3FA" Ref="#PWR016"  Part="1"
-F 0 "#PWR014" H 5275 4775 50  0001 C CNN
+F 0 "#PWR016" H 5275 4775 50  0001 C CNN
 F 1 "VCC" H 5275 5075 50  0000 C CNN
 F 2 "" H 5275 4925 50  0000 C CNN
@@
 	5275 4925 5600 4925
 $Comp
-L C C12
+L spice:C C12
 U 1 1 5AEB4A12
 P 5600 4450
 AR Path="/5AE62FB7/5AEA44C6/5AEB4A12" Ref="C12"  Part="1"
 AR Path="/5AE62FB7/5AE93FA0/5AEB4A12" Ref="C14"  Part="1"
-F 0 "C12" V 5450 4450 60  0000 C CNN
+F 0 "C14" V 5450 4450 60  0000 C CNN
 F 1 "100nF" V 5750 4450 60  0000 C CNN
 F 2 "" H 5600 4450 60  0000 C CNN
@@
 $EndComp
 $Comp
-L C C11
+L spice:C C11
 U 1 1 5AEB4A63
 P 2200 4450
 AR Path="/5AE62FB7/5AEA44C6/5AEB4A63" Ref="C11"  Part="1"
 AR Path="/5AE62FB7/5AE93FA0/5AEB4A63" Ref="C13"  Part="1"
-F 0 "C11" V 2050 4450 60  0000 C CNN
+F 0 "C13" V 2050 4450 60  0000 C CNN
 F 1 "100nF" V 2350 4450 60  0000 C CNN
 F 2 "" H 2200 4450 60  0000 C CNN
@@
 $EndComp
 $Comp
-L 0 #GND14
+L spice:0 #GND14
 U 1 1 5AEB4A84
 P 5850 4125
 AR Path="/5AE62FB7/5AEA44C6/5AEB4A84" Ref="#GND14"  Part="1"
 AR Path="/5AE62FB7/5AE93FA0/5AEB4A84" Ref="#GND16"  Part="1"
-F 0 "#GND14" H 5850 4025 60  0001 C CNN
+F 0 "#GND16" H 5850 4025 60  0001 C CNN
 F 1 "0" H 5850 4055 60  0000 C CNN
 F 2 "" H 5850 4125 60  0000 C CNN
@@
 $EndComp
 $Comp
-L 0 #GND13
+L spice:0 #GND13
 U 1 1 5AEB4AA0
 P 2300 4000
 AR Path="/5AE62FB7/5AEA44C6/5AEB4AA0" Ref="#GND13"  Part="1"
 AR Path="/5AE62FB7/5AE93FA0/5AEB4AA0" Ref="#GND15"  Part="1"
-F 0 "#GND13" H 2300 3900 60  0001 C CNN
+F 0 "#GND15" H 2300 3900 60  0001 C CNN
 F 1 "0" H 2300 3930 60  0000 C CNN
 F 2 "" H 2300 4000 60  0000 C CNN

Commit message: lots of work done
Parts:
- renumbered C12 to C?, C11 to C?, U13 to U?, U14 to U?
Changed lines of the file:
@@
 $Descr A4 11693 8268
 encoding utf-8
-Sheet 10 21
+Sheet 77 81
 Title ""
 Date ""
@@
 Z7
 $Comp
-L myCpu-rescue:74LS283 U13
+L myCpu-rescue:74LS283 U?
 U 1 1 5AEA474F
 P 3075 4500
-AR Path="/5AE62FB7/5AEA44C6/5AEA474F" Ref="U13"  Part="1"
-AR Path="/5AE62FB7/5AE93FA0/5AEA474F" Ref="U15"  Part="1"
-F 0 "U15" H 3075 4500 50  0000 C CNN
+F 0 "U?" H 3075 4500 50  0000 C CNN
 F 1 "74LS283" H 3125 4150 50  0000 C CNN
 F 2 "" H 3075 4500 50  0000 C CNN
@@
 $EndComp
 $Comp
-L myCpu-rescue:74LS283 U14
+L myCpu-rescue:74LS283 U?
 U 1 1 5AEA4880
 P 4525 4550
-AR Path="/5AE62FB7/5AEA44C6/5AEA4880" Ref="U14"  Part="1"
-AR Path="/5AE62FB7/5AE93FA0/5AEA4880" Ref="U16"  Part="1"
-F 0 "U16" H 4525 4550 50  0000 C CNN
+F 0 "U?" H 4525 4550 50  0000 C CNN
 F 1 "74LS283" H 4575 4200 50  0000 C CNN
 F 2 "" H 4525 4550 50  0000 C CNN
@@
 	5225 3850 5225 3800
 $Comp
-L myCpu-rescue:VCC #PWR013
+L myCpu-rescue:VCC #PWR?
 U 1 1 5AE8D3DE
 P 2050 4825
-AR Path="/5AE62FB7/5AEA44C6/5AE8D3DE" Ref="#PWR013"  Part="1"
-AR Path="/5AE62FB7/5AE93FA0/5AE8D3DE" Ref="#PWR015"  Part="1"
-F 0 "#PWR015" H 2050 4675 50  0001 C CNN
+F 0 "#PWR?" H 2050 4675 50  0001 C CNN
 F 1 "VCC" H 2050 4975 50  0000 C CNN
 F 2 "" H 2050 4825 50  0000 C CNN
@@
 $EndComp
 $Comp
-L myCpu-rescue:VCC #PWR014
+L myCpu-rescue:VCC #PWR?
 U 1 1 5AE8D3FA
 P 5275 4925
-AR Path="/5AE62FB7/5AEA44C6/5AE8D3FA" Ref="#PWR014"  Part="1"
-AR Path="/5AE62FB7/5AE93FA0/5AE8D3FA" Ref="#PWR016"  Part="1"
-F 0 "#PWR016" H 5275 4775 50  0001 C CNN
+F 0 "#PWR?" H 5275 4775 50  0001 C CNN
 F 1 "VCC" H 5275 5075 50  0000 C CNN
 F 2 "" H 5275 4925 50  0000 C CNN
@@
 	5275 4925 5600 4925
 $Comp
-L spice:C C12
+L spice:C C?
 U 1 1 5AEB4A12
 P 5600 4450
-AR Path="/5AE62FB7/5AEA44C6/5AEB4A12" Ref="C12"  Part="1"
-AR Path="/5AE62FB7/5AE93FA0/5AEB4A12" Ref="C14"  Part="1"
-F 0 "C14" V 5450 4450 60  0000 C CNN
+F 0 "C?" V 5450 4450 60  0000 C CNN
 F 1 "100nF" V 5750 4450 60  0000 C CNN
 F 2 "" H 5600 4450 60  0000 C CNN
@@
 $EndComp
 $Comp
-L spice:C C11
+L spice:C C?
 U 1 1 5AEB4A63
 P 2200 4450
-AR Path="/5AE62FB7/5AEA44C6/5AEB4A63" Ref="C11"  Part="1"
-AR Path="/5AE62FB7/5AE93FA0/5AEB4A63" Ref="C13"  Part="1"
-F 0 "C13" V 2050 4450 60  0000 C CNN
+F 0 "C?" V 2050 4450 60  0000 C CNN
 F 1 "100nF" V 2350 4450 60  0000 C CNN
 F 2 "" H 2200 4450 60  0000 C CNN
@@
 $EndComp
 $Comp
-L spice:0 #GND14
+L spice:0 #GND?
 U 1 1 5AEB4A84
 P 5850 4125
-AR Path="/5AE62FB7/5AEA44C6/5AEB4A84" Ref="#GND14"  Part="1"
-AR Path="/5AE62FB7/5AE93FA0/5AEB4A84" Ref="#GND16"  Part="1"
-F 0 "#GND16" H 5850 4025 60  0001 C CNN
+F 0 "#GND?" H 5850 4025 60  0001 C CNN
 F 1 "0" H 5850 4055 60  0000 C CNN
 F 2 "" H 5850 4125 60  0000 C CNN
@@
 $EndComp
 $Comp
-L spice:0 #GND13
+L spice:0 #GND?
 U 1 1 5AEB4AA0
 P 2300 4000
-AR Path="/5AE62FB7/5AEA44C6/5AEB4AA0" Ref="#GND13"  Part="1"
-AR Path="/5AE62FB7/5AE93FA0/5AEB4AA0" Ref="#GND15"  Part="1"
-F 0 "#GND15" H 2300 3900 60  0001 C CNN
+F 0 "#GND?" H 2300 3900 60  0001 C CNN
 F 1 "0" H 2300 3930 60  0000 C CNN
 F 2 "" H 2300 4000 60  0000 C CNN

Commit message: b
Parts:
- gave numbers to parts that had none: 4
Changed lines of the file:
@@
 $Descr A4 11693 8268
 encoding utf-8
-Sheet 77 90
+Sheet 10 92
 Title ""
 Date ""
@@
 Z7
 $Comp
-L myCpu-rescue:74LS283 U?
+L myCpu-rescue:74LS283 U16
 U 1 1 5AEA474F
 P 3075 4500
-F 0 "U?" H 3075 4500 50  0000 C CNN
+AR Path="/5AE62FB7/5AEA44C6/5AEA474F" Ref="U16"  Part="1"
+AR Path="/5AE62FB7/5AE93FA0/5AEA474F" Ref="U18"  Part="1"
+AR Path="/82611AC0/82611C89/82611C91/5AEA474F" Ref="U201"  Part="1"
+AR Path="/5D3014E7/82611C91/5AEA474F" Ref="U229"  Part="1"
+F 0 "U16" H 3075 4500 50  0000 C CNN
 F 1 "74LS283" H 3125 4150 50  0000 C CNN
 F 2 "" H 3075 4500 50  0000 C CNN
@@
 $EndComp
 $Comp
-L myCpu-rescue:74LS283 U?
+L myCpu-rescue:74LS283 U17
 U 1 1 5AEA4880
 P 4525 4550
-F 0 "U?" H 4525 4550 50  0000 C CNN
+AR Path="/5AE62FB7/5AEA44C6/5AEA4880" Ref="U17"  Part="1"
+AR Path="/5AE62FB7/5AE93FA0/5AEA4880" Ref="U19"  Part="1"
+AR Path="/82611AC0/82611C89/82611C91/5AEA4880" Ref="U202"  Part="1"
+AR Path="/5D3014E7/82611C91/5AEA4880" Ref="U230"  Part="1"
+F 0 "U17" H 4525 4550 50  0000 C CNN
 F 1 "74LS283" H 4575 4200 50  0000 C CNN
 F 2 "" H 4525 4550 50  0000 C CNN
@@
 	5225 3850 5225 3800
 $Comp
-L myCpu-rescue:VCC #PWR?
+L myCpu-rescue:VCC #PWR024
 U 1 1 5AE8D3DE
 P 2050 4825
-F 0 "#PWR?" H 2050 4675 50  0001 C CNN
+AR Path="/5AE62FB7/5AEA44C6/5AE8D3DE" Ref="#PWR024"  Part="1"
+AR Path="/5AE62FB7/5AE93FA0/5AE8D3DE" Ref="#PWR026"  Part="1"
+AR Path="/82611AC0/82611C89/82611C91/5AE8D3DE" Ref="#PWR0533"  Part="1"
+AR Path="/5D3014E7/82611C91/5AE8D3DE" Ref="#PWR0602"  Part="1"
+F 0 "#PWR0602" H 2050 4675 50  0001 C CNN
 F 1 "VCC" H 2050 4975 50  0000 C CNN
 F 2 "" H 2050 4825 50  0000 C CNN
@@
 $EndComp
 $Comp
-L myCpu-rescue:VCC #PWR?
+L myCpu-rescue:VCC #PWR025
 U 1 1 5AE8D3FA
 P 5275 4925
-F 0 "#PWR?" H 5275 4775 50  0001 C CNN
+AR Path="/5AE62FB7/5AEA44C6/5AE8D3FA" Ref="#PWR025"  Part="1"
+AR Path="/5AE62FB7/5AE93FA0/5AE8D3FA" Ref="#PWR027"  Part="1"
+AR Path="/82611AC0/82611C89/82611C91/5AE8D3FA" Ref="#PWR0534"  Part="1"
+AR Path="/5D3014E7/82611C91/5AE8D3FA" Ref="#PWR0603"  Part="1"
+F 0 "#PWR0603" H 5275 4775 50  0001 C CNN
 F 1 "VCC" H 5275 5075 50  0000 C CNN
 F 2 "" H 5275 4925 50  0000 C CNN
@@
 	5275 4925 5600 4925
 $Comp
-L spice:C C?
+L spice:C C15
 U 1 1 5AEB4A12
 P 5600 4450
-F 0 "C?" V 5450 4450 60  0000 C CNN
+AR Path="/5AE62FB7/5AEA44C6/5AEB4A12" Ref="C15"  Part="1"
+AR Path="/5AE62FB7/5AE93FA0/5AEB4A12" Ref="C17"  Part="1"
+AR Path="/82611AC0/82611C89/82611C91/5AEB4A12" Ref="C301"  Part="1"
+AR Path="/5D3014E7/82611C91/5AEB4A12" Ref="C329"  Part="1"
+F 0 "C15" V 5450 4450 60  0000 C CNN
 F 1 "100nF" V 5750 4450 60  0000 C CNN
 F 2 "" H 5600 4450 60  0000 C CNN
@@
 $EndComp
 $Comp
-L spice:C C?
+L spice:C C14
 U 1 1 5AEB4A63
 P 2200 4450
-F 0 "C?" V 2050 4450 60  0000 C CNN
+AR Path="/5AE62FB7/5AEA44C6/5AEB4A63" Ref="C14"  Part="1"
+AR Path="/5AE62FB7/5AE93FA0/5AEB4A63" Ref="C16"  Part="1"
+AR Path="/82611AC0/82611C89/82611C91/5AEB4A63" Ref="C300"  Part="1"
+AR Path="/5D3014E7/82611C91/5AEB4A63" Ref="C328"  Part="1"
+F 0 "C14" V 2050 4450 60  0000 C CNN
 F 1 "100nF" V 2350 4450 60  0000 C CNN
 F 2 "" H 2200 4450 60  0000 C CNN
@@
 $EndComp
 $Comp
-L spice:0 #GND?
+L spice:0 #GND16
 U 1 1 5AEB4A84
 P 5850 4125
-F 0 "#GND?" H 5850 4025 60  0001 C CNN
+AR Path="/5AE62FB7/5AEA44C6/5AEB4A84" Ref="#GND16"  Part="1"
+AR Path="/5AE62FB7/5AE93FA0/5AEB4A84" Ref="#GND18"  Part="1"
+AR Path="/82611AC0/82611C89/82611C91/5AEB4A84" Ref="#GND85"  Part="1"
+AR Path="/5D3014E7/82611C91/5AEB4A84" Ref="#GND91"  Part="1"
+F 0 "#GND16" H 5850 4025 60  0001 C CNN
 F 1 "0" H 5850 4055 60  0000 C CNN
 F 2 "" H 5850 4125 60  0000 C CNN
@@
 $EndComp
 $Comp
-L spice:0 #GND?
+L spice:0 #GND15
 U 1 1 5AEB4AA0
 P 2300 4000
-F 0 "#GND?" H 2300 3900 60  0001 C CNN
+AR Path="/5AE62FB7/5AEA44C6/5AEB4AA0" Ref="#GND15"  Part="1"
+AR Path="/5AE62FB7/5AE93FA0/5AEB4AA0" Ref="#GND17"  Part="1"
+AR Path="/82611AC0/82611C89/82611C91/5AEB4AA0" Ref="#GND84"  Part="1"
+AR Path="/5D3014E7/82611C91/5AEB4AA0" Ref="#GND90"  Part="1"
+F 0 "#GND15" H 2300 3900 60  0001 C CNN
 F 1 "0" H 2300 3930 60  0000 C CNN
 F 2 "" H 2300 4000 60  0000 C CNN
