File: ADD.sch (KiCad schematic (older format))
At the start: 4 parts, among them U16 74LS283, U17 74LS283

Commit message: fixed errors
Changed lines of the file:
@@
 AR Path="/82611AC0/82611C89/82611C91/5AEA474F" Ref="U201"  Part="1"
 AR Path="/5D3014E7/82611C91/5AEA474F" Ref="U229"  Part="1"
-F 0 "U16" H 3075 4500 50  0000 C CNN
+F 0 "U18" H 3075 4500 50  0000 C CNN
 F 1 "74LS283" H 3125 4150 50  0000 C CNN
 F 2 "" H 3075 4500 50  0000 C CNN
@@
 AR Path="/82611AC0/82611C89/82611C91/5AEA4880" Ref="U202"  Part="1"
 AR Path="/5D3014E7/82611C91/5AEA4880" Ref="U230"  Part="1"
-F 0 "U17" H 4525 4550 50  0000 C CNN
+F 0 "U19" H 4525 4550 50  0000 C CNN
 F 1 "74LS283" H 4575 4200 50  0000 C CNN
 F 2 "" H 4525 4550 50  0000 C CNN
@@
 AR Path="/82611AC0/82611C89/82611C91/5AEB4A12" Ref="C301"  Part="1"
 AR Path="/5D3014E7/82611C91/5AEB4A12" Ref="C329"  Part="1"
-F 0 "C15" V 5450 4450 60  0000 C CNN
+F 0 "C17" V 5450 4450 60  0000 C CNN
 F 1 "100nF" V 5750 4450 60  0000 C CNN
 F 2 "" H 5600 4450 60  0000 C CNN
@@
 AR Path="/82611AC0/82611C89/82611C91/5AEB4A63" Ref="C300"  Part="1"
 AR Path="/5D3014E7/82611C91/5AEB4A63" Ref="C328"  Part="1"
-F 0 "C14" V 2050 4450 60  0000 C CNN
+F 0 "C16" V 2050 4450 60  0000 C CNN
 F 1 "100nF" V 2350 4450 60  0000 C CNN
 F 2 "" H 2200 4450 60  0000 C CNN
@@
 AR Path="/82611AC0/82611C89/82611C91/5AEB4A84" Ref="#GND85"  Part="1"
 AR Path="/5D3014E7/82611C91/5AEB4A84" Ref="#GND91"  Part="1"
-F 0 "#GND16" H 5850 4025 60  0001 C CNN
+F 0 "#GND18" H 5850 4025 60  0001 C CNN
 F 1 "0" H 5850 4055 60  0000 C CNN
 F 2 "" H 5850 4125 60  0000 C CNN
@@
 AR Path="/82611AC0/82611C89/82611C91/5AEB4AA0" Ref="#GND84"  Part="1"
 AR Path="/5D3014E7/82611C91/5AEB4AA0" Ref="#GND90"  Part="1"
-F 0 "#GND15" H 2300 3900 60  0001 C CNN
+F 0 "#GND17" H 2300 3900 60  0001 C CNN
 F 1 "0" H 2300 3930 60  0000 C CNN
 F 2 "" H 2300 4000 60  0000 C CNN

Commit message: message
Parts:
- renumbered U16 to U29, U17 to U30
Changed lines of the file:
@@
 $Descr A4 11693 8268
 encoding utf-8
-Sheet 10 92
+Sheet 10 101
 Title ""
 Date ""
@@
 Z7
 $Comp
-L myCpu-rescue:74LS283 U16
+L myCpu-rescue:74LS283 U29
 U 1 1 5AEA474F
 P 3075 4500
-AR Path="/5AE62FB7/5AEA44C6/5AEA474F" Ref="U16"  Part="1"
-AR Path="/5AE62FB7/5AE93FA0/5AEA474F" Ref="U18"  Part="1"
-AR Path="/82611AC0/82611C89/82611C91/5AEA474F" Ref="U201"  Part="1"
-AR Path="/5D3014E7/82611C91/5AEA474F" Ref="U229"  Part="1"
-F 0 "U18" H 3075 4500 50  0000 C CNN
+AR Path="/5AE62FB7/5AEA44C6/5AEA474F" Ref="U29"  Part="1"
+AR Path="/5AE62FB7/5AE93FA0/5AEA474F" Ref="U31"  Part="1"
+AR Path="/82611AC0/82611C89/82611C91/5AEA474F" Ref="U248"  Part="1"
+AR Path="/5D3014E7/82611C91/5AEA474F" Ref="U276"  Part="1"
+F 0 "U276" H 3075 4500 50  0000 C CNN
 F 1 "74LS283" H 3125 4150 50  0000 C CNN
 F 2 "" H 3075 4500 50  0000 C CNN
@@
 $EndComp
 $Comp
-L myCpu-rescue:74LS283 U17
+L myCpu-rescue:74LS283 U30
 U 1 1 5AEA4880
 P 4525 4550
-AR Path="/5AE62FB7/5AEA44C6/5AEA4880" Ref="U17"  Part="1"
-AR Path="/5AE62FB7/5AE93FA0/5AEA4880" Ref="U19"  Part="1"
-AR Path="/82611AC0/82611C89/82611C91/5AEA4880" Ref="U202"  Part="1"
-AR Path="/5D3014E7/82611C91/5AEA4880" Ref="U230"  Part="1"
-F 0 "U19" H 4525 4550 50  0000 C CNN
+AR Path="/5AE62FB7/5AEA44C6/5AEA4880" Ref="U30"  Part="1"
+AR Path="/5AE62FB7/5AE93FA0/5AEA4880" Ref="U32"  Part="1"
+AR Path="/82611AC0/82611C89/82611C91/5AEA4880" Ref="U249"  Part="1"
+AR Path="/5D3014E7/82611C91/5AEA4880" Ref="U277"  Part="1"
+F 0 "U277" H 4525 4550 50  0000 C CNN
 F 1 "74LS283" H 4575 4200 50  0000 C CNN
 F 2 "" H 4525 4550 50  0000 C CNN
@@
 	5225 3850 5225 3800
 $Comp
-L myCpu-rescue:VCC #PWR024
+L myCpu-rescue:VCC #PWR030
 U 1 1 5AE8D3DE
 P 2050 4825
-AR Path="/5AE62FB7/5AEA44C6/5AE8D3DE" Ref="#PWR024"  Part="1"
-AR Path="/5AE62FB7/5AE93FA0/5AE8D3DE" Ref="#PWR026"  Part="1"
-AR Path="/82611AC0/82611C89/82611C91/5AE8D3DE" Ref="#PWR0533"  Part="1"
-AR Path="/5D3014E7/82611C91/5AE8D3DE" Ref="#PWR0602"  Part="1"
-F 0 "#PWR0602" H 2050 4675 50  0001 C CNN
+AR Path="/5AE62FB7/5AEA44C6/5AE8D3DE" Ref="#PWR030"  Part="1"
+AR Path="/5AE62FB7/5AE93FA0/5AE8D3DE" Ref="#PWR032"  Part="1"
+AR Path="/82611AC0/82611C89/82611C91/5AE8D3DE" Ref="#PWR0585"  Part="1"
+AR Path="/5D3014E7/82611C91/5AE8D3DE" Ref="#PWR0658"  Part="1"
+F 0 "#PWR0658" H 2050 4675 50  0001 C CNN
 F 1 "VCC" H 2050 4975 50  0000 C CNN
 F 2 "" H 2050 4825 50  0000 C CNN
@@
 $EndComp
 $Comp
-L myCpu-rescue:VCC #PWR025
+L myCpu-rescue:VCC #PWR031
 U 1 1 5AE8D3FA
 P 5275 4925
-AR Path="/5AE62FB7/5AEA44C6/5AE8D3FA" Ref="#PWR025"  Part="1"
-AR Path="/5AE62FB7/5AE93FA0/5AE8D3FA" Ref="#PWR027"  Part="1"
-AR Path="/82611AC0/82611C89/82611C91/5AE8D3FA" Ref="#PWR0534"  Part="1"
-AR Path="/5D3014E7/82611C91/5AE8D3FA" Ref="#PWR0603"  Part="1"
-F 0 "#PWR0603" H 5275 4775 50  0001 C CNN
+AR Path="/5AE62FB7/5AEA44C6/5AE8D3FA" Ref="#PWR031"  Part="1"
+AR Path="/5AE62FB7/5AE93FA0/5AE8D3FA" Ref="#PWR033"  Part="1"
+AR Path="/82611AC0/82611C89/82611C91/5AE8D3FA" Ref="#PWR0586"  Part="1"
+AR Path="/5D3014E7/82611C91/5AE8D3FA" Ref="#PWR0659"  Part="1"
+F 0 "#PWR0659" H 5275 4775 50  0001 C CNN
 F 1 "VCC" H 5275 5075 50  0000 C CNN
 F 2 "" H 5275 4925 50  0000 C CNN
@@
 AR Path="/5AE62FB7/5AEA44C6/5AEB4A12" Ref="C15"  Part="1"
 AR Path="/5AE62FB7/5AE93FA0/5AEB4A12" Ref="C17"  Part="1"
-AR Path="/82611AC0/82611C89/82611C91/5AEB4A12" Ref="C301"  Part="1"
-AR Path="/5D3014E7/82611C91/5AEB4A12" Ref="C329"  Part="1"
-F 0 "C17" V 5450 4450 60  0000 C CNN
+AR Path="/82611AC0/82611C89/82611C91/5AEB4A12" Ref="C325"  Part="1"
+AR Path="/5D3014E7/82611C91/5AEB4A12" Ref="C353"  Part="1"
+F 0 "C353" V 5450 4450 60  0000 C CNN
 F 1 "100nF" V 5750 4450 60  0000 C CNN
 F 2 "" H 5600 4450 60  0000 C CNN
@@
 AR Path="/5AE62FB7/5AEA44C6/5AEB4A63" Ref="C14"  Part="1"
 AR Path="/5AE62FB7/5AE93FA0/5AEB4A63" Ref="C16"  Part="1"
-AR Path="/82611AC0/82611C89/82611C91/5AEB4A63" Ref="C300"  Part="1"
-AR Path="/5D3014E7/82611C91/5AEB4A63" Ref="C328"  Part="1"
-F 0 "C16" V 2050 4450 60  0000 C CNN
+AR Path="/82611AC0/82611C89/82611C91/5AEB4A63" Ref="C324"  Part="1"
+AR Path="/5D3014E7/82611C91/5AEB4A63" Ref="C352"  Part="1"
+F 0 "C352" V 2050 4450 60  0000 C CNN
 F 1 "100nF" V 2350 4450 60  0000 C CNN
 F 2 "" H 2200 4450 60  0000 C CNN
@@
 $EndComp
 $Comp
-L spice:0 #GND16
+L spice:0 #GND11
 U 1 1 5AEB4A84
 P 5850 4125
-AR Path="/5AE62FB7/5AEA44C6/5AEB4A84" Ref="#GND16"  Part="1"
-AR Path="/5AE62FB7/5AE93FA0/5AEB4A84" Ref="#GND18"  Part="1"
-AR Path="/82611AC0/82611C89/82611C91/5AEB4A84" Ref="#GND85"  Part="1"
-AR Path="/5D3014E7/82611C91/5AEB4A84" Ref="#GND91"  Part="1"
-F 0 "#GND18" H 5850 4025 60  0001 C CNN
+AR Path="/5AE62FB7/5AEA44C6/5AEB4A84" Ref="#GND11"  Part="1"
+AR Path="/5AE62FB7/5AE93FA0/5AEB4A84" Ref="#GND13"  Part="1"
+AR Path="/82611AC0/82611C89/82611C91/5AEB4A84" Ref="#GND96"  Part="1"
+AR Path="/5D3014E7/82611C91/5AEB4A84" Ref="#GND98"  Part="1"
+F 0 "#GND98" H 5850 4025 60  0001 C CNN
 F 1 "0" H 5850 4055 60  0000 C CNN
 F 2 "" H 5850 4125 60  0000 C CNN
@@
 $EndComp
 $Comp
-L spice:0 #GND15
+L spice:0 #GND10
 U 1 1 5AEB4AA0
 P 2300 4000
-AR Path="/5AE62FB7/5AEA44C6/5AEB4AA0" Ref="#GND15"  Part="1"
-AR Path="/5AE62FB7/5AE93FA0/5AEB4AA0" Ref="#GND17"  Part="1"
-AR Path="/82611AC0/82611C89/82611C91/5AEB4AA0" Ref="#GND84"  Part="1"
-AR Path="/5D3014E7/82611C91/5AEB4AA0" Ref="#GND90"  Part="1"
-F 0 "#GND17" H 2300 3900 60  0001 C CNN
+AR Path="/5AE62FB7/5AEA44C6/5AEB4AA0" Ref="#GND10"  Part="1"
+AR Path="/5AE62FB7/5AE93FA0/5AEB4AA0" Ref="#GND12"  Part="1"
+AR Path="/82611AC0/82611C89/82611C91/5AEB4AA0" Ref="#GND95"  Part="1"
+AR Path="/5D3014E7/82611C91/5AEB4AA0" Ref="#GND97"  Part="1"
+F 0 "#GND97" H 2300 3900 60  0001 C CNN
 F 1 "0" H 2300 3930 60  0000 C CNN
 F 2 "" H 2300 4000 60  0000 C CNN

Commit message: .
Changed lines of the file:
@@
 $Descr A4 11693 8268
 encoding utf-8
-Sheet 10 101
+Sheet 10 75
 Title ""
 Date ""
@@
 AR Path="/5AE62FB7/5AEA44C6/5AEA474F" Ref="U29"  Part="1"
 AR Path="/5AE62FB7/5AE93FA0/5AEA474F" Ref="U31"  Part="1"
-AR Path="/82611AC0/82611C89/82611C91/5AEA474F" Ref="U248"  Part="1"
-AR Path="/5D3014E7/82611C91/5AEA474F" Ref="U276"  Part="1"
-F 0 "U276" H 3075 4500 50  0000 C CNN
+AR Path="/82611AC0/82611C89/82611C91/5AEA474F" Ref="U147"  Part="1"
+AR Path="/5D3014E7/82611C91/5AEA474F" Ref="U175"  Part="1"
+F 0 "U175" H 3075 4500 50  0000 C CNN
 F 1 "74LS283" H 3125 4150 50  0000 C CNN
 F 2 "" H 3075 4500 50  0000 C CNN
@@
 AR Path="/5AE62FB7/5AEA44C6/5AEA4880" Ref="U30"  Part="1"
 AR Path="/5AE62FB7/5AE93FA0/5AEA4880" Ref="U32"  Part="1"
-AR Path="/82611AC0/82611C89/82611C91/5AEA4880" Ref="U249"  Part="1"
-AR Path="/5D3014E7/82611C91/5AEA4880" Ref="U277"  Part="1"
-F 0 "U277" H 4525 4550 50  0000 C CNN
+AR Path="/82611AC0/82611C89/82611C91/5AEA4880" Ref="U148"  Part="1"
+AR Path="/5D3014E7/82611C91/5AEA4880" Ref="U176"  Part="1"
+F 0 "U176" H 4525 4550 50  0000 C CNN
 F 1 "74LS283" H 4575 4200 50  0000 C CNN
 F 2 "" H 4525 4550 50  0000 C CNN
@@
 	5225 3850 5225 3800
 $Comp
-L myCpu-rescue:VCC #PWR030
+L myCpu-rescue:VCC #PWR033
 U 1 1 5AE8D3DE
 P 2050 4825
-AR Path="/5AE62FB7/5AEA44C6/5AE8D3DE" Ref="#PWR030"  Part="1"
-AR Path="/5AE62FB7/5AE93FA0/5AE8D3DE" Ref="#PWR032"  Part="1"
-AR Path="/82611AC0/82611C89/82611C91/5AE8D3DE" Ref="#PWR0585"  Part="1"
-AR Path="/5D3014E7/82611C91/5AE8D3DE" Ref="#PWR0658"  Part="1"
-F 0 "#PWR0658" H 2050 4675 50  0001 C CNN
+AR Path="/5AE62FB7/5AEA44C6/5AE8D3DE" Ref="#PWR033"  Part="1"
+AR Path="/5AE62FB7/5AE93FA0/5AE8D3DE" Ref="#PWR035"  Part="1"
+AR Path="/82611AC0/82611C89/82611C91/5AE8D3DE" Ref="#PWR0175"  Part="1"
+AR Path="/5D3014E7/82611C91/5AE8D3DE" Ref="#PWR0248"  Part="1"
+F 0 "#PWR0248" H 2050 4675 50  0001 C CNN
 F 1 "VCC" H 2050 4975 50  0000 C CNN
 F 2 "" H 2050 4825 50  0000 C CNN
@@
 $EndComp
 $Comp
-L myCpu-rescue:VCC #PWR031
+L myCpu-rescue:VCC #PWR034
 U 1 1 5AE8D3FA
 P 5275 4925
-AR Path="/5AE62FB7/5AEA44C6/5AE8D3FA" Ref="#PWR031"  Part="1"
-AR Path="/5AE62FB7/5AE93FA0/5AE8D3FA" Ref="#PWR033"  Part="1"
-AR Path="/82611AC0/82611C89/82611C91/5AE8D3FA" Ref="#PWR0586"  Part="1"
-AR Path="/5D3014E7/82611C91/5AE8D3FA" Ref="#PWR0659"  Part="1"
-F 0 "#PWR0659" H 5275 4775 50  0001 C CNN
+AR Path="/5AE62FB7/5AEA44C6/5AE8D3FA" Ref="#PWR034"  Part="1"
+AR Path="/5AE62FB7/5AE93FA0/5AE8D3FA" Ref="#PWR036"  Part="1"
+AR Path="/82611AC0/82611C89/82611C91/5AE8D3FA" Ref="#PWR0176"  Part="1"
+AR Path="/5D3014E7/82611C91/5AE8D3FA" Ref="#PWR0249"  Part="1"
+F 0 "#PWR0249" H 5275 4775 50  0001 C CNN
 F 1 "VCC" H 5275 5075 50  0000 C CNN
 F 2 "" H 5275 4925 50  0000 C CNN
@@
 AR Path="/5AE62FB7/5AEA44C6/5AEB4A12" Ref="C15"  Part="1"
 AR Path="/5AE62FB7/5AE93FA0/5AEB4A12" Ref="C17"  Part="1"
-AR Path="/82611AC0/82611C89/82611C91/5AEB4A12" Ref="C325"  Part="1"
-AR Path="/5D3014E7/82611C91/5AEB4A12" Ref="C353"  Part="1"
-F 0 "C353" V 5450 4450 60  0000 C CNN
+AR Path="/82611AC0/82611C89/82611C91/5AEB4A12" Ref="C117"  Part="1"
+AR Path="/5D3014E7/82611C91/5AEB4A12" Ref="C145"  Part="1"
+F 0 "C145" V 5450 4450 60  0000 C CNN
 F 1 "100nF" V 5750 4450 60  0000 C CNN
 F 2 "" H 5600 4450 60  0000 C CNN
@@
 AR Path="/5AE62FB7/5AEA44C6/5AEB4A63" Ref="C14"  Part="1"
 AR Path="/5AE62FB7/5AE93FA0/5AEB4A63" Ref="C16"  Part="1"
-AR Path="/82611AC0/82611C89/82611C91/5AEB4A63" Ref="C324"  Part="1"
-AR Path="/5D3014E7/82611C91/5AEB4A63" Ref="C352"  Part="1"
-F 0 "C352" V 2050 4450 60  0000 C CNN
+AR Path="/82611AC0/82611C89/82611C91/5AEB4A63" Ref="C116"  Part="1"
+AR Path="/5D3014E7/82611C91/5AEB4A63" Ref="C144"  Part="1"
+F 0 "C144" V 2050 4450 60  0000 C CNN
 F 1 "100nF" V 2350 4450 60  0000 C CNN
 F 2 "" H 2200 4450 60  0000 C CNN
