File: AND.sch (KiCad schematic (older format))
At the start: 4 parts, among them U1 4081, U2 4081

Commit message: wiring
Parts:
- gave numbers to parts that had none: 2
Changed lines of the file:
@@
 $Descr A4 11693 8268
 encoding utf-8
-Sheet 3 8
+Sheet 3 20
 Title ""
 Date ""
@@
 	4775 2925 5850 2925
 $Comp
-L C C?
+L C C2
 U 1 1 5AE7579C
 P 750 3550
-F 0 "C?" H 775 3650 50  0000 L CNN
+F 0 "C2" H 775 3650 50  0000 L CNN
 F 1 "C" H 775 3450 50  0000 L CNN
 F 2 "" H 788 3400 50  0000 C CNN
@@
 $EndComp
 $Comp
-L C C?
+L C C3
 U 1 1 5AE75811
 P 6475 3550
-F 0 "C?" H 6500 3650 50  0000 L CNN
+F 0 "C3" H 6500 3650 50  0000 L CNN
 F 1 "C" H 6500 3450 50  0000 L CNN
 F 2 "" H 6513 3400 50  0000 C CNN
@@
 $EndComp
 $Comp
-L GND #PWR?
+L GND #PWR3
 U 1 1 5AE75904
 P 6500 3050
-F 0 "#PWR?" H 6500 2800 50  0001 C CNN
+F 0 "#PWR3" H 6500 2800 50  0001 C CNN
 F 1 "GND" H 6500 2900 50  0000 C CNN
 F 2 "" H 6500 3050 50  0000 C CNN
@@
 $EndComp
 $Comp
-L GND #PWR?
+L GND #PWR2
 U 1 1 5AE75968
 P 850 3125
-F 0 "#PWR?" H 850 2875 50  0001 C CNN
+F 0 "#PWR2" H 850 2875 50  0001 C CNN
 F 1 "GND" H 850 2975 50  0000 C CNN
 F 2 "" H 850 3125 50  0000 C CNN
@@
 $EndComp
 $Comp
-L VCC #PWR?
+L VCC #PWR1
 U 1 1 5AE75990
 P 775 4000
-F 0 "#PWR?" H 775 3850 50  0001 C CNN
+F 0 "#PWR1" H 775 3850 50  0001 C CNN
 F 1 "VCC" H 775 4150 50  0000 C CNN
 F 2 "" H 775 4000 50  0000 C CNN
@@
 $EndComp
 $Comp
-L VCC #PWR?
+L VCC #PWR4
 U 1 1 5AE759C2
 P 6500 4100
-F 0 "#PWR?" H 6500 3950 50  0001 C CNN
+F 0 "#PWR4" H 6500 3950 50  0001 C CNN
 F 1 "VCC" H 6500 4250 50  0000 C CNN
 F 2 "" H 6500 4100 50  0000 C CNN

Commit message: SPICE capacitance and ground symbols
Parts:
- removed C2, C3: C, symbol C
- added C? (x2): C, symbol C
Connections:
- net labels added: 0
- net labels removed: GND
- wire segments 69 -> 71
Changed lines of the file:
@@
 EESchema Schematic File Version 2
-LIBS:power
-LIBS:device
-LIBS:transistors
-LIBS:conn
-LIBS:linear
-LIBS:regul
-LIBS:74xx
-LIBS:cmos4000
-LIBS:adc-dac
-LIBS:memory
-LIBS:xilinx
-LIBS:microcontrollers
-LIBS:dsp
-LIBS:microchip
-LIBS:analog_switches
-LIBS:motorola
-LIBS:texas
-LIBS:intel
-LIBS:audio
-LIBS:interface
-LIBS:digital-audio
-LIBS:philips
-LIBS:display
-LIBS:cypress
-LIBS:siliconi
-LIBS:opto
-LIBS:atmel
-LIBS:contrib
-LIBS:valves
+LIBS:spice
+LIBS:pspice
 LIBS:myCpu-cache
 EELAYER 25 0
@@
 	4775 2925 5850 2925
 $Comp
-L C C2
-U 1 1 5AE7579C
-P 750 3550
-F 0 "C2" H 775 3650 50  0000 L CNN
-F 1 "C" H 775 3450 50  0000 L CNN
-F 2 "" H 788 3400 50  0000 C CNN
-F 3 "" H 750 3550 50  0000 C CNN
-	1    750  3550
-	1    0    0    -1
-$EndComp
-$Comp
-L C C3
-U 1 1 5AE75811
-P 6475 3550
-F 0 "C3" H 6500 3650 50  0000 L CNN
-F 1 "C" H 6500 3450 50  0000 L CNN
-F 2 "" H 6513 3400 50  0000 C CNN
-F 3 "" H 6475 3550 50  0000 C CNN
-	1    6475 3550
-	1    0    0    -1
-$EndComp
-$Comp
-L GND #PWR3
-U 1 1 5AE75904
-P 6500 3050
-F 0 "#PWR3" H 6500 2800 50  0001 C CNN
-F 1 "GND" H 6500 2900 50  0000 C CNN
-F 2 "" H 6500 3050 50  0000 C CNN
-F 3 "" H 6500 3050 50  0000 C CNN
-	1    6500 3050
-	1    0    0    -1
-$EndComp
-$Comp
-L GND #PWR2
-U 1 1 5AE75968
-P 850 3125
-F 0 "#PWR2" H 850 2875 50  0001 C CNN
-F 1 "GND" H 850 2975 50  0000 C CNN
-F 2 "" H 850 3125 50  0000 C CNN
-F 3 "" H 850 3125 50  0000 C CNN
-	1    850  3125
-	1    0    0    -1
-$EndComp
-$Comp
 L VCC #PWR1
 U 1 1 5AE75990
@@
 $EndComp
 Wire Wire Line
-	6500 4100 6500 3700
-Wire Wire Line
-	6500 3700 6475 3700
-Wire Wire Line
-	6475 3400 6475 3050
-Wire Wire Line
-	6475 3050 6500 3050
-Wire Wire Line
-	750  3400 750  3125
-Wire Wire Line
-	750  3125 850  3125
-Wire Wire Line
-	750  3700 750  4000
-Wire Wire Line
 	750  4000 775  4000
+$Comp
+L C C?
+U 1 1 5AEBB378
+P 750 3750
+F 0 "C?" V 600 3750 60  0000 C CNN
+F 1 "C" V 900 3750 60  0000 C CNN
+F 2 "" H 750 3750 60  0000 C CNN
+F 3 "" H 750 3750 60  0000 C CNN
+	1    750  3750
+	1    0    0    -1
+$EndComp
+$Comp
+L C C?
+U 1 1 5AEBB40C
+P 6375 3825
+F 0 "C?" V 6225 3825 60  0000 C CNN
+F 1 "C" V 6525 3825 60  0000 C CNN
+F 2 "" H 6375 3825 60  0000 C CNN
+F 3 "" H 6375 3825 60  0000 C CNN
+	1    6375 3825
+	1    0    0    -1
+$EndComp
+$Comp
+L 0 #GND?
+U 1 1 5AEBB4E1
+P 6250 3575
+F 0 "#GND?" H 6250 3475 60  0001 C CNN
+F 1 "0" H 6250 3505 60  0000 C CNN
+F 2 "" H 6250 3575 60  0000 C CNN
+F 3 "" H 6250 3575 60  0000 C CNN
+	1    6250 3575
+	1    0    0    -1
+$EndComp
+$Comp
+L 0 #GND?
+U 1 1 5AEBB527
+P 575 3550
+F 0 "#GND?" H 575 3450 60  0001 C CNN
+F 1 "0" H 575 3480 60  0000 C CNN
+F 2 "" H 575 3550 60  0000 C CNN
+F 3 "" H 575 3550 60  0000 C CNN
+	1    575  3550
+	1    0    0    -1
+$EndComp
+Wire Wire Line
+	575  3550 575  3425
+Wire Wire Line
+	575  3425 775  3425
+Wire Wire Line
+	775  3425 775  3500
+Wire Wire Line
+	775  3500 750  3500
+Wire Wire Line
+	6375 3575 6375 3525
+Wire Wire Line
+	6375 3525 6250 3525
+Wire Wire Line
+	6250 3525 6250 3575
+Wire Wire Line
+	6375 4075 6500 4075
+Wire Wire Line
+	6500 4075 6500 4100
 $EndSCHEMATC

Commit message: fixed duplicate names
Parts:
- gave numbers to parts that had none: 2
Changed lines of the file:
@@
 	4775 2925 5850 2925
 $Comp
-L VCC #PWR1
+L VCC #PWR01
 U 1 1 5AE75990
 P 775 4000
-F 0 "#PWR1" H 775 3850 50  0001 C CNN
+F 0 "#PWR01" H 775 3850 50  0001 C CNN
 F 1 "VCC" H 775 4150 50  0000 C CNN
 F 2 "" H 775 4000 50  0000 C CNN
@@
 $EndComp
 $Comp
-L VCC #PWR4
+L VCC #PWR02
 U 1 1 5AE759C2
 P 6500 4100
-F 0 "#PWR4" H 6500 3950 50  0001 C CNN
+F 0 "#PWR02" H 6500 3950 50  0001 C CNN
 F 1 "VCC" H 6500 4250 50  0000 C CNN
 F 2 "" H 6500 4100 50  0000 C CNN
@@
 	750  4000 775  4000
 $Comp
-L C C?
+L C C1
 U 1 1 5AEBB378
 P 750 3750
-F 0 "C?" V 600 3750 60  0000 C CNN
+F 0 "C1" V 600 3750 60  0000 C CNN
 F 1 "C" V 900 3750 60  0000 C CNN
 F 2 "" H 750 3750 60  0000 C CNN
@@
 $EndComp
 $Comp
-L C C?
+L C C2
 U 1 1 5AEBB40C
 P 6375 3825
-F 0 "C?" V 6225 3825 60  0000 C CNN
+F 0 "C2" V 6225 3825 60  0000 C CNN
 F 1 "C" V 6525 3825 60  0000 C CNN
 F 2 "" H 6375 3825 60  0000 C CNN
@@
 $EndComp
 $Comp
-L 0 #GND?
+L 0 #GND2
 U 1 1 5AEBB4E1
 P 6250 3575
-F 0 "#GND?" H 6250 3475 60  0001 C CNN
+F 0 "#GND2" H 6250 3475 60  0001 C CNN
 F 1 "0" H 6250 3505 60  0000 C CNN
 F 2 "" H 6250 3575 60  0000 C CNN
@@
 $EndComp
 $Comp
-L 0 #GND?
+L 0 #GND1
 U 1 1 5AEBB527
 P 575 3550
-F 0 "#GND?" H 575 3450 60  0001 C CNN
+F 0 "#GND1" H 575 3450 60  0001 C CNN
 F 1 "0" H 575 3480 60  0000 C CNN
 F 2 "" H 575 3550 60  0000 C CNN

Commit message: spice libs from the internet, opened with new kicad 5.0.0, added spice models to components
Parts:
- C1, C2: value C -> 100nF; symbol C -> spice:C
- U1: symbol 4081 -> myCpu-rescue:4081; Spice_Lib_File (none) -> cd4000.lib; Spice_Model (none) -> CD4081B; Spice_Netlist_Enabled (none) -> Y; Spice_Primitive (none) -> X
- U1, U2: symbol 4081 -> myCpu-rescue:4081
Changed lines of the file:
@@
-EESchema Schematic File Version 2
-LIBS:spice
-LIBS:pspice
+EESchema Schematic File Version 4
 LIBS:myCpu-cache
-EELAYER 25 0
+EELAYER 26 0
 EELAYER END
 $Descr A4 11693 8268
@@
 Z7
 $Comp
-L 4081 U1
+L myCpu-rescue:4081 U1
 U 1 1 5AE63E39
 P 1325 3650
@@
 F 2 "" H 1325 3650 60  0001 C CNN
 F 3 "" H 1325 3650 60  0001 C CNN
+F 4 "X" H 1325 3650 50  0001 C CNN "Spice_Primitive"
+F 5 "CD4081B" H 1325 3650 50  0001 C CNN "Spice_Model"
+F 6 "Y" H 1325 3650 50  0001 C CNN "Spice_Netlist_Enabled"
+F 7 "cd4000.lib" H 1325 3650 50  0001 C CNN "Spice_Lib_File"
 	1    1325 3650
 	0    -1   -1   0
 $EndComp
 $Comp
-L 4081 U1
+L myCpu-rescue:4081 U1
 U 2 1 5AE63EAA
 P 1925 3650
@@
 $EndComp
 $Comp
-L 4081 U1
+L myCpu-rescue:4081 U1
 U 3 1 5AE63F35
 P 2575 3575
@@
 $EndComp
 $Comp
-L 4081 U1
+L myCpu-rescue:4081 U1
 U 4 1 5AE63FD4
 P 3300 3525
@@
 	5950 7250 5950 4125
 $Comp
-L 4081 U2
+L myCpu-rescue:4081 U2
 U 1 1 5AE64A18
 P 3875 3650
@@
 $EndComp
 $Comp
-L 4081 U2
+L myCpu-rescue:4081 U2
 U 2 1 5AE64ABB
 P 4475 3650
@@
 $EndComp
 $Comp
-L 4081 U2
+L myCpu-rescue:4081 U2
 U 3 1 5AE64B4C
 P 5125 3575
@@
 $EndComp
 $Comp
-L 4081 U2
+L myCpu-rescue:4081 U2
 U 4 1 5AE64BBD
 P 5850 3525
@@
 	4775 2925 5850 2925
 $Comp
-L VCC #PWR01
+L myCpu-rescue:VCC #PWR01
 U 1 1 5AE75990
 P 775 4000
@@
 $EndComp
 $Comp
-L VCC #PWR02
+L myCpu-rescue:VCC #PWR02
 U 1 1 5AE759C2
 P 6500 4100
@@
 	750  4000 775  4000
 $Comp
-L C C1
+L spice:C C1
 U 1 1 5AEBB378
 P 750 3750
 F 0 "C1" V 600 3750 60  0000 C CNN
-F 1 "C" V 900 3750 60  0000 C CNN
+F 1 "100nF" V 900 3750 60  0000 C CNN
 F 2 "" H 750 3750 60  0000 C CNN
 F 3 "" H 750 3750 60  0000 C CNN
@@
 $EndComp
 $Comp
-L C C2
+L spice:C C2
 U 1 1 5AEBB40C
 P 6375 3825
 F 0 "C2" V 6225 3825 60  0000 C CNN
-F 1 "C" V 6525 3825 60  0000 C CNN
+F 1 "100nF" V 6525 3825 60  0000 C CNN
 F 2 "" H 6375 3825 60  0000 C CNN
 F 3 "" H 6375 3825 60  0000 C CNN
@@
 $EndComp
 $Comp
-L 0 #GND2
+L spice:0 #GND2
 U 1 1 5AEBB4E1
 P 6250 3575
@@
 $EndComp
 $Comp
-L 0 #GND1
+L spice:0 #GND1
 U 1 1 5AEBB527
 P 575 3550

Commit message: lots of work done
Parts:
- renumbered C1 to C2, C2 to C3, U1 to U2, U2 to U3
Changed lines of the file:
@@
 $Descr A4 11693 8268
 encoding utf-8
-Sheet 3 21
+Sheet 3 81
 Title ""
 Date ""
@@
 Z7
 $Comp
-L myCpu-rescue:4081 U1
+L myCpu-rescue:4081 U2
 U 1 1 5AE63E39
 P 1325 3650
-F 0 "U1" H 1325 3700 50  0000 C CNN
+F 0 "U2" H 1325 3700 50  0000 C CNN
 F 1 "4081" H 1325 3600 50  0000 C CNN
 F 2 "" H 1325 3650 60  0001 C CNN
@@
 $EndComp
 $Comp
-L myCpu-rescue:4081 U1
+L myCpu-rescue:4081 U2
 U 2 1 5AE63EAA
 P 1925 3650
-F 0 "U1" H 1925 3700 50  0000 C CNN
+F 0 "U2" H 1925 3700 50  0000 C CNN
 F 1 "4081" H 1925 3600 50  0000 C CNN
 F 2 "" H 1925 3650 60  0001 C CNN
@@
 $EndComp
 $Comp
-L myCpu-rescue:4081 U1
+L myCpu-rescue:4081 U2
 U 3 1 5AE63F35
 P 2575 3575
-F 0 "U1" H 2575 3625 50  0000 C CNN
+F 0 "U2" H 2575 3625 50  0000 C CNN
 F 1 "4081" H 2575 3525 50  0000 C CNN
 F 2 "" H 2575 3575 60  0001 C CNN
@@
 $EndComp
 $Comp
-L myCpu-rescue:4081 U1
+L myCpu-rescue:4081 U2
 U 4 1 5AE63FD4
 P 3300 3525
-F 0 "U1" H 3300 3575 50  0000 C CNN
+F 0 "U2" H 3300 3575 50  0000 C CNN
 F 1 "4081" H 3300 3475 50  0000 C CNN
 F 2 "" H 3300 3525 60  0001 C CNN
@@
 	5950 7250 5950 4125
 $Comp
-L myCpu-rescue:4081 U2
+L myCpu-rescue:4081 U3
 U 1 1 5AE64A18
 P 3875 3650
-F 0 "U2" H 3875 3700 50  0000 C CNN
+F 0 "U3" H 3875 3700 50  0000 C CNN
 F 1 "4081" H 3875 3600 50  0000 C CNN
 F 2 "" H 3875 3650 60  0001 C CNN
@@
 $EndComp
 $Comp
-L myCpu-rescue:4081 U2
+L myCpu-rescue:4081 U3
 U 2 1 5AE64ABB
 P 4475 3650
-F 0 "U2" H 4475 3700 50  0000 C CNN
+F 0 "U3" H 4475 3700 50  0000 C CNN
 F 1 "4081" H 4475 3600 50  0000 C CNN
 F 2 "" H 4475 3650 60  0001 C CNN
@@
 $EndComp
 $Comp
-L myCpu-rescue:4081 U2
+L myCpu-rescue:4081 U3
 U 3 1 5AE64B4C
 P 5125 3575
-F 0 "U2" H 5125 3625 50  0000 C CNN
+F 0 "U3" H 5125 3625 50  0000 C CNN
 F 1 "4081" H 5125 3525 50  0000 C CNN
 F 2 "" H 5125 3575 60  0001 C CNN
@@
 $EndComp
 $Comp
-L myCpu-rescue:4081 U2
+L myCpu-rescue:4081 U3
 U 4 1 5AE64BBD
 P 5850 3525
-F 0 "U2" H 5850 3575 50  0000 C CNN
+F 0 "U3" H 5850 3575 50  0000 C CNN
 F 1 "4081" H 5850 3475 50  0000 C CNN
 F 2 "" H 5850 3525 60  0001 C CNN
@@
 	4775 2925 5850 2925
 $Comp
-L myCpu-rescue:VCC #PWR01
+L myCpu-rescue:VCC #PWR05
 U 1 1 5AE75990
 P 775 4000
-F 0 "#PWR01" H 775 3850 50  0001 C CNN
+F 0 "#PWR05" H 775 3850 50  0001 C CNN
 F 1 "VCC" H 775 4150 50  0000 C CNN
 F 2 "" H 775 4000 50  0000 C CNN
@@
 $EndComp
 $Comp
-L myCpu-rescue:VCC #PWR02
+L myCpu-rescue:VCC #PWR06
 U 1 1 5AE759C2
 P 6500 4100
-F 0 "#PWR02" H 6500 3950 50  0001 C CNN
+F 0 "#PWR06" H 6500 3950 50  0001 C CNN
 F 1 "VCC" H 6500 4250 50  0000 C CNN
 F 2 "" H 6500 4100 50  0000 C CNN
@@
 	750  4000 775  4000
 $Comp
-L spice:C C1
+L spice:C C2
 U 1 1 5AEBB378
 P 750 3750
-F 0 "C1" V 600 3750 60  0000 C CNN
+F 0 "C2" V 600 3750 60  0000 C CNN
 F 1 "100nF" V 900 3750 60  0000 C CNN
 F 2 "" H 750 3750 60  0000 C CNN
@@
 $EndComp
 $Comp
-L spice:C C2
+L spice:C C3
 U 1 1 5AEBB40C
 P 6375 3825
-F 0 "C2" V 6225 3825 60  0000 C CNN
+F 0 "C3" V 6225 3825 60  0000 C CNN
 F 1 "100nF" V 6525 3825 60  0000 C CNN
 F 2 "" H 6375 3825 60  0000 C CNN
@@
 $EndComp
 $Comp
-L spice:0 #GND2
+L spice:0 #GND7
 U 1 1 5AEBB4E1
 P 6250 3575
-F 0 "#GND2" H 6250 3475 60  0001 C CNN
+F 0 "#GND7" H 6250 3475 60  0001 C CNN
 F 1 "0" H 6250 3505 60  0000 C CNN
 F 2 "" H 6250 3575 60  0000 C CNN
@@
 $EndComp
 $Comp
-L spice:0 #GND1
+L spice:0 #GND6
 U 1 1 5AEBB527
 P 575 3550
-F 0 "#GND1" H 575 3450 60  0001 C CNN
+F 0 "#GND6" H 575 3450 60  0001 C CNN
 F 1 "0" H 575 3480 60  0000 C CNN
 F 2 "" H 575 3550 60  0000 C CNN

Commit message: b
Parts:
- renumbered C2 to C4, C3 to C5, U2 to U4, U3 to U5
Changed lines of the file:
@@
 $Descr A4 11693 8268
 encoding utf-8
-Sheet 3 90
+Sheet 3 92
 Title ""
 Date ""
@@
 Z7
 $Comp
-L myCpu-rescue:4081 U2
+L myCpu-rescue:4081 U4
 U 1 1 5AE63E39
 P 1325 3650
-F 0 "U2" H 1325 3700 50  0000 C CNN
+F 0 "U4" H 1325 3700 50  0000 C CNN
 F 1 "4081" H 1325 3600 50  0000 C CNN
 F 2 "" H 1325 3650 60  0001 C CNN
@@
 $EndComp
 $Comp
-L myCpu-rescue:4081 U2
+L myCpu-rescue:4081 U4
 U 2 1 5AE63EAA
 P 1925 3650
-F 0 "U2" H 1925 3700 50  0000 C CNN
+F 0 "U4" H 1925 3700 50  0000 C CNN
 F 1 "4081" H 1925 3600 50  0000 C CNN
 F 2 "" H 1925 3650 60  0001 C CNN
@@
 $EndComp
 $Comp
-L myCpu-rescue:4081 U2
+L myCpu-rescue:4081 U4
 U 3 1 5AE63F35
 P 2575 3575
-F 0 "U2" H 2575 3625 50  0000 C CNN
+F 0 "U4" H 2575 3625 50  0000 C CNN
 F 1 "4081" H 2575 3525 50  0000 C CNN
 F 2 "" H 2575 3575 60  0001 C CNN
@@
 $EndComp
 $Comp
-L myCpu-rescue:4081 U2
+L myCpu-rescue:4081 U4
 U 4 1 5AE63FD4
 P 3300 3525
-F 0 "U2" H 3300 3575 50  0000 C CNN
+F 0 "U4" H 3300 3575 50  0000 C CNN
 F 1 "4081" H 3300 3475 50  0000 C CNN
 F 2 "" H 3300 3525 60  0001 C CNN
@@
 	5950 7250 5950 4125
 $Comp
-L myCpu-rescue:4081 U3
+L myCpu-rescue:4081 U5
 U 1 1 5AE64A18
 P 3875 3650
-F 0 "U3" H 3875 3700 50  0000 C CNN
+F 0 "U5" H 3875 3700 50  0000 C CNN
 F 1 "4081" H 3875 3600 50  0000 C CNN
 F 2 "" H 3875 3650 60  0001 C CNN
@@
 $EndComp
 $Comp
-L myCpu-rescue:4081 U3
+L myCpu-rescue:4081 U5
 U 2 1 5AE64ABB
 P 4475 3650
-F 0 "U3" H 4475 3700 50  0000 C CNN
+F 0 "U5" H 4475 3700 50  0000 C CNN
 F 1 "4081" H 4475 3600 50  0000 C CNN
 F 2 "" H 4475 3650 60  0001 C CNN
@@
 $EndComp
 $Comp
-L myCpu-rescue:4081 U3
+L myCpu-rescue:4081 U5
 U 3 1 5AE64B4C
 P 5125 3575
-F 0 "U3" H 5125 3625 50  0000 C CNN
+F 0 "U5" H 5125 3625 50  0000 C CNN
 F 1 "4081" H 5125 3525 50  0000 C CNN
 F 2 "" H 5125 3575 60  0001 C CNN
@@
 $EndComp
 $Comp
-L myCpu-rescue:4081 U3
+L myCpu-rescue:4081 U5
 U 4 1 5AE64BBD
 P 5850 3525
-F 0 "U3" H 5850 3575 50  0000 C CNN
+F 0 "U5" H 5850 3575 50  0000 C CNN
 F 1 "4081" H 5850 3475 50  0000 C CNN
 F 2 "" H 5850 3525 60  0001 C CNN
@@
 	4775 2925 5850 2925
 $Comp
-L myCpu-rescue:VCC #PWR05
+L myCpu-rescue:VCC #PWR08
 U 1 1 5AE75990
 P 775 4000
-F 0 "#PWR05" H 775 3850 50  0001 C CNN
+F 0 "#PWR08" H 775 3850 50  0001 C CNN
 F 1 "VCC" H 775 4150 50  0000 C CNN
 F 2 "" H 775 4000 50  0000 C CNN
@@
 $EndComp
 $Comp
-L myCpu-rescue:VCC #PWR06
+L myCpu-rescue:VCC #PWR09
 U 1 1 5AE759C2
 P 6500 4100
-F 0 "#PWR06" H 6500 3950 50  0001 C CNN
+F 0 "#PWR09" H 6500 3950 50  0001 C CNN
 F 1 "VCC" H 6500 4250 50  0000 C CNN
 F 2 "" H 6500 4100 50  0000 C CNN
@@
 	750  4000 775  4000
 $Comp
-L spice:C C2
+L spice:C C4
 U 1 1 5AEBB378
 P 750 3750
-F 0 "C2" V 600 3750 60  0000 C CNN
+F 0 "C4" V 600 3750 60  0000 C CNN
 F 1 "100nF" V 900 3750 60  0000 C CNN
 F 2 "" H 750 3750 60  0000 C CNN
@@
 $EndComp
 $Comp
-L spice:C C3
+L spice:C C5
 U 1 1 5AEBB40C
 P 6375 3825
-F 0 "C3" V 6225 3825 60  0000 C CNN
+F 0 "C5" V 6225 3825 60  0000 C CNN
 F 1 "100nF" V 6525 3825 60  0000 C CNN
 F 2 "" H 6375 3825 60  0000 C CNN
@@
 $EndComp
 $Comp
-L spice:0 #GND7
+L spice:0 #GND4
 U 1 1 5AEBB4E1
 P 6250 3575
-F 0 "#GND7" H 6250 3475 60  0001 C CNN
+F 0 "#GND4" H 6250 3475 60  0001 C CNN
 F 1 "0" H 6250 3505 60  0000 C CNN
 F 2 "" H 6250 3575 60  0000 C CNN
@@
 $EndComp
 $Comp
-L spice:0 #GND6
+L spice:0 #GND3
 U 1 1 5AEBB527
 P 575 3550
-F 0 "#GND6" H 575 3450 60  0001 C CNN
+F 0 "#GND3" H 575 3450 60  0001 C CNN
 F 1 "0" H 575 3480 60  0000 C CNN
 F 2 "" H 575 3550 60  0000 C CNN
