File: AND.sch (KiCad schematic (older format))
At the start: 4 parts, among them U4 4081, U5 4081

Commit message: message
Parts:
- renumbered U5 to U10, U4 to U7, U4 to U8, U5 to U9
Changed lines of the file:
@@
 $Descr A4 11693 8268
 encoding utf-8
-Sheet 3 92
+Sheet 3 101
 Title ""
 Date ""
@@
 Z7
 $Comp
-L myCpu-rescue:4081 U4
+L myCpu-rescue:4081 U7
 U 1 1 5AE63E39
 P 1325 3650
-F 0 "U4" H 1325 3700 50  0000 C CNN
+F 0 "U7" H 1325 3700 50  0000 C CNN
 F 1 "4081" H 1325 3600 50  0000 C CNN
 F 2 "" H 1325 3650 60  0001 C CNN
@@
 $EndComp
 $Comp
-L myCpu-rescue:4081 U4
+L myCpu-rescue:4081 U7
 U 2 1 5AE63EAA
 P 1925 3650
-F 0 "U4" H 1925 3700 50  0000 C CNN
+F 0 "U7" H 1925 3700 50  0000 C CNN
 F 1 "4081" H 1925 3600 50  0000 C CNN
 F 2 "" H 1925 3650 60  0001 C CNN
@@
 $EndComp
 $Comp
-L myCpu-rescue:4081 U4
+L myCpu-rescue:4081 U8
 U 3 1 5AE63F35
 P 2575 3575
-F 0 "U4" H 2575 3625 50  0000 C CNN
+F 0 "U8" H 2575 3625 50  0000 C CNN
 F 1 "4081" H 2575 3525 50  0000 C CNN
 F 2 "" H 2575 3575 60  0001 C CNN
@@
 $EndComp
 $Comp
-L myCpu-rescue:4081 U4
+L myCpu-rescue:4081 U8
 U 4 1 5AE63FD4
 P 3300 3525
-F 0 "U4" H 3300 3575 50  0000 C CNN
+F 0 "U8" H 3300 3575 50  0000 C CNN
 F 1 "4081" H 3300 3475 50  0000 C CNN
 F 2 "" H 3300 3525 60  0001 C CNN
@@
 	5950 7250 5950 4125
 $Comp
-L myCpu-rescue:4081 U5
+L myCpu-rescue:4081 U9
 U 1 1 5AE64A18
 P 3875 3650
-F 0 "U5" H 3875 3700 50  0000 C CNN
+F 0 "U9" H 3875 3700 50  0000 C CNN
 F 1 "4081" H 3875 3600 50  0000 C CNN
 F 2 "" H 3875 3650 60  0001 C CNN
@@
 $EndComp
 $Comp
-L myCpu-rescue:4081 U5
+L myCpu-rescue:4081 U9
 U 2 1 5AE64ABB
 P 4475 3650
-F 0 "U5" H 4475 3700 50  0000 C CNN
+F 0 "U9" H 4475 3700 50  0000 C CNN
 F 1 "4081" H 4475 3600 50  0000 C CNN
 F 2 "" H 4475 3650 60  0001 C CNN
@@
 $EndComp
 $Comp
-L myCpu-rescue:4081 U5
+L myCpu-rescue:4081 U10
 U 3 1 5AE64B4C
 P 5125 3575
-F 0 "U5" H 5125 3625 50  0000 C CNN
+F 0 "U10" H 5125 3625 50  0000 C CNN
 F 1 "4081" H 5125 3525 50  0000 C CNN
 F 2 "" H 5125 3575 60  0001 C CNN
@@
 $EndComp
 $Comp
-L myCpu-rescue:4081 U5
+L myCpu-rescue:4081 U10
 U 4 1 5AE64BBD
 P 5850 3525
-F 0 "U5" H 5850 3575 50  0000 C CNN
+F 0 "U10" H 5850 3575 50  0000 C CNN
 F 1 "4081" H 5850 3475 50  0000 C CNN
 F 2 "" H 5850 3525 60  0001 C CNN
@@
 	4775 2925 5850 2925
 $Comp
-L myCpu-rescue:VCC #PWR08
+L myCpu-rescue:VCC #PWR010
 U 1 1 5AE75990
 P 775 4000
-F 0 "#PWR08" H 775 3850 50  0001 C CNN
+F 0 "#PWR010" H 775 3850 50  0001 C CNN
 F 1 "VCC" H 775 4150 50  0000 C CNN
 F 2 "" H 775 4000 50  0000 C CNN
@@
 $EndComp
 $Comp
-L myCpu-rescue:VCC #PWR09
+L myCpu-rescue:VCC #PWR011
 U 1 1 5AE759C2
 P 6500 4100
-F 0 "#PWR09" H 6500 3950 50  0001 C CNN
+F 0 "#PWR011" H 6500 3950 50  0001 C CNN
 F 1 "VCC" H 6500 4250 50  0000 C CNN
 F 2 "" H 6500 4100 50  0000 C CNN
@@
 $EndComp
 $Comp
-L spice:0 #GND4
+L spice:0 #GND3
 U 1 1 5AEBB4E1
 P 6250 3575
-F 0 "#GND4" H 6250 3475 60  0001 C CNN
+F 0 "#GND3" H 6250 3475 60  0001 C CNN
 F 1 "0" H 6250 3505 60  0000 C CNN
 F 2 "" H 6250 3575 60  0000 C CNN
@@
 $EndComp
 $Comp
-L spice:0 #GND3
+L spice:0 #GND2
 U 1 1 5AEBB527
 P 575 3550
-F 0 "#GND3" H 575 3450 60  0001 C CNN
+F 0 "#GND2" H 575 3450 60  0001 C CNN
 F 1 "0" H 575 3480 60  0000 C CNN
 F 2 "" H 575 3550 60  0000 C CNN
