File: INC8.sch (KiCad schematic (older format))
At the start: 4 parts, among them U9 74LS283

Commit message: wiring
Parts:
- gave numbers to parts that had none: 2
Changed lines of the file:
@@
 $Descr A4 11693 8268
 encoding utf-8
-Sheet 7 8
+Sheet 7 20
 Title ""
 Date ""
@@
 $EndComp
 $Comp
-L GND #PWR4
+L GND #PWR8
 U 1 1 5AE74CA3
 P 1975 5475
-F 0 "#PWR4" H 1975 5225 50  0001 C CNN
+F 0 "#PWR8" H 1975 5225 50  0001 C CNN
 F 1 "GND" H 1975 5325 50  0000 C CNN
 F 2 "" H 1975 5475 50  0000 C CNN
@@
 $EndComp
 $Comp
-L VCC #PWR3
+L VCC #PWR7
 U 1 1 5AE74CB9
 P 875 5275
-F 0 "#PWR3" H 875 5125 50  0001 C CNN
+F 0 "#PWR7" H 875 5125 50  0001 C CNN
 F 1 "VCC" H 875 5425 50  0000 C CNN
 F 2 "" H 875 5275 50  0000 C CNN
@@
 	875  4675 875  5275
 $Comp
-L GND #PWR2
+L GND #PWR6
 U 1 1 5AE74F65
 P 875 4075
-F 0 "#PWR2" H 875 3825 50  0001 C CNN
+F 0 "#PWR6" H 875 3825 50  0001 C CNN
 F 1 "GND" H 875 3925 50  0000 C CNN
 F 2 "" H 875 4075 50  0000 C CNN
@@
 	875  4075 875  4375
 $Comp
-L 74LS283 U?
+L 74LS283 U10
 U 1 1 5AE74FBD
 P 3575 4700
-F 0 "U?" H 3575 4700 50  0000 C CNN
+F 0 "U10" H 3575 4700 50  0000 C CNN
 F 1 "74LS283" H 3625 4350 50  0000 C CNN
 F 2 "" H 3575 4700 50  0000 C CNN
@@
 $EndComp
 $Comp
-L C C?
+L C C4
 U 1 1 5AE75052
 P 2900 4600
-F 0 "C?" H 2925 4700 50  0000 L CNN
+F 0 "C4" H 2925 4700 50  0000 L CNN
 F 1 "100n" H 2925 4500 50  0000 L CNN
 F 2 "" H 2938 4450 50  0000 C CNN
@@
 $EndComp
 $Comp
-L GND #PWR?
+L GND #PWR9
 U 1 1 5AE750AB
 P 2875 4225
-F 0 "#PWR?" H 2875 3975 50  0001 C CNN
+F 0 "#PWR9" H 2875 3975 50  0001 C CNN
 F 1 "GND" H 2875 4075 50  0000 C CNN
 F 2 "" H 2875 4225 50  0000 C CNN
@@
 $EndComp
 $Comp
-L VCC #PWR?
+L VCC #PWR10
 U 1 1 5AE750C7
 P 2875 4975
-F 0 "#PWR?" H 2875 4825 50  0001 C CNN
+F 0 "#PWR10" H 2875 4825 50  0001 C CNN
 F 1 "VCC" H 2875 5125 50  0000 C CNN
 F 2 "" H 2875 4975 50  0000 C CNN
@@
 	2900 4225 2875 4225
 $Comp
-L GND #PWR?
+L GND #PWR11
 U 1 1 5AE7515A
 P 4125 5625
-F 0 "#PWR?" H 4125 5375 50  0001 C CNN
+F 0 "#PWR11" H 4125 5375 50  0001 C CNN
 F 1 "GND" H 4125 5475 50  0000 C CNN
 F 2 "" H 4125 5625 50  0000 C CNN

Commit message: SPICE capacitance and ground symbols
Parts:
- removed C1, C4: 100n, symbol C
- added C? (x2): 100nF, symbol C
Connections:
- net labels added: 0
- net labels removed: GND
- wire segments 61 -> 63
Changed lines of the file:
@@
 EESchema Schematic File Version 2
-LIBS:power
-LIBS:device
-LIBS:transistors
-LIBS:conn
-LIBS:linear
-LIBS:regul
-LIBS:74xx
-LIBS:cmos4000
-LIBS:adc-dac
-LIBS:memory
-LIBS:xilinx
-LIBS:microcontrollers
-LIBS:dsp
-LIBS:microchip
-LIBS:analog_switches
-LIBS:motorola
-LIBS:texas
-LIBS:intel
-LIBS:audio
-LIBS:interface
-LIBS:digital-audio
-LIBS:philips
-LIBS:display
-LIBS:cypress
-LIBS:siliconi
-LIBS:opto
-LIBS:atmel
-LIBS:contrib
-LIBS:valves
+LIBS:spice
+LIBS:pspice
 LIBS:myCpu-cache
 EELAYER 25 0
@@
 	0    -1   -1   0
 $EndComp
-$Comp
-L GND #PWR8
-U 1 1 5AE74CA3
-P 1975 5475
-F 0 "#PWR8" H 1975 5225 50  0001 C CNN
-F 1 "GND" H 1975 5325 50  0000 C CNN
-F 2 "" H 1975 5475 50  0000 C CNN
-F 3 "" H 1975 5475 50  0000 C CNN
-	1    1975 5475
-	1    0    0    -1
-$EndComp
-$Comp
-L VCC #PWR7
-U 1 1 5AE74CB9
-P 875 5275
-F 0 "#PWR7" H 875 5125 50  0001 C CNN
-F 1 "VCC" H 875 5425 50  0000 C CNN
-F 2 "" H 875 5275 50  0000 C CNN
-F 3 "" H 875 5275 50  0000 C CNN
-	1    875  5275
-	1    0    0    -1
-$EndComp
 Wire Wire Line
 	1075 6500 1075 5525
@@
 	2000 5475 2000 5275
 Wire Wire Line
-	875  5275 1100 5275
-$Comp
-L C C1
-U 1 1 5AE74D99
-P 875 4525
-F 0 "C1" H 900 4625 50  0000 L CNN
-F 1 "100n" H 900 4425 50  0000 L CNN
-F 2 "" H 913 4375 50  0000 C CNN
-F 3 "" H 875 4525 50  0000 C CNN
-	1    875  4525
-	1    0    0    -1
-$EndComp
-Wire Wire Line
-	875  4675 875  5275
-$Comp
-L GND #PWR6
-U 1 1 5AE74F65
-P 875 4075
-F 0 "#PWR6" H 875 3825 50  0001 C CNN
-F 1 "GND" H 875 3925 50  0000 C CNN
-F 2 "" H 875 4075 50  0000 C CNN
-F 3 "" H 875 4075 50  0000 C CNN
-	1    875  4075
-	1    0    0    -1
-$EndComp
-Wire Wire Line
-	875  4075 875  4375
+	775  5275 1100 5275
 $Comp
 L 74LS283 U10
@@
 	0    -1   -1   0
 $EndComp
-$Comp
-L C C4
-U 1 1 5AE75052
-P 2900 4600
-F 0 "C4" H 2925 4700 50  0000 L CNN
-F 1 "100n" H 2925 4500 50  0000 L CNN
-F 2 "" H 2938 4450 50  0000 C CNN
-F 3 "" H 2900 4600 50  0000 C CNN
-	1    2900 4600
-	1    0    0    -1
-$EndComp
-$Comp
-L GND #PWR9
-U 1 1 5AE750AB
-P 2875 4225
-F 0 "#PWR9" H 2875 3975 50  0001 C CNN
-F 1 "GND" H 2875 4075 50  0000 C CNN
-F 2 "" H 2875 4225 50  0000 C CNN
-F 3 "" H 2875 4225 50  0000 C CNN
-	1    2875 4225
-	1    0    0    -1
-$EndComp
-$Comp
-L VCC #PWR10
-U 1 1 5AE750C7
-P 2875 4975
-F 0 "#PWR10" H 2875 4825 50  0001 C CNN
-F 1 "VCC" H 2875 5125 50  0000 C CNN
-F 2 "" H 2875 4975 50  0000 C CNN
-F 3 "" H 2875 4975 50  0000 C CNN
-	1    2875 4975
-	1    0    0    -1
-$EndComp
-Wire Wire Line
-	2875 4975 2875 4750
-Wire Wire Line
-	2875 4750 2900 4750
-Wire Wire Line
-	2900 4450 2900 4225
-Wire Wire Line
-	2900 4225 2875 4225
-$Comp
-L GND #PWR11
-U 1 1 5AE7515A
-P 4125 5625
-F 0 "#PWR11" H 4125 5375 50  0001 C CNN
-F 1 "GND" H 4125 5475 50  0000 C CNN
-F 2 "" H 4125 5625 50  0000 C CNN
-F 3 "" H 4125 5625 50  0000 C CNN
-	1    4125 5625
-	1    0    0    -1
-$EndComp
 Wire Wire Line
 	3725 5400 4125 5400
@@
 Connection ~ 3925 5400
 Wire Wire Line
-	4125 5400 4125 5625
+	4125 5400 4125 5650
 Connection ~ 4025 5400
 Wire Wire Line
@@
 Wire Wire Line
 	4375 4000 4375 2800
+$Comp
+L 0 #GND?
+U 1 1 5AEB8305
+P 700 4200
+F 0 "#GND?" H 700 4100 60  0001 C CNN
+F 1 "0" H 700 4130 60  0000 C CNN
+F 2 "" H 700 4200 60  0000 C CNN
+F 3 "" H 700 4200 60  0000 C CNN
+	1    700  4200
+	1    0    0    -1
+$EndComp
+$Comp
+L 0 #GND?
+U 1 1 5AEB831D
+P 2850 4300
+F 0 "#GND?" H 2850 4200 60  0001 C CNN
+F 1 "0" H 2850 4230 60  0000 C CNN
+F 2 "" H 2850 4300 60  0000 C CNN
+F 3 "" H 2850 4300 60  0000 C CNN
+	1    2850 4300
+	1    0    0    -1
+$EndComp
+$Comp
+L C C?
+U 1 1 5AEB8335
+P 650 4675
+F 0 "C?" V 500 4675 60  0000 C CNN
+F 1 "100nF" V 800 4675 60  0000 C CNN
+F 2 "" H 650 4675 60  0000 C CNN
+F 3 "" H 650 4675 60  0000 C CNN
+	1    650  4675
+	1    0    0    -1
+$EndComp
+$Comp
+L C C?
+U 1 1 5AEB839C
+P 2675 4750
+F 0 "C?" V 2525 4750 60  0000 C CNN
+F 1 "100nF" V 2825 4750 60  0000 C CNN
+F 2 "" H 2675 4750 60  0000 C CNN
+F 3 "" H 2675 4750 60  0000 C CNN
+	1    2675 4750
+	1    0    0    -1
+$EndComp
+$Comp
+L 0 #GND?
+U 1 1 5AEB8401
+P 4125 5650
+F 0 "#GND?" H 4125 5550 60  0001 C CNN
+F 1 "0" H 4125 5580 60  0000 C CNN
+F 2 "" H 4125 5650 60  0000 C CNN
+F 3 "" H 4125 5650 60  0000 C CNN
+	1    4125 5650
+	1    0    0    -1
+$EndComp
+$Comp
+L 0 #GND?
+U 1 1 5AEB841D
+P 1975 5575
+F 0 "#GND?" H 1975 5475 60  0001 C CNN
+F 1 "0" H 1975 5505 60  0000 C CNN
+F 2 "" H 1975 5575 60  0000 C CNN
+F 3 "" H 1975 5575 60  0000 C CNN
+	1    1975 5575
+	1    0    0    -1
+$EndComp
+$Comp
+L VCC #PWR?
+U 1 1 5AEB8439
+P 2525 5000
+F 0 "#PWR?" H 2525 4850 50  0001 C CNN
+F 1 "VCC" H 2525 5150 50  0000 C CNN
+F 2 "" H 2525 5000 50  0000 C CNN
+F 3 "" H 2525 5000 50  0000 C CNN
+	1    2525 5000
+	1    0    0    -1
+$EndComp
+$Comp
+L VCC #PWR?
+U 1 1 5AEB8455
+P 775 4900
+F 0 "#PWR?" H 775 4750 50  0001 C CNN
+F 1 "VCC" H 775 5050 50  0000 C CNN
+F 2 "" H 775 4900 50  0000 C CNN
+F 3 "" H 775 4900 50  0000 C CNN
+	1    775  4900
+	1    0    0    -1
+$EndComp
+Wire Wire Line
+	775  4900 775  5275
+Wire Wire Line
+	650  4925 775  4925
+Connection ~ 775  4925
+Wire Wire Line
+	650  4425 700  4425
+Wire Wire Line
+	700  4425 700  4200
+Wire Wire Line
+	2850 4300 2675 4300
+Wire Wire Line
+	2675 4300 2675 4500
+Wire Wire Line
+	2675 5000 2525 5000
+Wire Wire Line
+	1975 5475 1975 5575
 $EndSCHEMATC

Commit message: fixed duplicate names
Parts:
- gave numbers to parts that had none: 2
Changed lines of the file:
@@
 $Descr A4 11693 8268
 encoding utf-8
-Sheet 7 21
+Sheet 20 21
 Title ""
 Date ""
@@
 U 1 1 5AE74BC6
 P 1550 4575
-F 0 "U9" H 1550 4575 50  0000 C CNN
+AR Path="/5AE62FB7/5AE74AF7/5AE74BC6" Ref="U9"  Part="1"
+AR Path="/5AE62FB7/5AF84E03/5AE74BC6" Ref="U35"  Part="1"
+F 0 "U35" H 1550 4575 50  0000 C CNN
 F 1 "74LS283" H 1600 4225 50  0000 C CNN
 F 2 "" H 1550 4575 50  0000 C CNN
@@
 U 1 1 5AE74FBD
 P 3575 4700
-F 0 "U10" H 3575 4700 50  0000 C CNN
+AR Path="/5AE62FB7/5AE74AF7/5AE74FBD" Ref="U10"  Part="1"
+AR Path="/5AE62FB7/5AF84E03/5AE74FBD" Ref="U36"  Part="1"
+F 0 "U36" H 3575 4700 50  0000 C CNN
 F 1 "74LS283" H 3625 4350 50  0000 C CNN
 F 2 "" H 3575 4700 50  0000 C CNN
@@
 	4375 4000 4375 2800
 $Comp
-L 0 #GND?
+L 0 #GND7
 U 1 1 5AEB8305
 P 700 4200
-F 0 "#GND?" H 700 4100 60  0001 C CNN
+AR Path="/5AE62FB7/5AE74AF7/5AEB8305" Ref="#GND7"  Part="1"
+AR Path="/5AE62FB7/5AF84E03/5AEB8305" Ref="#GND35"  Part="1"
+F 0 "#GND35" H 700 4100 60  0001 C CNN
 F 1 "0" H 700 4130 60  0000 C CNN
 F 2 "" H 700 4200 60  0000 C CNN
@@
 $EndComp
 $Comp
-L 0 #GND?
+L 0 #GND9
 U 1 1 5AEB831D
 P 2850 4300
-F 0 "#GND?" H 2850 4200 60  0001 C CNN
+AR Path="/5AE62FB7/5AE74AF7/5AEB831D" Ref="#GND9"  Part="1"
+AR Path="/5AE62FB7/5AF84E03/5AEB831D" Ref="#GND37"  Part="1"
+F 0 "#GND37" H 2850 4200 60  0001 C CNN
 F 1 "0" H 2850 4230 60  0000 C CNN
 F 2 "" H 2850 4300 60  0000 C CNN
@@
 $EndComp
 $Comp
-L C C?
+L C C7
 U 1 1 5AEB8335
 P 650 4675
-F 0 "C?" V 500 4675 60  0000 C CNN
+AR Path="/5AE62FB7/5AE74AF7/5AEB8335" Ref="C7"  Part="1"
+AR Path="/5AE62FB7/5AF84E03/5AEB8335" Ref="C33"  Part="1"
+F 0 "C33" V 500 4675 60  0000 C CNN
 F 1 "100nF" V 800 4675 60  0000 C CNN
 F 2 "" H 650 4675 60  0000 C CNN
@@
 $EndComp
 $Comp
-L C C?
+L C C8
 U 1 1 5AEB839C
 P 2675 4750
-F 0 "C?" V 2525 4750 60  0000 C CNN
+AR Path="/5AE62FB7/5AE74AF7/5AEB839C" Ref="C8"  Part="1"
+AR Path="/5AE62FB7/5AF84E03/5AEB839C" Ref="C34"  Part="1"
+F 0 "C34" V 2525 4750 60  0000 C CNN
 F 1 "100nF" V 2825 4750 60  0000 C CNN
 F 2 "" H 2675 4750 60  0000 C CNN
@@
 $EndComp
 $Comp
-L 0 #GND?
+L 0 #GND10
 U 1 1 5AEB8401
 P 4125 5650
-F 0 "#GND?" H 4125 5550 60  0001 C CNN
+AR Path="/5AE62FB7/5AE74AF7/5AEB8401" Ref="#GND10"  Part="1"
+AR Path="/5AE62FB7/5AF84E03/5AEB8401" Ref="#GND38"  Part="1"
+F 0 "#GND38" H 4125 5550 60  0001 C CNN
 F 1 "0" H 4125 5580 60  0000 C CNN
 F 2 "" H 4125 5650 60  0000 C CNN
@@
 $EndComp
 $Comp
-L 0 #GND?
+L 0 #GND8
 U 1 1 5AEB841D
 P 1975 5575
-F 0 "#GND?" H 1975 5475 60  0001 C CNN
+AR Path="/5AE62FB7/5AE74AF7/5AEB841D" Ref="#GND8"  Part="1"
+AR Path="/5AE62FB7/5AF84E03/5AEB841D" Ref="#GND36"  Part="1"
+F 0 "#GND36" H 1975 5475 60  0001 C CNN
 F 1 "0" H 1975 5505 60  0000 C CNN
 F 2 "" H 1975 5575 60  0000 C CNN
@@
 $EndComp
 $Comp
-L VCC #PWR?
+L VCC #PWR08
 U 1 1 5AEB8439
 P 2525 5000
-F 0 "#PWR?" H 2525 4850 50  0001 C CNN
+AR Path="/5AE62FB7/5AE74AF7/5AEB8439" Ref="#PWR08"  Part="1"
+AR Path="/5AE62FB7/5AF84E03/5AEB8439" Ref="#PWR035"  Part="1"
+F 0 "#PWR035" H 2525 4850 50  0001 C CNN
 F 1 "VCC" H 2525 5150 50  0000 C CNN
 F 2 "" H 2525 5000 50  0000 C CNN
@@
 $EndComp
 $Comp
-L VCC #PWR?
+L VCC #PWR09
 U 1 1 5AEB8455
 P 775 4900
-F 0 "#PWR?" H 775 4750 50  0001 C CNN
+AR Path="/5AE62FB7/5AE74AF7/5AEB8455" Ref="#PWR09"  Part="1"
+AR Path="/5AE62FB7/5AF84E03/5AEB8455" Ref="#PWR036"  Part="1"
+F 0 "#PWR036" H 775 4750 50  0001 C CNN
 F 1 "VCC" H 775 5050 50  0000 C CNN
 F 2 "" H 775 4900 50  0000 C CNN

Commit message: spice libs from the internet, opened with new kicad 5.0.0, added spice models to components
Parts:
- C7, C8: symbol C -> spice:C
- U10: symbol 74LS283 -> myCpu-rescue:74LS283
- U9: symbol 74LS283 -> myCpu-rescue:74LS283; Spice_Lib_File (none) -> 74hc.lib; Spice_Model (none) -> 74HC283; Spice_Netlist_Enabled (none) -> Y; Spice_Primitive (none) -> X
Connections:
- wire segments 63 -> 67
Changed lines of the file:
@@
-EESchema Schematic File Version 2
-LIBS:spice
-LIBS:pspice
+EESchema Schematic File Version 4
 LIBS:myCpu-cache
-EELAYER 25 0
+EELAYER 26 0
 EELAYER END
 $Descr A4 11693 8268
 encoding utf-8
-Sheet 20 21
+Sheet 21 21
 Title ""
 Date ""
@@
 Z7
 $Comp
-L 74LS283 U9
+L myCpu-rescue:74LS283 U9
 U 1 1 5AE74BC6
 P 1550 4575
@@
 F 2 "" H 1550 4575 50  0000 C CNN
 F 3 "" H 1550 4575 50  0000 C CNN
+F 4 "X" H 1550 4575 50  0001 C CNN "Spice_Primitive"
+F 5 "74HC283" H 1550 4575 50  0001 C CNN "Spice_Model"
+F 6 "Y" H 1550 4575 50  0001 C CNN "Spice_Netlist_Enabled"
+F 7 "74hc.lib" H 1550 4575 50  0001 C CNN "Spice_Lib_File"
 	1    1550 4575
 	0    -1   -1   0
@@
 	1875 5950 1875 6575
 Wire Wire Line
-	1700 5275 1900 5275
+	1700 5275 1800 5275
 Connection ~ 1800 5275
-Wire Wire Line
-	2000 5275 1875 5275
 Connection ~ 1875 5275
 Wire Wire Line
@@
 	775  5275 1100 5275
 $Comp
-L 74LS283 U10
+L myCpu-rescue:74LS283 U10
 U 1 1 5AE74FBD
 P 3575 4700
@@
 $EndComp
 Wire Wire Line
-	3725 5400 4125 5400
+	3725 5400 3825 5400
 Connection ~ 3825 5400
 Connection ~ 3925 5400
@@
 	4375 4000 4375 2800
 $Comp
-L 0 #GND7
+L spice:0 #GND7
 U 1 1 5AEB8305
 P 700 4200
@@
 $EndComp
 $Comp
-L 0 #GND9
+L spice:0 #GND9
 U 1 1 5AEB831D
 P 2850 4300
@@
 $EndComp
 $Comp
-L C C7
+L spice:C C7
 U 1 1 5AEB8335
 P 650 4675
@@
 $EndComp
 $Comp
-L C C8
+L spice:C C8
 U 1 1 5AEB839C
 P 2675 4750
@@
 $EndComp
 $Comp
-L 0 #GND10
+L spice:0 #GND10
 U 1 1 5AEB8401
 P 4125 5650
@@
 $EndComp
 $Comp
-L 0 #GND8
+L spice:0 #GND8
 U 1 1 5AEB841D
 P 1975 5575
@@
 $EndComp
 $Comp
-L VCC #PWR08
+L myCpu-rescue:VCC #PWR08
 U 1 1 5AEB8439
 P 2525 5000
@@
 $EndComp
 $Comp
-L VCC #PWR09
+L myCpu-rescue:VCC #PWR09
 U 1 1 5AEB8455
 P 775 4900
@@
 $EndComp
 Wire Wire Line
-	775  4900 775  5275
+	775  4900 775  4925
 Wire Wire Line
 	650  4925 775  4925
@@
 Wire Wire Line
 	1975 5475 1975 5575
+Wire Wire Line
+	3825 5400 3925 5400
+Wire Wire Line
+	3925 5400 4025 5400
+Wire Wire Line
+	4025 5400 4125 5400
+Wire Wire Line
+	775  4925 775  5275
+Wire Wire Line
+	1800 5275 2000 5275
 $EndSCHEMATC

Commit message: lots of work done
Parts:
- renumbered C7 to C?, C8 to C?, U9 to U?, U10 to U?
Changed lines of the file:
@@
 $Descr A4 11693 8268
 encoding utf-8
-Sheet 21 21
+Sheet 76 81
 Title ""
 Date ""
@@
 Z7
 $Comp
-L myCpu-rescue:74LS283 U9
+L myCpu-rescue:74LS283 U?
 U 1 1 5AE74BC6
 P 1550 4575
-AR Path="/5AE62FB7/5AE74AF7/5AE74BC6" Ref="U9"  Part="1"
-AR Path="/5AE62FB7/5AF84E03/5AE74BC6" Ref="U35"  Part="1"
-F 0 "U35" H 1550 4575 50  0000 C CNN
+F 0 "U?" H 1550 4575 50  0000 C CNN
 F 1 "74LS283" H 1600 4225 50  0000 C CNN
 F 2 "" H 1550 4575 50  0000 C CNN
@@
 	1700 5275 1800 5275
 Connection ~ 1800 5275
-Connection ~ 1875 5275
 Wire Wire Line
 	1975 5475 2000 5475
@@
 	775  5275 1100 5275
 $Comp
-L myCpu-rescue:74LS283 U10
+L myCpu-rescue:74LS283 U?
 U 1 1 5AE74FBD
 P 3575 4700
-AR Path="/5AE62FB7/5AE74AF7/5AE74FBD" Ref="U10"  Part="1"
-AR Path="/5AE62FB7/5AF84E03/5AE74FBD" Ref="U36"  Part="1"
-F 0 "U36" H 3575 4700 50  0000 C CNN
+F 0 "U?" H 3575 4700 50  0000 C CNN
 F 1 "74LS283" H 3625 4350 50  0000 C CNN
 F 2 "" H 3575 4700 50  0000 C CNN
@@
 	4375 4000 4375 2800
 $Comp
-L spice:0 #GND7
+L spice:0 #GND?
 U 1 1 5AEB8305
 P 700 4200
-AR Path="/5AE62FB7/5AE74AF7/5AEB8305" Ref="#GND7"  Part="1"
-AR Path="/5AE62FB7/5AF84E03/5AEB8305" Ref="#GND35"  Part="1"
-F 0 "#GND35" H 700 4100 60  0001 C CNN
+F 0 "#GND?" H 700 4100 60  0001 C CNN
 F 1 "0" H 700 4130 60  0000 C CNN
 F 2 "" H 700 4200 60  0000 C CNN
@@
 $EndComp
 $Comp
-L spice:0 #GND9
+L spice:0 #GND?
 U 1 1 5AEB831D
 P 2850 4300
-AR Path="/5AE62FB7/5AE74AF7/5AEB831D" Ref="#GND9"  Part="1"
-AR Path="/5AE62FB7/5AF84E03/5AEB831D" Ref="#GND37"  Part="1"
-F 0 "#GND37" H 2850 4200 60  0001 C CNN
+F 0 "#GND?" H 2850 4200 60  0001 C CNN
 F 1 "0" H 2850 4230 60  0000 C CNN
 F 2 "" H 2850 4300 60  0000 C CNN
@@
 $EndComp
 $Comp
-L spice:C C7
+L spice:C C?
 U 1 1 5AEB8335
 P 650 4675
-AR Path="/5AE62FB7/5AE74AF7/5AEB8335" Ref="C7"  Part="1"
-AR Path="/5AE62FB7/5AF84E03/5AEB8335" Ref="C33"  Part="1"
-F 0 "C33" V 500 4675 60  0000 C CNN
+F 0 "C?" V 500 4675 60  0000 C CNN
 F 1 "100nF" V 800 4675 60  0000 C CNN
 F 2 "" H 650 4675 60  0000 C CNN
@@
 $EndComp
 $Comp
-L spice:C C8
+L spice:C C?
 U 1 1 5AEB839C
 P 2675 4750
-AR Path="/5AE62FB7/5AE74AF7/5AEB839C" Ref="C8"  Part="1"
-AR Path="/5AE62FB7/5AF84E03/5AEB839C" Ref="C34"  Part="1"
-F 0 "C34" V 2525 4750 60  0000 C CNN
+F 0 "C?" V 2525 4750 60  0000 C CNN
 F 1 "100nF" V 2825 4750 60  0000 C CNN
 F 2 "" H 2675 4750 60  0000 C CNN
@@
 $EndComp
 $Comp
-L spice:0 #GND10
+L spice:0 #GND?
 U 1 1 5AEB8401
 P 4125 5650
-AR Path="/5AE62FB7/5AE74AF7/5AEB8401" Ref="#GND10"  Part="1"
-AR Path="/5AE62FB7/5AF84E03/5AEB8401" Ref="#GND38"  Part="1"
-F 0 "#GND38" H 4125 5550 60  0001 C CNN
+F 0 "#GND?" H 4125 5550 60  0001 C CNN
 F 1 "0" H 4125 5580 60  0000 C CNN
 F 2 "" H 4125 5650 60  0000 C CNN
@@
 $EndComp
 $Comp
-L spice:0 #GND8
+L spice:0 #GND?
 U 1 1 5AEB841D
 P 1975 5575
-AR Path="/5AE62FB7/5AE74AF7/5AEB841D" Ref="#GND8"  Part="1"
-AR Path="/5AE62FB7/5AF84E03/5AEB841D" Ref="#GND36"  Part="1"
-F 0 "#GND36" H 1975 5475 60  0001 C CNN
+F 0 "#GND?" H 1975 5475 60  0001 C CNN
 F 1 "0" H 1975 5505 60  0000 C CNN
 F 2 "" H 1975 5575 60  0000 C CNN
@@
 $EndComp
 $Comp
-L myCpu-rescue:VCC #PWR08
+L myCpu-rescue:VCC #PWR?
 U 1 1 5AEB8439
 P 2525 5000
-AR Path="/5AE62FB7/5AE74AF7/5AEB8439" Ref="#PWR08"  Part="1"
-AR Path="/5AE62FB7/5AF84E03/5AEB8439" Ref="#PWR035"  Part="1"
-F 0 "#PWR035" H 2525 4850 50  0001 C CNN
+F 0 "#PWR?" H 2525 4850 50  0001 C CNN
 F 1 "VCC" H 2525 5150 50  0000 C CNN
 F 2 "" H 2525 5000 50  0000 C CNN
@@
 $EndComp
 $Comp
-L myCpu-rescue:VCC #PWR09
+L myCpu-rescue:VCC #PWR?
 U 1 1 5AEB8455
 P 775 4900
-AR Path="/5AE62FB7/5AE74AF7/5AEB8455" Ref="#PWR09"  Part="1"
-AR Path="/5AE62FB7/5AF84E03/5AEB8455" Ref="#PWR036"  Part="1"
-F 0 "#PWR036" H 775 4750 50  0001 C CNN
+F 0 "#PWR?" H 775 4750 50  0001 C CNN
 F 1 "VCC" H 775 5050 50  0000 C CNN
 F 2 "" H 775 4900 50  0000 C CNN
