File: INC8.sch (KiCad schematic (older format))
At the start: 4 parts

Commit message: b
Parts:
- added R3: 0R1, symbol pspice:R
- C298, C299: renamed from C?; symbol spice:C -> pspice:C
- gave numbers to parts that had none: 2
Connections:
- net labels added: GND
- net labels removed: 0
- wire segments 67 -> 70
Changed lines of the file:
@@
 $Descr A4 11693 8268
 encoding utf-8
-Sheet 76 90
+Sheet 77 92
 Title ""
 Date ""
@@
 Z7
 $Comp
-L myCpu-rescue:74LS283 U?
+L myCpu-rescue:74LS283 U199
 U 1 1 5AE74BC6
 P 1550 4575
-F 0 "U?" H 1550 4575 50  0000 C CNN
+AR Path="/82611AC0/82611C89/82611C8C/5AE74BC6" Ref="U199"  Part="1"
+AR Path="/5AE62FB7/5AE74AF7/5AE74BC6" Ref="U12"  Part="1"
+AR Path="/5AE62FB7/5AF84E03/5AE74BC6" Ref="U40"  Part="1"
+AR Path="/5D3014E7/82611C8C/5AE74BC6" Ref="U227"  Part="1"
+F 0 "U12" H 1550 4575 50  0000 C CNN
 F 1 "74LS283" H 1600 4225 50  0000 C CNN
 F 2 "" H 1550 4575 50  0000 C CNN
@@
 Wire Wire Line
 	2000 5475 2000 5275
-Wire Wire Line
-	775  5275 1100 5275
-$Comp
-L myCpu-rescue:74LS283 U?
+$Comp
+L myCpu-rescue:74LS283 U200
 U 1 1 5AE74FBD
 P 3575 4700
-F 0 "U?" H 3575 4700 50  0000 C CNN
+AR Path="/82611AC0/82611C89/82611C8C/5AE74FBD" Ref="U200"  Part="1"
+AR Path="/5AE62FB7/5AE74AF7/5AE74FBD" Ref="U13"  Part="1"
+AR Path="/5AE62FB7/5AF84E03/5AE74FBD" Ref="U41"  Part="1"
+AR Path="/5D3014E7/82611C8C/5AE74FBD" Ref="U228"  Part="1"
+F 0 "U13" H 3575 4700 50  0000 C CNN
 F 1 "74LS283" H 3625 4350 50  0000 C CNN
 F 2 "" H 3575 4700 50  0000 C CNN
@@
 	4375 4000 4375 2800
 $Comp
-L spice:0 #GND?
-U 1 1 5AEB8305
-P 700 4200
-F 0 "#GND?" H 700 4100 60  0001 C CNN
-F 1 "0" H 700 4130 60  0000 C CNN
-F 2 "" H 700 4200 60  0000 C CNN
-F 3 "" H 700 4200 60  0000 C CNN
-	1    700  4200
-	1    0    0    -1
-$EndComp
-$Comp
-L spice:0 #GND?
-U 1 1 5AEB831D
-P 2850 4300
-F 0 "#GND?" H 2850 4200 60  0001 C CNN
-F 1 "0" H 2850 4230 60  0000 C CNN
-F 2 "" H 2850 4300 60  0000 C CNN
-F 3 "" H 2850 4300 60  0000 C CNN
-	1    2850 4300
-	1    0    0    -1
-$EndComp
-$Comp
-L spice:C C?
+L pspice:C C298
 U 1 1 5AEB8335
 P 650 4675
-F 0 "C?" V 500 4675 60  0000 C CNN
+AR Path="/82611AC0/82611C89/82611C8C/5AEB8335" Ref="C298"  Part="1"
+AR Path="/5AE62FB7/5AE74AF7/5AEB8335" Ref="C10"  Part="1"
+AR Path="/5AE62FB7/5AF84E03/5AEB8335" Ref="C36"  Part="1"
+AR Path="/5D3014E7/82611C8C/5AEB8335" Ref="C326"  Part="1"
+F 0 "C10" V 500 4675 60  0000 C CNN
 F 1 "100nF" V 800 4675 60  0000 C CNN
 F 2 "" H 650 4675 60  0000 C CNN
@@
 $EndComp
 $Comp
-L spice:C C?
+L pspice:C C299
 U 1 1 5AEB839C
 P 2675 4750
-F 0 "C?" V 2525 4750 60  0000 C CNN
+AR Path="/82611AC0/82611C89/82611C8C/5AEB839C" Ref="C299"  Part="1"
+AR Path="/5AE62FB7/5AE74AF7/5AEB839C" Ref="C11"  Part="1"
+AR Path="/5AE62FB7/5AF84E03/5AEB839C" Ref="C37"  Part="1"
+AR Path="/5D3014E7/82611C8C/5AEB839C" Ref="C327"  Part="1"
+F 0 "C11" V 2525 4750 60  0000 C CNN
 F 1 "100nF" V 2825 4750 60  0000 C CNN
 F 2 "" H 2675 4750 60  0000 C CNN
@@
 $EndComp
 $Comp
-L spice:0 #GND?
-U 1 1 5AEB8401
-P 4125 5650
-F 0 "#GND?" H 4125 5550 60  0001 C CNN
-F 1 "0" H 4125 5580 60  0000 C CNN
-F 2 "" H 4125 5650 60  0000 C CNN
-F 3 "" H 4125 5650 60  0000 C CNN
-	1    4125 5650
-	1    0    0    -1
-$EndComp
-$Comp
-L spice:0 #GND?
-U 1 1 5AEB841D
-P 1975 5575
-F 0 "#GND?" H 1975 5475 60  0001 C CNN
-F 1 "0" H 1975 5505 60  0000 C CNN
-F 2 "" H 1975 5575 60  0000 C CNN
-F 3 "" H 1975 5575 60  0000 C CNN
-	1    1975 5575
-	1    0    0    -1
-$EndComp
-$Comp
-L myCpu-rescue:VCC #PWR?
+L myCpu-rescue:VCC #PWR0532
 U 1 1 5AEB8439
 P 2525 5000
-F 0 "#PWR?" H 2525 4850 50  0001 C CNN
+AR Path="/82611AC0/82611C89/82611C8C/5AEB8439" Ref="#PWR0532"  Part="1"
+AR Path="/5AE62FB7/5AE74AF7/5AEB8439" Ref="#PWR020"  Part="1"
+AR Path="/5AE62FB7/5AF84E03/5AEB8439" Ref="#PWR052"  Part="1"
+AR Path="/5D3014E7/82611C8C/5AEB8439" Ref="#PWR0601"  Part="1"
+F 0 "#PWR020" H 2525 4850 50  0001 C CNN
 F 1 "VCC" H 2525 5150 50  0000 C CNN
 F 2 "" H 2525 5000 50  0000 C CNN
@@
 $EndComp
 $Comp
-L myCpu-rescue:VCC #PWR?
+L myCpu-rescue:VCC #PWR0531
 U 1 1 5AEB8455
 P 775 4900
-F 0 "#PWR?" H 775 4750 50  0001 C CNN
+AR Path="/82611AC0/82611C89/82611C8C/5AEB8455" Ref="#PWR0531"  Part="1"
+AR Path="/5AE62FB7/5AE74AF7/5AEB8455" Ref="#PWR019"  Part="1"
+AR Path="/5AE62FB7/5AF84E03/5AEB8455" Ref="#PWR051"  Part="1"
+AR Path="/5D3014E7/82611C8C/5AEB8455" Ref="#PWR0600"  Part="1"
+F 0 "#PWR019" H 775 4750 50  0001 C CNN
 F 1 "VCC" H 775 5050 50  0000 C CNN
 F 2 "" H 775 4900 50  0000 C CNN
@@
 	775  4925 775  5275
 Wire Wire Line
-	1800 5275 2000 5275
+	1800 5275 1900 5275
+Connection ~ 1900 5275
+Wire Wire Line
+	1900 5275 2000 5275
+$Comp
+L pspice:R R3
+U 1 1 5CBC5903
+P 775 5525
+AR Path="/82611AC0/82611C89/82611C8C/5CBC5903" Ref="R3"  Part="1"
+AR Path="/5AE62FB7/5AE74AF7/5CBC5903" Ref="R1"  Part="1"
+AR Path="/5AE62FB7/5AF84E03/5CBC5903" Ref="R2"  Part="1"
+AR Path="/5D3014E7/82611C8C/5CBC5903" Ref="R4"  Part="1"
+F 0 "R1" H 843 5571 50  0000 L CNN
+F 1 "0R1" H 843 5480 50  0000 L CNN
+F 2 "" H 775 5525 60  0001 C CNN
+F 3 "" H 775 5525 60  0001 C CNN
+	1    775  5525
+	1    0    0    -1
+$EndComp
+Wire Wire Line
+	775  5775 975  5775
+Wire Wire Line
+	975  5775 975  5275
+Wire Wire Line
+	975  5275 1100 5275
+$Comp
+L power:GND #PWR0684
+U 1 1 5CF197AB
+P 4125 5650
+AR Path="/5AE62FB7/5AE74AF7/5CF197AB" Ref="#PWR0684"  Part="1"
+AR Path="/5AE62FB7/5AF84E03/5CF197AB" Ref="#PWR0687"  Part="1"
+AR Path="/82611AC0/82611C89/82611C8C/5CF197AB" Ref="#PWR0690"  Part="1"
+AR Path="/5D3014E7/82611C8C/5CF197AB" Ref="#PWR0693"  Part="1"
+F 0 "#PWR0684" H 4125 5650 30  0001 C CNN
+F 1 "GND" H 4125 5580 30  0001 C CNN
+F 2 "" H 4125 5650 60  0001 C CNN
+F 3 "" H 4125 5650 60  0001 C CNN
+	1    4125 5650
+	1    0    0    -1
+$EndComp
+$Comp
+L power:GND #PWR0685
+U 1 1 5CF198E5
+P 1975 5575
+AR Path="/5AE62FB7/5AE74AF7/5CF198E5" Ref="#PWR0685"  Part="1"
+AR Path="/5AE62FB7/5AF84E03/5CF198E5" Ref="#PWR0688"  Part="1"
+AR Path="/82611AC0/82611C89/82611C8C/5CF198E5" Ref="#PWR0691"  Part="1"
+AR Path="/5D3014E7/82611C8C/5CF198E5" Ref="#PWR0694"  Part="1"
+F 0 "#PWR0685" H 1975 5575 30  0001 C CNN
+F 1 "GND" H 1975 5505 30  0001 C CNN
+F 2 "" H 1975 5575 60  0001 C CNN
+F 3 "" H 1975 5575 60  0001 C CNN
+	1    1975 5575
+	1    0    0    -1
+$EndComp
+$Comp
+L power:GND #PWR0686
+U 1 1 5CF199DA
+P 2850 4300
+AR Path="/5AE62FB7/5AE74AF7/5CF199DA" Ref="#PWR0686"  Part="1"
+AR Path="/5AE62FB7/5AF84E03/5CF199DA" Ref="#PWR0689"  Part="1"
+AR Path="/82611AC0/82611C89/82611C8C/5CF199DA" Ref="#PWR0692"  Part="1"
+AR Path="/5D3014E7/82611C8C/5CF199DA" Ref="#PWR0695"  Part="1"
+F 0 "#PWR0686" H 2850 4300 30  0001 C CNN
+F 1 "GND" H 2850 4230 30  0001 C CNN
+F 2 "" H 2850 4300 60  0001 C CNN
+F 3 "" H 2850 4300 60  0001 C CNN
+	1    2850 4300
+	1    0    0    -1
+$EndComp
+$Comp
+L power:GND #PWR?
+U 1 1 5CF19D18
+P 700 4200
+F 0 "#PWR?" H 700 4200 30  0001 C CNN
+F 1 "GND" H 700 4130 30  0001 C CNN
+F 2 "" H 700 4200 60  0001 C CNN
+F 3 "" H 700 4200 60  0001 C CNN
+	1    700  4200
+	1    0    0    -1
+$EndComp
 $EndSCHEMATC
