File: INC8.sch (KiCad schematic (older format))
At the start: 5 parts, among them U199 74LS283, U200 74LS283

Commit message: c)
Parts:
- removed R3: 0R1, symbol pspice:R
Connections:
- wire segments 70 -> 68
Other:
- moved on the sheet: C10
Changed lines of the file:
@@
 L pspice:C C298
 U 1 1 5AEB8335
-P 650 4675
+P 600 4625
 AR Path="/82611AC0/82611C89/82611C8C/5AEB8335" Ref="C298"  Part="1"
 AR Path="/5AE62FB7/5AE74AF7/5AEB8335" Ref="C10"  Part="1"
 AR Path="/5AE62FB7/5AF84E03/5AEB8335" Ref="C36"  Part="1"
 AR Path="/5D3014E7/82611C8C/5AEB8335" Ref="C326"  Part="1"
-F 0 "C10" V 500 4675 60  0000 C CNN
-F 1 "100nF" V 800 4675 60  0000 C CNN
-F 2 "" H 650 4675 60  0000 C CNN
-F 3 "" H 650 4675 60  0000 C CNN
-	1    650  4675
+F 0 "C10" V 450 4625 60  0000 C CNN
+F 1 "100nF" V 750 4625 60  0000 C CNN
+F 2 "" H 600 4625 60  0000 C CNN
+F 3 "" H 600 4625 60  0000 C CNN
+	1    600  4625
 	1    0    0    -1
 $EndComp
@@
 AR Path="/5AE62FB7/5AF84E03/5AEB8439" Ref="#PWR052"  Part="1"
 AR Path="/5D3014E7/82611C8C/5AEB8439" Ref="#PWR0601"  Part="1"
-F 0 "#PWR0601" H 2525 4850 50  0001 C CNN
+F 0 "#PWR020" H 2525 4850 50  0001 C CNN
 F 1 "VCC" H 2525 5150 50  0000 C CNN
 F 2 "" H 2525 5000 50  0000 C CNN
@@
 L myCpu-rescue:VCC #PWR0531
 U 1 1 5AEB8455
-P 775 4900
+P 875 4900
 AR Path="/82611AC0/82611C89/82611C8C/5AEB8455" Ref="#PWR0531"  Part="1"
 AR Path="/5AE62FB7/5AE74AF7/5AEB8455" Ref="#PWR019"  Part="1"
 AR Path="/5AE62FB7/5AF84E03/5AEB8455" Ref="#PWR051"  Part="1"
 AR Path="/5D3014E7/82611C8C/5AEB8455" Ref="#PWR0600"  Part="1"
-F 0 "#PWR0600" H 775 4750 50  0001 C CNN
-F 1 "VCC" H 775 5050 50  0000 C CNN
-F 2 "" H 775 4900 50  0000 C CNN
-F 3 "" H 775 4900 50  0000 C CNN
-	1    775  4900
+F 0 "#PWR019" H 875 4750 50  0001 C CNN
+F 1 "VCC" H 875 5050 50  0000 C CNN
+F 2 "" H 875 4900 50  0000 C CNN
+F 3 "" H 875 4900 50  0000 C CNN
+	1    875  4900
 	1    0    0    -1
 $EndComp
 Wire Wire Line
-	775  4900 775  4925
+	875  4900 775  4925
 Wire Wire Line
-	650  4925 775  4925
+	600  4875 775  4925
 Connection ~ 775  4925
 Wire Wire Line
-	650  4425 700  4425
+	600  4375 700  4425
 Wire Wire Line
 	700  4425 700  4200
@@
 Connection ~ 1900 5275
 $Comp
-L pspice:R R3
-U 1 1 5CBC5903
-P 775 5525
-AR Path="/82611AC0/82611C89/82611C8C/5CBC5903" Ref="R3"  Part="1"
-AR Path="/5AE62FB7/5AE74AF7/5CBC5903" Ref="R1"  Part="1"
-AR Path="/5AE62FB7/5AF84E03/5CBC5903" Ref="R2"  Part="1"
-AR Path="/5D3014E7/82611C8C/5CBC5903" Ref="R4"  Part="1"
-F 0 "R1" H 843 5571 50  0000 L CNN
-F 1 "0R1" H 843 5480 50  0000 L CNN
-F 2 "" H 775 5525 60  0001 C CNN
-F 3 "" H 775 5525 60  0001 C CNN
-	1    775  5525
-	1    0    0    -1
-$EndComp
-Wire Wire Line
-	775  5775 975  5775
-Wire Wire Line
-	975  5775 975  5275
-Wire Wire Line
-	975  5275 1100 5275
-$Comp
 L power:GND #PWR0684
 U 1 1 5CF197AB
@@
 AR Path="/82611AC0/82611C89/82611C8C/5CF197AB" Ref="#PWR0690"  Part="1"
 AR Path="/5D3014E7/82611C8C/5CF197AB" Ref="#PWR0693"  Part="1"
-F 0 "#PWR0693" H 4125 5650 30  0001 C CNN
+F 0 "#PWR0684" H 4125 5650 30  0001 C CNN
 F 1 "GND" H 4125 5580 30  0001 C CNN
 F 2 "" H 4125 5650 60  0001 C CNN
@@
 AR Path="/82611AC0/82611C89/82611C8C/5CF198E5" Ref="#PWR0691"  Part="1"
 AR Path="/5D3014E7/82611C8C/5CF198E5" Ref="#PWR0694"  Part="1"
-F 0 "#PWR0694" H 1975 5575 30  0001 C CNN
+F 0 "#PWR0685" H 1975 5575 30  0001 C CNN
 F 1 "GND" H 1975 5505 30  0001 C CNN
 F 2 "" H 1975 5575 60  0001 C CNN
@@
 AR Path="/82611AC0/82611C89/82611C8C/5CF199DA" Ref="#PWR0692"  Part="1"
 AR Path="/5D3014E7/82611C8C/5CF199DA" Ref="#PWR0695"  Part="1"
-F 0 "#PWR0695" H 2850 4300 30  0001 C CNN
+F 0 "#PWR0686" H 2850 4300 30  0001 C CNN
 F 1 "GND" H 2850 4230 30  0001 C CNN
 F 2 "" H 2850 4300 60  0001 C CNN
@@
 AR Path="/82611AC0/82611C89/82611C8C/5CF19D18" Ref="#PWR0698"  Part="1"
 AR Path="/5D3014E7/82611C8C/5CF19D18" Ref="#PWR0699"  Part="1"
-F 0 "#PWR0699" H 700 4200 30  0001 C CNN
+F 0 "#PWR0696" H 700 4200 30  0001 C CNN
 F 1 "GND" H 700 4130 30  0001 C CNN
 F 2 "" H 700 4200 60  0001 C CNN
@@
 Wire Wire Line
 	1900 5275 2000 5275
+Wire Wire Line
+	775  5275 1100 5275
 $EndSCHEMATC

Commit message: message
Parts:
- renumbered C298 to C10, C299 to C11, U199 to U25, U200 to U26
Changed lines of the file:
@@
 $Descr A4 11693 8268
 encoding utf-8
-Sheet 7 92
+Sheet 7 101
 Title ""
 Date ""
@@
 Z7
 $Comp
-L myCpu-rescue:74LS283 U199
+L myCpu-rescue:74LS283 U25
 U 1 1 5AE74BC6
 P 1550 4575
-AR Path="/82611AC0/82611C89/82611C8C/5AE74BC6" Ref="U199"  Part="1"
-AR Path="/5AE62FB7/5AE74AF7/5AE74BC6" Ref="U12"  Part="1"
-AR Path="/5AE62FB7/5AF84E03/5AE74BC6" Ref="U40"  Part="1"
-AR Path="/5D3014E7/82611C8C/5AE74BC6" Ref="U227"  Part="1"
-F 0 "U12" H 1550 4575 50  0000 C CNN
+AR Path="/5AE62FB7/5AE74AF7/5AE74BC6" Ref="U25"  Part="1"
+AR Path="/5AE62FB7/5AF84E03/5AE74BC6" Ref="U57"  Part="1"
+AR Path="/82611AC0/82611C89/82611C8C/5AE74BC6" Ref="U246"  Part="1"
+AR Path="/5D3014E7/82611C8C/5AE74BC6" Ref="U274"  Part="1"
+F 0 "U274" H 1550 4575 50  0000 C CNN
 F 1 "74LS283" H 1600 4225 50  0000 C CNN
 F 2 "" H 1550 4575 50  0000 C CNN
@@
 	2000 5475 2000 5275
 $Comp
-L myCpu-rescue:74LS283 U200
+L myCpu-rescue:74LS283 U26
 U 1 1 5AE74FBD
 P 3575 4700
-AR Path="/82611AC0/82611C89/82611C8C/5AE74FBD" Ref="U200"  Part="1"
-AR Path="/5AE62FB7/5AE74AF7/5AE74FBD" Ref="U13"  Part="1"
-AR Path="/5AE62FB7/5AF84E03/5AE74FBD" Ref="U41"  Part="1"
-AR Path="/5D3014E7/82611C8C/5AE74FBD" Ref="U228"  Part="1"
-F 0 "U13" H 3575 4700 50  0000 C CNN
+AR Path="/5AE62FB7/5AE74AF7/5AE74FBD" Ref="U26"  Part="1"
+AR Path="/5AE62FB7/5AF84E03/5AE74FBD" Ref="U58"  Part="1"
+AR Path="/82611AC0/82611C89/82611C8C/5AE74FBD" Ref="U247"  Part="1"
+AR Path="/5D3014E7/82611C8C/5AE74FBD" Ref="U275"  Part="1"
+F 0 "U275" H 3575 4700 50  0000 C CNN
 F 1 "74LS283" H 3625 4350 50  0000 C CNN
 F 2 "" H 3575 4700 50  0000 C CNN
@@
 	4375 4000 4375 2800
 $Comp
-L pspice:C C298
+L pspice:C C10
 U 1 1 5AEB8335
 P 600 4625
-AR Path="/82611AC0/82611C89/82611C8C/5AEB8335" Ref="C298"  Part="1"
 AR Path="/5AE62FB7/5AE74AF7/5AEB8335" Ref="C10"  Part="1"
 AR Path="/5AE62FB7/5AF84E03/5AEB8335" Ref="C36"  Part="1"
-AR Path="/5D3014E7/82611C8C/5AEB8335" Ref="C326"  Part="1"
-F 0 "C10" V 450 4625 60  0000 C CNN
+AR Path="/82611AC0/82611C89/82611C8C/5AEB8335" Ref="C322"  Part="1"
+AR Path="/5D3014E7/82611C8C/5AEB8335" Ref="C350"  Part="1"
+F 0 "C350" V 450 4625 60  0000 C CNN
 F 1 "100nF" V 750 4625 60  0000 C CNN
 F 2 "" H 600 4625 60  0000 C CNN
@@
 $EndComp
 $Comp
-L pspice:C C299
+L pspice:C C11
 U 1 1 5AEB839C
 P 2675 4750
-AR Path="/82611AC0/82611C89/82611C8C/5AEB839C" Ref="C299"  Part="1"
 AR Path="/5AE62FB7/5AE74AF7/5AEB839C" Ref="C11"  Part="1"
 AR Path="/5AE62FB7/5AF84E03/5AEB839C" Ref="C37"  Part="1"
-AR Path="/5D3014E7/82611C8C/5AEB839C" Ref="C327"  Part="1"
-F 0 "C11" V 2525 4750 60  0000 C CNN
+AR Path="/82611AC0/82611C89/82611C8C/5AEB839C" Ref="C323"  Part="1"
+AR Path="/5D3014E7/82611C8C/5AEB839C" Ref="C351"  Part="1"
+F 0 "C351" V 2525 4750 60  0000 C CNN
 F 1 "100nF" V 2825 4750 60  0000 C CNN
 F 2 "" H 2675 4750 60  0000 C CNN
@@
 $EndComp
 $Comp
-L myCpu-rescue:VCC #PWR0532
+L myCpu-rescue:VCC #PWR024
 U 1 1 5AEB8439
 P 2525 5000
-AR Path="/82611AC0/82611C89/82611C8C/5AEB8439" Ref="#PWR0532"  Part="1"
-AR Path="/5AE62FB7/5AE74AF7/5AEB8439" Ref="#PWR020"  Part="1"
-AR Path="/5AE62FB7/5AF84E03/5AEB8439" Ref="#PWR052"  Part="1"
-AR Path="/5D3014E7/82611C8C/5AEB8439" Ref="#PWR0601"  Part="1"
-F 0 "#PWR0601" H 2525 4850 50  0001 C CNN
+AR Path="/5AE62FB7/5AE74AF7/5AEB8439" Ref="#PWR024"  Part="1"
+AR Path="/5AE62FB7/5AF84E03/5AEB8439" Ref="#PWR060"  Part="1"
+AR Path="/82611AC0/82611C89/82611C8C/5AEB8439" Ref="#PWR0582"  Part="1"
+AR Path="/5D3014E7/82611C8C/5AEB8439" Ref="#PWR0655"  Part="1"
+F 0 "#PWR0655" H 2525 4850 50  0001 C CNN
 F 1 "VCC" H 2525 5150 50  0000 C CNN
 F 2 "" H 2525 5000 50  0000 C CNN
@@
 $EndComp
 $Comp
-L myCpu-rescue:VCC #PWR0531
+L myCpu-rescue:VCC #PWR022
 U 1 1 5AEB8455
 P 875 4900
-AR Path="/82611AC0/82611C89/82611C8C/5AEB8455" Ref="#PWR0531"  Part="1"
-AR Path="/5AE62FB7/5AE74AF7/5AEB8455" Ref="#PWR019"  Part="1"
-AR Path="/5AE62FB7/5AF84E03/5AEB8455" Ref="#PWR051"  Part="1"
-AR Path="/5D3014E7/82611C8C/5AEB8455" Ref="#PWR0600"  Part="1"
-F 0 "#PWR0600" H 875 4750 50  0001 C CNN
+AR Path="/5AE62FB7/5AE74AF7/5AEB8455" Ref="#PWR022"  Part="1"
+AR Path="/5AE62FB7/5AF84E03/5AEB8455" Ref="#PWR058"  Part="1"
+AR Path="/82611AC0/82611C89/82611C8C/5AEB8455" Ref="#PWR0580"  Part="1"
+AR Path="/5D3014E7/82611C8C/5AEB8455" Ref="#PWR0653"  Part="1"
+F 0 "#PWR0653" H 875 4750 50  0001 C CNN
 F 1 "VCC" H 875 5050 50  0000 C CNN
 F 2 "" H 875 4900 50  0000 C CNN
@@
 Connection ~ 1900 5275
 $Comp
-L power:GND #PWR0684
+L power:GND #PWR026
 U 1 1 5CF197AB
 P 4125 5650
-AR Path="/5AE62FB7/5AE74AF7/5CF197AB" Ref="#PWR0684"  Part="1"
-AR Path="/5AE62FB7/5AF84E03/5CF197AB" Ref="#PWR0687"  Part="1"
-AR Path="/82611AC0/82611C89/82611C8C/5CF197AB" Ref="#PWR0690"  Part="1"
-AR Path="/5D3014E7/82611C8C/5CF197AB" Ref="#PWR0693"  Part="1"
-F 0 "#PWR0693" H 4125 5650 30  0001 C CNN
+AR Path="/5AE62FB7/5AE74AF7/5CF197AB" Ref="#PWR026"  Part="1"
+AR Path="/5AE62FB7/5AF84E03/5CF197AB" Ref="#PWR062"  Part="1"
+AR Path="/82611AC0/82611C89/82611C8C/5CF197AB" Ref="#PWR0584"  Part="1"
+AR Path="/5D3014E7/82611C8C/5CF197AB" Ref="#PWR0657"  Part="1"
+F 0 "#PWR0657" H 4125 5650 30  0001 C CNN
 F 1 "GND" H 4125 5580 30  0001 C CNN
 F 2 "" H 4125 5650 60  0001 C CNN
@@
 $EndComp
 $Comp
-L power:GND #PWR0685
+L power:GND #PWR023
 U 1 1 5CF198E5
 P 1975 5575
-AR Path="/5AE62FB7/5AE74AF7/5CF198E5" Ref="#PWR0685"  Part="1"
-AR Path="/5AE62FB7/5AF84E03/5CF198E5" Ref="#PWR0688"  Part="1"
-AR Path="/82611AC0/82611C89/82611C8C/5CF198E5" Ref="#PWR0691"  Part="1"
-AR Path="/5D3014E7/82611C8C/5CF198E5" Ref="#PWR0694"  Part="1"
-F 0 "#PWR0694" H 1975 5575 30  0001 C CNN
+AR Path="/5AE62FB7/5AE74AF7/5CF198E5" Ref="#PWR023"  Part="1"
+AR Path="/5AE62FB7/5AF84E03/5CF198E5" Ref="#PWR059"  Part="1"
+AR Path="/82611AC0/82611C89/82611C8C/5CF198E5" Ref="#PWR0581"  Part="1"
+AR Path="/5D3014E7/82611C8C/5CF198E5" Ref="#PWR0654"  Part="1"
+F 0 "#PWR0654" H 1975 5575 30  0001 C CNN
 F 1 "GND" H 1975 5505 30  0001 C CNN
 F 2 "" H 1975 5575 60  0001 C CNN
@@
 $EndComp
 $Comp
-L power:GND #PWR0686
+L power:GND #PWR025
 U 1 1 5CF199DA
 P 2850 4300
-AR Path="/5AE62FB7/5AE74AF7/5CF199DA" Ref="#PWR0686"  Part="1"
-AR Path="/5AE62FB7/5AF84E03/5CF199DA" Ref="#PWR0689"  Part="1"
-AR Path="/82611AC0/82611C89/82611C8C/5CF199DA" Ref="#PWR0692"  Part="1"
-AR Path="/5D3014E7/82611C8C/5CF199DA" Ref="#PWR0695"  Part="1"
-F 0 "#PWR0695" H 2850 4300 30  0001 C CNN
+AR Path="/5AE62FB7/5AE74AF7/5CF199DA" Ref="#PWR025"  Part="1"
+AR Path="/5AE62FB7/5AF84E03/5CF199DA" Ref="#PWR061"  Part="1"
+AR Path="/82611AC0/82611C89/82611C8C/5CF199DA" Ref="#PWR0583"  Part="1"
+AR Path="/5D3014E7/82611C8C/5CF199DA" Ref="#PWR0656"  Part="1"
+F 0 "#PWR0656" H 2850 4300 30  0001 C CNN
 F 1 "GND" H 2850 4230 30  0001 C CNN
 F 2 "" H 2850 4300 60  0001 C CNN
@@
 $EndComp
 $Comp
-L power:GND #PWR0696
+L power:GND #PWR021
 U 1 1 5CF19D18
 P 700 4200
-AR Path="/5AE62FB7/5AE74AF7/5CF19D18" Ref="#PWR0696"  Part="1"
-AR Path="/5AE62FB7/5AF84E03/5CF19D18" Ref="#PWR0697"  Part="1"
-AR Path="/82611AC0/82611C89/82611C8C/5CF19D18" Ref="#PWR0698"  Part="1"
-AR Path="/5D3014E7/82611C8C/5CF19D18" Ref="#PWR0699"  Part="1"
-F 0 "#PWR0699" H 700 4200 30  0001 C CNN
+AR Path="/5AE62FB7/5AE74AF7/5CF19D18" Ref="#PWR021"  Part="1"
+AR Path="/5AE62FB7/5AF84E03/5CF19D18" Ref="#PWR057"  Part="1"
+AR Path="/82611AC0/82611C89/82611C8C/5CF19D18" Ref="#PWR0579"  Part="1"
+AR Path="/5D3014E7/82611C8C/5CF19D18" Ref="#PWR0652"  Part="1"
+F 0 "#PWR0652" H 700 4200 30  0001 C CNN
 F 1 "GND" H 700 4130 30  0001 C CNN
 F 2 "" H 700 4200 60  0001 C CNN

Commit message: .
Changed lines of the file:
@@
 $Descr A4 11693 8268
 encoding utf-8
-Sheet 7 101
+Sheet 7 75
 Title ""
 Date ""
@@
 AR Path="/5AE62FB7/5AE74AF7/5AE74BC6" Ref="U25"  Part="1"
 AR Path="/5AE62FB7/5AF84E03/5AE74BC6" Ref="U57"  Part="1"
-AR Path="/82611AC0/82611C89/82611C8C/5AE74BC6" Ref="U246"  Part="1"
-AR Path="/5D3014E7/82611C8C/5AE74BC6" Ref="U274"  Part="1"
-F 0 "U274" H 1550 4575 50  0000 C CNN
+AR Path="/82611AC0/82611C89/82611C8C/5AE74BC6" Ref="U145"  Part="1"
+AR Path="/5D3014E7/82611C8C/5AE74BC6" Ref="U173"  Part="1"
+F 0 "U173" H 1550 4575 50  0000 C CNN
 F 1 "74LS283" H 1600 4225 50  0000 C CNN
 F 2 "" H 1550 4575 50  0000 C CNN
@@
 AR Path="/5AE62FB7/5AE74AF7/5AE74FBD" Ref="U26"  Part="1"
 AR Path="/5AE62FB7/5AF84E03/5AE74FBD" Ref="U58"  Part="1"
-AR Path="/82611AC0/82611C89/82611C8C/5AE74FBD" Ref="U247"  Part="1"
-AR Path="/5D3014E7/82611C8C/5AE74FBD" Ref="U275"  Part="1"
-F 0 "U275" H 3575 4700 50  0000 C CNN
+AR Path="/82611AC0/82611C89/82611C8C/5AE74FBD" Ref="U146"  Part="1"
+AR Path="/5D3014E7/82611C8C/5AE74FBD" Ref="U174"  Part="1"
+F 0 "U174" H 3575 4700 50  0000 C CNN
 F 1 "74LS283" H 3625 4350 50  0000 C CNN
 F 2 "" H 3575 4700 50  0000 C CNN
@@
 AR Path="/5AE62FB7/5AE74AF7/5AEB8335" Ref="C10"  Part="1"
 AR Path="/5AE62FB7/5AF84E03/5AEB8335" Ref="C36"  Part="1"
-AR Path="/82611AC0/82611C89/82611C8C/5AEB8335" Ref="C322"  Part="1"
-AR Path="/5D3014E7/82611C8C/5AEB8335" Ref="C350"  Part="1"
-F 0 "C350" V 450 4625 60  0000 C CNN
+AR Path="/82611AC0/82611C89/82611C8C/5AEB8335" Ref="C114"  Part="1"
+AR Path="/5D3014E7/82611C8C/5AEB8335" Ref="C142"  Part="1"
+F 0 "C142" V 450 4625 60  0000 C CNN
 F 1 "100nF" V 750 4625 60  0000 C CNN
 F 2 "" H 600 4625 60  0000 C CNN
@@
 AR Path="/5AE62FB7/5AE74AF7/5AEB839C" Ref="C11"  Part="1"
 AR Path="/5AE62FB7/5AF84E03/5AEB839C" Ref="C37"  Part="1"
-AR Path="/82611AC0/82611C89/82611C8C/5AEB839C" Ref="C323"  Part="1"
-AR Path="/5D3014E7/82611C8C/5AEB839C" Ref="C351"  Part="1"
-F 0 "C351" V 2525 4750 60  0000 C CNN
+AR Path="/82611AC0/82611C89/82611C8C/5AEB839C" Ref="C115"  Part="1"
+AR Path="/5D3014E7/82611C8C/5AEB839C" Ref="C143"  Part="1"
+F 0 "C143" V 2525 4750 60  0000 C CNN
 F 1 "100nF" V 2825 4750 60  0000 C CNN
 F 2 "" H 2675 4750 60  0000 C CNN
@@
 $EndComp
 $Comp
-L myCpu-rescue:VCC #PWR024
+L myCpu-rescue:VCC #PWR027
 U 1 1 5AEB8439
 P 2525 5000
-AR Path="/5AE62FB7/5AE74AF7/5AEB8439" Ref="#PWR024"  Part="1"
-AR Path="/5AE62FB7/5AF84E03/5AEB8439" Ref="#PWR060"  Part="1"
-AR Path="/82611AC0/82611C89/82611C8C/5AEB8439" Ref="#PWR0582"  Part="1"
-AR Path="/5D3014E7/82611C8C/5AEB8439" Ref="#PWR0655"  Part="1"
-F 0 "#PWR0655" H 2525 4850 50  0001 C CNN
+AR Path="/5AE62FB7/5AE74AF7/5AEB8439" Ref="#PWR027"  Part="1"
+AR Path="/5AE62FB7/5AF84E03/5AEB8439" Ref="#PWR063"  Part="1"
+AR Path="/82611AC0/82611C89/82611C8C/5AEB8439" Ref="#PWR0172"  Part="1"
+AR Path="/5D3014E7/82611C8C/5AEB8439" Ref="#PWR0245"  Part="1"
+F 0 "#PWR0245" H 2525 4850 50  0001 C CNN
 F 1 "VCC" H 2525 5150 50  0000 C CNN
 F 2 "" H 2525 5000 50  0000 C CNN
@@
 $EndComp
 $Comp
-L myCpu-rescue:VCC #PWR022
+L myCpu-rescue:VCC #PWR025
 U 1 1 5AEB8455
 P 875 4900
-AR Path="/5AE62FB7/5AE74AF7/5AEB8455" Ref="#PWR022"  Part="1"
-AR Path="/5AE62FB7/5AF84E03/5AEB8455" Ref="#PWR058"  Part="1"
-AR Path="/82611AC0/82611C89/82611C8C/5AEB8455" Ref="#PWR0580"  Part="1"
-AR Path="/5D3014E7/82611C8C/5AEB8455" Ref="#PWR0653"  Part="1"
-F 0 "#PWR0653" H 875 4750 50  0001 C CNN
+AR Path="/5AE62FB7/5AE74AF7/5AEB8455" Ref="#PWR025"  Part="1"
+AR Path="/5AE62FB7/5AF84E03/5AEB8455" Ref="#PWR061"  Part="1"
+AR Path="/82611AC0/82611C89/82611C8C/5AEB8455" Ref="#PWR0170"  Part="1"
+AR Path="/5D3014E7/82611C8C/5AEB8455" Ref="#PWR0243"  Part="1"
+F 0 "#PWR0243" H 875 4750 50  0001 C CNN
 F 1 "VCC" H 875 5050 50  0000 C CNN
 F 2 "" H 875 4900 50  0000 C CNN
@@
 Connection ~ 1900 5275
 $Comp
-L power:GND #PWR026
+L power:GND #PWR029
 U 1 1 5CF197AB
 P 4125 5650
-AR Path="/5AE62FB7/5AE74AF7/5CF197AB" Ref="#PWR026"  Part="1"
-AR Path="/5AE62FB7/5AF84E03/5CF197AB" Ref="#PWR062"  Part="1"
-AR Path="/82611AC0/82611C89/82611C8C/5CF197AB" Ref="#PWR0584"  Part="1"
-AR Path="/5D3014E7/82611C8C/5CF197AB" Ref="#PWR0657"  Part="1"
-F 0 "#PWR0657" H 4125 5650 30  0001 C CNN
+AR Path="/5AE62FB7/5AE74AF7/5CF197AB" Ref="#PWR029"  Part="1"
+AR Path="/5AE62FB7/5AF84E03/5CF197AB" Ref="#PWR065"  Part="1"
+AR Path="/82611AC0/82611C89/82611C8C/5CF197AB" Ref="#PWR0174"  Part="1"
+AR Path="/5D3014E7/82611C8C/5CF197AB" Ref="#PWR0247"  Part="1"
+F 0 "#PWR0247" H 4125 5650 30  0001 C CNN
 F 1 "GND" H 4125 5580 30  0001 C CNN
 F 2 "" H 4125 5650 60  0001 C CNN
@@
 $EndComp
 $Comp
-L power:GND #PWR023
+L power:GND #PWR026
 U 1 1 5CF198E5
 P 1975 5575
-AR Path="/5AE62FB7/5AE74AF7/5CF198E5" Ref="#PWR023"  Part="1"
-AR Path="/5AE62FB7/5AF84E03/5CF198E5" Ref="#PWR059"  Part="1"
-AR Path="/82611AC0/82611C89/82611C8C/5CF198E5" Ref="#PWR0581"  Part="1"
-AR Path="/5D3014E7/82611C8C/5CF198E5" Ref="#PWR0654"  Part="1"
-F 0 "#PWR0654" H 1975 5575 30  0001 C CNN
+AR Path="/5AE62FB7/5AE74AF7/5CF198E5" Ref="#PWR026"  Part="1"
+AR Path="/5AE62FB7/5AF84E03/5CF198E5" Ref="#PWR062"  Part="1"
+AR Path="/82611AC0/82611C89/82611C8C/5CF198E5" Ref="#PWR0171"  Part="1"
+AR Path="/5D3014E7/82611C8C/5CF198E5" Ref="#PWR0244"  Part="1"
+F 0 "#PWR0244" H 1975 5575 30  0001 C CNN
 F 1 "GND" H 1975 5505 30  0001 C CNN
 F 2 "" H 1975 5575 60  0001 C CNN
@@
 $EndComp
 $Comp
-L power:GND #PWR025
+L power:GND #PWR028
 U 1 1 5CF199DA
 P 2850 4300
-AR Path="/5AE62FB7/5AE74AF7/5CF199DA" Ref="#PWR025"  Part="1"
-AR Path="/5AE62FB7/5AF84E03/5CF199DA" Ref="#PWR061"  Part="1"
-AR Path="/82611AC0/82611C89/82611C8C/5CF199DA" Ref="#PWR0583"  Part="1"
-AR Path="/5D3014E7/82611C8C/5CF199DA" Ref="#PWR0656"  Part="1"
-F 0 "#PWR0656" H 2850 4300 30  0001 C CNN
+AR Path="/5AE62FB7/5AE74AF7/5CF199DA" Ref="#PWR028"  Part="1"
+AR Path="/5AE62FB7/5AF84E03/5CF199DA" Ref="#PWR064"  Part="1"
+AR Path="/82611AC0/82611C89/82611C8C/5CF199DA" Ref="#PWR0173"  Part="1"
+AR Path="/5D3014E7/82611C8C/5CF199DA" Ref="#PWR0246"  Part="1"
+F 0 "#PWR0246" H 2850 4300 30  0001 C CNN
 F 1 "GND" H 2850 4230 30  0001 C CNN
 F 2 "" H 2850 4300 60  0001 C CNN
@@
 $EndComp
 $Comp
-L power:GND #PWR021
+L power:GND #PWR024
 U 1 1 5CF19D18
 P 700 4200
-AR Path="/5AE62FB7/5AE74AF7/5CF19D18" Ref="#PWR021"  Part="1"
-AR Path="/5AE62FB7/5AF84E03/5CF19D18" Ref="#PWR057"  Part="1"
-AR Path="/82611AC0/82611C89/82611C8C/5CF19D18" Ref="#PWR0579"  Part="1"
-AR Path="/5D3014E7/82611C8C/5CF19D18" Ref="#PWR0652"  Part="1"
-F 0 "#PWR0652" H 700 4200 30  0001 C CNN
+AR Path="/5AE62FB7/5AE74AF7/5CF19D18" Ref="#PWR024"  Part="1"
+AR Path="/5AE62FB7/5AF84E03/5CF19D18" Ref="#PWR060"  Part="1"
+AR Path="/82611AC0/82611C89/82611C8C/5CF19D18" Ref="#PWR0169"  Part="1"
+AR Path="/5D3014E7/82611C8C/5CF19D18" Ref="#PWR0242"  Part="1"
+F 0 "#PWR0242" H 700 4200 30  0001 C CNN
 F 1 "GND" H 700 4130 30  0001 C CNN
 F 2 "" H 700 4200 60  0001 C CNN
