File: OR.sch (KiCad schematic (older format))
At the start: 2 parts, among them U3 4071, U4 4071

Commit message: SPICE capacitance and ground symbols
Parts:
- added C? (x2): 100nF, symbol C
Connections:
- net labels added: 0, VCC
- wire segments 67 -> 75
Changed lines of the file:
@@
 EESchema Schematic File Version 2
-LIBS:power
-LIBS:device
-LIBS:transistors
-LIBS:conn
-LIBS:linear
-LIBS:regul
-LIBS:74xx
-LIBS:cmos4000
-LIBS:adc-dac
-LIBS:memory
-LIBS:xilinx
-LIBS:microcontrollers
-LIBS:dsp
-LIBS:microchip
-LIBS:analog_switches
-LIBS:motorola
-LIBS:texas
-LIBS:intel
-LIBS:audio
-LIBS:interface
-LIBS:digital-audio
-LIBS:philips
-LIBS:display
-LIBS:cypress
-LIBS:siliconi
-LIBS:opto
-LIBS:atmel
-LIBS:contrib
-LIBS:valves
+LIBS:spice
+LIBS:pspice
 LIBS:myCpu-cache
 EELAYER 25 0
@@
 Wire Wire Line
 	6100 850  6100 1625
+$Comp
+L 0 #GND?
+U 1 1 5AEBC873
+P 7400 1700
+F 0 "#GND?" H 7400 1600 60  0001 C CNN
+F 1 "0" H 7400 1630 60  0000 C CNN
+F 2 "" H 7400 1700 60  0000 C CNN
+F 3 "" H 7400 1700 60  0000 C CNN
+	1    7400 1700
+	1    0    0    -1
+$EndComp
+$Comp
+L C C?
+U 1 1 5AEBC897
+P 7300 2150
+F 0 "C?" V 7150 2150 60  0000 C CNN
+F 1 "100nF" V 7450 2150 60  0000 C CNN
+F 2 "" H 7300 2150 60  0000 C CNN
+F 3 "" H 7300 2150 60  0000 C CNN
+	1    7300 2150
+	1    0    0    -1
+$EndComp
+$Comp
+L VCC #PWR?
+U 1 1 5AEBC8FE
+P 6925 2500
+F 0 "#PWR?" H 6925 2350 50  0001 C CNN
+F 1 "VCC" H 6925 2650 50  0000 C CNN
+F 2 "" H 6925 2500 50  0000 C CNN
+F 3 "" H 6925 2500 50  0000 C CNN
+	1    6925 2500
+	1    0    0    -1
+$EndComp
+Wire Wire Line
+	7300 1900 7400 1900
+Wire Wire Line
+	7400 1900 7400 1700
+Wire Wire Line
+	6925 2500 7300 2500
+Wire Wire Line
+	7300 2500 7300 2400
+$Comp
+L 0 #GND?
+U 1 1 5AEBCAF9
+P 1025 1850
+F 0 "#GND?" H 1025 1750 60  0001 C CNN
+F 1 "0" H 1025 1780 60  0000 C CNN
+F 2 "" H 1025 1850 60  0000 C CNN
+F 3 "" H 1025 1850 60  0000 C CNN
+	1    1025 1850
+	1    0    0    -1
+$EndComp
+$Comp
+L C C?
+U 1 1 5AEBCAFF
+P 925 2300
+F 0 "C?" V 775 2300 60  0000 C CNN
+F 1 "100nF" V 1075 2300 60  0000 C CNN
+F 2 "" H 925 2300 60  0000 C CNN
+F 3 "" H 925 2300 60  0000 C CNN
+	1    925  2300
+	1    0    0    -1
+$EndComp
+$Comp
+L VCC #PWR?
+U 1 1 5AEBCB05
+P 550 2650
+F 0 "#PWR?" H 550 2500 50  0001 C CNN
+F 1 "VCC" H 550 2800 50  0000 C CNN
+F 2 "" H 550 2650 50  0000 C CNN
+F 3 "" H 550 2650 50  0000 C CNN
+	1    550  2650
+	1    0    0    -1
+$EndComp
+Wire Wire Line
+	925  2050 1025 2050
+Wire Wire Line
+	1025 2050 1025 1850
+Wire Wire Line
+	550  2650 925  2650
+Wire Wire Line
+	925  2650 925  2550
 $EndSCHEMATC

Commit message: fixed duplicate names
Parts:
- gave numbers to parts that had none: 2
Changed lines of the file:
@@
 	6100 850  6100 1625
 $Comp
-L 0 #GND?
+L 0 #GND4
 U 1 1 5AEBC873
 P 7400 1700
-F 0 "#GND?" H 7400 1600 60  0001 C CNN
+F 0 "#GND4" H 7400 1600 60  0001 C CNN
 F 1 "0" H 7400 1630 60  0000 C CNN
 F 2 "" H 7400 1700 60  0000 C CNN
@@
 $EndComp
 $Comp
-L C C?
+L C C4
 U 1 1 5AEBC897
 P 7300 2150
-F 0 "C?" V 7150 2150 60  0000 C CNN
+F 0 "C4" V 7150 2150 60  0000 C CNN
 F 1 "100nF" V 7450 2150 60  0000 C CNN
 F 2 "" H 7300 2150 60  0000 C CNN
@@
 $EndComp
 $Comp
-L VCC #PWR?
+L VCC #PWR03
 U 1 1 5AEBC8FE
 P 6925 2500
-F 0 "#PWR?" H 6925 2350 50  0001 C CNN
+F 0 "#PWR03" H 6925 2350 50  0001 C CNN
 F 1 "VCC" H 6925 2650 50  0000 C CNN
 F 2 "" H 6925 2500 50  0000 C CNN
@@
 	7300 2500 7300 2400
 $Comp
-L 0 #GND?
+L 0 #GND3
 U 1 1 5AEBCAF9
 P 1025 1850
-F 0 "#GND?" H 1025 1750 60  0001 C CNN
+F 0 "#GND3" H 1025 1750 60  0001 C CNN
 F 1 "0" H 1025 1780 60  0000 C CNN
 F 2 "" H 1025 1850 60  0000 C CNN
@@
 $EndComp
 $Comp
-L C C?
+L C C3
 U 1 1 5AEBCAFF
 P 925 2300
-F 0 "C?" V 775 2300 60  0000 C CNN
+F 0 "C3" V 775 2300 60  0000 C CNN
 F 1 "100nF" V 1075 2300 60  0000 C CNN
 F 2 "" H 925 2300 60  0000 C CNN
@@
 $EndComp
 $Comp
-L VCC #PWR?
+L VCC #PWR04
 U 1 1 5AEBCB05
 P 550 2650
-F 0 "#PWR?" H 550 2500 50  0001 C CNN
+F 0 "#PWR04" H 550 2500 50  0001 C CNN
 F 1 "VCC" H 550 2800 50  0000 C CNN
 F 2 "" H 550 2650 50  0000 C CNN

Commit message: spice libs from the internet, opened with new kicad 5.0.0, added spice models to components
Parts:
- C3, C4: symbol C -> spice:C
- U3: symbol 4071 -> myCpu-rescue:4071; Spice_Lib_File (none) -> cd4000.lib; Spice_Model (none) -> CD4071B; Spice_Netlist_Enabled (none) -> Y; Spice_Primitive (none) -> X
- U3, U4: symbol 4071 -> myCpu-rescue:4071
Changed lines of the file:
@@
-EESchema Schematic File Version 2
-LIBS:spice
-LIBS:pspice
+EESchema Schematic File Version 4
 LIBS:myCpu-cache
-EELAYER 25 0
+EELAYER 26 0
 EELAYER END
 $Descr A4 11693 8268
@@
 Z7
 $Comp
-L 4071 U3
+L myCpu-rescue:4071 U3
 U 1 1 5AE65623
 P 1500 2200
@@
 F 2 "" H 1500 2200 60  0001 C CNN
 F 3 "" H 1500 2200 60  0001 C CNN
+F 4 "X" H 1500 2200 50  0001 C CNN "Spice_Primitive"
+F 5 "CD4071B" H 1500 2200 50  0001 C CNN "Spice_Model"
+F 6 "Y" H 1500 2200 50  0001 C CNN "Spice_Netlist_Enabled"
+F 7 "cd4000.lib" H 1500 2200 50  0001 C CNN "Spice_Lib_File"
 	1    1500 2200
 	0    -1   -1   0
 $EndComp
 $Comp
-L 4071 U3
+L myCpu-rescue:4071 U3
 U 2 1 5AE656B0
 P 2100 2200
@@
 $EndComp
 $Comp
-L 4071 U3
+L myCpu-rescue:4071 U3
 U 3 1 5AE6574D
 P 2750 2250
@@
 $EndComp
 $Comp
-L 4071 U3
+L myCpu-rescue:4071 U3
 U 4 1 5AE657EA
 P 3400 2250
@@
 $EndComp
 $Comp
-L 4071 U4
+L myCpu-rescue:4071 U4
 U 1 1 5AE65887
 P 4350 2225
@@
 $EndComp
 $Comp
-L 4071 U4
+L myCpu-rescue:4071 U4
 U 2 1 5AE658F8
 P 4925 2200
@@
 $EndComp
 $Comp
-L 4071 U4
+L myCpu-rescue:4071 U4
 U 3 1 5AE65977
 P 5450 2175
@@
 $EndComp
 $Comp
-L 4071 U4
+L myCpu-rescue:4071 U4
 U 4 1 5AE65A2C
 P 6100 2225
@@
 	3525 5000 3525 5475
 Wire Wire Line
-	3750 3300 3750 5550
-Wire Wire Line
 	3750 3300 2850 3300
 Wire Wire Line
 	2850 3300 2850 2850
-Connection ~ 3750 5500
 Wire Wire Line
 	3500 2850 3500 4900
@@
 	6100 850  6100 1625
 $Comp
-L 0 #GND4
+L spice:0 #GND4
 U 1 1 5AEBC873
 P 7400 1700
@@
 $EndComp
 $Comp
-L C C4
+L spice:C C4
 U 1 1 5AEBC897
 P 7300 2150
@@
 $EndComp
 $Comp
-L VCC #PWR03
+L myCpu-rescue:VCC #PWR03
 U 1 1 5AEBC8FE
 P 6925 2500
@@
 	7300 2500 7300 2400
 $Comp
-L 0 #GND3
+L spice:0 #GND3
 U 1 1 5AEBCAF9
 P 1025 1850
@@
 $EndComp
 $Comp
-L C C3
+L spice:C C3
 U 1 1 5AEBCAFF
 P 925 2300
@@
 $EndComp
 $Comp
-L VCC #PWR04
+L myCpu-rescue:VCC #PWR04
 U 1 1 5AEBCB05
 P 550 2650
@@
 Wire Wire Line
 	925  2650 925  2550
+Wire Wire Line
+	3750 3300 3750 5550
 $EndSCHEMATC

Commit message: lots of work done
Parts:
- renumbered C3 to C4, C4 to C5, U3 to U4, U4 to U5
Changed lines of the file:
@@
 $Descr A4 11693 8268
 encoding utf-8
-Sheet 4 21
+Sheet 4 81
 Title ""
 Date ""
@@
 Z7
 $Comp
-L myCpu-rescue:4071 U3
+L myCpu-rescue:4071 U4
 U 1 1 5AE65623
 P 1500 2200
-F 0 "U3" H 1500 2250 50  0000 C CNN
+F 0 "U4" H 1500 2250 50  0000 C CNN
 F 1 "4071" H 1500 2150 50  0000 C CNN
 F 2 "" H 1500 2200 60  0001 C CNN
@@
 $EndComp
 $Comp
-L myCpu-rescue:4071 U3
+L myCpu-rescue:4071 U4
 U 2 1 5AE656B0
 P 2100 2200
-F 0 "U3" H 2100 2250 50  0000 C CNN
+F 0 "U4" H 2100 2250 50  0000 C CNN
 F 1 "4071" H 2100 2150 50  0000 C CNN
 F 2 "" H 2100 2200 60  0001 C CNN
@@
 $EndComp
 $Comp
-L myCpu-rescue:4071 U3
+L myCpu-rescue:4071 U4
 U 3 1 5AE6574D
 P 2750 2250
-F 0 "U3" H 2750 2300 50  0000 C CNN
+F 0 "U4" H 2750 2300 50  0000 C CNN
 F 1 "4071" H 2750 2200 50  0000 C CNN
 F 2 "" H 2750 2250 60  0001 C CNN
@@
 $EndComp
 $Comp
-L myCpu-rescue:4071 U3
+L myCpu-rescue:4071 U4
 U 4 1 5AE657EA
 P 3400 2250
-F 0 "U3" H 3400 2300 50  0000 C CNN
+F 0 "U4" H 3400 2300 50  0000 C CNN
 F 1 "4071" H 3400 2200 50  0000 C CNN
 F 2 "" H 3400 2250 60  0001 C CNN
@@
 $EndComp
 $Comp
-L myCpu-rescue:4071 U4
+L myCpu-rescue:4071 U5
 U 1 1 5AE65887
 P 4350 2225
-F 0 "U4" H 4350 2275 50  0000 C CNN
+F 0 "U5" H 4350 2275 50  0000 C CNN
 F 1 "4071" H 4350 2175 50  0000 C CNN
 F 2 "" H 4350 2225 60  0001 C CNN
@@
 $EndComp
 $Comp
-L myCpu-rescue:4071 U4
+L myCpu-rescue:4071 U5
 U 2 1 5AE658F8
 P 4925 2200
-F 0 "U4" H 4925 2250 50  0000 C CNN
+F 0 "U5" H 4925 2250 50  0000 C CNN
 F 1 "4071" H 4925 2150 50  0000 C CNN
 F 2 "" H 4925 2200 60  0001 C CNN
@@
 $EndComp
 $Comp
-L myCpu-rescue:4071 U4
+L myCpu-rescue:4071 U5
 U 3 1 5AE65977
 P 5450 2175
-F 0 "U4" H 5450 2225 50  0000 C CNN
+F 0 "U5" H 5450 2225 50  0000 C CNN
 F 1 "4071" H 5450 2125 50  0000 C CNN
 F 2 "" H 5450 2175 60  0001 C CNN
@@
 $EndComp
 $Comp
-L myCpu-rescue:4071 U4
+L myCpu-rescue:4071 U5
 U 4 1 5AE65A2C
 P 6100 2225
-F 0 "U4" H 6100 2275 50  0000 C CNN
+F 0 "U5" H 6100 2275 50  0000 C CNN
 F 1 "4071" H 6100 2175 50  0000 C CNN
 F 2 "" H 6100 2225 60  0001 C CNN
@@
 	6100 850  6100 1625
 $Comp
-L spice:0 #GND4
+L spice:0 #GND9
 U 1 1 5AEBC873
 P 7400 1700
-F 0 "#GND4" H 7400 1600 60  0001 C CNN
+F 0 "#GND9" H 7400 1600 60  0001 C CNN
 F 1 "0" H 7400 1630 60  0000 C CNN
 F 2 "" H 7400 1700 60  0000 C CNN
@@
 $EndComp
 $Comp
-L spice:C C4
+L spice:C C5
 U 1 1 5AEBC897
 P 7300 2150
-F 0 "C4" V 7150 2150 60  0000 C CNN
+F 0 "C5" V 7150 2150 60  0000 C CNN
 F 1 "100nF" V 7450 2150 60  0000 C CNN
 F 2 "" H 7300 2150 60  0000 C CNN
@@
 $EndComp
 $Comp
-L myCpu-rescue:VCC #PWR03
+L myCpu-rescue:VCC #PWR08
 U 1 1 5AEBC8FE
 P 6925 2500
-F 0 "#PWR03" H 6925 2350 50  0001 C CNN
+F 0 "#PWR08" H 6925 2350 50  0001 C CNN
 F 1 "VCC" H 6925 2650 50  0000 C CNN
 F 2 "" H 6925 2500 50  0000 C CNN
@@
 	7300 2500 7300 2400
 $Comp
-L spice:0 #GND3
+L spice:0 #GND8
 U 1 1 5AEBCAF9
 P 1025 1850
-F 0 "#GND3" H 1025 1750 60  0001 C CNN
+F 0 "#GND8" H 1025 1750 60  0001 C CNN
 F 1 "0" H 1025 1780 60  0000 C CNN
 F 2 "" H 1025 1850 60  0000 C CNN
@@
 $EndComp
 $Comp
-L spice:C C3
+L spice:C C4
 U 1 1 5AEBCAFF
 P 925 2300
-F 0 "C3" V 775 2300 60  0000 C CNN
+F 0 "C4" V 775 2300 60  0000 C CNN
 F 1 "100nF" V 1075 2300 60  0000 C CNN
 F 2 "" H 925 2300 60  0000 C CNN
@@
 $EndComp
 $Comp
-L myCpu-rescue:VCC #PWR04
+L myCpu-rescue:VCC #PWR07
 U 1 1 5AEBCB05
 P 550 2650
-F 0 "#PWR04" H 550 2500 50  0001 C CNN
+F 0 "#PWR07" H 550 2500 50  0001 C CNN
 F 1 "VCC" H 550 2800 50  0000 C CNN
 F 2 "" H 550 2650 50  0000 C CNN

Commit message: b
Parts:
- renumbered C4 to C6, C5 to C7, U4 to U6, U5 to U7
Changed lines of the file:
@@
 $Descr A4 11693 8268
 encoding utf-8
-Sheet 4 90
+Sheet 4 92
 Title ""
 Date ""
@@
 Text HLabel 1750 875  1    60   Output ~ 0
 Z2
-Text HLabel 2075 850  1    60   Output ~ 0
+Text HLabel 2100 875  1    60   Output ~ 0
 Z4
 Text HLabel 1925 875  1    60   Output ~ 0
@@
 Z7
 $Comp
-L myCpu-rescue:4071 U4
+L myCpu-rescue:4071 U6
 U 1 1 5AE65623
 P 1500 2200
-F 0 "U4" H 1500 2250 50  0000 C CNN
+F 0 "U6" H 1500 2250 50  0000 C CNN
 F 1 "4071" H 1500 2150 50  0000 C CNN
 F 2 "" H 1500 2200 60  0001 C CNN
@@
 $EndComp
 $Comp
-L myCpu-rescue:4071 U4
+L myCpu-rescue:4071 U6
 U 2 1 5AE656B0
 P 2100 2200
-F 0 "U4" H 2100 2250 50  0000 C CNN
+F 0 "U6" H 2100 2250 50  0000 C CNN
 F 1 "4071" H 2100 2150 50  0000 C CNN
 F 2 "" H 2100 2200 60  0001 C CNN
@@
 $EndComp
 $Comp
-L myCpu-rescue:4071 U4
+L myCpu-rescue:4071 U6
 U 3 1 5AE6574D
 P 2750 2250
-F 0 "U4" H 2750 2300 50  0000 C CNN
+F 0 "U6" H 2750 2300 50  0000 C CNN
 F 1 "4071" H 2750 2200 50  0000 C CNN
 F 2 "" H 2750 2250 60  0001 C CNN
@@
 $EndComp
 $Comp
-L myCpu-rescue:4071 U4
+L myCpu-rescue:4071 U6
 U 4 1 5AE657EA
 P 3400 2250
-F 0 "U4" H 3400 2300 50  0000 C CNN
+F 0 "U6" H 3400 2300 50  0000 C CNN
 F 1 "4071" H 3400 2200 50  0000 C CNN
 F 2 "" H 3400 2250 60  0001 C CNN
@@
 $EndComp
 $Comp
-L myCpu-rescue:4071 U5
+L myCpu-rescue:4071 U7
 U 1 1 5AE65887
 P 4350 2225
-F 0 "U5" H 4350 2275 50  0000 C CNN
+F 0 "U7" H 4350 2275 50  0000 C CNN
 F 1 "4071" H 4350 2175 50  0000 C CNN
 F 2 "" H 4350 2225 60  0001 C CNN
@@
 $EndComp
 $Comp
-L myCpu-rescue:4071 U5
+L myCpu-rescue:4071 U7
 U 2 1 5AE658F8
 P 4925 2200
-F 0 "U5" H 4925 2250 50  0000 C CNN
+F 0 "U7" H 4925 2250 50  0000 C CNN
 F 1 "4071" H 4925 2150 50  0000 C CNN
 F 2 "" H 4925 2200 60  0001 C CNN
@@
 $EndComp
 $Comp
-L myCpu-rescue:4071 U5
+L myCpu-rescue:4071 U7
 U 3 1 5AE65977
 P 5450 2175
-F 0 "U5" H 5450 2225 50  0000 C CNN
+F 0 "U7" H 5450 2225 50  0000 C CNN
 F 1 "4071" H 5450 2125 50  0000 C CNN
 F 2 "" H 5450 2175 60  0001 C CNN
@@
 $EndComp
 $Comp
-L myCpu-rescue:4071 U5
+L myCpu-rescue:4071 U7
 U 4 1 5AE65A2C
 P 6100 2225
-F 0 "U5" H 6100 2275 50  0000 C CNN
+F 0 "U7" H 6100 2275 50  0000 C CNN
 F 1 "4071" H 6100 2175 50  0000 C CNN
 F 2 "" H 6100 2225 60  0001 C CNN
@@
 	6100 850  6100 1625
 $Comp
-L spice:0 #GND9
+L spice:0 #GND6
 U 1 1 5AEBC873
 P 7400 1700
-F 0 "#GND9" H 7400 1600 60  0001 C CNN
+F 0 "#GND6" H 7400 1600 60  0001 C CNN
 F 1 "0" H 7400 1630 60  0000 C CNN
 F 2 "" H 7400 1700 60  0000 C CNN
@@
 $EndComp
 $Comp
-L spice:C C5
+L spice:C C7
 U 1 1 5AEBC897
 P 7300 2150
-F 0 "C5" V 7150 2150 60  0000 C CNN
+F 0 "C7" V 7150 2150 60  0000 C CNN
 F 1 "100nF" V 7450 2150 60  0000 C CNN
 F 2 "" H 7300 2150 60  0000 C CNN
@@
 $EndComp
 $Comp
-L myCpu-rescue:VCC #PWR08
+L myCpu-rescue:VCC #PWR011
 U 1 1 5AEBC8FE
 P 6925 2500
-F 0 "#PWR08" H 6925 2350 50  0001 C CNN
+F 0 "#PWR011" H 6925 2350 50  0001 C CNN
 F 1 "VCC" H 6925 2650 50  0000 C CNN
 F 2 "" H 6925 2500 50  0000 C CNN
@@
 	7300 2500 7300 2400
 $Comp
-L spice:0 #GND8
+L spice:0 #GND5
 U 1 1 5AEBCAF9
 P 1025 1850
-F 0 "#GND8" H 1025 1750 60  0001 C CNN
+F 0 "#GND5" H 1025 1750 60  0001 C CNN
 F 1 "0" H 1025 1780 60  0000 C CNN
 F 2 "" H 1025 1850 60  0000 C CNN
@@
 $EndComp
 $Comp
-L spice:C C4
+L spice:C C6
 U 1 1 5AEBCAFF
 P 925 2300
-F 0 "C4" V 775 2300 60  0000 C CNN
+F 0 "C6" V 775 2300 60  0000 C CNN
 F 1 "100nF" V 1075 2300 60  0000 C CNN
 F 2 "" H 925 2300 60  0000 C CNN
@@
 $EndComp
 $Comp
-L myCpu-rescue:VCC #PWR07
+L myCpu-rescue:VCC #PWR010
 U 1 1 5AEBCB05
 P 550 2650
-F 0 "#PWR07" H 550 2500 50  0001 C CNN
+F 0 "#PWR010" H 550 2500 50  0001 C CNN
 F 1 "VCC" H 550 2800 50  0000 C CNN
 F 2 "" H 550 2650 50  0000 C CNN
