File: OR.sch (KiCad schematic (older format))
At the start: 4 parts, among them U6 4071, U7 4071

Commit message: message
Parts:
- renumbered U6 to U11, U6 to U12, U7 to U13, U7 to U14
Changed lines of the file:
@@
 $Descr A4 11693 8268
 encoding utf-8
-Sheet 4 92
+Sheet 4 101
 Title ""
 Date ""
@@
 Z7
 $Comp
-L myCpu-rescue:4071 U6
+L myCpu-rescue:4071 U11
 U 1 1 5AE65623
 P 1500 2200
-F 0 "U6" H 1500 2250 50  0000 C CNN
+F 0 "U11" H 1500 2250 50  0000 C CNN
 F 1 "4071" H 1500 2150 50  0000 C CNN
 F 2 "" H 1500 2200 60  0001 C CNN
@@
 $EndComp
 $Comp
-L myCpu-rescue:4071 U6
+L myCpu-rescue:4071 U11
 U 2 1 5AE656B0
 P 2100 2200
-F 0 "U6" H 2100 2250 50  0000 C CNN
+F 0 "U11" H 2100 2250 50  0000 C CNN
 F 1 "4071" H 2100 2150 50  0000 C CNN
 F 2 "" H 2100 2200 60  0001 C CNN
@@
 $EndComp
 $Comp
-L myCpu-rescue:4071 U6
+L myCpu-rescue:4071 U12
 U 3 1 5AE6574D
 P 2750 2250
-F 0 "U6" H 2750 2300 50  0000 C CNN
+F 0 "U12" H 2750 2300 50  0000 C CNN
 F 1 "4071" H 2750 2200 50  0000 C CNN
 F 2 "" H 2750 2250 60  0001 C CNN
@@
 $EndComp
 $Comp
-L myCpu-rescue:4071 U6
+L myCpu-rescue:4071 U12
 U 4 1 5AE657EA
 P 3400 2250
-F 0 "U6" H 3400 2300 50  0000 C CNN
+F 0 "U12" H 3400 2300 50  0000 C CNN
 F 1 "4071" H 3400 2200 50  0000 C CNN
 F 2 "" H 3400 2250 60  0001 C CNN
@@
 $EndComp
 $Comp
-L myCpu-rescue:4071 U7
+L myCpu-rescue:4071 U13
 U 1 1 5AE65887
 P 4350 2225
-F 0 "U7" H 4350 2275 50  0000 C CNN
+F 0 "U13" H 4350 2275 50  0000 C CNN
 F 1 "4071" H 4350 2175 50  0000 C CNN
 F 2 "" H 4350 2225 60  0001 C CNN
@@
 $EndComp
 $Comp
-L myCpu-rescue:4071 U7
+L myCpu-rescue:4071 U13
 U 2 1 5AE658F8
 P 4925 2200
-F 0 "U7" H 4925 2250 50  0000 C CNN
+F 0 "U13" H 4925 2250 50  0000 C CNN
 F 1 "4071" H 4925 2150 50  0000 C CNN
 F 2 "" H 4925 2200 60  0001 C CNN
@@
 $EndComp
 $Comp
-L myCpu-rescue:4071 U7
+L myCpu-rescue:4071 U14
 U 3 1 5AE65977
 P 5450 2175
-F 0 "U7" H 5450 2225 50  0000 C CNN
+F 0 "U14" H 5450 2225 50  0000 C CNN
 F 1 "4071" H 5450 2125 50  0000 C CNN
 F 2 "" H 5450 2175 60  0001 C CNN
@@
 $EndComp
 $Comp
-L myCpu-rescue:4071 U7
+L myCpu-rescue:4071 U14
 U 4 1 5AE65A2C
 P 6100 2225
-F 0 "U7" H 6100 2275 50  0000 C CNN
+F 0 "U14" H 6100 2275 50  0000 C CNN
 F 1 "4071" H 6100 2175 50  0000 C CNN
 F 2 "" H 6100 2225 60  0001 C CNN
@@
 	6100 850  6100 1625
 $Comp
-L spice:0 #GND6
+L spice:0 #GND5
 U 1 1 5AEBC873
 P 7400 1700
-F 0 "#GND6" H 7400 1600 60  0001 C CNN
+F 0 "#GND5" H 7400 1600 60  0001 C CNN
 F 1 "0" H 7400 1630 60  0000 C CNN
 F 2 "" H 7400 1700 60  0000 C CNN
@@
 $EndComp
 $Comp
-L myCpu-rescue:VCC #PWR011
+L myCpu-rescue:VCC #PWR013
 U 1 1 5AEBC8FE
 P 6925 2500
-F 0 "#PWR011" H 6925 2350 50  0001 C CNN
+F 0 "#PWR013" H 6925 2350 50  0001 C CNN
 F 1 "VCC" H 6925 2650 50  0000 C CNN
 F 2 "" H 6925 2500 50  0000 C CNN
@@
 	7300 2500 7300 2400
 $Comp
-L spice:0 #GND5
+L spice:0 #GND4
 U 1 1 5AEBCAF9
 P 1025 1850
-F 0 "#GND5" H 1025 1750 60  0001 C CNN
+F 0 "#GND4" H 1025 1750 60  0001 C CNN
 F 1 "0" H 1025 1780 60  0000 C CNN
 F 2 "" H 1025 1850 60  0000 C CNN
@@
 $EndComp
 $Comp
-L myCpu-rescue:VCC #PWR010
+L myCpu-rescue:VCC #PWR012
 U 1 1 5AEBCB05
 P 550 2650
-F 0 "#PWR010" H 550 2500 50  0001 C CNN
+F 0 "#PWR012" H 550 2500 50  0001 C CNN
 F 1 "VCC" H 550 2800 50  0000 C CNN
 F 2 "" H 550 2650 50  0000 C CNN
