File: XOR.sch (KiCad schematic (older format))
At the start: 2 parts, among them U7 4070, U8 4070

Commit message: SPICE capacitance and ground symbols
Parts:
- added C? (x2): 100nF, symbol C
Connections:
- net labels added: 0, VCC
- wire segments 78 -> 86

Commit message: fixed duplicate names
Parts:
- gave numbers to parts that had none: 2
Changed lines of the file:
@@
 	5800 1600 4150 1600
 $Comp
-L VCC #PWR?
+L VCC #PWR06
 U 1 1 5AEBE631
 P 8300 4525
-F 0 "#PWR?" H 8300 4375 50  0001 C CNN
+F 0 "#PWR06" H 8300 4375 50  0001 C CNN
 F 1 "VCC" H 8300 4675 50  0000 C CNN
 F 2 "" H 8300 4525 50  0000 C CNN
@@
 $EndComp
 $Comp
-L C C?
+L C C6
 U 1 1 5AEBE655
 P 8025 3975
-F 0 "C?" V 7875 3975 60  0000 C CNN
+F 0 "C6" V 7875 3975 60  0000 C CNN
 F 1 "100nF" V 8175 3975 60  0000 C CNN
 F 2 "" H 8025 3975 60  0000 C CNN
@@
 $EndComp
 $Comp
-L 0 #GND?
+L 0 #GND6
 U 1 1 5AEBE6D2
 P 8100 3275
-F 0 "#GND?" H 8100 3175 60  0001 C CNN
+F 0 "#GND6" H 8100 3175 60  0001 C CNN
 F 1 "0" H 8100 3205 60  0000 C CNN
 F 2 "" H 8100 3275 60  0000 C CNN
@@
 	8100 3725 8100 3275
 $Comp
-L VCC #PWR?
+L VCC #PWR07
 U 1 1 5AEBE8CD
 P 1525 4575
-F 0 "#PWR?" H 1525 4425 50  0001 C CNN
+F 0 "#PWR07" H 1525 4425 50  0001 C CNN
 F 1 "VCC" H 1525 4725 50  0000 C CNN
 F 2 "" H 1525 4575 50  0000 C CNN
@@
 $EndComp
 $Comp
-L C C?
+L C C5
 U 1 1 5AEBE8D3
 P 1250 4025
-F 0 "C?" V 1100 4025 60  0000 C CNN
+F 0 "C5" V 1100 4025 60  0000 C CNN
 F 1 "100nF" V 1400 4025 60  0000 C CNN
 F 2 "" H 1250 4025 60  0000 C CNN
@@
 $EndComp
 $Comp
-L 0 #GND?
+L 0 #GND5
 U 1 1 5AEBE8D9
 P 1325 3325
-F 0 "#GND?" H 1325 3225 60  0001 C CNN
+F 0 "#GND5" H 1325 3225 60  0001 C CNN
 F 1 "0" H 1325 3255 60  0000 C CNN
 F 2 "" H 1325 3325 60  0000 C CNN

Commit message: spice libs from the internet, opened with new kicad 5.0.0, added spice models to components
Parts:
- C5, C6: symbol C -> spice:C
- U7: symbol 4070 -> myCpu-rescue:4070; Spice_Lib_File (none) -> cd4000.lib; Spice_Model (none) -> CD4070B; Spice_Netlist_Enabled (none) -> Y; Spice_Primitive (none) -> X
- U7, U8: symbol 4070 -> myCpu-rescue:4070
Changed lines of the file:
@@
-EESchema Schematic File Version 2
-LIBS:spice
-LIBS:pspice
+EESchema Schematic File Version 4
 LIBS:myCpu-cache
-EELAYER 25 0
+EELAYER 26 0
 EELAYER END
 $Descr A4 11693 8268
@@
 Z7
 $Comp
-L 4070 U7
+L myCpu-rescue:4070 U7
 U 1 1 5AE671E3
 P 2350 3975
@@
 F 2 "" H 2350 3975 60  0001 C CNN
 F 3 "" H 2350 3975 60  0001 C CNN
+F 4 "X" H 2350 3975 50  0001 C CNN "Spice_Primitive"
+F 5 "CD4070B" H 2350 3975 50  0001 C CNN "Spice_Model"
+F 6 "Y" H 2350 3975 50  0001 C CNN "Spice_Netlist_Enabled"
+F 7 "cd4000.lib" H 2350 3975 50  0001 C CNN "Spice_Lib_File"
 	1    2350 3975
 	0    -1   -1   0
 $EndComp
 $Comp
-L 4070 U7
+L myCpu-rescue:4070 U7
 U 2 1 5AE67266
 P 3050 3950
@@
 $EndComp
 $Comp
-L 4070 U7
+L myCpu-rescue:4070 U7
 U 3 1 5AE672EB
 P 3750 3950
@@
 $EndComp
 $Comp
-L 4070 U7
+L myCpu-rescue:4070 U7
 U 4 1 5AE6737A
 P 4450 3925
@@
 $EndComp
 $Comp
-L 4070 U8
+L myCpu-rescue:4070 U8
 U 1 1 5AE67413
 P 5150 3950
@@
 $EndComp
 $Comp
-L 4070 U8
+L myCpu-rescue:4070 U8
 U 2 1 5AE6749C
 P 5825 3950
@@
 $EndComp
 $Comp
-L 4070 U8
+L myCpu-rescue:4070 U8
 U 3 1 5AE67535
 P 6550 3975
@@
 $EndComp
 $Comp
-L 4070 U8
+L myCpu-rescue:4070 U8
 U 4 1 5AE675DA
 P 7250 3975
@@
 	5800 1600 4150 1600
 $Comp
-L VCC #PWR06
+L myCpu-rescue:VCC #PWR06
 U 1 1 5AEBE631
 P 8300 4525
@@
 $EndComp
 $Comp
-L C C6
+L spice:C C6
 U 1 1 5AEBE655
 P 8025 3975
@@
 $EndComp
 $Comp
-L 0 #GND6
+L spice:0 #GND6
 U 1 1 5AEBE6D2
 P 8100 3275
@@
 	8100 3725 8100 3275
 $Comp
-L VCC #PWR07
+L myCpu-rescue:VCC #PWR07
 U 1 1 5AEBE8CD
 P 1525 4575
@@
 $EndComp
 $Comp
-L C C5
+L spice:C C5
 U 1 1 5AEBE8D3
 P 1250 4025
@@
 $EndComp
 $Comp
-L 0 #GND5
+L spice:0 #GND5
 U 1 1 5AEBE8D9
 P 1325 3325

Commit message: lots of work done
Parts:
- renumbered C5 to C6, C6 to C7, U7 to U8, U8 to U9
Changed lines of the file:
@@
 $Descr A4 11693 8268
 encoding utf-8
-Sheet 6 21
+Sheet 6 81
 Title ""
 Date ""
@@
 Z7
 $Comp
-L myCpu-rescue:4070 U7
+L myCpu-rescue:4070 U8
 U 1 1 5AE671E3
 P 2350 3975
-F 0 "U7" H 2350 4025 50  0000 C CNN
+F 0 "U8" H 2350 4025 50  0000 C CNN
 F 1 "4070" H 2350 3925 50  0000 C CNN
 F 2 "" H 2350 3975 60  0001 C CNN
@@
 $EndComp
 $Comp
-L myCpu-rescue:4070 U7
+L myCpu-rescue:4070 U8
 U 2 1 5AE67266
 P 3050 3950
-F 0 "U7" H 3050 4000 50  0000 C CNN
+F 0 "U8" H 3050 4000 50  0000 C CNN
 F 1 "4070" H 3050 3900 50  0000 C CNN
 F 2 "" H 3050 3950 60  0001 C CNN
@@
 $EndComp
 $Comp
-L myCpu-rescue:4070 U7
+L myCpu-rescue:4070 U8
 U 3 1 5AE672EB
 P 3750 3950
-F 0 "U7" H 3750 4000 50  0000 C CNN
+F 0 "U8" H 3750 4000 50  0000 C CNN
 F 1 "4070" H 3750 3900 50  0000 C CNN
 F 2 "" H 3750 3950 60  0001 C CNN
@@
 $EndComp
 $Comp
-L myCpu-rescue:4070 U7
+L myCpu-rescue:4070 U8
 U 4 1 5AE6737A
 P 4450 3925
-F 0 "U7" H 4450 3975 50  0000 C CNN
+F 0 "U8" H 4450 3975 50  0000 C CNN
 F 1 "4070" H 4450 3875 50  0000 C CNN
 F 2 "" H 4450 3925 60  0001 C CNN
@@
 $EndComp
 $Comp
-L myCpu-rescue:4070 U8
+L myCpu-rescue:4070 U9
 U 1 1 5AE67413
 P 5150 3950
-F 0 "U8" H 5150 4000 50  0000 C CNN
+F 0 "U9" H 5150 4000 50  0000 C CNN
 F 1 "4070" H 5150 3900 50  0000 C CNN
 F 2 "" H 5150 3950 60  0001 C CNN
@@
 $EndComp
 $Comp
-L myCpu-rescue:4070 U8
+L myCpu-rescue:4070 U9
 U 2 1 5AE6749C
 P 5825 3950
-F 0 "U8" H 5825 4000 50  0000 C CNN
+F 0 "U9" H 5825 4000 50  0000 C CNN
 F 1 "4070" H 5825 3900 50  0000 C CNN
 F 2 "" H 5825 3950 60  0001 C CNN
@@
 $EndComp
 $Comp
-L myCpu-rescue:4070 U8
+L myCpu-rescue:4070 U9
 U 3 1 5AE67535
 P 6550 3975
-F 0 "U8" H 6550 4025 50  0000 C CNN
+F 0 "U9" H 6550 4025 50  0000 C CNN
 F 1 "4070" H 6550 3925 50  0000 C CNN
 F 2 "" H 6550 3975 60  0001 C CNN
@@
 $EndComp
 $Comp
-L myCpu-rescue:4070 U8
+L myCpu-rescue:4070 U9
 U 4 1 5AE675DA
 P 7250 3975
-F 0 "U8" H 7250 4025 50  0000 C CNN
+F 0 "U9" H 7250 4025 50  0000 C CNN
 F 1 "4070" H 7250 3925 50  0000 C CNN
 F 2 "" H 7250 3975 60  0001 C CNN
@@
 	5800 1600 4150 1600
 $Comp
-L myCpu-rescue:VCC #PWR06
+L myCpu-rescue:VCC #PWR011
 U 1 1 5AEBE631
 P 8300 4525
-F 0 "#PWR06" H 8300 4375 50  0001 C CNN
+F 0 "#PWR011" H 8300 4375 50  0001 C CNN
 F 1 "VCC" H 8300 4675 50  0000 C CNN
 F 2 "" H 8300 4525 50  0000 C CNN
@@
 $EndComp
 $Comp
-L spice:C C6
+L spice:C C7
 U 1 1 5AEBE655
 P 8025 3975
-F 0 "C6" V 7875 3975 60  0000 C CNN
+F 0 "C7" V 7875 3975 60  0000 C CNN
 F 1 "100nF" V 8175 3975 60  0000 C CNN
 F 2 "" H 8025 3975 60  0000 C CNN
@@
 $EndComp
 $Comp
-L spice:0 #GND6
+L spice:0 #GND11
 U 1 1 5AEBE6D2
 P 8100 3275
-F 0 "#GND6" H 8100 3175 60  0001 C CNN
+F 0 "#GND11" H 8100 3175 60  0001 C CNN
 F 1 "0" H 8100 3205 60  0000 C CNN
 F 2 "" H 8100 3275 60  0000 C CNN
@@
 	8100 3725 8100 3275
 $Comp
-L myCpu-rescue:VCC #PWR07
+L myCpu-rescue:VCC #PWR010
 U 1 1 5AEBE8CD
 P 1525 4575
-F 0 "#PWR07" H 1525 4425 50  0001 C CNN
+F 0 "#PWR010" H 1525 4425 50  0001 C CNN
 F 1 "VCC" H 1525 4725 50  0000 C CNN
 F 2 "" H 1525 4575 50  0000 C CNN
@@
 $EndComp
 $Comp
-L spice:C C5
+L spice:C C6
 U 1 1 5AEBE8D3
 P 1250 4025
-F 0 "C5" V 1100 4025 60  0000 C CNN
+F 0 "C6" V 1100 4025 60  0000 C CNN
 F 1 "100nF" V 1400 4025 60  0000 C CNN
 F 2 "" H 1250 4025 60  0000 C CNN
@@
 $EndComp
 $Comp
-L spice:0 #GND5
+L spice:0 #GND10
 U 1 1 5AEBE8D9
 P 1325 3325
-F 0 "#GND5" H 1325 3225 60  0001 C CNN
+F 0 "#GND10" H 1325 3225 60  0001 C CNN
 F 1 "0" H 1325 3255 60  0000 C CNN
 F 2 "" H 1325 3325 60  0000 C CNN

Commit message: b
Parts:
- renumbered C6 to C8, C7 to C9, U8 to U10, U9 to U11
Changed lines of the file:
@@
 $Descr A4 11693 8268
 encoding utf-8
-Sheet 6 90
+Sheet 6 92
 Title ""
 Date ""
@@
 Z7
 $Comp
-L myCpu-rescue:4070 U8
+L myCpu-rescue:4070 U10
 U 1 1 5AE671E3
 P 2350 3975
-F 0 "U8" H 2350 4025 50  0000 C CNN
+F 0 "U10" H 2350 4025 50  0000 C CNN
 F 1 "4070" H 2350 3925 50  0000 C CNN
 F 2 "" H 2350 3975 60  0001 C CNN
@@
 $EndComp
 $Comp
-L myCpu-rescue:4070 U8
+L myCpu-rescue:4070 U10
 U 2 1 5AE67266
 P 3050 3950
-F 0 "U8" H 3050 4000 50  0000 C CNN
+F 0 "U10" H 3050 4000 50  0000 C CNN
 F 1 "4070" H 3050 3900 50  0000 C CNN
 F 2 "" H 3050 3950 60  0001 C CNN
@@
 $EndComp
 $Comp
-L myCpu-rescue:4070 U8
+L myCpu-rescue:4070 U10
 U 3 1 5AE672EB
 P 3750 3950
-F 0 "U8" H 3750 4000 50  0000 C CNN
+F 0 "U10" H 3750 4000 50  0000 C CNN
 F 1 "4070" H 3750 3900 50  0000 C CNN
 F 2 "" H 3750 3950 60  0001 C CNN
@@
 $EndComp
 $Comp
-L myCpu-rescue:4070 U8
+L myCpu-rescue:4070 U10
 U 4 1 5AE6737A
 P 4450 3925
-F 0 "U8" H 4450 3975 50  0000 C CNN
+F 0 "U10" H 4450 3975 50  0000 C CNN
 F 1 "4070" H 4450 3875 50  0000 C CNN
 F 2 "" H 4450 3925 60  0001 C CNN
@@
 $EndComp
 $Comp
-L myCpu-rescue:4070 U9
+L myCpu-rescue:4070 U11
 U 1 1 5AE67413
 P 5150 3950
-F 0 "U9" H 5150 4000 50  0000 C CNN
+F 0 "U11" H 5150 4000 50  0000 C CNN
 F 1 "4070" H 5150 3900 50  0000 C CNN
 F 2 "" H 5150 3950 60  0001 C CNN
@@
 $EndComp
 $Comp
-L myCpu-rescue:4070 U9
+L myCpu-rescue:4070 U11
 U 2 1 5AE6749C
 P 5825 3950
-F 0 "U9" H 5825 4000 50  0000 C CNN
+F 0 "U11" H 5825 4000 50  0000 C CNN
 F 1 "4070" H 5825 3900 50  0000 C CNN
 F 2 "" H 5825 3950 60  0001 C CNN
@@
 $EndComp
 $Comp
-L myCpu-rescue:4070 U9
+L myCpu-rescue:4070 U11
 U 3 1 5AE67535
 P 6550 3975
-F 0 "U9" H 6550 4025 50  0000 C CNN
+F 0 "U11" H 6550 4025 50  0000 C CNN
 F 1 "4070" H 6550 3925 50  0000 C CNN
 F 2 "" H 6550 3975 60  0001 C CNN
@@
 $EndComp
 $Comp
-L myCpu-rescue:4070 U9
+L myCpu-rescue:4070 U11
 U 4 1 5AE675DA
 P 7250 3975
-F 0 "U9" H 7250 4025 50  0000 C CNN
+F 0 "U11" H 7250 4025 50  0000 C CNN
 F 1 "4070" H 7250 3925 50  0000 C CNN
 F 2 "" H 7250 3975 60  0001 C CNN
@@
 	5800 1600 4150 1600
 $Comp
-L myCpu-rescue:VCC #PWR011
+L myCpu-rescue:VCC #PWR018
 U 1 1 5AEBE631
 P 8300 4525
-F 0 "#PWR011" H 8300 4375 50  0001 C CNN
+F 0 "#PWR018" H 8300 4375 50  0001 C CNN
 F 1 "VCC" H 8300 4675 50  0000 C CNN
 F 2 "" H 8300 4525 50  0000 C CNN
@@
 $EndComp
 $Comp
-L spice:C C7
+L spice:C C9
 U 1 1 5AEBE655
 P 8025 3975
-F 0 "C7" V 7875 3975 60  0000 C CNN
+F 0 "C9" V 7875 3975 60  0000 C CNN
 F 1 "100nF" V 8175 3975 60  0000 C CNN
 F 2 "" H 8025 3975 60  0000 C CNN
@@
 $EndComp
 $Comp
-L spice:0 #GND11
+L spice:0 #GND8
 U 1 1 5AEBE6D2
 P 8100 3275
-F 0 "#GND11" H 8100 3175 60  0001 C CNN
+F 0 "#GND8" H 8100 3175 60  0001 C CNN
 F 1 "0" H 8100 3205 60  0000 C CNN
 F 2 "" H 8100 3275 60  0000 C CNN
@@
 	8100 3725 8100 3275
 $Comp
-L myCpu-rescue:VCC #PWR010
+L myCpu-rescue:VCC #PWR017
 U 1 1 5AEBE8CD
 P 1525 4575
-F 0 "#PWR010" H 1525 4425 50  0001 C CNN
+F 0 "#PWR017" H 1525 4425 50  0001 C CNN
 F 1 "VCC" H 1525 4725 50  0000 C CNN
 F 2 "" H 1525 4575 50  0000 C CNN
@@
 $EndComp
 $Comp
-L spice:C C6
+L spice:C C8
 U 1 1 5AEBE8D3
 P 1250 4025
-F 0 "C6" V 1100 4025 60  0000 C CNN
+F 0 "C8" V 1100 4025 60  0000 C CNN
 F 1 "100nF" V 1400 4025 60  0000 C CNN
 F 2 "" H 1250 4025 60  0000 C CNN
@@
 $EndComp
 $Comp
-L spice:0 #GND10
+L spice:0 #GND7
 U 1 1 5AEBE8D9
 P 1325 3325
-F 0 "#GND10" H 1325 3225 60  0001 C CNN
+F 0 "#GND7" H 1325 3225 60  0001 C CNN
 F 1 "0" H 1325 3255 60  0000 C CNN
 F 2 "" H 1325 3325 60  0000 C CNN
