File: XOR.sch (KiCad schematic (older format))
At the start: 4 parts, among them U10 4070, U11 4070

Commit message: message
Parts:
- renumbered U10 to U21, U10 to U22, U11 to U23, U11 to U24
Changed lines of the file:
@@
 $Descr A4 11693 8268
 encoding utf-8
-Sheet 6 92
+Sheet 6 101
 Title ""
 Date ""
@@
 Z7
 $Comp
-L myCpu-rescue:4070 U10
+L myCpu-rescue:4070 U21
 U 1 1 5AE671E3
 P 2350 3975
-F 0 "U10" H 2350 4025 50  0000 C CNN
+F 0 "U21" H 2350 4025 50  0000 C CNN
 F 1 "4070" H 2350 3925 50  0000 C CNN
 F 2 "" H 2350 3975 60  0001 C CNN
@@
 $EndComp
 $Comp
-L myCpu-rescue:4070 U10
+L myCpu-rescue:4070 U21
 U 2 1 5AE67266
 P 3050 3950
-F 0 "U10" H 3050 4000 50  0000 C CNN
+F 0 "U21" H 3050 4000 50  0000 C CNN
 F 1 "4070" H 3050 3900 50  0000 C CNN
 F 2 "" H 3050 3950 60  0001 C CNN
@@
 $EndComp
 $Comp
-L myCpu-rescue:4070 U10
+L myCpu-rescue:4070 U22
 U 3 1 5AE672EB
 P 3750 3950
-F 0 "U10" H 3750 4000 50  0000 C CNN
+F 0 "U22" H 3750 4000 50  0000 C CNN
 F 1 "4070" H 3750 3900 50  0000 C CNN
 F 2 "" H 3750 3950 60  0001 C CNN
@@
 $EndComp
 $Comp
-L myCpu-rescue:4070 U10
+L myCpu-rescue:4070 U22
 U 4 1 5AE6737A
 P 4450 3925
-F 0 "U10" H 4450 3975 50  0000 C CNN
+F 0 "U22" H 4450 3975 50  0000 C CNN
 F 1 "4070" H 4450 3875 50  0000 C CNN
 F 2 "" H 4450 3925 60  0001 C CNN
@@
 $EndComp
 $Comp
-L myCpu-rescue:4070 U11
+L myCpu-rescue:4070 U23
 U 1 1 5AE67413
 P 5150 3950
-F 0 "U11" H 5150 4000 50  0000 C CNN
+F 0 "U23" H 5150 4000 50  0000 C CNN
 F 1 "4070" H 5150 3900 50  0000 C CNN
 F 2 "" H 5150 3950 60  0001 C CNN
@@
 $EndComp
 $Comp
-L myCpu-rescue:4070 U11
+L myCpu-rescue:4070 U23
 U 2 1 5AE6749C
 P 5825 3950
-F 0 "U11" H 5825 4000 50  0000 C CNN
+F 0 "U23" H 5825 4000 50  0000 C CNN
 F 1 "4070" H 5825 3900 50  0000 C CNN
 F 2 "" H 5825 3950 60  0001 C CNN
@@
 $EndComp
 $Comp
-L myCpu-rescue:4070 U11
+L myCpu-rescue:4070 U24
 U 3 1 5AE67535
 P 6550 3975
-F 0 "U11" H 6550 4025 50  0000 C CNN
+F 0 "U24" H 6550 4025 50  0000 C CNN
 F 1 "4070" H 6550 3925 50  0000 C CNN
 F 2 "" H 6550 3975 60  0001 C CNN
@@
 $EndComp
 $Comp
-L myCpu-rescue:4070 U11
+L myCpu-rescue:4070 U24
 U 4 1 5AE675DA
 P 7250 3975
-F 0 "U11" H 7250 4025 50  0000 C CNN
+F 0 "U24" H 7250 4025 50  0000 C CNN
 F 1 "4070" H 7250 3925 50  0000 C CNN
 F 2 "" H 7250 3975 60  0001 C CNN
@@
 	5800 1600 4150 1600
 $Comp
-L myCpu-rescue:VCC #PWR018
+L myCpu-rescue:VCC #PWR020
 U 1 1 5AEBE631
 P 8300 4525
-F 0 "#PWR018" H 8300 4375 50  0001 C CNN
+F 0 "#PWR020" H 8300 4375 50  0001 C CNN
 F 1 "VCC" H 8300 4675 50  0000 C CNN
 F 2 "" H 8300 4525 50  0000 C CNN
@@
 $EndComp
 $Comp
-L spice:0 #GND8
+L spice:0 #GND7
 U 1 1 5AEBE6D2
 P 8100 3275
-F 0 "#GND8" H 8100 3175 60  0001 C CNN
+F 0 "#GND7" H 8100 3175 60  0001 C CNN
 F 1 "0" H 8100 3205 60  0000 C CNN
 F 2 "" H 8100 3275 60  0000 C CNN
@@
 	8100 3725 8100 3275
 $Comp
-L myCpu-rescue:VCC #PWR017
+L myCpu-rescue:VCC #PWR019
 U 1 1 5AEBE8CD
 P 1525 4575
-F 0 "#PWR017" H 1525 4425 50  0001 C CNN
+F 0 "#PWR019" H 1525 4425 50  0001 C CNN
 F 1 "VCC" H 1525 4725 50  0000 C CNN
 F 2 "" H 1525 4575 50  0000 C CNN
@@
 $EndComp
 $Comp
-L spice:0 #GND7
+L spice:0 #GND6
 U 1 1 5AEBE8D9
 P 1325 3325
-F 0 "#GND7" H 1325 3225 60  0001 C CNN
+F 0 "#GND6" H 1325 3225 60  0001 C CNN
 F 1 "0" H 1325 3255 60  0000 C CNN
 F 2 "" H 1325 3325 60  0000 C CNN
