File: 8-BIT_16-1MUX.sch (KiCad schematic (older format))
At the start: 4 parts

Commit message: SPICE capacitance and ground symbols
Parts:
- removed C? (x2): 100n, symbol C_Small
- added C? (x2): 100nF, symbol C
Connections:
- net labels added: 0
- net labels removed: GND
- wire segments 482 -> 479
Changed lines of the file:
@@
 EESchema Schematic File Version 2
-LIBS:power
-LIBS:device
-LIBS:transistors
-LIBS:conn
-LIBS:linear
-LIBS:regul
-LIBS:74xx
-LIBS:cmos4000
-LIBS:adc-dac
-LIBS:memory
-LIBS:xilinx
-LIBS:microcontrollers
-LIBS:dsp
-LIBS:microchip
-LIBS:analog_switches
-LIBS:motorola
-LIBS:texas
-LIBS:intel
-LIBS:audio
-LIBS:interface
-LIBS:digital-audio
-LIBS:philips
-LIBS:display
-LIBS:cypress
-LIBS:siliconi
-LIBS:opto
-LIBS:atmel
-LIBS:contrib
-LIBS:valves
+LIBS:spice
+LIBS:pspice
 LIBS:myCpu-cache
 EELAYER 25 0
@@
 	11975 28950 11975 29000
 $Comp
-L C_Small C?
-U 1 1 5AF37E2A
-P 16200 19475
-F 0 "C?" H 16210 19545 50  0000 L CNN
-F 1 "100n" H 16210 19395 50  0000 L CNN
-F 2 "" H 16200 19475 50  0000 C CNN
-F 3 "" H 16200 19475 50  0000 C CNN
-	1    16200 19475
-	1    0    0    -1
-$EndComp
-$Comp
-L C_Small C?
-U 1 1 5AF38A47
-P 15000 7225
-F 0 "C?" H 15010 7295 50  0000 L CNN
-F 1 "100n" H 15010 7145 50  0000 L CNN
-F 2 "" H 15000 7225 50  0000 C CNN
-F 3 "" H 15000 7225 50  0000 C CNN
-	1    15000 7225
-	1    0    0    -1
-$EndComp
-$Comp
 L VCC #PWR?
 U 1 1 5AF3D664
@@
 F 3 "" H 15800 19500 50  0000 C CNN
 	1    15800 19500
-	1    0    0    -1
-$EndComp
-$Comp
-L GND #PWR?
-U 1 1 5AF3DA70
-P 16625 19475
-F 0 "#PWR?" H 16625 19225 50  0001 C CNN
-F 1 "GND" H 16625 19325 50  0000 C CNN
-F 2 "" H 16625 19475 50  0000 C CNN
-F 3 "" H 16625 19475 50  0000 C CNN
-	1    16625 19475
-	1    0    0    -1
-$EndComp
-$Comp
-L GND #PWR?
-U 1 1 5AF3F64C
-P 15075 7575
-F 0 "#PWR?" H 15075 7325 50  0001 C CNN
-F 1 "GND" H 15075 7425 50  0000 C CNN
-F 2 "" H 15075 7575 50  0000 C CNN
-F 3 "" H 15075 7575 50  0000 C CNN
-	1    15075 7575
 	1    0    0    -1
 $EndComp
@@
 	14600 7050 15000 7050
 Wire Wire Line
-	15000 7050 15000 7125
-Wire Wire Line
-	15000 7325 15000 7575
-Wire Wire Line
-	15000 7575 15075 7575
-Wire Wire Line
 	15400 19175 15400 19500
 Wire Wire Line
@@
 	16050 19375 16200 19375
 Connection ~ 15800 19500
-Wire Wire Line
-	16200 19575 16450 19575
-Wire Wire Line
-	16450 19575 16450 19475
-Wire Wire Line
-	16450 19475 16625 19475
 Wire Wire Line
 	15100 19075 15400 19075
@@
 Wire Wire Line
 	9825 15875 9450 15875
+$Comp
+L C C?
+U 1 1 5AE9ADCE
+P 15000 7400
+F 0 "C?" V 14850 7400 60  0000 C CNN
+F 1 "100nF" V 15150 7400 60  0000 C CNN
+F 2 "" H 15000 7400 60  0000 C CNN
+F 3 "" H 15000 7400 60  0000 C CNN
+	1    15000 7400
+	1    0    0    -1
+$EndComp
+Wire Wire Line
+	15000 7050 15000 7150
+Wire Wire Line
+	15025 7650 15000 7650
+$Comp
+L 0 #GND?
+U 1 1 5AEA4D0B
+P 15025 7775
+F 0 "#GND?" H 15025 7675 60  0001 C CNN
+F 1 "0" H 15025 7705 60  0000 C CNN
+F 2 "" H 15025 7775 60  0000 C CNN
+F 3 "" H 15025 7775 60  0000 C CNN
+	1    15025 7775
+	1    0    0    -1
+$EndComp
+Wire Wire Line
+	15025 7650 15025 7775
+$Comp
+L C C?
+U 1 1 5AEAE0FD
+P 16200 19625
+F 0 "C?" V 16050 19625 60  0000 C CNN
+F 1 "100nF" V 16350 19625 60  0000 C CNN
+F 2 "" H 16200 19625 60  0000 C CNN
+F 3 "" H 16200 19625 60  0000 C CNN
+	1    16200 19625
+	1    0    0    -1
+$EndComp
+$Comp
+L 0 #GND?
+U 1 1 5AEAE570
+P 16200 19875
+F 0 "#GND?" H 16200 19775 60  0001 C CNN
+F 1 "0" H 16200 19805 60  0000 C CNN
+F 2 "" H 16200 19875 60  0000 C CNN
+F 3 "" H 16200 19875 60  0000 C CNN
+	1    16200 19875
+	1    0    0    -1
+$EndComp
 $EndSCHEMATC

Commit message: fixed duplicate names
Parts:
- gave numbers to parts that had none: 4
Changed lines of the file:
@@
 S 9350 1650 1675 2550
 U 5AE9E178
-F0 "16-2MUX" 60
+F0 "16-2MUX0" 60
 F1 "16-2MUX.sch" 60
 F2 "X0" I L 9350 1850 60
@@
 S 9400 4550 1675 2550
 U 5AEA87F7
-F0 "16-2MUX" 60
+F0 "16-2MUX1" 60
 F1 "16-2MUX.sch" 60
 F2 "X0" I L 9400 4750 60
@@
 S 9375 7700 1675 2550
 U 5AEB0026
-F0 "16-2MUX" 60
+F0 "16-2MUX2" 60
 F1 "16-2MUX.sch" 60
 F2 "X0" I L 9375 7900 60
@@
 S 9425 10600 1675 2550
 U 5AEB003D
-F0 "16-2MUX" 60
+F0 "16-2MUX3" 60
 F1 "16-2MUX.sch" 60
 F2 "X0" I L 9425 10800 60
@@
 S 9825 14175 1675 2550
 U 5AEC7274
-F0 "16-2MUX" 60
+F0 "16-2MUX4" 60
 F1 "16-2MUX.sch" 60
 F2 "X0" I L 9825 14375 60
@@
 S 9875 17075 1675 2550
 U 5AEC728B
-F0 "16-2MUX" 60
+F0 "16-2MUX5" 60
 F1 "16-2MUX.sch" 60
 F2 "X0" I L 9875 17275 60
@@
 S 9850 20225 1675 2550
 U 5AEC72A2
-F0 "16-2MUX" 60
+F0 "16-2MUX6" 60
 F1 "16-2MUX.sch" 60
 F2 "X0" I L 9850 20425 60
@@
 S 9900 23125 1675 2550
 U 5AEC72B9
-F0 "16-2MUX" 60
+F0 "16-2MUX7" 60
 F1 "16-2MUX.sch" 60
 F2 "X0" I L 9900 23325 60
@@
 $EndSheet
 $Comp
-L 74LS158 U?
+L 74LS158 U17
 U 1 1 5AECFE89
 P 15350 6025
-F 0 "U?" H 15400 6175 50  0000 C CNN
+F 0 "U17" H 15400 6175 50  0000 C CNN
 F 1 "74LS158" H 15400 5875 50  0000 C CNN
 F 2 "" H 15350 6025 50  0000 C CNN
@@
 $EndComp
 $Comp
-L 74LS158 U?
+L 74LS158 U18
 U 1 1 5AED0336
 P 16150 18625
-F 0 "U?" H 16200 18775 50  0000 C CNN
+F 0 "U18" H 16200 18775 50  0000 C CNN
 F 1 "74LS158" H 16200 18475 50  0000 C CNN
 F 2 "" H 16150 18625 50  0000 C CNN
@@
 	11975 28950 11975 29000
 $Comp
-L VCC #PWR?
+L VCC #PWR017
 U 1 1 5AF3D664
 P 15800 19500
-F 0 "#PWR?" H 15800 19350 50  0001 C CNN
+F 0 "#PWR017" H 15800 19350 50  0001 C CNN
 F 1 "VCC" H 15800 19650 50  0000 C CNN
 F 2 "" H 15800 19500 50  0000 C CNN
@@
 $EndComp
 $Comp
-L VCC #PWR?
+L VCC #PWR018
 U 1 1 5AF3FA58
 P 15000 7050
-F 0 "#PWR?" H 15000 6900 50  0001 C CNN
+F 0 "#PWR018" H 15000 6900 50  0001 C CNN
 F 1 "VCC" H 15000 7200 50  0000 C CNN
 F 2 "" H 15000 7050 50  0000 C CNN
@@
 	9825 15875 9450 15875
 $Comp
-L C C?
+L C C15
 U 1 1 5AE9ADCE
 P 15000 7400
-F 0 "C?" V 14850 7400 60  0000 C CNN
+F 0 "C15" V 14850 7400 60  0000 C CNN
 F 1 "100nF" V 15150 7400 60  0000 C CNN
 F 2 "" H 15000 7400 60  0000 C CNN
@@
 	15025 7650 15000 7650
 $Comp
-L 0 #GND?
+L 0 #GND17
 U 1 1 5AEA4D0B
 P 15025 7775
-F 0 "#GND?" H 15025 7675 60  0001 C CNN
+F 0 "#GND17" H 15025 7675 60  0001 C CNN
 F 1 "0" H 15025 7705 60  0000 C CNN
 F 2 "" H 15025 7775 60  0000 C CNN
@@
 	15025 7650 15025 7775
 $Comp
-L C C?
+L C C16
 U 1 1 5AEAE0FD
 P 16200 19625
-F 0 "C?" V 16050 19625 60  0000 C CNN
+F 0 "C16" V 16050 19625 60  0000 C CNN
 F 1 "100nF" V 16350 19625 60  0000 C CNN
 F 2 "" H 16200 19625 60  0000 C CNN
@@
 $EndComp
 $Comp
-L 0 #GND?
+L 0 #GND18
 U 1 1 5AEAE570
 P 16200 19875
-F 0 "#GND?" H 16200 19775 60  0001 C CNN
+F 0 "#GND18" H 16200 19775 60  0001 C CNN
 F 1 "0" H 16200 19805 60  0000 C CNN
 F 2 "" H 16200 19875 60  0000 C CNN

Commit message: spice libs from the internet, opened with new kicad 5.0.0, added spice models to components
Parts:
- C15, C16: symbol C -> spice:C
- U17: symbol 74LS158 -> myCpu-rescue:74LS158; Spice_Lib_File (none) -> 74hc.lib; Spice_Model (none) -> 74HC158; Spice_Netlist_Enabled (none) -> Y; Spice_Primitive (none) -> X
- U18: symbol 74LS158 -> myCpu-rescue:74LS158
Connections:
- wire segments 479 -> 480
Changed lines of the file:
@@
-EESchema Schematic File Version 2
-LIBS:spice
-LIBS:pspice
+EESchema Schematic File Version 4
 LIBS:myCpu-cache
-EELAYER 25 0
+EELAYER 26 0
 EELAYER END
 $Descr A0 46811 33110
@@
 $EndSheet
 $Comp
-L 74LS158 U17
+L myCpu-rescue:74LS158 U17
 U 1 1 5AECFE89
 P 15350 6025
@@
 F 2 "" H 15350 6025 50  0000 C CNN
 F 3 "" H 15350 6025 50  0000 C CNN
+F 4 "X" H 15350 6025 50  0001 C CNN "Spice_Primitive"
+F 5 "74HC158" H 15350 6025 50  0001 C CNN "Spice_Model"
+F 6 "Y" H 15350 6025 50  0001 C CNN "Spice_Netlist_Enabled"
+F 7 "74hc.lib" H 15350 6025 50  0001 C CNN "Spice_Lib_File"
 	1    15350 6025
 	1    0    0    -1
 $EndComp
 $Comp
-L 74LS158 U18
+L myCpu-rescue:74LS158 U18
 U 1 1 5AED0336
 P 16150 18625
@@
 	11975 28950 11975 29000
 $Comp
-L VCC #PWR017
+L myCpu-rescue:VCC #PWR017
 U 1 1 5AF3D664
 P 15800 19500
@@
 $EndComp
 $Comp
-L VCC #PWR018
+L myCpu-rescue:VCC #PWR018
 U 1 1 5AF3FA58
 P 15000 7050
@@
 	15400 19175 15400 19500
 Wire Wire Line
-	15400 19500 16050 19500
+	15400 19500 15800 19500
 Wire Wire Line
 	16050 19500 16050 19375
@@
 	9825 15875 9450 15875
 $Comp
-L C C15
+L spice:C C15
 U 1 1 5AE9ADCE
 P 15000 7400
@@
 	15025 7650 15000 7650
 $Comp
-L 0 #GND17
+L spice:0 #GND17
 U 1 1 5AEA4D0B
 P 15025 7775
@@
 	15025 7650 15025 7775
 $Comp
-L C C16
+L spice:C C16
 U 1 1 5AEAE0FD
 P 16200 19625
@@
 $EndComp
 $Comp
-L 0 #GND18
+L spice:0 #GND18
 U 1 1 5AEAE570
 P 16200 19875
@@
 	1    0    0    -1
 $EndComp
+Wire Wire Line
+	15800 19500 16050 19500
 $EndSCHEMATC

Commit message: lots of work done
Parts:
- renumbered C15 to C16, C16 to C17, U17 to U18, U18 to U19
Changed lines of the file:
@@
 $Descr A0 46811 33110
 encoding utf-8
-Sheet 11 21
+Sheet 40 81
 Title ""
 Date ""
@@
 $EndSheet
 $Comp
-L myCpu-rescue:74LS158 U17
+L myCpu-rescue:74LS158 U18
 U 1 1 5AECFE89
 P 15350 6025
-F 0 "U17" H 15400 6175 50  0000 C CNN
+AR Path="/5AE62FB7/5AE9DF6E/5AECFE89" Ref="U18"  Part="1"
+AR Path="/5B1119BA/5BE38555/5AECFE89" Ref="U111"  Part="1"
+AR Path="/5B1119BA/5C00E21C/5AECFE89" Ref="U129"  Part="1"
+F 0 "U111" H 15400 6175 50  0000 C CNN
 F 1 "74LS158" H 15400 5875 50  0000 C CNN
 F 2 "" H 15350 6025 50  0000 C CNN
@@
 $EndComp
 $Comp
-L myCpu-rescue:74LS158 U18
+L myCpu-rescue:74LS158 U19
 U 1 1 5AED0336
 P 16150 18625
-F 0 "U18" H 16200 18775 50  0000 C CNN
+AR Path="/5AE62FB7/5AE9DF6E/5AED0336" Ref="U19"  Part="1"
+AR Path="/5B1119BA/5BE38555/5AED0336" Ref="U112"  Part="1"
+AR Path="/5B1119BA/5C00E21C/5AED0336" Ref="U130"  Part="1"
+F 0 "U112" H 16200 18775 50  0000 C CNN
 F 1 "74LS158" H 16200 18475 50  0000 C CNN
 F 2 "" H 16150 18625 50  0000 C CNN
@@
 	11975 28950 11975 29000
 $Comp
-L myCpu-rescue:VCC #PWR017
+L myCpu-rescue:VCC #PWR022
 U 1 1 5AF3D664
 P 15800 19500
-F 0 "#PWR017" H 15800 19350 50  0001 C CNN
+AR Path="/5AE62FB7/5AE9DF6E/5AF3D664" Ref="#PWR022"  Part="1"
+AR Path="/5B1119BA/5BE38555/5AF3D664" Ref="#PWR0304"  Part="1"
+AR Path="/5B1119BA/5C00E21C/5AF3D664" Ref="#PWR0322"  Part="1"
+F 0 "#PWR0304" H 15800 19350 50  0001 C CNN
 F 1 "VCC" H 15800 19650 50  0000 C CNN
 F 2 "" H 15800 19500 50  0000 C CNN
@@
 $EndComp
 $Comp
-L myCpu-rescue:VCC #PWR018
+L myCpu-rescue:VCC #PWR021
 U 1 1 5AF3FA58
 P 15000 7050
-F 0 "#PWR018" H 15000 6900 50  0001 C CNN
+AR Path="/5AE62FB7/5AE9DF6E/5AF3FA58" Ref="#PWR021"  Part="1"
+AR Path="/5B1119BA/5BE38555/5AF3FA58" Ref="#PWR0303"  Part="1"
+AR Path="/5B1119BA/5C00E21C/5AF3FA58" Ref="#PWR0321"  Part="1"
+F 0 "#PWR0303" H 15000 6900 50  0001 C CNN
 F 1 "VCC" H 15000 7200 50  0000 C CNN
 F 2 "" H 15000 7050 50  0000 C CNN
@@
 	9825 15875 9450 15875
 $Comp
-L spice:C C15
+L spice:C C16
 U 1 1 5AE9ADCE
 P 15000 7400
-F 0 "C15" V 14850 7400 60  0000 C CNN
+AR Path="/5AE62FB7/5AE9DF6E/5AE9ADCE" Ref="C16"  Part="1"
+AR Path="/5B1119BA/5BE38555/5AE9ADCE" Ref="C170"  Part="1"
+AR Path="/5B1119BA/5C00E21C/5AE9ADCE" Ref="C188"  Part="1"
+F 0 "C170" V 14850 7400 60  0000 C CNN
 F 1 "100nF" V 15150 7400 60  0000 C CNN
 F 2 "" H 15000 7400 60  0000 C CNN
@@
 	15025 7650 15000 7650
 $Comp
-L spice:0 #GND17
+L spice:0 #GND22
 U 1 1 5AEA4D0B
 P 15025 7775
-F 0 "#GND17" H 15025 7675 60  0001 C CNN
+AR Path="/5AE62FB7/5AE9DF6E/5AEA4D0B" Ref="#GND22"  Part="1"
+AR Path="/5B1119BA/5BE38555/5AEA4D0B" Ref="#GND47"  Part="1"
+AR Path="/5B1119BA/5C00E21C/5AEA4D0B" Ref="#GND65"  Part="1"
+F 0 "#GND47" H 15025 7675 60  0001 C CNN
 F 1 "0" H 15025 7705 60  0000 C CNN
 F 2 "" H 15025 7775 60  0000 C CNN
@@
 	15025 7650 15025 7775
 $Comp
-L spice:C C16
+L spice:C C17
 U 1 1 5AEAE0FD
 P 16200 19625
-F 0 "C16" V 16050 19625 60  0000 C CNN
+AR Path="/5AE62FB7/5AE9DF6E/5AEAE0FD" Ref="C17"  Part="1"
+AR Path="/5B1119BA/5BE38555/5AEAE0FD" Ref="C171"  Part="1"
+AR Path="/5B1119BA/5C00E21C/5AEAE0FD" Ref="C189"  Part="1"
+F 0 "C171" V 16050 19625 60  0000 C CNN
 F 1 "100nF" V 16350 19625 60  0000 C CNN
 F 2 "" H 16200 19625 60  0000 C CNN
@@
 $EndComp
 $Comp
-L spice:0 #GND18
+L spice:0 #GND23
 U 1 1 5AEAE570
 P 16200 19875
-F 0 "#GND18" H 16200 19775 60  0001 C CNN
+AR Path="/5AE62FB7/5AE9DF6E/5AEAE570" Ref="#GND23"  Part="1"
+AR Path="/5B1119BA/5BE38555/5AEAE570" Ref="#GND48"  Part="1"
+AR Path="/5B1119BA/5C00E21C/5AEAE570" Ref="#GND66"  Part="1"
+F 0 "#GND48" H 16200 19775 60  0001 C CNN
 F 1 "0" H 16200 19805 60  0000 C CNN
 F 2 "" H 16200 19875 60  0000 C CNN

Commit message: b
Parts:
- renumbered C16 to C18, C17 to C19, U18 to U20, U19 to U21
Changed lines of the file:
@@
 $Descr A0 46811 33110
 encoding utf-8
-Sheet 40 90
+Sheet 11 92
 Title ""
 Date ""
@@
 $EndSheet
 $Comp
-L myCpu-rescue:74LS158 U18
+L myCpu-rescue:74LS158 U20
 U 1 1 5AECFE89
 P 15350 6025
-AR Path="/5AE62FB7/5AE9DF6E/5AECFE89" Ref="U18"  Part="1"
-AR Path="/5B1119BA/5BE38555/5AECFE89" Ref="U111"  Part="1"
-AR Path="/5B1119BA/5C00E21C/5AECFE89" Ref="U129"  Part="1"
-F 0 "U111" H 15400 6175 50  0000 C CNN
+AR Path="/5AE62FB7/5AE9DF6E/5AECFE89" Ref="U20"  Part="1"
+AR Path="/5B1119BA/5BE38555/5AECFE89" Ref="U113"  Part="1"
+AR Path="/5B1119BA/5C00E21C/5AECFE89" Ref="U131"  Part="1"
+F 0 "U20" H 15400 6175 50  0000 C CNN
 F 1 "74LS158" H 15400 5875 50  0000 C CNN
 F 2 "" H 15350 6025 50  0000 C CNN
@@
 $EndComp
 $Comp
-L myCpu-rescue:74LS158 U19
+L myCpu-rescue:74LS158 U21
 U 1 1 5AED0336
 P 16150 18625
-AR Path="/5AE62FB7/5AE9DF6E/5AED0336" Ref="U19"  Part="1"
-AR Path="/5B1119BA/5BE38555/5AED0336" Ref="U112"  Part="1"
-AR Path="/5B1119BA/5C00E21C/5AED0336" Ref="U130"  Part="1"
-F 0 "U112" H 16200 18775 50  0000 C CNN
+AR Path="/5AE62FB7/5AE9DF6E/5AED0336" Ref="U21"  Part="1"
+AR Path="/5B1119BA/5BE38555/5AED0336" Ref="U114"  Part="1"
+AR Path="/5B1119BA/5C00E21C/5AED0336" Ref="U132"  Part="1"
+F 0 "U21" H 16200 18775 50  0000 C CNN
 F 1 "74LS158" H 16200 18475 50  0000 C CNN
 F 2 "" H 16150 18625 50  0000 C CNN
@@
 Text HLabel 35700 8000 2    60   Output ~ 0
 Z7
-Wire Wire Line
-	16125 5525 35625 5525
 Wire Wire Line
 	35625 5525 35625 6075
@@
 	11975 28950 11975 29000
 $Comp
-L myCpu-rescue:VCC #PWR022
+L myCpu-rescue:VCC #PWR029
 U 1 1 5AF3D664
 P 15800 19500
-AR Path="/5AE62FB7/5AE9DF6E/5AF3D664" Ref="#PWR022"  Part="1"
-AR Path="/5B1119BA/5BE38555/5AF3D664" Ref="#PWR0304"  Part="1"
-AR Path="/5B1119BA/5C00E21C/5AF3D664" Ref="#PWR0322"  Part="1"
-F 0 "#PWR0304" H 15800 19350 50  0001 C CNN
+AR Path="/5AE62FB7/5AE9DF6E/5AF3D664" Ref="#PWR029"  Part="1"
+AR Path="/5B1119BA/5BE38555/5AF3D664" Ref="#PWR0315"  Part="1"
+AR Path="/5B1119BA/5C00E21C/5AF3D664" Ref="#PWR0333"  Part="1"
+F 0 "#PWR0333" H 15800 19350 50  0001 C CNN
 F 1 "VCC" H 15800 19650 50  0000 C CNN
 F 2 "" H 15800 19500 50  0000 C CNN
@@
 $EndComp
 $Comp
-L myCpu-rescue:VCC #PWR021
+L myCpu-rescue:VCC #PWR028
 U 1 1 5AF3FA58
 P 15000 7050
-AR Path="/5AE62FB7/5AE9DF6E/5AF3FA58" Ref="#PWR021"  Part="1"
-AR Path="/5B1119BA/5BE38555/5AF3FA58" Ref="#PWR0303"  Part="1"
-AR Path="/5B1119BA/5C00E21C/5AF3FA58" Ref="#PWR0321"  Part="1"
-F 0 "#PWR0303" H 15000 6900 50  0001 C CNN
+AR Path="/5AE62FB7/5AE9DF6E/5AF3FA58" Ref="#PWR028"  Part="1"
+AR Path="/5B1119BA/5BE38555/5AF3FA58" Ref="#PWR0314"  Part="1"
+AR Path="/5B1119BA/5C00E21C/5AF3FA58" Ref="#PWR0332"  Part="1"
+F 0 "#PWR0332" H 15000 6900 50  0001 C CNN
 F 1 "VCC" H 15000 7200 50  0000 C CNN
 F 2 "" H 15000 7050 50  0000 C CNN
@@
 	9825 15875 9450 15875
 $Comp
-L spice:C C16
+L spice:C C18
 U 1 1 5AE9ADCE
 P 15000 7400
-AR Path="/5AE62FB7/5AE9DF6E/5AE9ADCE" Ref="C16"  Part="1"
-AR Path="/5B1119BA/5BE38555/5AE9ADCE" Ref="C170"  Part="1"
-AR Path="/5B1119BA/5C00E21C/5AE9ADCE" Ref="C188"  Part="1"
-F 0 "C170" V 14850 7400 60  0000 C CNN
+AR Path="/5AE62FB7/5AE9DF6E/5AE9ADCE" Ref="C18"  Part="1"
+AR Path="/5B1119BA/5BE38555/5AE9ADCE" Ref="C172"  Part="1"
+AR Path="/5B1119BA/5C00E21C/5AE9ADCE" Ref="C190"  Part="1"
+F 0 "C18" V 14850 7400 60  0000 C CNN
 F 1 "100nF" V 15150 7400 60  0000 C CNN
 F 2 "" H 15000 7400 60  0000 C CNN
@@
 	15025 7650 15000 7650
 $Comp
-L spice:0 #GND22
+L spice:0 #GND19
 U 1 1 5AEA4D0B
 P 15025 7775
-AR Path="/5AE62FB7/5AE9DF6E/5AEA4D0B" Ref="#GND22"  Part="1"
-AR Path="/5B1119BA/5BE38555/5AEA4D0B" Ref="#GND47"  Part="1"
-AR Path="/5B1119BA/5C00E21C/5AEA4D0B" Ref="#GND65"  Part="1"
-F 0 "#GND47" H 15025 7675 60  0001 C CNN
+AR Path="/5AE62FB7/5AE9DF6E/5AEA4D0B" Ref="#GND19"  Part="1"
+AR Path="/5B1119BA/5BE38555/5AEA4D0B" Ref="#GND44"  Part="1"
+AR Path="/5B1119BA/5C00E21C/5AEA4D0B" Ref="#GND62"  Part="1"
+F 0 "#GND19" H 15025 7675 60  0001 C CNN
 F 1 "0" H 15025 7705 60  0000 C CNN
 F 2 "" H 15025 7775 60  0000 C CNN
@@
 	15025 7650 15025 7775
 $Comp
-L spice:C C17
+L spice:C C19
 U 1 1 5AEAE0FD
 P 16200 19625
-AR Path="/5AE62FB7/5AE9DF6E/5AEAE0FD" Ref="C17"  Part="1"
-AR Path="/5B1119BA/5BE38555/5AEAE0FD" Ref="C171"  Part="1"
-AR Path="/5B1119BA/5C00E21C/5AEAE0FD" Ref="C189"  Part="1"
-F 0 "C171" V 16050 19625 60  0000 C CNN
+AR Path="/5AE62FB7/5AE9DF6E/5AEAE0FD" Ref="C19"  Part="1"
+AR Path="/5B1119BA/5BE38555/5AEAE0FD" Ref="C173"  Part="1"
+AR Path="/5B1119BA/5C00E21C/5AEAE0FD" Ref="C191"  Part="1"
+F 0 "C19" V 16050 19625 60  0000 C CNN
 F 1 "100nF" V 16350 19625 60  0000 C CNN
 F 2 "" H 16200 19625 60  0000 C CNN
@@
 $EndComp
 $Comp
-L spice:0 #GND23
+L spice:0 #GND20
 U 1 1 5AEAE570
 P 16200 19875
-AR Path="/5AE62FB7/5AE9DF6E/5AEAE570" Ref="#GND23"  Part="1"
-AR Path="/5B1119BA/5BE38555/5AEAE570" Ref="#GND48"  Part="1"
-AR Path="/5B1119BA/5C00E21C/5AEAE570" Ref="#GND66"  Part="1"
-F 0 "#GND48" H 16200 19775 60  0001 C CNN
+AR Path="/5AE62FB7/5AE9DF6E/5AEAE570" Ref="#GND20"  Part="1"
+AR Path="/5B1119BA/5BE38555/5AEAE570" Ref="#GND45"  Part="1"
+AR Path="/5B1119BA/5C00E21C/5AEAE570" Ref="#GND63"  Part="1"
+F 0 "#GND20" H 16200 19775 60  0001 C CNN
 F 1 "0" H 16200 19805 60  0000 C CNN
 F 2 "" H 16200 19875 60  0000 C CNN
@@
 Wire Wire Line
 	15800 19500 16050 19500
+Wire Wire Line
+	16100 5525 35625 5525
 $EndSCHEMATC

Commit message: tst
Changed lines of the file:
@@
 L myCpu-rescue:74LS158 U21
 U 1 1 5AED0336
-P 16150 18625
+P 16125 18625
 AR Path="/5AE62FB7/5AE9DF6E/5AED0336" Ref="U21"  Part="1"
 AR Path="/5B1119BA/5BE38555/5AED0336" Ref="U114"  Part="1"
 AR Path="/5B1119BA/5C00E21C/5AED0336" Ref="U132"  Part="1"
-F 0 "U21" H 16200 18775 50  0000 C CNN
-F 1 "74LS158" H 16200 18475 50  0000 C CNN
-F 2 "" H 16150 18625 50  0000 C CNN
-F 3 "" H 16150 18625 50  0000 C CNN
-	1    16150 18625
+F 0 "U21" H 16175 18775 50  0000 C CNN
+F 1 "74LS158" H 16175 18475 50  0000 C CNN
+F 2 "" H 16125 18625 50  0000 C CNN
+F 3 "" H 16125 18625 50  0000 C CNN
+	1    16125 18625
 	1    0    0    -1
 $EndComp
@@
 	13875 15000 13875 18075
 Wire Wire Line
-	13875 18075 15400 18075
+	13875 18075 15375 18075
 Wire Wire Line
 	11500 15100 13775 15100
@@
 	13775 15100 13775 18175
 Wire Wire Line
-	13775 18175 15400 18175
+	13775 18175 15375 18175
 Wire Wire Line
 	11550 17900 13575 17900
@@
 	13575 17900 13575 18325
 Wire Wire Line
-	13575 18325 15400 18325
+	13575 18325 15375 18325
 Wire Wire Line
 	11550 18000 13400 18000
@@
 	13400 18000 13400 18425
 Wire Wire Line
-	13400 18425 15400 18425
-Wire Wire Line
-	15400 18575 13350 18575
+	13400 18425 15375 18425
+Wire Wire Line
+	15375 18575 13350 18575
 Wire Wire Line
 	13350 18575 13350 21050
@@
 	13550 21150 13550 18675
 Wire Wire Line
-	13550 18675 15400 18675
-Wire Wire Line
-	15400 18825 13925 18825
+	13550 18675 15375 18675
+Wire Wire Line
+	15375 18825 13925 18825
 Wire Wire Line
 	13925 18825 13925 23950
@@
 	14250 24050 14250 18925
 Wire Wire Line
-	14250 18925 15400 18925
+	14250 18925 15375 18925
 Text HLabel 35625 6075 2    60   Output ~ 0
 Z0
@@
 	16100 7100 16100 6275
 Wire Wire Line
-	16900 18125 30475 18125
+	16875 18125 30475 18125
 Wire Wire Line
 	30475 18125 30475 7275
@@
 	30800 7475 30800 18375
 Wire Wire Line
-	30800 18375 16900 18375
-Wire Wire Line
-	16900 18625 31475 18625
+	30800 18375 16875 18375
+Wire Wire Line
+	16875 18625 31475 18625
 Wire Wire Line
 	31475 18625 31475 7725
@@
 	32100 8000 32100 18875
 Wire Wire Line
-	32100 18875 16900 18875
+	32100 18875 16875 18875
 Text HLabel 16075 21425 3    60   Input ~ 0
 S0
@@
 AR Path="/5B1119BA/5BE38555/5AF3D664" Ref="#PWR0315"  Part="1"
 AR Path="/5B1119BA/5C00E21C/5AF3D664" Ref="#PWR0333"  Part="1"
-F 0 "#PWR0333" H 15800 19350 50  0001 C CNN
+F 0 "#PWR029" H 15800 19350 50  0001 C CNN
 F 1 "VCC" H 15800 19650 50  0000 C CNN
 F 2 "" H 15800 19500 50  0000 C CNN
@@
 AR Path="/5B1119BA/5BE38555/5AF3FA58" Ref="#PWR0314"  Part="1"
 AR Path="/5B1119BA/5C00E21C/5AF3FA58" Ref="#PWR0332"  Part="1"
-F 0 "#PWR0332" H 15000 6900 50  0001 C CNN
+F 0 "#PWR028" H 15000 6900 50  0001 C CNN
 F 1 "VCC" H 15000 7200 50  0000 C CNN
 F 2 "" H 15000 7050 50  0000 C CNN
@@
 	14600 7050 15000 7050
 Wire Wire Line
-	15400 19175 15400 19500
+	15375 19175 15400 19500
 Wire Wire Line
 	15400 19500 15800 19500
@@
 Connection ~ 15800 19500
 Wire Wire Line
-	15100 19075 15400 19075
+	15100 19075 15375 19075
 Text HLabel 7925 1675 0    60   Input ~ 0
 Bit0_X0
