File: 8-BIT_16-1MUX.sch (KiCad schematic (older format))
At the start: 4 parts, among them U20 74LS158, U21 74LS158

Commit message: message
Parts:
- renumbered U20 to U33, U21 to U34
Changed lines of the file:
@@
 $Descr A0 46811 33110
 encoding utf-8
-Sheet 11 92
+Sheet 11 101
 Title ""
 Date ""
@@
 $EndSheet
 $Comp
-L myCpu-rescue:74LS158 U20
+L myCpu-rescue:74LS158 U33
 U 1 1 5AECFE89
 P 15350 6025
-AR Path="/5AE62FB7/5AE9DF6E/5AECFE89" Ref="U20"  Part="1"
-AR Path="/5B1119BA/5BE38555/5AECFE89" Ref="U113"  Part="1"
-AR Path="/5B1119BA/5C00E21C/5AECFE89" Ref="U131"  Part="1"
-F 0 "U20" H 15400 6175 50  0000 C CNN
+AR Path="/5AE62FB7/5AE9DF6E/5AECFE89" Ref="U33"  Part="1"
+AR Path="/5B1119BA/5BE38555/5AECFE89" Ref="U160"  Part="1"
+AR Path="/5B1119BA/5C00E21C/5AECFE89" Ref="U178"  Part="1"
+F 0 "U178" H 15400 6175 50  0000 C CNN
 F 1 "74LS158" H 15400 5875 50  0000 C CNN
 F 2 "" H 15350 6025 50  0000 C CNN
@@
 $EndComp
 $Comp
-L myCpu-rescue:74LS158 U21
+L myCpu-rescue:74LS158 U34
 U 1 1 5AED0336
 P 16125 18625
-AR Path="/5AE62FB7/5AE9DF6E/5AED0336" Ref="U21"  Part="1"
-AR Path="/5B1119BA/5BE38555/5AED0336" Ref="U114"  Part="1"
-AR Path="/5B1119BA/5C00E21C/5AED0336" Ref="U132"  Part="1"
-F 0 "U21" H 16175 18775 50  0000 C CNN
+AR Path="/5AE62FB7/5AE9DF6E/5AED0336" Ref="U34"  Part="1"
+AR Path="/5B1119BA/5BE38555/5AED0336" Ref="U161"  Part="1"
+AR Path="/5B1119BA/5C00E21C/5AED0336" Ref="U179"  Part="1"
+F 0 "U179" H 16175 18775 50  0000 C CNN
 F 1 "74LS158" H 16175 18475 50  0000 C CNN
 F 2 "" H 16125 18625 50  0000 C CNN
@@
 	11975 28950 11975 29000
 $Comp
-L myCpu-rescue:VCC #PWR029
+L myCpu-rescue:VCC #PWR035
 U 1 1 5AF3D664
 P 15800 19500
-AR Path="/5AE62FB7/5AE9DF6E/5AF3D664" Ref="#PWR029"  Part="1"
-AR Path="/5B1119BA/5BE38555/5AF3D664" Ref="#PWR0315"  Part="1"
-AR Path="/5B1119BA/5C00E21C/5AF3D664" Ref="#PWR0333"  Part="1"
-F 0 "#PWR0333" H 15800 19350 50  0001 C CNN
+AR Path="/5AE62FB7/5AE9DF6E/5AF3D664" Ref="#PWR035"  Part="1"
+AR Path="/5B1119BA/5BE38555/5AF3D664" Ref="#PWR0363"  Part="1"
+AR Path="/5B1119BA/5C00E21C/5AF3D664" Ref="#PWR0381"  Part="1"
+F 0 "#PWR0381" H 15800 19350 50  0001 C CNN
 F 1 "VCC" H 15800 19650 50  0000 C CNN
 F 2 "" H 15800 19500 50  0000 C CNN
@@
 $EndComp
 $Comp
-L myCpu-rescue:VCC #PWR028
+L myCpu-rescue:VCC #PWR034
 U 1 1 5AF3FA58
 P 15000 7050
-AR Path="/5AE62FB7/5AE9DF6E/5AF3FA58" Ref="#PWR028"  Part="1"
-AR Path="/5B1119BA/5BE38555/5AF3FA58" Ref="#PWR0314"  Part="1"
-AR Path="/5B1119BA/5C00E21C/5AF3FA58" Ref="#PWR0332"  Part="1"
-F 0 "#PWR0332" H 15000 6900 50  0001 C CNN
+AR Path="/5AE62FB7/5AE9DF6E/5AF3FA58" Ref="#PWR034"  Part="1"
+AR Path="/5B1119BA/5BE38555/5AF3FA58" Ref="#PWR0362"  Part="1"
+AR Path="/5B1119BA/5C00E21C/5AF3FA58" Ref="#PWR0380"  Part="1"
+F 0 "#PWR0380" H 15000 6900 50  0001 C CNN
 F 1 "VCC" H 15000 7200 50  0000 C CNN
 F 2 "" H 15000 7050 50  0000 C CNN
@@
 P 15000 7400
 AR Path="/5AE62FB7/5AE9DF6E/5AE9ADCE" Ref="C18"  Part="1"
-AR Path="/5B1119BA/5BE38555/5AE9ADCE" Ref="C172"  Part="1"
-AR Path="/5B1119BA/5C00E21C/5AE9ADCE" Ref="C190"  Part="1"
-F 0 "C18" V 14850 7400 60  0000 C CNN
+AR Path="/5B1119BA/5BE38555/5AE9ADCE" Ref="C196"  Part="1"
+AR Path="/5B1119BA/5C00E21C/5AE9ADCE" Ref="C214"  Part="1"
+F 0 "C214" V 14850 7400 60  0000 C CNN
 F 1 "100nF" V 15150 7400 60  0000 C CNN
 F 2 "" H 15000 7400 60  0000 C CNN
@@
 	15025 7650 15000 7650
 $Comp
-L spice:0 #GND19
+L spice:0 #GND14
 U 1 1 5AEA4D0B
 P 15025 7775
-AR Path="/5AE62FB7/5AE9DF6E/5AEA4D0B" Ref="#GND19"  Part="1"
-AR Path="/5B1119BA/5BE38555/5AEA4D0B" Ref="#GND44"  Part="1"
-AR Path="/5B1119BA/5C00E21C/5AEA4D0B" Ref="#GND62"  Part="1"
-F 0 "#GND19" H 15025 7675 60  0001 C CNN
+AR Path="/5AE62FB7/5AE9DF6E/5AEA4D0B" Ref="#GND14"  Part="1"
+AR Path="/5B1119BA/5BE38555/5AEA4D0B" Ref="#GND59"  Part="1"
+AR Path="/5B1119BA/5C00E21C/5AEA4D0B" Ref="#GND77"  Part="1"
+F 0 "#GND77" H 15025 7675 60  0001 C CNN
 F 1 "0" H 15025 7705 60  0000 C CNN
 F 2 "" H 15025 7775 60  0000 C CNN
@@
 P 16200 19625
 AR Path="/5AE62FB7/5AE9DF6E/5AEAE0FD" Ref="C19"  Part="1"
-AR Path="/5B1119BA/5BE38555/5AEAE0FD" Ref="C173"  Part="1"
-AR Path="/5B1119BA/5C00E21C/5AEAE0FD" Ref="C191"  Part="1"
-F 0 "C19" V 16050 19625 60  0000 C CNN
+AR Path="/5B1119BA/5BE38555/5AEAE0FD" Ref="C197"  Part="1"
+AR Path="/5B1119BA/5C00E21C/5AEAE0FD" Ref="C215"  Part="1"
+F 0 "C215" V 16050 19625 60  0000 C CNN
 F 1 "100nF" V 16350 19625 60  0000 C CNN
 F 2 "" H 16200 19625 60  0000 C CNN
@@
 $EndComp
 $Comp
-L spice:0 #GND20
+L spice:0 #GND15
 U 1 1 5AEAE570
 P 16200 19875
-AR Path="/5AE62FB7/5AE9DF6E/5AEAE570" Ref="#GND20"  Part="1"
-AR Path="/5B1119BA/5BE38555/5AEAE570" Ref="#GND45"  Part="1"
-AR Path="/5B1119BA/5C00E21C/5AEAE570" Ref="#GND63"  Part="1"
-F 0 "#GND20" H 16200 19775 60  0001 C CNN
+AR Path="/5AE62FB7/5AE9DF6E/5AEAE570" Ref="#GND15"  Part="1"
+AR Path="/5B1119BA/5BE38555/5AEAE570" Ref="#GND60"  Part="1"
+AR Path="/5B1119BA/5C00E21C/5AEAE570" Ref="#GND78"  Part="1"
+F 0 "#GND78" H 16200 19775 60  0001 C CNN
 F 1 "0" H 16200 19805 60  0000 C CNN
 F 2 "" H 16200 19875 60  0000 C CNN

Commit message: .
Changed lines of the file:
@@
 $Descr A0 46811 33110
 encoding utf-8
-Sheet 11 101
+Sheet 50 75
 Title ""
 Date ""
@@
 P 15350 6025
 AR Path="/5AE62FB7/5AE9DF6E/5AECFE89" Ref="U33"  Part="1"
-AR Path="/5B1119BA/5BE38555/5AECFE89" Ref="U160"  Part="1"
-AR Path="/5B1119BA/5C00E21C/5AECFE89" Ref="U178"  Part="1"
-F 0 "U178" H 15400 6175 50  0000 C CNN
+AR Path="/5B1119BA/5BE38555/5AECFE89" Ref="U99"  Part="1"
+AR Path="/5B1119BA/5C00E21C/5AECFE89" Ref="U117"  Part="1"
+F 0 "U117" H 15400 6175 50  0000 C CNN
 F 1 "74LS158" H 15400 5875 50  0000 C CNN
 F 2 "" H 15350 6025 50  0000 C CNN
@@
 P 16125 18625
 AR Path="/5AE62FB7/5AE9DF6E/5AED0336" Ref="U34"  Part="1"
-AR Path="/5B1119BA/5BE38555/5AED0336" Ref="U161"  Part="1"
-AR Path="/5B1119BA/5C00E21C/5AED0336" Ref="U179"  Part="1"
-F 0 "U179" H 16175 18775 50  0000 C CNN
+AR Path="/5B1119BA/5BE38555/5AED0336" Ref="U100"  Part="1"
+AR Path="/5B1119BA/5C00E21C/5AED0336" Ref="U118"  Part="1"
+F 0 "U118" H 16175 18775 50  0000 C CNN
 F 1 "74LS158" H 16175 18475 50  0000 C CNN
 F 2 "" H 16125 18625 50  0000 C CNN
@@
 	11975 28950 11975 29000
 $Comp
-L myCpu-rescue:VCC #PWR035
+L myCpu-rescue:VCC #PWR038
 U 1 1 5AF3D664
 P 15800 19500
-AR Path="/5AE62FB7/5AE9DF6E/5AF3D664" Ref="#PWR035"  Part="1"
-AR Path="/5B1119BA/5BE38555/5AF3D664" Ref="#PWR0363"  Part="1"
-AR Path="/5B1119BA/5C00E21C/5AF3D664" Ref="#PWR0381"  Part="1"
-F 0 "#PWR0381" H 15800 19350 50  0001 C CNN
+AR Path="/5AE62FB7/5AE9DF6E/5AF3D664" Ref="#PWR038"  Part="1"
+AR Path="/5B1119BA/5BE38555/5AF3D664" Ref="#PWR0113"  Part="1"
+AR Path="/5B1119BA/5C00E21C/5AF3D664" Ref="#PWR0131"  Part="1"
+F 0 "#PWR0131" H 15800 19350 50  0001 C CNN
 F 1 "VCC" H 15800 19650 50  0000 C CNN
 F 2 "" H 15800 19500 50  0000 C CNN
@@
 $EndComp
 $Comp
-L myCpu-rescue:VCC #PWR034
+L myCpu-rescue:VCC #PWR037
 U 1 1 5AF3FA58
 P 15000 7050
-AR Path="/5AE62FB7/5AE9DF6E/5AF3FA58" Ref="#PWR034"  Part="1"
-AR Path="/5B1119BA/5BE38555/5AF3FA58" Ref="#PWR0362"  Part="1"
-AR Path="/5B1119BA/5C00E21C/5AF3FA58" Ref="#PWR0380"  Part="1"
-F 0 "#PWR0380" H 15000 6900 50  0001 C CNN
+AR Path="/5AE62FB7/5AE9DF6E/5AF3FA58" Ref="#PWR037"  Part="1"
+AR Path="/5B1119BA/5BE38555/5AF3FA58" Ref="#PWR0112"  Part="1"
+AR Path="/5B1119BA/5C00E21C/5AF3FA58" Ref="#PWR0130"  Part="1"
+F 0 "#PWR0130" H 15000 6900 50  0001 C CNN
 F 1 "VCC" H 15000 7200 50  0000 C CNN
 F 2 "" H 15000 7050 50  0000 C CNN
@@
 P 15000 7400
 AR Path="/5AE62FB7/5AE9DF6E/5AE9ADCE" Ref="C18"  Part="1"
-AR Path="/5B1119BA/5BE38555/5AE9ADCE" Ref="C196"  Part="1"
-AR Path="/5B1119BA/5C00E21C/5AE9ADCE" Ref="C214"  Part="1"
-F 0 "C214" V 14850 7400 60  0000 C CNN
+AR Path="/5B1119BA/5BE38555/5AE9ADCE" Ref="C68"  Part="1"
+AR Path="/5B1119BA/5C00E21C/5AE9ADCE" Ref="C86"  Part="1"
+F 0 "C86" V 14850 7400 60  0000 C CNN
 F 1 "100nF" V 15150 7400 60  0000 C CNN
 F 2 "" H 15000 7400 60  0000 C CNN
@@
 P 16200 19625
 AR Path="/5AE62FB7/5AE9DF6E/5AEAE0FD" Ref="C19"  Part="1"
-AR Path="/5B1119BA/5BE38555/5AEAE0FD" Ref="C197"  Part="1"
-AR Path="/5B1119BA/5C00E21C/5AEAE0FD" Ref="C215"  Part="1"
-F 0 "C215" V 16050 19625 60  0000 C CNN
+AR Path="/5B1119BA/5BE38555/5AEAE0FD" Ref="C69"  Part="1"
+AR Path="/5B1119BA/5C00E21C/5AEAE0FD" Ref="C87"  Part="1"
+F 0 "C87" V 16050 19625 60  0000 C CNN
 F 1 "100nF" V 16350 19625 60  0000 C CNN
 F 2 "" H 16200 19625 60  0000 C CNN
