File: myCpu.sch (KiCad schematic (older format))
At the start: 0 parts

Commit message: lots of work done
Parts:
- added 5V1: V, symbol spice:V
Connections:
- net labels added: 0, GNDPWR, VCC
- wire segments 0 -> 146

Commit message: X
Parts:
- added P?: INSTRUCTION, symbol conn:CONN_12X2
- added P?: ROM_ADDR, symbol conn:CONN_17
- added P?: RAM_READ, symbol conn:CONN_8
- added P?: RAM_WRITE, symbol conn:CONN_9
- added P?: RAM_ADDR, symbol conn:CONN_17
Connections:
- net labels added: ADDR0, ADDR1, ADDR10, ADDR11, ADDR12, ADDR13, ADDR14, ADDR15, ADDR2, ADDR3, ADDR4, ADDR5, ADDR6, ADDR7, ADDR8, ADDR9, ADDR_ENABLE, ADDR_X_S0, ADDR_X_S1, ADDR_Z_S0, ADDR_Z_S1, ALU_S0, ALU_S1, ALU_S2, ALU_S3, ALU_X0, ALU_X1, ALU_X2, ALU_X3, ALU_X4, ALU_X5, ALU_X6, ALU_X7, ALU_Y0, ALU_Y1, ALU_Y2, ALU_Y3, ALU_Y4, ALU_Y5, ALU_Y6, ALU_Y7, ALU_Z0, ALU_Z1, ALU_Z2, ALU_Z3, ALU_Z4, ALU_Z5, ALU_Z6, ALU_Z7, CARRY, CLK, CLK_PC, CarryEnable, IM0, IM1, IM2, IM3, IM4, IM5, IM6, IM7, IN0, IN1, IN10, IN11, IN12, IN13, IN14, IN15, IN16, IN17, IN18, IN19, IN2, IN20, IN21, IN22, IN23, IN3, IN4, IN5, IN6, IN7, IN8, IN9, LADDR, LOAD, LOD, PCINC, PCSTACK, RAM0, RAM1, RAM10, RAM11, RAM12, RAM13, RAM14, RAM15, RAM2, RAM3, RAM4, RAM5, RAM6, RAM7, RAM8, RAM9, READ, REG_ENABLE, RX_S0, RX_S1, RX_S2, RX_S3, RY_S0, RY_S1, RY_S2, RY_S3, RZ_S0, RZ_S1, RZ_S2, RZ_S3, WRITE, ZFLAG
- wire segments 146 -> 852
- no-connect marks 0 -> 2

Commit message: b
Parts:
- removed 5V1: V, symbol spice:V
- added K1: CONN_3, symbol conn:CONN_3
- gave numbers to parts that had none: 5
Connections:
- net labels added: CALL, CARRY_S, CMP, GND, JMP, RET, UNCOND, ZFLAG_S, Z_FLAG, Z_FLAG_S
- net labels removed: LOD, PCSTACK
- wire segments 852 -> 834
- no-connect marks 2 -> 7

Commit message: fixed errors
Parts:
- P1: symbol conn:CONN_12X2 -> myCpu-rescue:CONN_12X2-conn
- P4: symbol conn:CONN_8 -> myCpu-rescue:CONN_8-conn
Changed lines of the file:
@@
 	7650 21325 7725 21325
 $Comp
-L conn:CONN_12X2 P1
+L myCpu-rescue:CONN_12X2-conn P1
 U 1 1 60A9395A
 P 1975 25300
@@
 	11525 5175 12550 5175
 $Comp
-L conn:CONN_8 P4
+L myCpu-rescue:CONN_8-conn P4
 U 1 1 652660C6
 P 6700 21975
@@
 F77 "ADDR_X_S0" O R 14800 30250 60
 F78 "ADDR_X_S1" O R 14800 30350 60
-F79 "CALL" O R 14800 28150 60
+F79 "CALL_ANY" O R 14800 28150 60
 F80 "RET" O R 14800 28550 60
-F81 "JMP" O R 14800 28450 60
+F81 "JMP_ANY" O R 14800 28450 60
 F82 "CMP" O L 11225 28475 60
 F83 "WRITE" O L 11225 27900 60
