File: myCpu.sch (KiCad schematic (older format))
At the start: 6 parts, among them K1 CONN_3, P1 INSTRUCTION, P2 RAM_ADDR, P3 RAM_WRITE, P4 RAM_READ, P5 ROM_ADDR

Commit message: .
Changed lines of the file:
@@
 $Descr A0 46811 33110
 encoding utf-8
-Sheet 1 101
+Sheet 1 75
 Title ""
 Date ""
@@
 Connection ~ 28400 10475
 NoConn ~ 28975 11050
-$Sheet
-S 15525 6500 1250 1325
-U 64EF26C6
-F0 "SREG" 59
-F1 "SREG.sch" 59
-F2 "CLK" I L 15525 7775 60
-F3 "Cin" I L 15525 6800 60
-F4 "Zin" I L 15525 6925 60
-F5 "Zout" O R 16775 6900 60
-F6 "Cout" O R 16775 7050 60
-$EndSheet
 Wire Wire Line
 	16075 4600 16625 4600

Commit message: .
Connections:
- wire segments 834 -> 841
Changed lines of the file:
@@
 $Descr A0 46811 33110
 encoding utf-8
-Sheet 1 75
+Sheet 1 100
 Title ""
 Date ""
@@
 Wire Wire Line
 	25075 10775 25425 10775
-$Sheet
-S 23000 10450 800  1350
-U 5B4927F7
-F0 "CALL_SELELCTOR" 60
-F1 "CALL_SELECTOR.sch" 60
-F2 "CALL" I L 23000 10575 60
-F3 "UNCOND" I L 23000 10675 60
-F4 "Z_FLAG" I L 23000 10775 60
-F5 "ZFLAG_S" I L 23000 10900 60
-F6 "Cin" I L 23000 11000 60
-F7 "CARRY_S" I L 23000 11075 60
-F8 "CALL_ENABLE" O R 23800 11225 60
-$EndSheet
 Wire Wire Line
 	23800 11225 24400 11225
@@
 Wire Wire Line
 	24400 10850 25425 10850
-Text Label 23000 10900 2    60   ~ 0
+Text Label 22850 10775 2    60   ~ 0
 Z_FLAG
 Text Label 23000 11000 2    60   ~ 0
@@
 Text Label 23000 11075 2    60   ~ 0
 CARRY_S
-Text Label 23000 10775 2    60   ~ 0
+Text Label 22850 10875 2    60   ~ 0
 Z_FLAG_S
 Text Label 23000 10675 2    60   ~ 0
@@
 Text Label 23000 10575 2    60   ~ 0
 CALL
-Text Label 16775 6900 0    60   ~ 0
+Text Label 17075 6875 0    60   ~ 0
 Z_FLAG
 $Sheet
@@
 CARRY_S
 Text Label 14800 25850 0    60   ~ 0
-ZFLAG_S
+Z_FLAG_S
 Text Label 14875 25950 0    60   ~ 0
 UNCOND
+Text Label 14800 28550 0    60   ~ 0
+RET
+Text Label 14800 28450 0    60   ~ 0
+JMP
+Text Label 14800 28150 0    60   ~ 0
+CALL
+Text Label 18975 8725 2    60   ~ 0
+RET
+Wire Wire Line
+	11425 1525 11425 1300
+Connection ~ 11425 1525
+$Comp
+L power:GND #PWR02
+U 1 1 5C3953FD
+P 11425 1300
+F 0 "#PWR02" H 11425 1300 30  0001 C CNN
+F 1 "GND" H 11425 1230 30  0001 C CNN
+F 2 "" H 11425 1300 60  0001 C CNN
+F 3 "" H 11425 1300 60  0001 C CNN
+	1    11425 1300
+	1    0    0    -1
+$EndComp
+Text Label 11550 1025 2    60   ~ 0
+CLK
+Text Label 11225 27900 2    60   ~ 0
+WRITE
+Text Label 11225 28475 2    60   ~ 0
+CMP
+NoConn ~ 2375 25550
+NoConn ~ 2375 25850
+NoConn ~ 1575 25550
+$Comp
+L conn:CONN_3 K1
+U 1 1 5C2C3063
+P 11900 1025
+F 0 "K1" H 12027 1053 50  0000 L CNN
+F 1 "CONN_3" H 12027 969 40  0000 L CNN
+F 2 "" H 11900 1025 60  0001 C CNN
+F 3 "" H 11900 1025 60  0001 C CNN
+	1    11900 1025
+	1    0    0    -1
+$EndComp
+Wire Wire Line
+	11325 675  11775 675
+NoConn ~ 11550 925
+NoConn ~ 11550 1125
+$Comp
+L power:GNDPWR #PWR03
+U 1 1 5CF0EF7A
+P 11775 1675
+F 0 "#PWR03" H 11775 1725 40  0001 C CNN
+F 1 "GNDPWR" H 11770 1743 40  0000 C CNN
+F 2 "" H 11775 1675 60  0001 C CNN
+F 3 "" H 11775 1675 60  0001 C CNN
+	1    11775 1675
+	1    0    0    -1
+$EndComp
 $Sheet
-S 11225 22600 3575 9750
-U 83254C33
+S 15525 6725 1250 350
+U 5BC3891B
+F0 "SREG" 60
+F1 "SREG.sch" 60
+F2 "CLK" I L 15525 7000 60
+F3 "Cin" I L 15525 6800 60
+F4 "Zin" I L 15525 6925 60
+F5 "Zout" O R 16775 6900 60
+F6 "Cout" O R 16775 7050 60
+$EndSheet
+Text Label 15375 7000 2    60   ~ 0
+CLK
+Wire Wire Line
+	15375 7000 15525 7000
+Wire Wire Line
+	16775 6900 17075 6900
+Wire Wire Line
+	17075 6900 17075 6875
+Wire Wire Line
+	22850 10875 22950 10875
+Wire Wire Line
+	22950 10875 22950 10900
+Wire Wire Line
+	22950 10900 23000 10900
+Wire Wire Line
+	22850 10775 23000 10775
+$Sheet
+S 23000 10500 800  850
+U 5C13542F
+F0 "CALL_SELECTOR" 60
+F1 "CALL_SELECTOR.sch" 60
+F2 "CALL" I L 23000 10575 60
+F3 "UNCOND" I L 23000 10675 60
+F4 "Z_FLAG" I L 23000 10775 60
+F5 "ZFLAG_S" I L 23000 10900 60
+F6 "Cin" I L 23000 11000 60
+F7 "CARRY_S" I L 23000 11075 60
+F8 "CALL_ENABLE" O R 23800 11225 60
+$EndSheet
+$Sheet
+S 11225 22575 3575 7875
+U 5C13587C
 F0 "DECODER" 60
 F1 "DECODER.sch" 60
@@
 F83 "WRITE" O L 11225 27900 60
 $EndSheet
-Text Label 14800 28550 0    60   ~ 0
-RET
-Text Label 14800 28450 0    60   ~ 0
-JMP
-Text Label 14800 28150 0    60   ~ 0
-CALL
-Text Label 18975 8725 2    60   ~ 0
-RET
-Wire Wire Line
-	11425 1525 11425 1300
-Connection ~ 11425 1525
-$Comp
-L power:GND #PWR02
-U 1 1 5C3953FD
-P 11425 1300
-F 0 "#PWR02" H 11425 1300 30  0001 C CNN
-F 1 "GND" H 11425 1230 30  0001 C CNN
-F 2 "" H 11425 1300 60  0001 C CNN
-F 3 "" H 11425 1300 60  0001 C CNN
-	1    11425 1300
-	1    0    0    -1
-$EndComp
-Text Label 11550 1025 2    60   ~ 0
-CLK
-Text Label 11225 27900 2    60   ~ 0
-WRITE
-Text Label 11225 28475 2    60   ~ 0
-CMP
-NoConn ~ 2375 25550
-NoConn ~ 2375 25850
-NoConn ~ 1575 25550
-$Comp
-L conn:CONN_3 K1
-U 1 1 5C2C3063
-P 11900 1025
-F 0 "K1" H 12027 1053 50  0000 L CNN
-F 1 "CONN_3" H 12027 969 40  0000 L CNN
-F 2 "" H 11900 1025 60  0001 C CNN
-F 3 "" H 11900 1025 60  0001 C CNN
-	1    11900 1025
-	1    0    0    -1
-$EndComp
-Wire Wire Line
-	11325 675  11775 675
-NoConn ~ 11550 925
-NoConn ~ 11550 1125
-$Comp
-L power:GNDPWR #PWR03
-U 1 1 5CF0EF7A
-P 11775 1675
-F 0 "#PWR03" H 11775 1725 40  0001 C CNN
-F 1 "GNDPWR" H 11770 1743 40  0000 C CNN
-F 2 "" H 11775 1675 60  0001 C CNN
-F 3 "" H 11775 1675 60  0001 C CNN
-	1    11775 1675
-	1    0    0    -1
-$EndComp
 $EndSCHEMATC
