File: 16-1MUX.sch (KiCad schematic (older format))
At the start: 4 parts

Commit message: lots of work done
Parts:
- removed C? (x2): 100n, symbol C_Small
- removed U? (x2): 74LS151, symbol 74LS151
- added C36: C, symbol spice:C
- added C37, C38: 100nF, symbol spice:C
- added U40, U42: 74LS151, symbol 74xx:74LS151
- added U41: 74LS157, symbol 74xx:74LS157
Connections:
- net labels added: 0, Cout, S0
- net labels removed: GND, Z0, Z1
- wire segments 70 -> 131
- no-connect marks 0 -> 5

Commit message: b
Parts:
- renumbered C36 to C38, C37 to C39, C38 to C40, U40 to U42, U41 to U43, U42 to U44
Changed lines of the file:
@@
 $Descr A4 11693 8268
 encoding utf-8
-Sheet 22 90
+Sheet 22 92
 Title ""
 Date ""
@@
 S3
 $Comp
-L 74xx:74LS151 U40
+L 74xx:74LS151 U42
 U 1 1 5CEE5429
 P 2425 4650
-F 0 "U40" V 2478 5398 60  0000 L CNN
+F 0 "U42" V 2478 5398 60  0000 L CNN
 F 1 "74LS151" V 2372 5398 60  0000 L CNN
 F 2 "" H 2425 4650 60  0001 C CNN
@@
 $EndComp
 $Comp
-L 74xx:74LS151 U42
+L 74xx:74LS151 U44
 U 1 1 5CEE54B0
 P 4300 4600
-F 0 "U42" V 4353 5348 60  0000 L CNN
+F 0 "U44" V 4353 5348 60  0000 L CNN
 F 1 "74LS151" V 4247 5348 60  0000 L CNN
 F 2 "" H 4300 4600 60  0001 C CNN
@@
 	2975 7250 2975 5350
 $Comp
-L spice:0 #GND44
+L spice:0 #GND41
 U 1 1 5CF007F5
 P 3225 4950
-F 0 "#GND44" H 3225 4850 60  0001 C CNN
+F 0 "#GND41" H 3225 4850 60  0001 C CNN
 F 1 "0" H 3225 5044 60  0000 C CNN
 F 2 "" H 3225 4950 60  0000 C CNN
@@
 $EndComp
 $Comp
-L spice:0 #GND46
+L spice:0 #GND43
 U 1 1 5CF0081D
 P 5100 4925
-F 0 "#GND46" H 5100 4825 60  0001 C CNN
+F 0 "#GND43" H 5100 4825 60  0001 C CNN
 F 1 "0" H 5100 5019 60  0000 C CNN
 F 2 "" H 5100 4925 60  0000 C CNN
@@
 Connection ~ 5100 4925
 $Comp
-L spice:C C38
+L spice:C C40
 U 1 1 5CF0AB17
 P 5600 4600
-F 0 "C38" H 5728 4653 60  0000 L CNN
+F 0 "C40" H 5728 4653 60  0000 L CNN
 F 1 "100nF" H 5728 4547 60  0000 L CNN
 F 2 "" H 5600 4600 60  0000 C CNN
@@
 $EndComp
 $Comp
-L spice:C C36
+L spice:C C38
 U 1 1 5CF0AB7E
 P 3400 4600
-F 0 "C36" H 3528 4653 60  0000 L CNN
+F 0 "C38" H 3528 4653 60  0000 L CNN
 F 1 "C" H 3528 4547 60  0000 L CNN
 F 2 "" H 3400 4600 60  0000 C CNN
@@
 Connection ~ 5100 4900
 $Comp
-L myCpu-rescue:VCC #PWR044
+L myCpu-rescue:VCC #PWR055
 U 1 1 5CF105EB
 P 5600 4350
-F 0 "#PWR044" H 5600 4200 50  0001 C CNN
+F 0 "#PWR055" H 5600 4200 50  0001 C CNN
 F 1 "VCC" H 5617 4523 50  0000 C CNN
 F 2 "" H 5600 4350 50  0000 C CNN
@@
 $EndComp
 $Comp
-L myCpu-rescue:VCC #PWR042
+L myCpu-rescue:VCC #PWR053
 U 1 1 5CF10619
 P 3400 4350
-F 0 "#PWR042" H 3400 4200 50  0001 C CNN
+F 0 "#PWR053" H 3400 4200 50  0001 C CNN
 F 1 "VCC" H 3417 4523 50  0000 C CNN
 F 2 "" H 3400 4350 50  0000 C CNN
@@
 NoConn ~ 3900 3900
 $Comp
-L 74xx:74LS157 U41
+L 74xx:74LS157 U43
 U 1 1 5CF16234
 P 3000 2625
-F 0 "U41" V 3053 1966 60  0000 R CNN
+F 0 "U43" V 3053 1966 60  0000 R CNN
 F 1 "74LS157" V 2947 1966 60  0000 R CNN
 F 2 "" H 3000 2625 60  0001 C CNN
@@
 	2550 3900 2550 3375
 $Comp
-L myCpu-rescue:VCC #PWR043
+L myCpu-rescue:VCC #PWR054
 U 1 1 5CF22AD6
 P 4125 2600
-F 0 "#PWR043" H 4125 2450 50  0001 C CNN
+F 0 "#PWR054" H 4125 2450 50  0001 C CNN
 F 1 "VCC" H 4142 2773 50  0000 C CNN
 F 2 "" H 4125 2600 50  0000 C CNN
@@
 $EndComp
 $Comp
-L spice:0 #GND45
+L spice:0 #GND42
 U 1 1 5CF22B0E
 P 4000 3000
-F 0 "#GND45" H 4000 2900 60  0001 C CNN
+F 0 "#GND42" H 4000 2900 60  0001 C CNN
 F 1 "0" H 4000 3094 60  0000 C CNN
 F 2 "" H 4000 3000 60  0000 C CNN
@@
 $EndComp
 $Comp
-L spice:C C37
+L spice:C C39
 U 1 1 5CF22B4B
 P 4375 2825
-F 0 "C37" H 4503 2878 60  0000 L CNN
+F 0 "C39" H 4503 2878 60  0000 L CNN
 F 1 "100nF" H 4503 2772 60  0000 L CNN
 F 2 "" H 4375 2825 60  0000 C CNN

Commit message: tst
Changed lines of the file:
@@
 Text HLabel 2350 6500 3    60   Input ~ 0
 X3
-Text HLabel 2475 6425 3    60   Input ~ 0
+Text HLabel 2475 6500 3    60   Input ~ 0
 X4
 Text HLabel 2575 6425 3    60   Input ~ 0
@@
 	2350 5925 2350 6500
 Wire Wire Line
-	2375 6425 2575 6425
-Wire Wire Line
 	2575 6325 2675 6325
 Wire Wire Line
@@
 	2325 5775 2475 5775
 Wire Wire Line
-	2475 5775 2475 6425
-Wire Wire Line
 	2375 5350 2400 5350
 Wire Wire Line
@@
 NoConn ~ 3000 1875
 NoConn ~ 3250 1875
+Wire Wire Line
+	2475 5775 2475 6500
+Wire Wire Line
+	2575 6425 2375 6425
 $EndSCHEMATC

Commit message: message
Parts:
- renumbered U42 to U59, U43 to U60, U44 to U61
