File: 16-Bit4-1Mux.sch (KiCad schematic (older format))
At the start: 16 parts

Commit message: b
Parts:
- gave numbers to parts that had none: 16
Changed lines of the file:
@@
 $Descr A0 33110 46811 portrait
 encoding utf-8
-Sheet 71 90
+Sheet 71 92
 Title ""
 Date ""
@@
 $EndDescr
 $Comp
-L 74xx:74LS153 U?
+L 74xx:74LS153 U187
 U 1 1 812F095F
 P 8075 4150
-F 0 "U?" H 8075 5108 60  0000 C CNN
+F 0 "U187" H 8075 5108 60  0000 C CNN
 F 1 "74LS153" H 8075 5002 60  0000 C CNN
 F 2 "" H 8075 4150 60  0001 C CNN
@@
 $EndComp
 $Comp
-L 74xx:74LS153 U?
+L 74xx:74LS153 U183
 U 1 1 812F09E7
 P 7950 7350
-F 0 "U?" H 7950 8308 60  0000 C CNN
+F 0 "U183" H 7950 8308 60  0000 C CNN
 F 1 "74LS153" H 7950 8202 60  0000 C CNN
 F 2 "" H 7950 7350 60  0001 C CNN
@@
 $EndComp
 $Comp
-L 74xx:74LS153 U?
+L 74xx:74LS153 U185
 U 1 1 812F0A85
 P 7975 10225
-F 0 "U?" H 7975 11183 60  0000 C CNN
+F 0 "U185" H 7975 11183 60  0000 C CNN
 F 1 "74LS153" H 7975 11077 60  0000 C CNN
 F 2 "" H 7975 10225 60  0001 C CNN
@@
 $EndComp
 $Comp
-L 74xx:74LS153 U?
+L 74xx:74LS153 U186
 U 1 1 812F0D4A
 P 7975 12650
-F 0 "U?" H 7975 13608 60  0000 C CNN
+F 0 "U186" H 7975 13608 60  0000 C CNN
 F 1 "74LS153" H 7975 13502 60  0000 C CNN
 F 2 "" H 7975 12650 60  0001 C CNN
@@
 $EndComp
 $Comp
-L 74xx:74LS153 U?
+L 74xx:74LS153 U184
 U 1 1 812F0D51
 P 7950 15500
-F 0 "U?" H 7950 16458 60  0000 C CNN
+F 0 "U184" H 7950 16458 60  0000 C CNN
 F 1 "74LS153" H 7950 16352 60  0000 C CNN
 F 2 "" H 7950 15500 60  0001 C CNN
@@
 $EndComp
 $Comp
-L 74xx:74LS153 U?
+L 74xx:74LS153 U188
 U 1 1 812F0D58
 P 8300 18525
-F 0 "U?" H 8300 19483 60  0000 C CNN
+F 0 "U188" H 8300 19483 60  0000 C CNN
 F 1 "74LS153" H 8300 19377 60  0000 C CNN
 F 2 "" H 8300 18525 60  0001 C CNN
@@
 $EndComp
 $Comp
-L 74xx:74LS153 U?
+L 74xx:74LS153 U189
 U 1 1 812F1353
 P 8300 20925
-F 0 "U?" H 8300 21883 60  0000 C CNN
+F 0 "U189" H 8300 21883 60  0000 C CNN
 F 1 "74LS153" H 8300 21777 60  0000 C CNN
 F 2 "" H 8300 20925 60  0001 C CNN
@@
 $EndComp
 $Comp
-L 74xx:74LS153 U?
+L 74xx:74LS153 U190
 U 1 1 812F135A
 P 8325 23800
-F 0 "U?" H 8325 24758 60  0000 C CNN
+F 0 "U190" H 8325 24758 60  0000 C CNN
 F 1 "74LS153" H 8325 24652 60  0000 C CNN
 F 2 "" H 8325 23800 60  0001 C CNN
@@
 $EndComp
 $Comp
-L power:GND #PWR?
+L power:GND #PWR0486
 U 1 1 812F1AD5
 P 7850 5275
-F 0 "#PWR?" H 7850 5275 30  0001 C CNN
+F 0 "#PWR0486" H 7850 5275 30  0001 C CNN
 F 1 "GND" H 7850 5205 30  0001 C CNN
 F 2 "" H 7850 5275 60  0001 C CNN
@@
 $EndComp
 $Comp
-L power:VCC #PWR?
+L power:VCC #PWR0494
 U 1 1 812F1B16
 P 8350 5275
-F 0 "#PWR?" H 8350 5375 30  0001 C CNN
+F 0 "#PWR0494" H 8350 5375 30  0001 C CNN
 F 1 "VCC" H 8354 5402 30  0000 C CNN
 F 2 "" H 8350 5275 60  0001 C CNN
@@
 $EndComp
 $Comp
-L spice:C C?
+L spice:C C278
 U 1 1 812F1B57
 P 8100 5275
-F 0 "C?" V 7813 5275 60  0000 C CNN
+F 0 "C278" V 7813 5275 60  0000 C CNN
 F 1 "100nF" V 7919 5275 60  0000 C CNN
 F 2 "" H 8100 5275 60  0000 C CNN
@@
 $EndComp
 $Comp
-L power:GND #PWR?
+L power:GND #PWR0484
 U 1 1 812F1CB2
 P 7775 8500
-F 0 "#PWR?" H 7775 8500 30  0001 C CNN
+F 0 "#PWR0484" H 7775 8500 30  0001 C CNN
 F 1 "GND" H 7775 8430 30  0001 C CNN
 F 2 "" H 7775 8500 60  0001 C CNN
@@
 $EndComp
 $Comp
-L power:VCC #PWR?
+L power:VCC #PWR0492
 U 1 1 812F1CB8
 P 8275 8500
-F 0 "#PWR?" H 8275 8600 30  0001 C CNN
+F 0 "#PWR0492" H 8275 8600 30  0001 C CNN
 F 1 "VCC" H 8279 8627 30  0000 C CNN
 F 2 "" H 8275 8500 60  0001 C CNN
@@
 $EndComp
 $Comp
-L spice:C C?
+L spice:C C276
 U 1 1 812F1CBE
 P 8025 8500
-F 0 "C?" V 7738 8500 60  0000 C CNN
+F 0 "C276" V 7738 8500 60  0000 C CNN
 F 1 "100nF" V 7844 8500 60  0000 C CNN
 F 2 "" H 8025 8500 60  0000 C CNN
@@
 $EndComp
 $Comp
-L power:GND #PWR?
+L power:GND #PWR0485
 U 1 1 812F1D0D
 P 7800 11425
-F 0 "#PWR?" H 7800 11425 30  0001 C CNN
+F 0 "#PWR0485" H 7800 11425 30  0001 C CNN
 F 1 "GND" H 7800 11355 30  0001 C CNN
 F 2 "" H 7800 11425 60  0001 C CNN
@@
 $EndComp
 $Comp
-L power:VCC #PWR?
+L power:VCC #PWR0493
 U 1 1 812F1D13
 P 8300 11425
-F 0 "#PWR?" H 8300 11525 30  0001 C CNN
+F 0 "#PWR0493" H 8300 11525 30  0001 C CNN
 F 1 "VCC" H 8304 11552 30  0000 C CNN
 F 2 "" H 8300 11425 60  0001 C CNN
@@
 $EndComp
 $Comp
-L spice:C C?
+L spice:C C277
 U 1 1 812F1D19
 P 8050 11425
-F 0 "C?" V 7763 11425 60  0000 C CNN
+F 0 "C277" V 7763 11425 60  0000 C CNN
 F 1 "100nF" V 7869 11425 60  0000 C CNN
 F 2 "" H 8050 11425 60  0000 C CNN
@@
 $EndComp
 $Comp
-L power:GND #PWR?
+L power:GND #PWR0482
 U 1 1 812F1E44
 P 7700 13950
-F 0 "#PWR?" H 7700 13950 30  0001 C CNN
+F 0 "#PWR0482" H 7700 13950 30  0001 C CNN
 F 1 "GND" H 7700 13880 30  0001 C CNN
 F 2 "" H 7700 13950 60  0001 C CNN
@@
 $EndComp
 $Comp
-L power:VCC #PWR?
+L power:VCC #PWR0490
 U 1 1 812F1E4A
 P 8200 13950
-F 0 "#PWR?" H 8200 14050 30  0001 C CNN
+F 0 "#PWR0490" H 8200 14050 30  0001 C CNN
 F 1 "VCC" H 8204 14077 30  0000 C CNN
 F 2 "" H 8200 13950 60  0001 C CNN
@@
 $EndComp
 $Comp
-L spice:C C?
+L spice:C C274
 U 1 1 812F1E50
 P 7950 13950
-F 0 "C?" V 7663 13950 60  0000 C CNN
+F 0 "C274" V 7663 13950 60  0000 C CNN
 F 1 "100nF" V 7769 13950 60  0000 C CNN
 F 2 "" H 7950 13950 60  0000 C CNN
@@
 $EndComp
 $Comp
-L power:GND #PWR?
+L power:GND #PWR0483
 U 1 1 812F1FAD
 P 7725 16825
-F 0 "#PWR?" H 7725 16825 30  0001 C CNN
+F 0 "#PWR0483" H 7725 16825 30  0001 C CNN
 F 1 "GND" H 7725 16755 30  0001 C CNN
 F 2 "" H 7725 16825 60  0001 C CNN
@@
 $EndComp
 $Comp
-L power:VCC #PWR?
+L power:VCC #PWR0491
 U 1 1 812F1FB3
 P 8225 16825
-F 0 "#PWR?" H 8225 16925 30  0001 C CNN
+F 0 "#PWR0491" H 8225 16925 30  0001 C CNN
 F 1 "VCC" H 8229 16952 30  0000 C CNN
 F 2 "" H 8225 16825 60  0001 C CNN
@@
 $EndComp
 $Comp
-L spice:C C?
+L spice:C C275
 U 1 1 812F1FB9
 P 7975 16825
-F 0 "C?" V 7688 16825 60  0000 C CNN
+F 0 "C275" V 7688 16825 60  0000 C CNN
 F 1 "100nF" V 7794 16825 60  0000 C CNN
 F 2 "" H 7975 16825 60  0000 C CNN
@@
 $EndComp
 $Comp
-L power:GND #PWR?
+L power:GND #PWR0489
 U 1 1 812F22A6
 P 8050 19625
-F 0 "#PWR?" H 8050 19625 30  0001 C CNN
+F 0 "#PWR0489" H 8050 19625 30  0001 C CNN
 F 1 "GND" H 8050 19555 30  0001 C CNN
 F 2 "" H 8050 19625 60  0001 C CNN
@@
 $EndComp
 $Comp
-L power:VCC #PWR?
+L power:VCC #PWR0497
 U 1 1 812F22AC
 P 8550 19625
-F 0 "#PWR?" H 8550 19725 30  0001 C CNN
+F 0 "#PWR0497" H 8550 19725 30  0001 C CNN
 F 1 "VCC" H 8554 19752 30  0000 C CNN
 F 2 "" H 8550 19625 60  0001 C CNN
@@
 $EndComp
 $Comp
-L spice:C C?
+L spice:C C281
 U 1 1 812F22B2
 P 8300 19625
-F 0 "C?" V 8013 19625 60  0000 C CNN
+F 0 "C281" V 8013 19625 60  0000 C CNN
 F 1 "100nF" V 8119 19625 60  0000 C CNN
 F 2 "" H 8300 19625 60  0000 C CNN
@@
 $EndComp
 $Comp
-L power:GND #PWR?
+L power:GND #PWR0488
 U 1 1 812F2465
 P 8025 22150
-F 0 "#PWR?" H 8025 22150 30  0001 C CNN
+F 0 "#PWR0488" H 8025 22150 30  0001 C CNN
 F 1 "GND" H 8025 22080 30  0001 C CNN
 F 2 "" H 8025 22150 60  0001 C CNN
@@
 $EndComp
 $Comp
-L power:VCC #PWR?
+L power:VCC #PWR0496
 U 1 1 812F246B
 P 8525 22150
-F 0 "#PWR?" H 8525 22250 30  0001 C CNN
+F 0 "#PWR0496" H 8525 22250 30  0001 C CNN
 F 1 "VCC" H 8529 22277 30  0000 C CNN
 F 2 "" H 8525 22150 60  0001 C CNN
@@
 $EndComp
 $Comp
-L spice:C C?
+L spice:C C280
 U 1 1 812F2471
 P 8275 22150
-F 0 "C?" V 7988 22150 60  0000 C CNN
+F 0 "C280" V 7988 22150 60  0000 C CNN
 F 1 "100nF" V 8094 22150 60  0000 C CNN
 F 2 "" H 8275 22150 60  0000 C CNN
@@
 $EndComp
 $Comp
-L power:GND #PWR?
+L power:GND #PWR0487
 U 1 1 812F263B
 P 8000 25075
-F 0 "#PWR?" H 8000 25075 30  0001 C CNN
+F 0 "#PWR0487" H 8000 25075 30  0001 C CNN
 F 1 "GND" H 8000 25005 30  0001 C CNN
 F 2 "" H 8000 25075 60  0001 C CNN
@@
 $EndComp
 $Comp
-L power:VCC #PWR?
+L power:VCC #PWR0495
 U 1 1 812F2641
 P 8500 25075
-F 0 "#PWR?" H 8500 25175 30  0001 C CNN
+F 0 "#PWR0495" H 8500 25175 30  0001 C CNN
 F 1 "VCC" H 8504 25202 30  0000 C CNN
 F 2 "" H 8500 25075 60  0001 C CNN
@@
 $EndComp
 $Comp
-L spice:C C?
+L spice:C C279
 U 1 1 812F2647
 P 8250 25075
-F 0 "C?" V 7963 25075 60  0000 C CNN
+F 0 "C279" V 7963 25075 60  0000 C CNN
 F 1 "100nF" V 8069 25075 60  0000 C CNN
 F 2 "" H 8250 25075 60  0000 C CNN

Commit message: message
Parts:
- renumbered C274 to C298, C275 to C299, C276 to C300, C277 to C301, C278 to C302, C279 to C303, C280 to C304, C281 to C305, U183 to U230, U184 to U231, U185 to U232, U186 to U233, U187 to U234, U188 to U235, U189 to U236, U190 to U237
Changed lines of the file:
@@
 $Descr A0 33110 46811 portrait
 encoding utf-8
-Sheet 71 92
+Sheet 71 101
 Title ""
 Date ""
@@
 $EndDescr
 $Comp
-L 74xx:74LS153 U187
+L 74xx:74LS153 U234
 U 1 1 812F095F
 P 8075 4150
-F 0 "U187" H 8075 5108 60  0000 C CNN
+F 0 "U234" H 8075 5108 60  0000 C CNN
 F 1 "74LS153" H 8075 5002 60  0000 C CNN
 F 2 "" H 8075 4150 60  0001 C CNN
@@
 $EndComp
 $Comp
-L 74xx:74LS153 U183
+L 74xx:74LS153 U230
 U 1 1 812F09E7
 P 7950 7350
-F 0 "U183" H 7950 8308 60  0000 C CNN
+F 0 "U230" H 7950 8308 60  0000 C CNN
 F 1 "74LS153" H 7950 8202 60  0000 C CNN
 F 2 "" H 7950 7350 60  0001 C CNN
@@
 $EndComp
 $Comp
-L 74xx:74LS153 U185
+L 74xx:74LS153 U232
 U 1 1 812F0A85
 P 7975 10225
-F 0 "U185" H 7975 11183 60  0000 C CNN
+F 0 "U232" H 7975 11183 60  0000 C CNN
 F 1 "74LS153" H 7975 11077 60  0000 C CNN
 F 2 "" H 7975 10225 60  0001 C CNN
@@
 $EndComp
 $Comp
-L 74xx:74LS153 U186
+L 74xx:74LS153 U233
 U 1 1 812F0D4A
 P 7975 12650
-F 0 "U186" H 7975 13608 60  0000 C CNN
+F 0 "U233" H 7975 13608 60  0000 C CNN
 F 1 "74LS153" H 7975 13502 60  0000 C CNN
 F 2 "" H 7975 12650 60  0001 C CNN
@@
 $EndComp
 $Comp
-L 74xx:74LS153 U184
+L 74xx:74LS153 U231
 U 1 1 812F0D51
 P 7950 15500
-F 0 "U184" H 7950 16458 60  0000 C CNN
+F 0 "U231" H 7950 16458 60  0000 C CNN
 F 1 "74LS153" H 7950 16352 60  0000 C CNN
 F 2 "" H 7950 15500 60  0001 C CNN
@@
 $EndComp
 $Comp
-L 74xx:74LS153 U188
+L 74xx:74LS153 U235
 U 1 1 812F0D58
 P 8300 18525
-F 0 "U188" H 8300 19483 60  0000 C CNN
+F 0 "U235" H 8300 19483 60  0000 C CNN
 F 1 "74LS153" H 8300 19377 60  0000 C CNN
 F 2 "" H 8300 18525 60  0001 C CNN
@@
 $EndComp
 $Comp
-L 74xx:74LS153 U189
+L 74xx:74LS153 U236
 U 1 1 812F1353
 P 8300 20925
-F 0 "U189" H 8300 21883 60  0000 C CNN
+F 0 "U236" H 8300 21883 60  0000 C CNN
 F 1 "74LS153" H 8300 21777 60  0000 C CNN
 F 2 "" H 8300 20925 60  0001 C CNN
@@
 $EndComp
 $Comp
-L 74xx:74LS153 U190
+L 74xx:74LS153 U237
 U 1 1 812F135A
 P 8325 23800
-F 0 "U190" H 8325 24758 60  0000 C CNN
+F 0 "U237" H 8325 24758 60  0000 C CNN
 F 1 "74LS153" H 8325 24652 60  0000 C CNN
 F 2 "" H 8325 23800 60  0001 C CNN
@@
 $EndComp
 $Comp
-L power:GND #PWR0486
+L power:GND #PWR0534
 U 1 1 812F1AD5
 P 7850 5275
-F 0 "#PWR0486" H 7850 5275 30  0001 C CNN
+F 0 "#PWR0534" H 7850 5275 30  0001 C CNN
 F 1 "GND" H 7850 5205 30  0001 C CNN
 F 2 "" H 7850 5275 60  0001 C CNN
@@
 $EndComp
 $Comp
-L power:VCC #PWR0494
+L power:VCC #PWR0542
 U 1 1 812F1B16
 P 8350 5275
-F 0 "#PWR0494" H 8350 5375 30  0001 C CNN
+F 0 "#PWR0542" H 8350 5375 30  0001 C CNN
 F 1 "VCC" H 8354 5402 30  0000 C CNN
 F 2 "" H 8350 5275 60  0001 C CNN
@@
 $EndComp
 $Comp
-L spice:C C278
+L spice:C C302
 U 1 1 812F1B57
 P 8100 5275
-F 0 "C278" V 7813 5275 60  0000 C CNN
+F 0 "C302" V 7813 5275 60  0000 C CNN
 F 1 "100nF" V 7919 5275 60  0000 C CNN
 F 2 "" H 8100 5275 60  0000 C CNN
@@
 $EndComp
 $Comp
-L power:GND #PWR0484
+L power:GND #PWR0532
 U 1 1 812F1CB2
 P 7775 8500
-F 0 "#PWR0484" H 7775 8500 30  0001 C CNN
+F 0 "#PWR0532" H 7775 8500 30  0001 C CNN
 F 1 "GND" H 7775 8430 30  0001 C CNN
 F 2 "" H 7775 8500 60  0001 C CNN
@@
 $EndComp
 $Comp
-L power:VCC #PWR0492
+L power:VCC #PWR0540
 U 1 1 812F1CB8
 P 8275 8500
-F 0 "#PWR0492" H 8275 8600 30  0001 C CNN
+F 0 "#PWR0540" H 8275 8600 30  0001 C CNN
 F 1 "VCC" H 8279 8627 30  0000 C CNN
 F 2 "" H 8275 8500 60  0001 C CNN
@@
 $EndComp
 $Comp
-L spice:C C276
+L spice:C C300
 U 1 1 812F1CBE
 P 8025 8500
-F 0 "C276" V 7738 8500 60  0000 C CNN
+F 0 "C300" V 7738 8500 60  0000 C CNN
 F 1 "100nF" V 7844 8500 60  0000 C CNN
 F 2 "" H 8025 8500 60  0000 C CNN
@@
 $EndComp
 $Comp
-L power:GND #PWR0485
+L power:GND #PWR0533
 U 1 1 812F1D0D
 P 7800 11425
-F 0 "#PWR0485" H 7800 11425 30  0001 C CNN
+F 0 "#PWR0533" H 7800 11425 30  0001 C CNN
 F 1 "GND" H 7800 11355 30  0001 C CNN
 F 2 "" H 7800 11425 60  0001 C CNN
@@
 $EndComp
 $Comp
-L power:VCC #PWR0493
+L power:VCC #PWR0541
 U 1 1 812F1D13
 P 8300 11425
-F 0 "#PWR0493" H 8300 11525 30  0001 C CNN
+F 0 "#PWR0541" H 8300 11525 30  0001 C CNN
 F 1 "VCC" H 8304 11552 30  0000 C CNN
 F 2 "" H 8300 11425 60  0001 C CNN
@@
 $EndComp
 $Comp
-L spice:C C277
+L spice:C C301
 U 1 1 812F1D19
 P 8050 11425
-F 0 "C277" V 7763 11425 60  0000 C CNN
+F 0 "C301" V 7763 11425 60  0000 C CNN
 F 1 "100nF" V 7869 11425 60  0000 C CNN
 F 2 "" H 8050 11425 60  0000 C CNN
@@
 $EndComp
 $Comp
-L power:GND #PWR0482
+L power:GND #PWR0530
 U 1 1 812F1E44
 P 7700 13950
-F 0 "#PWR0482" H 7700 13950 30  0001 C CNN
+F 0 "#PWR0530" H 7700 13950 30  0001 C CNN
 F 1 "GND" H 7700 13880 30  0001 C CNN
 F 2 "" H 7700 13950 60  0001 C CNN
@@
 $EndComp
 $Comp
-L power:VCC #PWR0490
+L power:VCC #PWR0538
 U 1 1 812F1E4A
 P 8200 13950
-F 0 "#PWR0490" H 8200 14050 30  0001 C CNN
+F 0 "#PWR0538" H 8200 14050 30  0001 C CNN
 F 1 "VCC" H 8204 14077 30  0000 C CNN
 F 2 "" H 8200 13950 60  0001 C CNN
@@
 $EndComp
 $Comp
-L spice:C C274
+L spice:C C298
 U 1 1 812F1E50
 P 7950 13950
-F 0 "C274" V 7663 13950 60  0000 C CNN
+F 0 "C298" V 7663 13950 60  0000 C CNN
 F 1 "100nF" V 7769 13950 60  0000 C CNN
 F 2 "" H 7950 13950 60  0000 C CNN
@@
 $EndComp
 $Comp
-L power:GND #PWR0483
+L power:GND #PWR0531
 U 1 1 812F1FAD
 P 7725 16825
-F 0 "#PWR0483" H 7725 16825 30  0001 C CNN
+F 0 "#PWR0531" H 7725 16825 30  0001 C CNN
 F 1 "GND" H 7725 16755 30  0001 C CNN
 F 2 "" H 7725 16825 60  0001 C CNN
@@
 $EndComp
 $Comp
-L power:VCC #PWR0491
+L power:VCC #PWR0539
 U 1 1 812F1FB3
 P 8225 16825
-F 0 "#PWR0491" H 8225 16925 30  0001 C CNN
+F 0 "#PWR0539" H 8225 16925 30  0001 C CNN
 F 1 "VCC" H 8229 16952 30  0000 C CNN
 F 2 "" H 8225 16825 60  0001 C CNN
@@
 $EndComp
 $Comp
-L spice:C C275
+L spice:C C299
 U 1 1 812F1FB9
 P 7975 16825
-F 0 "C275" V 7688 16825 60  0000 C CNN
+F 0 "C299" V 7688 16825 60  0000 C CNN
 F 1 "100nF" V 7794 16825 60  0000 C CNN
 F 2 "" H 7975 16825 60  0000 C CNN
@@
 $EndComp
 $Comp
-L power:GND #PWR0489
+L power:GND #PWR0537
 U 1 1 812F22A6
 P 8050 19625
-F 0 "#PWR0489" H 8050 19625 30  0001 C CNN
+F 0 "#PWR0537" H 8050 19625 30  0001 C CNN
 F 1 "GND" H 8050 19555 30  0001 C CNN
 F 2 "" H 8050 19625 60  0001 C CNN
@@
 $EndComp
 $Comp
-L power:VCC #PWR0497
+L power:VCC #PWR0545
 U 1 1 812F22AC
 P 8550 19625
-F 0 "#PWR0497" H 8550 19725 30  0001 C CNN
+F 0 "#PWR0545" H 8550 19725 30  0001 C CNN
 F 1 "VCC" H 8554 19752 30  0000 C CNN
 F 2 "" H 8550 19625 60  0001 C CNN
@@
 $EndComp
 $Comp
-L spice:C C281
+L spice:C C305
 U 1 1 812F22B2
 P 8300 19625
-F 0 "C281" V 8013 19625 60  0000 C CNN
+F 0 "C305" V 8013 19625 60  0000 C CNN
 F 1 "100nF" V 8119 19625 60  0000 C CNN
 F 2 "" H 8300 19625 60  0000 C CNN
@@
 $EndComp
 $Comp
-L power:GND #PWR0488
+L power:GND #PWR0536
 U 1 1 812F2465
 P 8025 22150
-F 0 "#PWR0488" H 8025 22150 30  0001 C CNN
+F 0 "#PWR0536" H 8025 22150 30  0001 C CNN
 F 1 "GND" H 8025 22080 30  0001 C CNN
 F 2 "" H 8025 22150 60  0001 C CNN
@@
 $EndComp
 $Comp
-L power:VCC #PWR0496
+L power:VCC #PWR0544
 U 1 1 812F246B
 P 8525 22150
-F 0 "#PWR0496" H 8525 22250 30  0001 C CNN
+F 0 "#PWR0544" H 8525 22250 30  0001 C CNN
 F 1 "VCC" H 8529 22277 30  0000 C CNN
 F 2 "" H 8525 22150 60  0001 C CNN
@@
 $EndComp
 $Comp
-L spice:C C280
+L spice:C C304
 U 1 1 812F2471
 P 8275 22150
-F 0 "C280" V 7988 22150 60  0000 C CNN
+F 0 "C304" V 7988 22150 60  0000 C CNN
 F 1 "100nF" V 8094 22150 60  0000 C CNN
 F 2 "" H 8275 22150 60  0000 C CNN
@@
 $EndComp
 $Comp
-L power:GND #PWR0487
+L power:GND #PWR0535
 U 1 1 812F263B
 P 8000 25075
-F 0 "#PWR0487" H 8000 25075 30  0001 C CNN
+F 0 "#PWR0535" H 8000 25075 30  0001 C CNN
 F 1 "GND" H 8000 25005 30  0001 C CNN
 F 2 "" H 8000 25075 60  0001 C CNN
@@
 $EndComp
 $Comp
-L power:VCC #PWR0495
+L power:VCC #PWR0543
 U 1 1 812F2641
 P 8500 25075
-F 0 "#PWR0495" H 8500 25175 30  0001 C CNN
+F 0 "#PWR0543" H 8500 25175 30  0001 C CNN
 F 1 "VCC" H 8504 25202 30  0000 C CNN
 F 2 "" H 8500 25075 60  0001 C CNN
@@
 $EndComp
 $Comp
-L spice:C C279
+L spice:C C303
 U 1 1 812F2647
 P 8250 25075
-F 0 "C279" V 7963 25075 60  0000 C CNN
+F 0 "C303" V 7963 25075 60  0000 C CNN
 F 1 "100nF" V 8069 25075 60  0000 C CNN
 F 2 "" H 8250 25075 60  0000 C CNN
