File: 16-Bit4-1Mux.sch (KiCad schematic (older format))
At the start: 16 parts, among them U230 74LS153, U231 74LS153, U232 74LS153, U233 74LS153, U234 74LS153, U235 74LS153, U236 74LS153, U237 74LS153

Commit message: .
Parts:
- renumbered C298 to C106, C299 to C107, C300 to C108, C301 to C109, C302 to C110, C303 to C111, C304 to C112, C305 to C113, U230 to U137, U231 to U138, U232 to U139, U233 to U140, U234 to U141, U235 to U142, U236 to U143, U237 to U144
Changed lines of the file:
@@
 $Descr A0 33110 46811 portrait
 encoding utf-8
-Sheet 71 101
+Sheet 71 75
 Title ""
 Date ""
@@
 $EndDescr
 $Comp
-L 74xx:74LS153 U234
+L 74xx:74LS153 U141
 U 1 1 812F095F
 P 8075 4150
-F 0 "U234" H 8075 5108 60  0000 C CNN
+F 0 "U141" H 8075 5108 60  0000 C CNN
 F 1 "74LS153" H 8075 5002 60  0000 C CNN
 F 2 "" H 8075 4150 60  0001 C CNN
@@
 $EndComp
 $Comp
-L 74xx:74LS153 U230
+L 74xx:74LS153 U137
 U 1 1 812F09E7
 P 7950 7350
-F 0 "U230" H 7950 8308 60  0000 C CNN
+F 0 "U137" H 7950 8308 60  0000 C CNN
 F 1 "74LS153" H 7950 8202 60  0000 C CNN
 F 2 "" H 7950 7350 60  0001 C CNN
@@
 $EndComp
 $Comp
-L 74xx:74LS153 U232
+L 74xx:74LS153 U139
 U 1 1 812F0A85
 P 7975 10225
-F 0 "U232" H 7975 11183 60  0000 C CNN
+F 0 "U139" H 7975 11183 60  0000 C CNN
 F 1 "74LS153" H 7975 11077 60  0000 C CNN
 F 2 "" H 7975 10225 60  0001 C CNN
@@
 $EndComp
 $Comp
-L 74xx:74LS153 U233
+L 74xx:74LS153 U140
 U 1 1 812F0D4A
 P 7975 12650
-F 0 "U233" H 7975 13608 60  0000 C CNN
+F 0 "U140" H 7975 13608 60  0000 C CNN
 F 1 "74LS153" H 7975 13502 60  0000 C CNN
 F 2 "" H 7975 12650 60  0001 C CNN
@@
 $EndComp
 $Comp
-L 74xx:74LS153 U231
+L 74xx:74LS153 U138
 U 1 1 812F0D51
 P 7950 15500
-F 0 "U231" H 7950 16458 60  0000 C CNN
+F 0 "U138" H 7950 16458 60  0000 C CNN
 F 1 "74LS153" H 7950 16352 60  0000 C CNN
 F 2 "" H 7950 15500 60  0001 C CNN
@@
 $EndComp
 $Comp
-L 74xx:74LS153 U235
+L 74xx:74LS153 U142
 U 1 1 812F0D58
 P 8300 18525
-F 0 "U235" H 8300 19483 60  0000 C CNN
+F 0 "U142" H 8300 19483 60  0000 C CNN
 F 1 "74LS153" H 8300 19377 60  0000 C CNN
 F 2 "" H 8300 18525 60  0001 C CNN
@@
 $EndComp
 $Comp
-L 74xx:74LS153 U236
+L 74xx:74LS153 U143
 U 1 1 812F1353
 P 8300 20925
-F 0 "U236" H 8300 21883 60  0000 C CNN
+F 0 "U143" H 8300 21883 60  0000 C CNN
 F 1 "74LS153" H 8300 21777 60  0000 C CNN
 F 2 "" H 8300 20925 60  0001 C CNN
@@
 $EndComp
 $Comp
-L 74xx:74LS153 U237
+L 74xx:74LS153 U144
 U 1 1 812F135A
 P 8325 23800
-F 0 "U237" H 8325 24758 60  0000 C CNN
+F 0 "U144" H 8325 24758 60  0000 C CNN
 F 1 "74LS153" H 8325 24652 60  0000 C CNN
 F 2 "" H 8325 23800 60  0001 C CNN
@@
 $EndComp
 $Comp
-L power:GND #PWR0534
+L power:GND #PWR0156
 U 1 1 812F1AD5
 P 7850 5275
-F 0 "#PWR0534" H 7850 5275 30  0001 C CNN
+F 0 "#PWR0156" H 7850 5275 30  0001 C CNN
 F 1 "GND" H 7850 5205 30  0001 C CNN
 F 2 "" H 7850 5275 60  0001 C CNN
@@
 $EndComp
 $Comp
-L power:VCC #PWR0542
+L power:VCC #PWR0164
 U 1 1 812F1B16
 P 8350 5275
-F 0 "#PWR0542" H 8350 5375 30  0001 C CNN
+F 0 "#PWR0164" H 8350 5375 30  0001 C CNN
 F 1 "VCC" H 8354 5402 30  0000 C CNN
 F 2 "" H 8350 5275 60  0001 C CNN
@@
 $EndComp
 $Comp
-L spice:C C302
+L spice:C C110
 U 1 1 812F1B57
 P 8100 5275
-F 0 "C302" V 7813 5275 60  0000 C CNN
+F 0 "C110" V 7813 5275 60  0000 C CNN
 F 1 "100nF" V 7919 5275 60  0000 C CNN
 F 2 "" H 8100 5275 60  0000 C CNN
@@
 $EndComp
 $Comp
-L power:GND #PWR0532
+L power:GND #PWR0154
 U 1 1 812F1CB2
 P 7775 8500
-F 0 "#PWR0532" H 7775 8500 30  0001 C CNN
+F 0 "#PWR0154" H 7775 8500 30  0001 C CNN
 F 1 "GND" H 7775 8430 30  0001 C CNN
 F 2 "" H 7775 8500 60  0001 C CNN
@@
 $EndComp
 $Comp
-L power:VCC #PWR0540
+L power:VCC #PWR0162
 U 1 1 812F1CB8
 P 8275 8500
-F 0 "#PWR0540" H 8275 8600 30  0001 C CNN
+F 0 "#PWR0162" H 8275 8600 30  0001 C CNN
 F 1 "VCC" H 8279 8627 30  0000 C CNN
 F 2 "" H 8275 8500 60  0001 C CNN
@@
 $EndComp
 $Comp
-L spice:C C300
+L spice:C C108
 U 1 1 812F1CBE
 P 8025 8500
-F 0 "C300" V 7738 8500 60  0000 C CNN
+F 0 "C108" V 7738 8500 60  0000 C CNN
 F 1 "100nF" V 7844 8500 60  0000 C CNN
 F 2 "" H 8025 8500 60  0000 C CNN
@@
 $EndComp
 $Comp
-L power:GND #PWR0533
+L power:GND #PWR0155
 U 1 1 812F1D0D
 P 7800 11425
-F 0 "#PWR0533" H 7800 11425 30  0001 C CNN
+F 0 "#PWR0155" H 7800 11425 30  0001 C CNN
 F 1 "GND" H 7800 11355 30  0001 C CNN
 F 2 "" H 7800 11425 60  0001 C CNN
@@
 $EndComp
 $Comp
-L power:VCC #PWR0541
+L power:VCC #PWR0163
 U 1 1 812F1D13
 P 8300 11425
-F 0 "#PWR0541" H 8300 11525 30  0001 C CNN
+F 0 "#PWR0163" H 8300 11525 30  0001 C CNN
 F 1 "VCC" H 8304 11552 30  0000 C CNN
 F 2 "" H 8300 11425 60  0001 C CNN
@@
 $EndComp
 $Comp
-L spice:C C301
+L spice:C C109
 U 1 1 812F1D19
 P 8050 11425
-F 0 "C301" V 7763 11425 60  0000 C CNN
+F 0 "C109" V 7763 11425 60  0000 C CNN
 F 1 "100nF" V 7869 11425 60  0000 C CNN
 F 2 "" H 8050 11425 60  0000 C CNN
@@
 $EndComp
 $Comp
-L power:GND #PWR0530
+L power:GND #PWR0152
 U 1 1 812F1E44
 P 7700 13950
-F 0 "#PWR0530" H 7700 13950 30  0001 C CNN
+F 0 "#PWR0152" H 7700 13950 30  0001 C CNN
 F 1 "GND" H 7700 13880 30  0001 C CNN
 F 2 "" H 7700 13950 60  0001 C CNN
@@
 $EndComp
 $Comp
-L power:VCC #PWR0538
+L power:VCC #PWR0160
 U 1 1 812F1E4A
 P 8200 13950
-F 0 "#PWR0538" H 8200 14050 30  0001 C CNN
+F 0 "#PWR0160" H 8200 14050 30  0001 C CNN
 F 1 "VCC" H 8204 14077 30  0000 C CNN
 F 2 "" H 8200 13950 60  0001 C CNN
@@
 $EndComp
 $Comp
-L spice:C C298
+L spice:C C106
 U 1 1 812F1E50
 P 7950 13950
-F 0 "C298" V 7663 13950 60  0000 C CNN
+F 0 "C106" V 7663 13950 60  0000 C CNN
 F 1 "100nF" V 7769 13950 60  0000 C CNN
 F 2 "" H 7950 13950 60  0000 C CNN
@@
 $EndComp
 $Comp
-L power:GND #PWR0531
+L power:GND #PWR0153
 U 1 1 812F1FAD
 P 7725 16825
-F 0 "#PWR0531" H 7725 16825 30  0001 C CNN
+F 0 "#PWR0153" H 7725 16825 30  0001 C CNN
 F 1 "GND" H 7725 16755 30  0001 C CNN
 F 2 "" H 7725 16825 60  0001 C CNN
@@
 $EndComp
 $Comp
-L power:VCC #PWR0539
+L power:VCC #PWR0161
 U 1 1 812F1FB3
 P 8225 16825
-F 0 "#PWR0539" H 8225 16925 30  0001 C CNN
+F 0 "#PWR0161" H 8225 16925 30  0001 C CNN
 F 1 "VCC" H 8229 16952 30  0000 C CNN
 F 2 "" H 8225 16825 60  0001 C CNN
@@
 $EndComp
 $Comp
-L spice:C C299
+L spice:C C107
 U 1 1 812F1FB9
 P 7975 16825
-F 0 "C299" V 7688 16825 60  0000 C CNN
+F 0 "C107" V 7688 16825 60  0000 C CNN
 F 1 "100nF" V 7794 16825 60  0000 C CNN
 F 2 "" H 7975 16825 60  0000 C CNN
@@
 $EndComp
 $Comp
-L power:GND #PWR0537
+L power:GND #PWR0159
 U 1 1 812F22A6
 P 8050 19625
-F 0 "#PWR0537" H 8050 19625 30  0001 C CNN
+F 0 "#PWR0159" H 8050 19625 30  0001 C CNN
 F 1 "GND" H 8050 19555 30  0001 C CNN
 F 2 "" H 8050 19625 60  0001 C CNN
@@
 $EndComp
 $Comp
-L power:VCC #PWR0545
+L power:VCC #PWR0167
 U 1 1 812F22AC
 P 8550 19625
-F 0 "#PWR0545" H 8550 19725 30  0001 C CNN
+F 0 "#PWR0167" H 8550 19725 30  0001 C CNN
 F 1 "VCC" H 8554 19752 30  0000 C CNN
 F 2 "" H 8550 19625 60  0001 C CNN
@@
 $EndComp
 $Comp
-L spice:C C305
+L spice:C C113
 U 1 1 812F22B2
 P 8300 19625
-F 0 "C305" V 8013 19625 60  0000 C CNN
+F 0 "C113" V 8013 19625 60  0000 C CNN
 F 1 "100nF" V 8119 19625 60  0000 C CNN
 F 2 "" H 8300 19625 60  0000 C CNN
@@
 $EndComp
 $Comp
-L power:GND #PWR0536
+L power:GND #PWR0158
 U 1 1 812F2465
 P 8025 22150
-F 0 "#PWR0536" H 8025 22150 30  0001 C CNN
+F 0 "#PWR0158" H 8025 22150 30  0001 C CNN
 F 1 "GND" H 8025 22080 30  0001 C CNN
 F 2 "" H 8025 22150 60  0001 C CNN
@@
 $EndComp
 $Comp
-L power:VCC #PWR0544
+L power:VCC #PWR0166
 U 1 1 812F246B
 P 8525 22150
-F 0 "#PWR0544" H 8525 22250 30  0001 C CNN
+F 0 "#PWR0166" H 8525 22250 30  0001 C CNN
 F 1 "VCC" H 8529 22277 30  0000 C CNN
 F 2 "" H 8525 22150 60  0001 C CNN
@@
 $EndComp
 $Comp
-L spice:C C304
+L spice:C C112
 U 1 1 812F2471
 P 8275 22150
-F 0 "C304" V 7988 22150 60  0000 C CNN
+F 0 "C112" V 7988 22150 60  0000 C CNN
 F 1 "100nF" V 8094 22150 60  0000 C CNN
 F 2 "" H 8275 22150 60  0000 C CNN
@@
 $EndComp
 $Comp
-L power:GND #PWR0535
+L power:GND #PWR0157
 U 1 1 812F263B
 P 8000 25075
-F 0 "#PWR0535" H 8000 25075 30  0001 C CNN
+F 0 "#PWR0157" H 8000 25075 30  0001 C CNN
 F 1 "GND" H 8000 25005 30  0001 C CNN
 F 2 "" H 8000 25075 60  0001 C CNN
@@
 $EndComp
 $Comp
-L power:VCC #PWR0543
+L power:VCC #PWR0165
 U 1 1 812F2641
 P 8500 25075
-F 0 "#PWR0543" H 8500 25175 30  0001 C CNN
+F 0 "#PWR0165" H 8500 25175 30  0001 C CNN
 F 1 "VCC" H 8504 25202 30  0000 C CNN
 F 2 "" H 8500 25075 60  0001 C CNN
@@
 $EndComp
 $Comp
-L spice:C C303
+L spice:C C111
 U 1 1 812F2647
 P 8250 25075
-F 0 "C303" V 7963 25075 60  0000 C CNN
+F 0 "C111" V 7963 25075 60  0000 C CNN
 F 1 "100nF" V 8069 25075 60  0000 C CNN
 F 2 "" H 8250 25075 60  0000 C CNN
