File: 16Bit2-1Mux.sch (KiCad schematic (older format))
At the start: 8 parts

Commit message: b
Parts:
- gave numbers to parts that had none: 8
Changed lines of the file:
@@
 $Descr A4 11693 8268
 encoding utf-8
-Sheet 80 90
+Sheet 80 92
 Title ""
 Date ""
@@
 $EndDescr
 $Comp
-L 74xx:74LS157 U?
+L 74xx:74LS157 U203
 U 1 1 82641704
 P 3075 1825
-F 0 "U?" H 3075 2633 60  0000 C CNN
+AR Path="/82611AC0/82641637/82641704" Ref="U203"  Part="1"
+AR Path="/831A25D1/82641704" Ref="U223"  Part="1"
+AR Path="/5D50CA86/82641704" Ref="U231"  Part="1"
+F 0 "U231" H 3075 2633 60  0000 C CNN
 F 1 "74LS157" H 3075 2527 60  0000 C CNN
 F 2 "" H 3075 1825 60  0001 C CNN
@@
 $EndComp
 $Comp
-L 74xx:74LS157 U?
+L 74xx:74LS157 U204
 U 1 1 826417B3
 P 3125 3500
-F 0 "U?" H 3125 4308 60  0000 C CNN
+AR Path="/82611AC0/82641637/826417B3" Ref="U204"  Part="1"
+AR Path="/831A25D1/826417B3" Ref="U224"  Part="1"
+AR Path="/5D50CA86/826417B3" Ref="U232"  Part="1"
+F 0 "U232" H 3125 4308 60  0000 C CNN
 F 1 "74LS157" H 3125 4202 60  0000 C CNN
 F 2 "" H 3125 3500 60  0001 C CNN
@@
 $EndComp
 $Comp
-L 74xx:74LS157 U?
+L 74xx:74LS157 U205
 U 1 1 8264184D
 P 3175 5200
-F 0 "U?" H 3175 6008 60  0000 C CNN
+AR Path="/82611AC0/82641637/8264184D" Ref="U205"  Part="1"
+AR Path="/831A25D1/8264184D" Ref="U225"  Part="1"
+AR Path="/5D50CA86/8264184D" Ref="U233"  Part="1"
+F 0 "U233" H 3175 6008 60  0000 C CNN
 F 1 "74LS157" H 3175 5902 60  0000 C CNN
 F 2 "" H 3175 5200 60  0001 C CNN
@@
 $EndComp
 $Comp
-L 74xx:74LS157 U?
+L 74xx:74LS157 U206
 U 1 1 826418D6
 P 3275 6925
-F 0 "U?" H 3275 7733 60  0000 C CNN
+AR Path="/82611AC0/82641637/826418D6" Ref="U206"  Part="1"
+AR Path="/831A25D1/826418D6" Ref="U226"  Part="1"
+AR Path="/5D50CA86/826418D6" Ref="U234"  Part="1"
+F 0 "U234" H 3275 7733 60  0000 C CNN
 F 1 "74LS157" H 3275 7627 60  0000 C CNN
 F 2 "" H 3275 6925 60  0001 C CNN
@@
 $EndComp
 $Comp
-L power:GND #PWR?
+L power:GND #PWR0535
 U 1 1 82641B85
 P 2425 2600
-F 0 "#PWR?" H 2425 2600 30  0001 C CNN
+AR Path="/82611AC0/82641637/82641B85" Ref="#PWR0535"  Part="1"
+AR Path="/831A25D1/82641B85" Ref="#PWR0591"  Part="1"
+AR Path="/5D50CA86/82641B85" Ref="#PWR0604"  Part="1"
+F 0 "#PWR0604" H 2425 2600 30  0001 C CNN
 F 1 "GND" H 2425 2530 30  0001 C CNN
 F 2 "" H 2425 2600 60  0001 C CNN
@@
 $EndComp
 $Comp
-L power:VCC #PWR?
+L power:VCC #PWR0539
 U 1 1 82641B8B
 P 3625 2550
-F 0 "#PWR?" H 3625 2650 30  0001 C CNN
+AR Path="/82611AC0/82641637/82641B8B" Ref="#PWR0539"  Part="1"
+AR Path="/831A25D1/82641B8B" Ref="#PWR0595"  Part="1"
+AR Path="/5D50CA86/82641B8B" Ref="#PWR0608"  Part="1"
+F 0 "#PWR0608" H 3625 2650 30  0001 C CNN
 F 1 "VCC" H 3629 2677 30  0000 C CNN
 F 2 "" H 3625 2550 60  0001 C CNN
@@
 $EndComp
 $Comp
-L spice:C C?
+L spice:C C302
 U 1 1 82641B91
 P 3075 2600
-F 0 "C?" V 2788 2600 60  0000 C CNN
+AR Path="/82611AC0/82641637/82641B91" Ref="C302"  Part="1"
+AR Path="/831A25D1/82641B91" Ref="C322"  Part="1"
+AR Path="/5D50CA86/82641B91" Ref="C330"  Part="1"
+F 0 "C330" V 2788 2600 60  0000 C CNN
 F 1 "100nF" V 2894 2600 60  0000 C CNN
 F 2 "" H 3075 2600 60  0000 C CNN
@@
 	3625 2600 3625 2550
 $Comp
-L power:GND #PWR?
+L power:GND #PWR0537
 U 1 1 82641BF1
 P 2600 4275
-F 0 "#PWR?" H 2600 4275 30  0001 C CNN
+AR Path="/82611AC0/82641637/82641BF1" Ref="#PWR0537"  Part="1"
+AR Path="/831A25D1/82641BF1" Ref="#PWR0593"  Part="1"
+AR Path="/5D50CA86/82641BF1" Ref="#PWR0606"  Part="1"
+F 0 "#PWR0606" H 2600 4275 30  0001 C CNN
 F 1 "GND" H 2600 4205 30  0001 C CNN
 F 2 "" H 2600 4275 60  0001 C CNN
@@
 $EndComp
 $Comp
-L power:VCC #PWR?
+L power:VCC #PWR0541
 U 1 1 82641BF7
 P 3800 4225
-F 0 "#PWR?" H 3800 4325 30  0001 C CNN
+AR Path="/82611AC0/82641637/82641BF7" Ref="#PWR0541"  Part="1"
+AR Path="/831A25D1/82641BF7" Ref="#PWR0597"  Part="1"
+AR Path="/5D50CA86/82641BF7" Ref="#PWR0610"  Part="1"
+F 0 "#PWR0610" H 3800 4325 30  0001 C CNN
 F 1 "VCC" H 3804 4352 30  0000 C CNN
 F 2 "" H 3800 4225 60  0001 C CNN
@@
 $EndComp
 $Comp
-L spice:C C?
+L spice:C C304
 U 1 1 82641BFD
 P 3250 4275
-F 0 "C?" V 2963 4275 60  0000 C CNN
+AR Path="/82611AC0/82641637/82641BFD" Ref="C304"  Part="1"
+AR Path="/831A25D1/82641BFD" Ref="C324"  Part="1"
+AR Path="/5D50CA86/82641BFD" Ref="C332"  Part="1"
+F 0 "C332" V 2963 4275 60  0000 C CNN
 F 1 "100nF" V 3069 4275 60  0000 C CNN
 F 2 "" H 3250 4275 60  0000 C CNN
@@
 	3800 4275 3800 4225
 $Comp
-L power:GND #PWR?
+L power:GND #PWR0536
 U 1 1 82641CA4
 P 2575 5975
-F 0 "#PWR?" H 2575 5975 30  0001 C CNN
+AR Path="/82611AC0/82641637/82641CA4" Ref="#PWR0536"  Part="1"
+AR Path="/831A25D1/82641CA4" Ref="#PWR0592"  Part="1"
+AR Path="/5D50CA86/82641CA4" Ref="#PWR0605"  Part="1"
+F 0 "#PWR0605" H 2575 5975 30  0001 C CNN
 F 1 "GND" H 2575 5905 30  0001 C CNN
 F 2 "" H 2575 5975 60  0001 C CNN
@@
 $EndComp
 $Comp
-L power:VCC #PWR?
+L power:VCC #PWR0540
 U 1 1 82641CAA
 P 3775 5925
-F 0 "#PWR?" H 3775 6025 30  0001 C CNN
+AR Path="/82611AC0/82641637/82641CAA" Ref="#PWR0540"  Part="1"
+AR Path="/831A25D1/82641CAA" Ref="#PWR0596"  Part="1"
+AR Path="/5D50CA86/82641CAA" Ref="#PWR0609"  Part="1"
+F 0 "#PWR0609" H 3775 6025 30  0001 C CNN
 F 1 "VCC" H 3779 6052 30  0000 C CNN
 F 2 "" H 3775 5925 60  0001 C CNN
@@
 $EndComp
 $Comp
-L spice:C C?
+L spice:C C303
 U 1 1 82641CB0
 P 3225 5975
-F 0 "C?" V 2938 5975 60  0000 C CNN
+AR Path="/82611AC0/82641637/82641CB0" Ref="C303"  Part="1"
+AR Path="/831A25D1/82641CB0" Ref="C323"  Part="1"
+AR Path="/5D50CA86/82641CB0" Ref="C331"  Part="1"
+F 0 "C331" V 2938 5975 60  0000 C CNN
 F 1 "100nF" V 3044 5975 60  0000 C CNN
 F 2 "" H 3225 5975 60  0000 C CNN
@@
 	3775 5975 3775 5925
 $Comp
-L power:GND #PWR?
+L power:GND #PWR0538
 U 1 1 82641D95
 P 2675 7700
-F 0 "#PWR?" H 2675 7700 30  0001 C CNN
+AR Path="/82611AC0/82641637/82641D95" Ref="#PWR0538"  Part="1"
+AR Path="/831A25D1/82641D95" Ref="#PWR0594"  Part="1"
+AR Path="/5D50CA86/82641D95" Ref="#PWR0607"  Part="1"
+F 0 "#PWR0607" H 2675 7700 30  0001 C CNN
 F 1 "GND" H 2675 7630 30  0001 C CNN
 F 2 "" H 2675 7700 60  0001 C CNN
@@
 $EndComp
 $Comp
-L power:VCC #PWR?
+L power:VCC #PWR0542
 U 1 1 82641D9B
 P 3875 7650
-F 0 "#PWR?" H 3875 7750 30  0001 C CNN
+AR Path="/82611AC0/82641637/82641D9B" Ref="#PWR0542"  Part="1"
+AR Path="/831A25D1/82641D9B" Ref="#PWR0598"  Part="1"
+AR Path="/5D50CA86/82641D9B" Ref="#PWR0611"  Part="1"
+F 0 "#PWR0611" H 3875 7750 30  0001 C CNN
 F 1 "VCC" H 3879 7777 30  0000 C CNN
 F 2 "" H 3875 7650 60  0001 C CNN
@@
 $EndComp
 $Comp
-L spice:C C?
+L spice:C C305
 U 1 1 82641DA1
 P 3325 7700
-F 0 "C?" V 3038 7700 60  0000 C CNN
+AR Path="/82611AC0/82641637/82641DA1" Ref="C305"  Part="1"
+AR Path="/831A25D1/82641DA1" Ref="C325"  Part="1"
+AR Path="/5D50CA86/82641DA1" Ref="C333"  Part="1"
+F 0 "C333" V 3038 7700 60  0000 C CNN
 F 1 "100nF" V 3144 7700 60  0000 C CNN
 F 2 "" H 3325 7700 60  0000 C CNN

Commit message: message
Parts:
- renumbered C302 to C326, C303 to C327, C304 to C328, C305 to C329, U203 to U250, U204 to U251, U205 to U252, U206 to U253
Changed lines of the file:
@@
 $Descr A4 11693 8268
 encoding utf-8
-Sheet 80 92
+Sheet 80 101
 Title ""
 Date ""
@@
 $EndDescr
 $Comp
-L 74xx:74LS157 U203
+L 74xx:74LS157 U250
 U 1 1 82641704
 P 3075 1825
-AR Path="/82611AC0/82641637/82641704" Ref="U203"  Part="1"
-AR Path="/831A25D1/82641704" Ref="U223"  Part="1"
-AR Path="/5D50CA86/82641704" Ref="U231"  Part="1"
-F 0 "U231" H 3075 2633 60  0000 C CNN
+AR Path="/82611AC0/82641637/82641704" Ref="U250"  Part="1"
+AR Path="/831A25D1/82641704" Ref="U270"  Part="1"
+AR Path="/5D50CA86/82641704" Ref="U278"  Part="1"
+F 0 "U278" H 3075 2633 60  0000 C CNN
 F 1 "74LS157" H 3075 2527 60  0000 C CNN
 F 2 "" H 3075 1825 60  0001 C CNN
@@
 $EndComp
 $Comp
-L 74xx:74LS157 U204
+L 74xx:74LS157 U251
 U 1 1 826417B3
 P 3125 3500
-AR Path="/82611AC0/82641637/826417B3" Ref="U204"  Part="1"
-AR Path="/831A25D1/826417B3" Ref="U224"  Part="1"
-AR Path="/5D50CA86/826417B3" Ref="U232"  Part="1"
-F 0 "U232" H 3125 4308 60  0000 C CNN
+AR Path="/82611AC0/82641637/826417B3" Ref="U251"  Part="1"
+AR Path="/831A25D1/826417B3" Ref="U271"  Part="1"
+AR Path="/5D50CA86/826417B3" Ref="U279"  Part="1"
+F 0 "U279" H 3125 4308 60  0000 C CNN
 F 1 "74LS157" H 3125 4202 60  0000 C CNN
 F 2 "" H 3125 3500 60  0001 C CNN
@@
 $EndComp
 $Comp
-L 74xx:74LS157 U205
+L 74xx:74LS157 U252
 U 1 1 8264184D
 P 3175 5200
-AR Path="/82611AC0/82641637/8264184D" Ref="U205"  Part="1"
-AR Path="/831A25D1/8264184D" Ref="U225"  Part="1"
-AR Path="/5D50CA86/8264184D" Ref="U233"  Part="1"
-F 0 "U233" H 3175 6008 60  0000 C CNN
+AR Path="/82611AC0/82641637/8264184D" Ref="U252"  Part="1"
+AR Path="/831A25D1/8264184D" Ref="U272"  Part="1"
+AR Path="/5D50CA86/8264184D" Ref="U280"  Part="1"
+F 0 "U280" H 3175 6008 60  0000 C CNN
 F 1 "74LS157" H 3175 5902 60  0000 C CNN
 F 2 "" H 3175 5200 60  0001 C CNN
@@
 $EndComp
 $Comp
-L 74xx:74LS157 U206
+L 74xx:74LS157 U253
 U 1 1 826418D6
 P 3275 6925
-AR Path="/82611AC0/82641637/826418D6" Ref="U206"  Part="1"
-AR Path="/831A25D1/826418D6" Ref="U226"  Part="1"
-AR Path="/5D50CA86/826418D6" Ref="U234"  Part="1"
-F 0 "U234" H 3275 7733 60  0000 C CNN
+AR Path="/82611AC0/82641637/826418D6" Ref="U253"  Part="1"
+AR Path="/831A25D1/826418D6" Ref="U273"  Part="1"
+AR Path="/5D50CA86/826418D6" Ref="U281"  Part="1"
+F 0 "U281" H 3275 7733 60  0000 C CNN
 F 1 "74LS157" H 3275 7627 60  0000 C CNN
 F 2 "" H 3275 6925 60  0001 C CNN
@@
 $EndComp
 $Comp
-L power:GND #PWR0535
+L power:GND #PWR0587
 U 1 1 82641B85
 P 2425 2600
-AR Path="/82611AC0/82641637/82641B85" Ref="#PWR0535"  Part="1"
-AR Path="/831A25D1/82641B85" Ref="#PWR0591"  Part="1"
-AR Path="/5D50CA86/82641B85" Ref="#PWR0604"  Part="1"
-F 0 "#PWR0604" H 2425 2600 30  0001 C CNN
+AR Path="/82611AC0/82641637/82641B85" Ref="#PWR0587"  Part="1"
+AR Path="/831A25D1/82641B85" Ref="#PWR0643"  Part="1"
+AR Path="/5D50CA86/82641B85" Ref="#PWR0660"  Part="1"
+F 0 "#PWR0660" H 2425 2600 30  0001 C CNN
 F 1 "GND" H 2425 2530 30  0001 C CNN
 F 2 "" H 2425 2600 60  0001 C CNN
@@
 $EndComp
 $Comp
-L power:VCC #PWR0539
+L power:VCC #PWR0591
 U 1 1 82641B8B
 P 3625 2550
-AR Path="/82611AC0/82641637/82641B8B" Ref="#PWR0539"  Part="1"
-AR Path="/831A25D1/82641B8B" Ref="#PWR0595"  Part="1"
-AR Path="/5D50CA86/82641B8B" Ref="#PWR0608"  Part="1"
-F 0 "#PWR0608" H 3625 2650 30  0001 C CNN
+AR Path="/82611AC0/82641637/82641B8B" Ref="#PWR0591"  Part="1"
+AR Path="/831A25D1/82641B8B" Ref="#PWR0647"  Part="1"
+AR Path="/5D50CA86/82641B8B" Ref="#PWR0664"  Part="1"
+F 0 "#PWR0664" H 3625 2650 30  0001 C CNN
 F 1 "VCC" H 3629 2677 30  0000 C CNN
 F 2 "" H 3625 2550 60  0001 C CNN
@@
 $EndComp
 $Comp
-L spice:C C302
+L spice:C C326
 U 1 1 82641B91
 P 3075 2600
-AR Path="/82611AC0/82641637/82641B91" Ref="C302"  Part="1"
-AR Path="/831A25D1/82641B91" Ref="C322"  Part="1"
-AR Path="/5D50CA86/82641B91" Ref="C330"  Part="1"
-F 0 "C330" V 2788 2600 60  0000 C CNN
+AR Path="/82611AC0/82641637/82641B91" Ref="C326"  Part="1"
+AR Path="/831A25D1/82641B91" Ref="C346"  Part="1"
+AR Path="/5D50CA86/82641B91" Ref="C354"  Part="1"
+F 0 "C354" V 2788 2600 60  0000 C CNN
 F 1 "100nF" V 2894 2600 60  0000 C CNN
 F 2 "" H 3075 2600 60  0000 C CNN
@@
 	3625 2600 3625 2550
 $Comp
-L power:GND #PWR0537
+L power:GND #PWR0589
 U 1 1 82641BF1
 P 2600 4275
-AR Path="/82611AC0/82641637/82641BF1" Ref="#PWR0537"  Part="1"
-AR Path="/831A25D1/82641BF1" Ref="#PWR0593"  Part="1"
-AR Path="/5D50CA86/82641BF1" Ref="#PWR0606"  Part="1"
-F 0 "#PWR0606" H 2600 4275 30  0001 C CNN
+AR Path="/82611AC0/82641637/82641BF1" Ref="#PWR0589"  Part="1"
+AR Path="/831A25D1/82641BF1" Ref="#PWR0645"  Part="1"
+AR Path="/5D50CA86/82641BF1" Ref="#PWR0662"  Part="1"
+F 0 "#PWR0662" H 2600 4275 30  0001 C CNN
 F 1 "GND" H 2600 4205 30  0001 C CNN
 F 2 "" H 2600 4275 60  0001 C CNN
@@
 $EndComp
 $Comp
-L power:VCC #PWR0541
+L power:VCC #PWR0593
 U 1 1 82641BF7
 P 3800 4225
-AR Path="/82611AC0/82641637/82641BF7" Ref="#PWR0541"  Part="1"
-AR Path="/831A25D1/82641BF7" Ref="#PWR0597"  Part="1"
-AR Path="/5D50CA86/82641BF7" Ref="#PWR0610"  Part="1"
-F 0 "#PWR0610" H 3800 4325 30  0001 C CNN
+AR Path="/82611AC0/82641637/82641BF7" Ref="#PWR0593"  Part="1"
+AR Path="/831A25D1/82641BF7" Ref="#PWR0649"  Part="1"
+AR Path="/5D50CA86/82641BF7" Ref="#PWR0666"  Part="1"
+F 0 "#PWR0666" H 3800 4325 30  0001 C CNN
 F 1 "VCC" H 3804 4352 30  0000 C CNN
 F 2 "" H 3800 4225 60  0001 C CNN
@@
 $EndComp
 $Comp
-L spice:C C304
+L spice:C C328
 U 1 1 82641BFD
 P 3250 4275
-AR Path="/82611AC0/82641637/82641BFD" Ref="C304"  Part="1"
-AR Path="/831A25D1/82641BFD" Ref="C324"  Part="1"
-AR Path="/5D50CA86/82641BFD" Ref="C332"  Part="1"
-F 0 "C332" V 2963 4275 60  0000 C CNN
+AR Path="/82611AC0/82641637/82641BFD" Ref="C328"  Part="1"
+AR Path="/831A25D1/82641BFD" Ref="C348"  Part="1"
+AR Path="/5D50CA86/82641BFD" Ref="C356"  Part="1"
+F 0 "C356" V 2963 4275 60  0000 C CNN
 F 1 "100nF" V 3069 4275 60  0000 C CNN
 F 2 "" H 3250 4275 60  0000 C CNN
@@
 	3800 4275 3800 4225
 $Comp
-L power:GND #PWR0536
+L power:GND #PWR0588
 U 1 1 82641CA4
 P 2575 5975
-AR Path="/82611AC0/82641637/82641CA4" Ref="#PWR0536"  Part="1"
-AR Path="/831A25D1/82641CA4" Ref="#PWR0592"  Part="1"
-AR Path="/5D50CA86/82641CA4" Ref="#PWR0605"  Part="1"
-F 0 "#PWR0605" H 2575 5975 30  0001 C CNN
+AR Path="/82611AC0/82641637/82641CA4" Ref="#PWR0588"  Part="1"
+AR Path="/831A25D1/82641CA4" Ref="#PWR0644"  Part="1"
+AR Path="/5D50CA86/82641CA4" Ref="#PWR0661"  Part="1"
+F 0 "#PWR0661" H 2575 5975 30  0001 C CNN
 F 1 "GND" H 2575 5905 30  0001 C CNN
 F 2 "" H 2575 5975 60  0001 C CNN
@@
 $EndComp
 $Comp
-L power:VCC #PWR0540
+L power:VCC #PWR0592
 U 1 1 82641CAA
 P 3775 5925
-AR Path="/82611AC0/82641637/82641CAA" Ref="#PWR0540"  Part="1"
-AR Path="/831A25D1/82641CAA" Ref="#PWR0596"  Part="1"
-AR Path="/5D50CA86/82641CAA" Ref="#PWR0609"  Part="1"
-F 0 "#PWR0609" H 3775 6025 30  0001 C CNN
+AR Path="/82611AC0/82641637/82641CAA" Ref="#PWR0592"  Part="1"
+AR Path="/831A25D1/82641CAA" Ref="#PWR0648"  Part="1"
+AR Path="/5D50CA86/82641CAA" Ref="#PWR0665"  Part="1"
+F 0 "#PWR0665" H 3775 6025 30  0001 C CNN
 F 1 "VCC" H 3779 6052 30  0000 C CNN
 F 2 "" H 3775 5925 60  0001 C CNN
@@
 $EndComp
 $Comp
-L spice:C C303
+L spice:C C327
 U 1 1 82641CB0
 P 3225 5975
-AR Path="/82611AC0/82641637/82641CB0" Ref="C303"  Part="1"
-AR Path="/831A25D1/82641CB0" Ref="C323"  Part="1"
-AR Path="/5D50CA86/82641CB0" Ref="C331"  Part="1"
-F 0 "C331" V 2938 5975 60  0000 C CNN
+AR Path="/82611AC0/82641637/82641CB0" Ref="C327"  Part="1"
+AR Path="/831A25D1/82641CB0" Ref="C347"  Part="1"
+AR Path="/5D50CA86/82641CB0" Ref="C355"  Part="1"
+F 0 "C355" V 2938 5975 60  0000 C CNN
 F 1 "100nF" V 3044 5975 60  0000 C CNN
 F 2 "" H 3225 5975 60  0000 C CNN
@@
 	3775 5975 3775 5925
 $Comp
-L power:GND #PWR0538
+L power:GND #PWR0590
 U 1 1 82641D95
 P 2675 7700
-AR Path="/82611AC0/82641637/82641D95" Ref="#PWR0538"  Part="1"
-AR Path="/831A25D1/82641D95" Ref="#PWR0594"  Part="1"
-AR Path="/5D50CA86/82641D95" Ref="#PWR0607"  Part="1"
-F 0 "#PWR0607" H 2675 7700 30  0001 C CNN
+AR Path="/82611AC0/82641637/82641D95" Ref="#PWR0590"  Part="1"
+AR Path="/831A25D1/82641D95" Ref="#PWR0646"  Part="1"
+AR Path="/5D50CA86/82641D95" Ref="#PWR0663"  Part="1"
+F 0 "#PWR0663" H 2675 7700 30  0001 C CNN
 F 1 "GND" H 2675 7630 30  0001 C CNN
 F 2 "" H 2675 7700 60  0001 C CNN
@@
 $EndComp
 $Comp
-L power:VCC #PWR0542
+L power:VCC #PWR0594
 U 1 1 82641D9B
 P 3875 7650
-AR Path="/82611AC0/82641637/82641D9B" Ref="#PWR0542"  Part="1"
-AR Path="/831A25D1/82641D9B" Ref="#PWR0598"  Part="1"
-AR Path="/5D50CA86/82641D9B" Ref="#PWR0611"  Part="1"
-F 0 "#PWR0611" H 3875 7750 30  0001 C CNN
+AR Path="/82611AC0/82641637/82641D9B" Ref="#PWR0594"  Part="1"
+AR Path="/831A25D1/82641D9B" Ref="#PWR0650"  Part="1"
+AR Path="/5D50CA86/82641D9B" Ref="#PWR0667"  Part="1"
+F 0 "#PWR0667" H 3875 7750 30  0001 C CNN
 F 1 "VCC" H 3879 7777 30  0000 C CNN
 F 2 "" H 3875 7650 60  0001 C CNN
@@
 $EndComp
 $Comp
-L spice:C C305
+L spice:C C329
 U 1 1 82641DA1
 P 3325 7700
-AR Path="/82611AC0/82641637/82641DA1" Ref="C305"  Part="1"
-AR Path="/831A25D1/82641DA1" Ref="C325"  Part="1"
-AR Path="/5D50CA86/82641DA1" Ref="C333"  Part="1"
-F 0 "C333" V 3038 7700 60  0000 C CNN
+AR Path="/82611AC0/82641637/82641DA1" Ref="C329"  Part="1"
+AR Path="/831A25D1/82641DA1" Ref="C349"  Part="1"
+AR Path="/5D50CA86/82641DA1" Ref="C357"  Part="1"
+F 0 "C357" V 3038 7700 60  0000 C CNN
 F 1 "100nF" V 3144 7700 60  0000 C CNN
 F 2 "" H 3325 7700 60  0000 C CNN
