File: 16Bit2-1Mux.sch (KiCad schematic (older format))
At the start: 8 parts, among them U250 74LS157, U251 74LS157, U252 74LS157, U253 74LS157

Commit message: .
Parts:
- renumbered C326 to C118, C327 to C119, C328 to C120, C329 to C121, U250 to U149, U251 to U150, U252 to U151, U253 to U152
Changed lines of the file:
@@
 $Descr A4 11693 8268
 encoding utf-8
-Sheet 80 101
+Sheet 80 75
 Title ""
 Date ""
@@
 $EndDescr
 $Comp
-L 74xx:74LS157 U250
+L 74xx:74LS157 U149
 U 1 1 82641704
 P 3075 1825
-AR Path="/82611AC0/82641637/82641704" Ref="U250"  Part="1"
-AR Path="/831A25D1/82641704" Ref="U270"  Part="1"
-AR Path="/5D50CA86/82641704" Ref="U278"  Part="1"
-F 0 "U278" H 3075 2633 60  0000 C CNN
+AR Path="/82611AC0/82641637/82641704" Ref="U149"  Part="1"
+AR Path="/831A25D1/82641704" Ref="U169"  Part="1"
+AR Path="/5D50CA86/82641704" Ref="U177"  Part="1"
+F 0 "U177" H 3075 2633 60  0000 C CNN
 F 1 "74LS157" H 3075 2527 60  0000 C CNN
 F 2 "" H 3075 1825 60  0001 C CNN
@@
 $EndComp
 $Comp
-L 74xx:74LS157 U251
+L 74xx:74LS157 U150
 U 1 1 826417B3
 P 3125 3500
-AR Path="/82611AC0/82641637/826417B3" Ref="U251"  Part="1"
-AR Path="/831A25D1/826417B3" Ref="U271"  Part="1"
-AR Path="/5D50CA86/826417B3" Ref="U279"  Part="1"
-F 0 "U279" H 3125 4308 60  0000 C CNN
+AR Path="/82611AC0/82641637/826417B3" Ref="U150"  Part="1"
+AR Path="/831A25D1/826417B3" Ref="U170"  Part="1"
+AR Path="/5D50CA86/826417B3" Ref="U178"  Part="1"
+F 0 "U178" H 3125 4308 60  0000 C CNN
 F 1 "74LS157" H 3125 4202 60  0000 C CNN
 F 2 "" H 3125 3500 60  0001 C CNN
@@
 $EndComp
 $Comp
-L 74xx:74LS157 U252
+L 74xx:74LS157 U151
 U 1 1 8264184D
 P 3175 5200
-AR Path="/82611AC0/82641637/8264184D" Ref="U252"  Part="1"
-AR Path="/831A25D1/8264184D" Ref="U272"  Part="1"
-AR Path="/5D50CA86/8264184D" Ref="U280"  Part="1"
-F 0 "U280" H 3175 6008 60  0000 C CNN
+AR Path="/82611AC0/82641637/8264184D" Ref="U151"  Part="1"
+AR Path="/831A25D1/8264184D" Ref="U171"  Part="1"
+AR Path="/5D50CA86/8264184D" Ref="U179"  Part="1"
+F 0 "U179" H 3175 6008 60  0000 C CNN
 F 1 "74LS157" H 3175 5902 60  0000 C CNN
 F 2 "" H 3175 5200 60  0001 C CNN
@@
 $EndComp
 $Comp
-L 74xx:74LS157 U253
+L 74xx:74LS157 U152
 U 1 1 826418D6
 P 3275 6925
-AR Path="/82611AC0/82641637/826418D6" Ref="U253"  Part="1"
-AR Path="/831A25D1/826418D6" Ref="U273"  Part="1"
-AR Path="/5D50CA86/826418D6" Ref="U281"  Part="1"
-F 0 "U281" H 3275 7733 60  0000 C CNN
+AR Path="/82611AC0/82641637/826418D6" Ref="U152"  Part="1"
+AR Path="/831A25D1/826418D6" Ref="U172"  Part="1"
+AR Path="/5D50CA86/826418D6" Ref="U180"  Part="1"
+F 0 "U180" H 3275 7733 60  0000 C CNN
 F 1 "74LS157" H 3275 7627 60  0000 C CNN
 F 2 "" H 3275 6925 60  0001 C CNN
@@
 $EndComp
 $Comp
-L power:GND #PWR0587
+L power:GND #PWR0177
 U 1 1 82641B85
 P 2425 2600
-AR Path="/82611AC0/82641637/82641B85" Ref="#PWR0587"  Part="1"
-AR Path="/831A25D1/82641B85" Ref="#PWR0643"  Part="1"
-AR Path="/5D50CA86/82641B85" Ref="#PWR0660"  Part="1"
-F 0 "#PWR0660" H 2425 2600 30  0001 C CNN
+AR Path="/82611AC0/82641637/82641B85" Ref="#PWR0177"  Part="1"
+AR Path="/831A25D1/82641B85" Ref="#PWR0233"  Part="1"
+AR Path="/5D50CA86/82641B85" Ref="#PWR0250"  Part="1"
+F 0 "#PWR0250" H 2425 2600 30  0001 C CNN
 F 1 "GND" H 2425 2530 30  0001 C CNN
 F 2 "" H 2425 2600 60  0001 C CNN
@@
 $EndComp
 $Comp
-L power:VCC #PWR0591
+L power:VCC #PWR0181
 U 1 1 82641B8B
 P 3625 2550
-AR Path="/82611AC0/82641637/82641B8B" Ref="#PWR0591"  Part="1"
-AR Path="/831A25D1/82641B8B" Ref="#PWR0647"  Part="1"
-AR Path="/5D50CA86/82641B8B" Ref="#PWR0664"  Part="1"
-F 0 "#PWR0664" H 3625 2650 30  0001 C CNN
+AR Path="/82611AC0/82641637/82641B8B" Ref="#PWR0181"  Part="1"
+AR Path="/831A25D1/82641B8B" Ref="#PWR0237"  Part="1"
+AR Path="/5D50CA86/82641B8B" Ref="#PWR0254"  Part="1"
+F 0 "#PWR0254" H 3625 2650 30  0001 C CNN
 F 1 "VCC" H 3629 2677 30  0000 C CNN
 F 2 "" H 3625 2550 60  0001 C CNN
@@
 $EndComp
 $Comp
-L spice:C C326
+L spice:C C118
 U 1 1 82641B91
 P 3075 2600
-AR Path="/82611AC0/82641637/82641B91" Ref="C326"  Part="1"
-AR Path="/831A25D1/82641B91" Ref="C346"  Part="1"
-AR Path="/5D50CA86/82641B91" Ref="C354"  Part="1"
-F 0 "C354" V 2788 2600 60  0000 C CNN
+AR Path="/82611AC0/82641637/82641B91" Ref="C118"  Part="1"
+AR Path="/831A25D1/82641B91" Ref="C138"  Part="1"
+AR Path="/5D50CA86/82641B91" Ref="C146"  Part="1"
+F 0 "C146" V 2788 2600 60  0000 C CNN
 F 1 "100nF" V 2894 2600 60  0000 C CNN
 F 2 "" H 3075 2600 60  0000 C CNN
@@
 	3625 2600 3625 2550
 $Comp
-L power:GND #PWR0589
+L power:GND #PWR0179
 U 1 1 82641BF1
 P 2600 4275
-AR Path="/82611AC0/82641637/82641BF1" Ref="#PWR0589"  Part="1"
-AR Path="/831A25D1/82641BF1" Ref="#PWR0645"  Part="1"
-AR Path="/5D50CA86/82641BF1" Ref="#PWR0662"  Part="1"
-F 0 "#PWR0662" H 2600 4275 30  0001 C CNN
+AR Path="/82611AC0/82641637/82641BF1" Ref="#PWR0179"  Part="1"
+AR Path="/831A25D1/82641BF1" Ref="#PWR0235"  Part="1"
+AR Path="/5D50CA86/82641BF1" Ref="#PWR0252"  Part="1"
+F 0 "#PWR0252" H 2600 4275 30  0001 C CNN
 F 1 "GND" H 2600 4205 30  0001 C CNN
 F 2 "" H 2600 4275 60  0001 C CNN
@@
 $EndComp
 $Comp
-L power:VCC #PWR0593
+L power:VCC #PWR0183
 U 1 1 82641BF7
 P 3800 4225
-AR Path="/82611AC0/82641637/82641BF7" Ref="#PWR0593"  Part="1"
-AR Path="/831A25D1/82641BF7" Ref="#PWR0649"  Part="1"
-AR Path="/5D50CA86/82641BF7" Ref="#PWR0666"  Part="1"
-F 0 "#PWR0666" H 3800 4325 30  0001 C CNN
+AR Path="/82611AC0/82641637/82641BF7" Ref="#PWR0183"  Part="1"
+AR Path="/831A25D1/82641BF7" Ref="#PWR0239"  Part="1"
+AR Path="/5D50CA86/82641BF7" Ref="#PWR0256"  Part="1"
+F 0 "#PWR0256" H 3800 4325 30  0001 C CNN
 F 1 "VCC" H 3804 4352 30  0000 C CNN
 F 2 "" H 3800 4225 60  0001 C CNN
@@
 $EndComp
 $Comp
-L spice:C C328
+L spice:C C120
 U 1 1 82641BFD
 P 3250 4275
-AR Path="/82611AC0/82641637/82641BFD" Ref="C328"  Part="1"
-AR Path="/831A25D1/82641BFD" Ref="C348"  Part="1"
-AR Path="/5D50CA86/82641BFD" Ref="C356"  Part="1"
-F 0 "C356" V 2963 4275 60  0000 C CNN
+AR Path="/82611AC0/82641637/82641BFD" Ref="C120"  Part="1"
+AR Path="/831A25D1/82641BFD" Ref="C140"  Part="1"
+AR Path="/5D50CA86/82641BFD" Ref="C148"  Part="1"
+F 0 "C148" V 2963 4275 60  0000 C CNN
 F 1 "100nF" V 3069 4275 60  0000 C CNN
 F 2 "" H 3250 4275 60  0000 C CNN
@@
 	3800 4275 3800 4225
 $Comp
-L power:GND #PWR0588
+L power:GND #PWR0178
 U 1 1 82641CA4
 P 2575 5975
-AR Path="/82611AC0/82641637/82641CA4" Ref="#PWR0588"  Part="1"
-AR Path="/831A25D1/82641CA4" Ref="#PWR0644"  Part="1"
-AR Path="/5D50CA86/82641CA4" Ref="#PWR0661"  Part="1"
-F 0 "#PWR0661" H 2575 5975 30  0001 C CNN
+AR Path="/82611AC0/82641637/82641CA4" Ref="#PWR0178"  Part="1"
+AR Path="/831A25D1/82641CA4" Ref="#PWR0234"  Part="1"
+AR Path="/5D50CA86/82641CA4" Ref="#PWR0251"  Part="1"
+F 0 "#PWR0251" H 2575 5975 30  0001 C CNN
 F 1 "GND" H 2575 5905 30  0001 C CNN
 F 2 "" H 2575 5975 60  0001 C CNN
@@
 $EndComp
 $Comp
-L power:VCC #PWR0592
+L power:VCC #PWR0182
 U 1 1 82641CAA
 P 3775 5925
-AR Path="/82611AC0/82641637/82641CAA" Ref="#PWR0592"  Part="1"
-AR Path="/831A25D1/82641CAA" Ref="#PWR0648"  Part="1"
-AR Path="/5D50CA86/82641CAA" Ref="#PWR0665"  Part="1"
-F 0 "#PWR0665" H 3775 6025 30  0001 C CNN
+AR Path="/82611AC0/82641637/82641CAA" Ref="#PWR0182"  Part="1"
+AR Path="/831A25D1/82641CAA" Ref="#PWR0238"  Part="1"
+AR Path="/5D50CA86/82641CAA" Ref="#PWR0255"  Part="1"
+F 0 "#PWR0255" H 3775 6025 30  0001 C CNN
 F 1 "VCC" H 3779 6052 30  0000 C CNN
 F 2 "" H 3775 5925 60  0001 C CNN
@@
 $EndComp
 $Comp
-L spice:C C327
+L spice:C C119
 U 1 1 82641CB0
 P 3225 5975
-AR Path="/82611AC0/82641637/82641CB0" Ref="C327"  Part="1"
-AR Path="/831A25D1/82641CB0" Ref="C347"  Part="1"
-AR Path="/5D50CA86/82641CB0" Ref="C355"  Part="1"
-F 0 "C355" V 2938 5975 60  0000 C CNN
+AR Path="/82611AC0/82641637/82641CB0" Ref="C119"  Part="1"
+AR Path="/831A25D1/82641CB0" Ref="C139"  Part="1"
+AR Path="/5D50CA86/82641CB0" Ref="C147"  Part="1"
+F 0 "C147" V 2938 5975 60  0000 C CNN
 F 1 "100nF" V 3044 5975 60  0000 C CNN
 F 2 "" H 3225 5975 60  0000 C CNN
@@
 	3775 5975 3775 5925
 $Comp
-L power:GND #PWR0590
+L power:GND #PWR0180
 U 1 1 82641D95
 P 2675 7700
-AR Path="/82611AC0/82641637/82641D95" Ref="#PWR0590"  Part="1"
-AR Path="/831A25D1/82641D95" Ref="#PWR0646"  Part="1"
-AR Path="/5D50CA86/82641D95" Ref="#PWR0663"  Part="1"
-F 0 "#PWR0663" H 2675 7700 30  0001 C CNN
+AR Path="/82611AC0/82641637/82641D95" Ref="#PWR0180"  Part="1"
+AR Path="/831A25D1/82641D95" Ref="#PWR0236"  Part="1"
+AR Path="/5D50CA86/82641D95" Ref="#PWR0253"  Part="1"
+F 0 "#PWR0253" H 2675 7700 30  0001 C CNN
 F 1 "GND" H 2675 7630 30  0001 C CNN
 F 2 "" H 2675 7700 60  0001 C CNN
@@
 $EndComp
 $Comp
-L power:VCC #PWR0594
+L power:VCC #PWR0184
 U 1 1 82641D9B
 P 3875 7650
-AR Path="/82611AC0/82641637/82641D9B" Ref="#PWR0594"  Part="1"
-AR Path="/831A25D1/82641D9B" Ref="#PWR0650"  Part="1"
-AR Path="/5D50CA86/82641D9B" Ref="#PWR0667"  Part="1"
-F 0 "#PWR0667" H 3875 7750 30  0001 C CNN
+AR Path="/82611AC0/82641637/82641D9B" Ref="#PWR0184"  Part="1"
+AR Path="/831A25D1/82641D9B" Ref="#PWR0240"  Part="1"
+AR Path="/5D50CA86/82641D9B" Ref="#PWR0257"  Part="1"
+F 0 "#PWR0257" H 3875 7750 30  0001 C CNN
 F 1 "VCC" H 3879 7777 30  0000 C CNN
 F 2 "" H 3875 7650 60  0001 C CNN
@@
 $EndComp
 $Comp
-L spice:C C329
+L spice:C C121
 U 1 1 82641DA1
 P 3325 7700
-AR Path="/82611AC0/82641637/82641DA1" Ref="C329"  Part="1"
-AR Path="/831A25D1/82641DA1" Ref="C349"  Part="1"
-AR Path="/5D50CA86/82641DA1" Ref="C357"  Part="1"
-F 0 "C357" V 3038 7700 60  0000 C CNN
+AR Path="/82611AC0/82641637/82641DA1" Ref="C121"  Part="1"
+AR Path="/831A25D1/82641DA1" Ref="C141"  Part="1"
+AR Path="/5D50CA86/82641DA1" Ref="C149"  Part="1"
+F 0 "C149" V 3038 7700 60  0000 C CNN
 F 1 "100nF" V 3144 7700 60  0000 C CNN
 F 2 "" H 3325 7700 60  0000 C CNN
