File: 5-32Decoder.sch (KiCad schematic (older format))
At the start: 46 parts

Commit message: b
Parts:
- gave numbers to parts that had none: 16
Connections:
- wire segments 107 -> 108
- no-connect marks 6 -> 8

Commit message: message
Parts:
- renumbered C361 to C385, C362 to C386, C363 to C387, C364 to C388, C365 to C389, C366 to C390, C367 to C391, C368 to C392, U259 to U325, U259 to U326, U259 to U327, U259 to U328, U260 to U329, U260 to U330, U261 to U331, U260 to U332, U262 to U333, U262 to U334, U263 to U335, U262 to U336, U262 to U337, U264 to U338, U264 to U339, U264 to U340, U265 to U341, U265 to U342, U265 to U343, U266 to U344, U266 to U345, U266 to U346

Commit message: .
Parts:
- renumbered C385 to C169, C386 to C170, C387 to C171, C388 to C172, C389 to C173, C390 to C174, C391 to C175, C392 to C176, U325 to U221, U326 to U222, U327 to U223, U328 to U224, U329 to U225, U330 to U226, U331 to U227, U332 to U228, U333 to U229, U334 to U230, U335 to U231, U336 to U232, U337 to U233, U338 to U234, U339 to U235, U340 to U236, U341 to U237, U342 to U238, U343 to U239, U344 to U240, U345 to U241, U346 to U242

Commit message: .
Parts:
- renumbered U222 to U15, U223 to U15, U221 to U15, U224 to U16, U223 to U16, U225 to U16, U228 to U17, U226 to U17, U229 to U18, U230 to U18, U232 to U18, U232 to U19, U234 to U19, U233 to U19, U235 to U19, U235 to U20, U236 to U20, U227 to U200, U231 to U201, U237 to U51, U238 to U51, U239 to U52, U240 to U52, U241 to U53, U242 to U53
