File: 8Bit3-1MUX.sch (KiCad schematic (older format))
At the start: 8 parts

Commit message: b
Parts:
- gave numbers to parts that had none: 8
Changed lines of the file:
@@
 $Descr A4 11693 8268
 encoding utf-8
-Sheet 88 90
+Sheet 86 92
 Title ""
 Date ""
@@
 Z7
 $Comp
-L 74xx:74LS157 U?
+L 74xx:74LS157 U235
 U 1 1 5E7947E7
 P 2650 1550
-F 0 "U?" H 2650 2358 60  0000 C CNN
+F 0 "U235" H 2650 2358 60  0000 C CNN
 F 1 "74LS157" H 2650 2252 60  0000 C CNN
 F 2 "" H 2650 1550 60  0001 C CNN
@@
 $EndComp
 $Comp
-L 74xx:74LS157 U?
+L 74xx:74LS157 U237
 U 1 1 5E7948A6
 P 5400 1975
-F 0 "U?" H 5400 2783 60  0000 C CNN
+F 0 "U237" H 5400 2783 60  0000 C CNN
 F 1 "74LS157" H 5400 2677 60  0000 C CNN
 F 2 "" H 5400 1975 60  0001 C CNN
@@
 $EndComp
 $Comp
-L pspice:C C?
+L pspice:C C335
 U 1 1 5E794931
 P 2600 650
-F 0 "C?" V 2285 650 50  0000 C CNN
+F 0 "C335" V 2285 650 50  0000 C CNN
 F 1 "100nF" V 2376 650 50  0000 C CNN
 F 2 "" H 2600 650 60  0001 C CNN
@@
 $EndComp
 $Comp
-L power:VCC #PWR?
+L power:VCC #PWR0615
 U 1 1 5E794A79
 P 2850 650
-F 0 "#PWR?" H 2850 750 30  0001 C CNN
+F 0 "#PWR0615" H 2850 750 30  0001 C CNN
 F 1 "VCC" H 2854 777 30  0000 C CNN
 F 2 "" H 2850 650 60  0001 C CNN
@@
 $EndComp
 $Comp
-L power:GND #PWR?
+L power:GND #PWR0613
 U 1 1 5E794AC0
 P 2350 650
-F 0 "#PWR?" H 2350 650 30  0001 C CNN
+F 0 "#PWR0613" H 2350 650 30  0001 C CNN
 F 1 "GND" H 2350 580 30  0001 C CNN
 F 2 "" H 2350 650 60  0001 C CNN
@@
 $EndComp
 $Comp
-L pspice:C C?
+L pspice:C C336
 U 1 1 5E794B20
 P 5425 2975
-F 0 "C?" V 5110 2975 50  0000 C CNN
+F 0 "C336" V 5110 2975 50  0000 C CNN
 F 1 "100nF" V 5201 2975 50  0000 C CNN
 F 2 "" H 5425 2975 60  0001 C CNN
@@
 $EndComp
 $Comp
-L power:VCC #PWR?
+L power:VCC #PWR0618
 U 1 1 5E794B27
 P 5675 2975
-F 0 "#PWR?" H 5675 3075 30  0001 C CNN
+F 0 "#PWR0618" H 5675 3075 30  0001 C CNN
 F 1 "VCC" H 5679 3102 30  0000 C CNN
 F 2 "" H 5675 2975 60  0001 C CNN
@@
 $EndComp
 $Comp
-L power:GND #PWR?
+L power:GND #PWR0616
 U 1 1 5E794B2D
 P 5175 2975
-F 0 "#PWR?" H 5175 2975 30  0001 C CNN
+F 0 "#PWR0616" H 5175 2975 30  0001 C CNN
 F 1 "GND" H 5175 2905 30  0001 C CNN
 F 2 "" H 5175 2975 60  0001 C CNN
@@
 	1250 1750 1900 1750
 $Comp
-L 74xx:74LS157 U?
+L 74xx:74LS157 U236
 U 1 1 5E794ED0
 P 2700 3575
-F 0 "U?" H 2700 4383 60  0000 C CNN
+F 0 "U236" H 2700 4383 60  0000 C CNN
 F 1 "74LS157" H 2700 4277 60  0000 C CNN
 F 2 "" H 2700 3575 60  0001 C CNN
@@
 $EndComp
 $Comp
-L 74xx:74LS157 U?
+L 74xx:74LS157 U238
 U 1 1 5E794ED7
 P 5425 3975
-F 0 "U?" H 5425 4783 60  0000 C CNN
+F 0 "U238" H 5425 4783 60  0000 C CNN
 F 1 "74LS157" H 5425 4677 60  0000 C CNN
 F 2 "" H 5425 3975 60  0001 C CNN
@@
 $EndComp
 $Comp
-L pspice:C C?
+L pspice:C C337
 U 1 1 5E794EE5
 P 5450 4975
-F 0 "C?" V 5135 4975 50  0000 C CNN
+F 0 "C337" V 5135 4975 50  0000 C CNN
 F 1 "100nF" V 5226 4975 50  0000 C CNN
 F 2 "" H 5450 4975 60  0001 C CNN
@@
 $EndComp
 $Comp
-L power:VCC #PWR?
+L power:VCC #PWR0619
 U 1 1 5E794EEC
 P 5700 4975
-F 0 "#PWR?" H 5700 5075 30  0001 C CNN
+F 0 "#PWR0619" H 5700 5075 30  0001 C CNN
 F 1 "VCC" H 5704 5102 30  0000 C CNN
 F 2 "" H 5700 4975 60  0001 C CNN
@@
 $EndComp
 $Comp
-L power:GND #PWR?
+L power:GND #PWR0617
 U 1 1 5E794EF2
 P 5200 4975
-F 0 "#PWR?" H 5200 4975 30  0001 C CNN
+F 0 "#PWR0617" H 5200 4975 30  0001 C CNN
 F 1 "GND" H 5200 4905 30  0001 C CNN
 F 2 "" H 5200 4975 60  0001 C CNN
@@
 	3925 4275 4675 4275
 $Comp
-L pspice:C C?
+L pspice:C C334
 U 1 1 5E7B19D4
 P 2550 4550
-F 0 "C?" V 2235 4550 50  0000 C CNN
+F 0 "C334" V 2235 4550 50  0000 C CNN
 F 1 "100nF" V 2326 4550 50  0000 C CNN
 F 2 "" H 2550 4550 60  0001 C CNN
@@
 $EndComp
 $Comp
-L power:VCC #PWR?
+L power:VCC #PWR0614
 U 1 1 5E7B19DB
 P 2800 4550
-F 0 "#PWR?" H 2800 4650 30  0001 C CNN
+F 0 "#PWR0614" H 2800 4650 30  0001 C CNN
 F 1 "VCC" H 2804 4677 30  0000 C CNN
 F 2 "" H 2800 4550 60  0001 C CNN
@@
 $EndComp
 $Comp
-L power:GND #PWR?
+L power:GND #PWR0612
 U 1 1 5E7B19E1
 P 2300 4550
-F 0 "#PWR?" H 2300 4550 30  0001 C CNN
+F 0 "#PWR0612" H 2300 4550 30  0001 C CNN
 F 1 "GND" H 2300 4480 30  0001 C CNN
 F 2 "" H 2300 4550 60  0001 C CNN

Commit message: message
Parts:
- renumbered C334 to C358, C335 to C359, C336 to C360, C337 to C361, U235 to U282, U236 to U283, U237 to U284, U238 to U285
Changed lines of the file:
@@
 $Descr A4 11693 8268
 encoding utf-8
-Sheet 86 92
+Sheet 86 101
 Title ""
 Date ""
@@
 Z7
 $Comp
-L 74xx:74LS157 U235
+L 74xx:74LS157 U282
 U 1 1 5E7947E7
 P 2650 1550
-F 0 "U235" H 2650 2358 60  0000 C CNN
+F 0 "U282" H 2650 2358 60  0000 C CNN
 F 1 "74LS157" H 2650 2252 60  0000 C CNN
 F 2 "" H 2650 1550 60  0001 C CNN
@@
 $EndComp
 $Comp
-L 74xx:74LS157 U237
+L 74xx:74LS157 U284
 U 1 1 5E7948A6
 P 5400 1975
-F 0 "U237" H 5400 2783 60  0000 C CNN
+F 0 "U284" H 5400 2783 60  0000 C CNN
 F 1 "74LS157" H 5400 2677 60  0000 C CNN
 F 2 "" H 5400 1975 60  0001 C CNN
@@
 $EndComp
 $Comp
-L pspice:C C335
+L pspice:C C359
 U 1 1 5E794931
 P 2600 650
-F 0 "C335" V 2285 650 50  0000 C CNN
+F 0 "C359" V 2285 650 50  0000 C CNN
 F 1 "100nF" V 2376 650 50  0000 C CNN
 F 2 "" H 2600 650 60  0001 C CNN
@@
 $EndComp
 $Comp
-L power:VCC #PWR0615
+L power:VCC #PWR0671
 U 1 1 5E794A79
 P 2850 650
-F 0 "#PWR0615" H 2850 750 30  0001 C CNN
+F 0 "#PWR0671" H 2850 750 30  0001 C CNN
 F 1 "VCC" H 2854 777 30  0000 C CNN
 F 2 "" H 2850 650 60  0001 C CNN
@@
 $EndComp
 $Comp
-L power:GND #PWR0613
+L power:GND #PWR0669
 U 1 1 5E794AC0
 P 2350 650
-F 0 "#PWR0613" H 2350 650 30  0001 C CNN
+F 0 "#PWR0669" H 2350 650 30  0001 C CNN
 F 1 "GND" H 2350 580 30  0001 C CNN
 F 2 "" H 2350 650 60  0001 C CNN
@@
 $EndComp
 $Comp
-L pspice:C C336
+L pspice:C C360
 U 1 1 5E794B20
 P 5425 2975
-F 0 "C336" V 5110 2975 50  0000 C CNN
+F 0 "C360" V 5110 2975 50  0000 C CNN
 F 1 "100nF" V 5201 2975 50  0000 C CNN
 F 2 "" H 5425 2975 60  0001 C CNN
@@
 $EndComp
 $Comp
-L power:VCC #PWR0618
+L power:VCC #PWR0674
 U 1 1 5E794B27
 P 5675 2975
-F 0 "#PWR0618" H 5675 3075 30  0001 C CNN
+F 0 "#PWR0674" H 5675 3075 30  0001 C CNN
 F 1 "VCC" H 5679 3102 30  0000 C CNN
 F 2 "" H 5675 2975 60  0001 C CNN
@@
 $EndComp
 $Comp
-L power:GND #PWR0616
+L power:GND #PWR0672
 U 1 1 5E794B2D
 P 5175 2975
-F 0 "#PWR0616" H 5175 2975 30  0001 C CNN
+F 0 "#PWR0672" H 5175 2975 30  0001 C CNN
 F 1 "GND" H 5175 2905 30  0001 C CNN
 F 2 "" H 5175 2975 60  0001 C CNN
@@
 	1250 1750 1900 1750
 $Comp
-L 74xx:74LS157 U236
+L 74xx:74LS157 U283
 U 1 1 5E794ED0
 P 2700 3575
-F 0 "U236" H 2700 4383 60  0000 C CNN
+F 0 "U283" H 2700 4383 60  0000 C CNN
 F 1 "74LS157" H 2700 4277 60  0000 C CNN
 F 2 "" H 2700 3575 60  0001 C CNN
@@
 $EndComp
 $Comp
-L 74xx:74LS157 U238
+L 74xx:74LS157 U285
 U 1 1 5E794ED7
 P 5425 3975
-F 0 "U238" H 5425 4783 60  0000 C CNN
+F 0 "U285" H 5425 4783 60  0000 C CNN
 F 1 "74LS157" H 5425 4677 60  0000 C CNN
 F 2 "" H 5425 3975 60  0001 C CNN
@@
 $EndComp
 $Comp
-L pspice:C C337
+L pspice:C C361
 U 1 1 5E794EE5
 P 5450 4975
-F 0 "C337" V 5135 4975 50  0000 C CNN
+F 0 "C361" V 5135 4975 50  0000 C CNN
 F 1 "100nF" V 5226 4975 50  0000 C CNN
 F 2 "" H 5450 4975 60  0001 C CNN
@@
 $EndComp
 $Comp
-L power:VCC #PWR0619
+L power:VCC #PWR0675
 U 1 1 5E794EEC
 P 5700 4975
-F 0 "#PWR0619" H 5700 5075 30  0001 C CNN
+F 0 "#PWR0675" H 5700 5075 30  0001 C CNN
 F 1 "VCC" H 5704 5102 30  0000 C CNN
 F 2 "" H 5700 4975 60  0001 C CNN
@@
 $EndComp
 $Comp
-L power:GND #PWR0617
+L power:GND #PWR0673
 U 1 1 5E794EF2
 P 5200 4975
-F 0 "#PWR0617" H 5200 4975 30  0001 C CNN
+F 0 "#PWR0673" H 5200 4975 30  0001 C CNN
 F 1 "GND" H 5200 4905 30  0001 C CNN
 F 2 "" H 5200 4975 60  0001 C CNN
@@
 	3925 4275 4675 4275
 $Comp
-L pspice:C C334
+L pspice:C C358
 U 1 1 5E7B19D4
 P 2550 4550
-F 0 "C334" V 2235 4550 50  0000 C CNN
+F 0 "C358" V 2235 4550 50  0000 C CNN
 F 1 "100nF" V 2326 4550 50  0000 C CNN
 F 2 "" H 2550 4550 60  0001 C CNN
@@
 $EndComp
 $Comp
-L power:VCC #PWR0614
+L power:VCC #PWR0670
 U 1 1 5E7B19DB
 P 2800 4550
-F 0 "#PWR0614" H 2800 4650 30  0001 C CNN
+F 0 "#PWR0670" H 2800 4650 30  0001 C CNN
 F 1 "VCC" H 2804 4677 30  0000 C CNN
 F 2 "" H 2800 4550 60  0001 C CNN
@@
 $EndComp
 $Comp
-L power:GND #PWR0612
+L power:GND #PWR0668
 U 1 1 5E7B19E1
 P 2300 4550
-F 0 "#PWR0612" H 2300 4550 30  0001 C CNN
+F 0 "#PWR0668" H 2300 4550 30  0001 C CNN
 F 1 "GND" H 2300 4480 30  0001 C CNN
 F 2 "" H 2300 4550 60  0001 C CNN

Commit message: .
Parts:
- renumbered C358 to C150, C359 to C151, C360 to C152, C361 to C153, U282 to U181, U283 to U182, U284 to U183, U285 to U184
Connections:
- wire segments 102 -> 124
Changed lines of the file:
@@
 $Descr A4 11693 8268
 encoding utf-8
-Sheet 86 101
+Sheet 95 75
 Title ""
 Date ""
@@
 Comment4 ""
 $EndDescr
-Text HLabel 875  1000 2    59   Input ~ 0
+Text HLabel 875  1000 0    59   Input ~ 0
 X0
-Text HLabel 875  1100 2    59   Input ~ 0
+Text HLabel 875  1100 0    59   Input ~ 0
 X1
-Text HLabel 875  1200 2    59   Input ~ 0
+Text HLabel 875  1200 0    59   Input ~ 0
 X2
-Text HLabel 875  1300 2    59   Input ~ 0
+Text HLabel 875  1300 0    59   Input ~ 0
 X3
-Text HLabel 1650 3025 2    59   Input ~ 0
+Text HLabel 1650 3025 0    59   Input ~ 0
 X4
-Text HLabel 1650 3125 2    59   Input ~ 0
+Text HLabel 1650 3125 0    59   Input ~ 0
 X5
-Text HLabel 1650 3225 2    59   Input ~ 0
+Text HLabel 1650 3225 0    59   Input ~ 0
 X6
-Text HLabel 1650 3325 2    59   Input ~ 0
+Text HLabel 1650 3325 0    59   Input ~ 0
 X7
-Text HLabel 575  1050 2    59   Input ~ 0
+Text HLabel 650  1050 0    59   Input ~ 0
 Y0
-Text HLabel 575  1150 2    59   Input ~ 0
+Text HLabel 650  1150 0    59   Input ~ 0
 Y1
-Text HLabel 575  1250 2    59   Input ~ 0
+Text HLabel 675  1250 0    59   Input ~ 0
 Y2
-Text HLabel 575  1350 2    59   Input ~ 0
+Text HLabel 675  1350 0    59   Input ~ 0
 Y3
-Text HLabel 1275 3100 2    59   Input ~ 0
+Text HLabel 1275 3100 0    59   Input ~ 0
 Y4
-Text HLabel 1275 3200 2    59   Input ~ 0
+Text HLabel 1275 3200 0    59   Input ~ 0
 Y5
-Text HLabel 1275 3300 2    59   Input ~ 0
+Text HLabel 1275 3300 0    59   Input ~ 0
 Y6
-Text HLabel 1275 3400 2    59   Input ~ 0
+Text HLabel 1275 3400 0    59   Input ~ 0
 Y7
 Text HLabel 3975 1575 2    59   Input ~ 0
@@
 Text HLabel 6475 1950 2    59   Output ~ 0
 Z3
-Text HLabel 6475 2050 2    59   Output ~ 0
+Text HLabel 6700 3675 2    59   Output ~ 0
 Z4
-Text HLabel 6475 2150 2    59   Output ~ 0
+Text HLabel 6700 3775 2    59   Output ~ 0
 Z5
-Text HLabel 6475 2250 2    59   Output ~ 0
+Text HLabel 6700 3875 2    59   Output ~ 0
 Z6
-Text HLabel 6475 2350 2    59   Output ~ 0
+Text HLabel 6700 3975 2    59   Output ~ 0
 Z7
 $Comp
-L 74xx:74LS157 U282
+L 74xx:74LS157 U181
 U 1 1 5E7947E7
 P 2650 1550
-F 0 "U282" H 2650 2358 60  0000 C CNN
+F 0 "U181" H 2650 2358 60  0000 C CNN
 F 1 "74LS157" H 2650 2252 60  0000 C CNN
 F 2 "" H 2650 1550 60  0001 C CNN
@@
 $EndComp
 $Comp
-L 74xx:74LS157 U284
+L 74xx:74LS157 U183
 U 1 1 5E7948A6
 P 5400 1975
-F 0 "U284" H 5400 2783 60  0000 C CNN
+F 0 "U183" H 5400 2783 60  0000 C CNN
 F 1 "74LS157" H 5400 2677 60  0000 C CNN
 F 2 "" H 5400 1975 60  0001 C CNN
@@
 $EndComp
 $Comp
-L pspice:C C359
+L pspice:C C151
 U 1 1 5E794931
 P 2600 650
-F 0 "C359" V 2285 650 50  0000 C CNN
+F 0 "C151" V 2285 650 50  0000 C CNN
 F 1 "100nF" V 2376 650 50  0000 C CNN
 F 2 "" H 2600 650 60  0001 C CNN
@@
 $EndComp
 $Comp
-L power:VCC #PWR0671
+L power:VCC #PWR0261
 U 1 1 5E794A79
 P 2850 650
-F 0 "#PWR0671" H 2850 750 30  0001 C CNN
+F 0 "#PWR0261" H 2850 750 30  0001 C CNN
 F 1 "VCC" H 2854 777 30  0000 C CNN
 F 2 "" H 2850 650 60  0001 C CNN
@@
 $EndComp
 $Comp
-L power:GND #PWR0669
+L power:GND #PWR0259
 U 1 1 5E794AC0
 P 2350 650
-F 0 "#PWR0669" H 2350 650 30  0001 C CNN
+F 0 "#PWR0259" H 2350 650 30  0001 C CNN
 F 1 "GND" H 2350 580 30  0001 C CNN
 F 2 "" H 2350 650 60  0001 C CNN
@@
 $EndComp
 $Comp
-L pspice:C C360
+L pspice:C C152
 U 1 1 5E794B20
 P 5425 2975
-F 0 "C360" V 5110 2975 50  0000 C CNN
+F 0 "C152" V 5110 2975 50  0000 C CNN
 F 1 "100nF" V 5201 2975 50  0000 C CNN
 F 2 "" H 5425 2975 60  0001 C CNN
@@
 $EndComp
 $Comp
-L power:VCC #PWR0674
+L power:VCC #PWR0264
 U 1 1 5E794B27
 P 5675 2975
-F 0 "#PWR0674" H 5675 3075 30  0001 C CNN
+F 0 "#PWR0264" H 5675 3075 30  0001 C CNN
 F 1 "VCC" H 5679 3102 30  0000 C CNN
 F 2 "" H 5675 2975 60  0001 C CNN
@@
 $EndComp
 $Comp
-L power:GND #PWR0672
+L power:GND #PWR0262
 U 1 1 5E794B2D
 P 5175 2975
-F 0 "#PWR0672" H 5175 2975 30  0001 C CNN
+F 0 "#PWR0262" H 5175 2975 30  0001 C CNN
 F 1 "GND" H 5175 2905 30  0001 C CNN
 F 2 "" H 5175 2975 60  0001 C CNN
@@
 	1250 1750 1900 1750
 $Comp
-L 74xx:74LS157 U283
+L 74xx:74LS157 U182
 U 1 1 5E794ED0
 P 2700 3575
-F 0 "U283" H 2700 4383 60  0000 C CNN
+F 0 "U182" H 2700 4383 60  0000 C CNN
 F 1 "74LS157" H 2700 4277 60  0000 C CNN
 F 2 "" H 2700 3575 60  0001 C CNN
@@
 $EndComp
 $Comp
-L 74xx:74LS157 U285
+L 74xx:74LS157 U184
 U 1 1 5E794ED7
 P 5425 3975
-F 0 "U285" H 5425 4783 60  0000 C CNN
+F 0 "U184" H 5425 4783 60  0000 C CNN
 F 1 "74LS157" H 5425 4677 60  0000 C CNN
 F 2 "" H 5425 3975 60  0001 C CNN
@@
 $EndComp
 $Comp
-L pspice:C C361
+L pspice:C C153
 U 1 1 5E794EE5
 P 5450 4975
-F 0 "C361" V 5135 4975 50  0000 C CNN
+F 0 "C153" V 5135 4975 50  0000 C CNN
 F 1 "100nF" V 5226 4975 50  0000 C CNN
 F 2 "" H 5450 4975 60  0001 C CNN
@@
 $EndComp
 $Comp
-L power:VCC #PWR0675
+L power:VCC #PWR0265
 U 1 1 5E794EEC
 P 5700 4975
-F 0 "#PWR0675" H 5700 5075 30  0001 C CNN
+F 0 "#PWR0265" H 5700 5075 30  0001 C CNN
 F 1 "VCC" H 5704 5102 30  0000 C CNN
 F 2 "" H 5700 4975 60  0001 C CNN
@@
 $EndComp
 $Comp
-L power:GND #PWR0673
+L power:GND #PWR0263
 U 1 1 5E794EF2
 P 5200 4975
-F 0 "#PWR0673" H 5200 4975 30  0001 C CNN
+F 0 "#PWR0263" H 5200 4975 30  0001 C CNN
 F 1 "GND" H 5200 4905 30  0001 C CNN
 F 2 "" H 5200 4975 60  0001 C CNN
@@
 	1250 1300 1250 1750
 Wire Wire Line
-	575  1050 1900 1050
+	650  1050 1900 1050
 Wire Wire Line
 	1900 1050 1900 1100
 Wire Wire Line
-	575  1150 1550 1150
+	650  1150 1550 1150
 Wire Wire Line
 	1550 1150 1550 1350
@@
 	1550 1350 1900 1350
 Wire Wire Line
-	600  1250 1325 1250
-Wire Wire Line
 	1325 1250 1325 1600
 Wire Wire Line
 	1325 1600 1900 1600
 Wire Wire Line
-	575  1350 1075 1350
+	675  1350 1075 1350
 Wire Wire Line
 	1075 1350 1075 1850
@@
 	3925 4275 4675 4275
 $Comp
-L pspice:C C358
+L pspice:C C150
 U 1 1 5E7B19D4
 P 2550 4550
-F 0 "C358" V 2235 4550 50  0000 C CNN
+F 0 "C150" V 2235 4550 50  0000 C CNN
 F 1 "100nF" V 2326 4550 50  0000 C CNN
 F 2 "" H 2550 4550 60  0001 C CNN
@@
 $EndComp
 $Comp
-L power:VCC #PWR0670
+L power:VCC #PWR0260
 U 1 1 5E7B19DB
 P 2800 4550
-F 0 "#PWR0670" H 2800 4650 30  0001 C CNN
+F 0 "#PWR0260" H 2800 4650 30  0001 C CNN
 F 1 "VCC" H 2804 4677 30  0000 C CNN
 F 2 "" H 2800 4550 60  0001 C CNN
@@
 $EndComp
 $Comp
-L power:GND #PWR0668
+L power:GND #PWR0258
 U 1 1 5E7B19E1
 P 2300 4550
-F 0 "#PWR0668" H 2300 4550 30  0001 C CNN
+F 0 "#PWR0258" H 2300 4550 30  0001 C CNN
 F 1 "GND" H 2300 4480 30  0001 C CNN
 F 2 "" H 2300 4550 60  0001 C CNN
@@
 Text Label 750  2450 0    59   ~ 0
 S1
+Wire Wire Line
+	675  1250 1325 1250
+Wire Wire Line
+	6150 1475 6425 1475
+Wire Wire Line
+	6425 1475 6425 1650
+Wire Wire Line
+	6425 1650 6475 1650
+Wire Wire Line
+	6475 1750 6150 1750
+Wire Wire Line
+	6150 1750 6150 1725
+Wire Wire Line
+	6475 1850 6150 1850
+Wire Wire Line
+	6150 1850 6150 1975
+Wire Wire Line
+	6475 1950 6350 1950
+Wire Wire Line
+	6350 1950 6350 2225
+Wire Wire Line
+	6350 2225 6150 2225
+Wire Wire Line
+	6700 3675 6325 3675
+Wire Wire Line
+	6325 3675 6325 3475
+Wire Wire Line
+	6325 3475 6175 3475
+Wire Wire Line
+	6675 3725 6675 3775
+Wire Wire Line
+	6675 3775 6700 3775
+Wire Wire Line
+	6175 3725 6675 3725
+Wire Wire Line
+	6175 3975 6500 3975
+Wire Wire Line
+	6500 3975 6500 3875
+Wire Wire Line
+	6500 3875 6700 3875
+Wire Wire Line
+	6700 3975 6550 3975
+Wire Wire Line
+	6550 3975 6550 4225
+Wire Wire Line
+	6550 4225 6175 4225
 $EndSCHEMATC

Commit message: .
Changed lines of the file:
@@
 $Descr A4 11693 8268
 encoding utf-8
-Sheet 95 75
+Sheet 95 100
 Title ""
 Date ""
@@
 Text HLabel 1275 3400 0    59   Input ~ 0
 Y7
-Text HLabel 3975 1575 2    59   Input ~ 0
+Text HLabel 3975 1575 0    59   Input ~ 0
 W0
-Text HLabel 3975 1675 2    59   Input ~ 0
+Text HLabel 3975 1675 0    59   Input ~ 0
 W1
-Text HLabel 3975 1775 2    59   Input ~ 0
+Text HLabel 3975 1775 0    59   Input ~ 0
 W2
-Text HLabel 3975 1875 2    59   Input ~ 0
+Text HLabel 3975 1875 0    59   Input ~ 0
 W3
-Text HLabel 3925 3350 2    59   Input ~ 0
+Text HLabel 3925 3350 0    59   Input ~ 0
 W4
-Text HLabel 3925 3450 2    59   Input ~ 0
+Text HLabel 3925 3450 0    59   Input ~ 0
 W5
-Text HLabel 3925 3550 2    59   Input ~ 0
+Text HLabel 3925 3550 0    59   Input ~ 0
 W6
-Text HLabel 3925 3650 2    59   Input ~ 0
+Text HLabel 3925 3650 0    59   Input ~ 0
 W7
 Text HLabel 6475 1650 2    59   Output ~ 0
