File: AdressReg.sch (KiCad schematic (older format))
At the start: 2 parts

Commit message: X
Parts:
- added C?: 100nF, symbol spice:C
- added U?: 74LS04, symbol 74xx:74LS04
Connections:
- net labels added: ENABLE
- wire segments 434 -> 432
Other:
- moved on the sheet: C?

Commit message: b
Parts:
- gave numbers to parts that had none: 4
Changed lines of the file:
@@
 $Descr A2 23386 16535
 encoding utf-8
-Sheet 58 90
+Sheet 58 92
 Title ""
 Date ""
@@
 	5450 5450 5525 5450
 $Comp
-L 74xx:74LS155 U?
+L 74xx:74LS155 U150
 U 1 1 81235F00
 P 3125 3475
-F 0 "U?" H 3125 4133 60  0000 C CNN
+F 0 "U150" H 3125 4133 60  0000 C CNN
 F 1 "74LS155" H 3125 4027 60  0000 C CNN
 F 2 "" H 3125 3475 60  0001 C CNN
@@
 $EndComp
 $Comp
-L power:VCC #PWR?
+L power:VCC #PWR0352
 U 1 1 812B1ACA
 P 2900 4300
-F 0 "#PWR?" H 2900 4400 30  0001 C CNN
+F 0 "#PWR0352" H 2900 4400 30  0001 C CNN
 F 1 "VCC" H 2904 4427 30  0000 C CNN
 F 2 "" H 2900 4300 60  0001 C CNN
@@
 $EndComp
 $Comp
-L power:GND #PWR?
+L power:GND #PWR0353
 U 1 1 812B1AF6
 P 3400 4300
-F 0 "#PWR?" H 3400 4300 30  0001 C CNN
+F 0 "#PWR0353" H 3400 4300 30  0001 C CNN
 F 1 "GND" H 3400 4230 30  0001 C CNN
 F 2 "" H 3400 4300 60  0001 C CNN
@@
 $EndComp
 $Comp
-L spice:C C?
+L spice:C C209
 U 1 1 812B1B42
 P 3150 4300
-F 0 "C?" V 2863 4300 60  0000 C CNN
+F 0 "C209" V 2863 4300 60  0000 C CNN
 F 1 "100nF" V 2969 4300 60  0000 C CNN
 F 2 "" H 3150 4300 60  0000 C CNN
@@
 	12125 6475 12475 6475
 $Comp
-L 74xx:74LS04 U?
+L 74xx:74LS04 U149
 U 1 1 5D22A95E
 P 1925 3250
-F 0 "U?" H 1925 3587 60  0000 C CNN
+F 0 "U149" H 1925 3587 60  0000 C CNN
 F 1 "74LS04" H 1925 3481 60  0000 C CNN
 F 2 "" H 1925 3250 60  0001 C CNN
@@
 ENABLE
 $Comp
-L power:VCC #PWR?
+L power:VCC #PWR0350
 U 1 1 5D25ADDB
 P 1500 3600
-F 0 "#PWR?" H 1500 3700 30  0001 C CNN
+F 0 "#PWR0350" H 1500 3700 30  0001 C CNN
 F 1 "VCC" H 1504 3727 30  0000 C CNN
 F 2 "" H 1500 3600 60  0001 C CNN
@@
 $EndComp
 $Comp
-L power:GND #PWR?
+L power:GND #PWR0351
 U 1 1 5D25ADE1
 P 2000 3600
-F 0 "#PWR?" H 2000 3600 30  0001 C CNN
+F 0 "#PWR0351" H 2000 3600 30  0001 C CNN
 F 1 "GND" H 2000 3530 30  0001 C CNN
 F 2 "" H 2000 3600 60  0001 C CNN
@@
 $EndComp
 $Comp
-L spice:C C?
+L spice:C C208
 U 1 1 5D25ADE7
 P 1750 3600
-F 0 "C?" V 1463 3600 60  0000 C CNN
+F 0 "C208" V 1463 3600 60  0000 C CNN
 F 1 "100nF" V 1569 3600 60  0000 C CNN
 F 2 "" H 1750 3600 60  0000 C CNN

Commit message: message
Parts:
- renumbered C208 to C232, C209 to C233, U149 to U196, U150 to U197
Changed lines of the file:
@@
 $Descr A2 23386 16535
 encoding utf-8
-Sheet 59 92
+Sheet 59 101
 Title ""
 Date ""
@@
 	5450 5450 5525 5450
 $Comp
-L 74xx:74LS155 U150
+L 74xx:74LS155 U197
 U 1 1 81235F00
 P 3125 3475
-F 0 "U150" H 3125 4133 60  0000 C CNN
+F 0 "U197" H 3125 4133 60  0000 C CNN
 F 1 "74LS155" H 3125 4027 60  0000 C CNN
 F 2 "" H 3125 3475 60  0001 C CNN
@@
 $EndComp
 $Comp
-L power:VCC #PWR0352
+L power:VCC #PWR0400
 U 1 1 812B1ACA
 P 2900 4300
-F 0 "#PWR0352" H 2900 4400 30  0001 C CNN
+F 0 "#PWR0400" H 2900 4400 30  0001 C CNN
 F 1 "VCC" H 2904 4427 30  0000 C CNN
 F 2 "" H 2900 4300 60  0001 C CNN
@@
 $EndComp
 $Comp
-L power:GND #PWR0353
+L power:GND #PWR0401
 U 1 1 812B1AF6
 P 3400 4300
-F 0 "#PWR0353" H 3400 4300 30  0001 C CNN
+F 0 "#PWR0401" H 3400 4300 30  0001 C CNN
 F 1 "GND" H 3400 4230 30  0001 C CNN
 F 2 "" H 3400 4300 60  0001 C CNN
@@
 $EndComp
 $Comp
-L spice:C C209
+L spice:C C233
 U 1 1 812B1B42
 P 3150 4300
-F 0 "C209" V 2863 4300 60  0000 C CNN
+F 0 "C233" V 2863 4300 60  0000 C CNN
 F 1 "100nF" V 2969 4300 60  0000 C CNN
 F 2 "" H 3150 4300 60  0000 C CNN
@@
 	12125 6475 12475 6475
 $Comp
-L 74xx:74LS04 U149
+L 74xx:74LS04 U196
 U 1 1 5D22A95E
 P 1925 3250
-F 0 "U149" H 1925 3587 60  0000 C CNN
+F 0 "U196" H 1925 3587 60  0000 C CNN
 F 1 "74LS04" H 1925 3481 60  0000 C CNN
 F 2 "" H 1925 3250 60  0001 C CNN
@@
 ENABLE
 $Comp
-L power:VCC #PWR0350
+L power:VCC #PWR0398
 U 1 1 5D25ADDB
 P 1500 3600
-F 0 "#PWR0350" H 1500 3700 30  0001 C CNN
+F 0 "#PWR0398" H 1500 3700 30  0001 C CNN
 F 1 "VCC" H 1504 3727 30  0000 C CNN
 F 2 "" H 1500 3600 60  0001 C CNN
@@
 $EndComp
 $Comp
-L power:GND #PWR0351
+L power:GND #PWR0399
 U 1 1 5D25ADE1
 P 2000 3600
-F 0 "#PWR0351" H 2000 3600 30  0001 C CNN
+F 0 "#PWR0399" H 2000 3600 30  0001 C CNN
 F 1 "GND" H 2000 3530 30  0001 C CNN
 F 2 "" H 2000 3600 60  0001 C CNN
@@
 $EndComp
 $Comp
-L spice:C C208
+L spice:C C232
 U 1 1 5D25ADE7
 P 1750 3600
-F 0 "C208" V 1463 3600 60  0000 C CNN
+F 0 "C232" V 1463 3600 60  0000 C CNN
 F 1 "100nF" V 1569 3600 60  0000 C CNN
 F 2 "" H 1750 3600 60  0000 C CNN

Commit message: .
Parts:
- renumbered C232 to C104, C233 to C105, U196 to U135, U197 to U136
Changed lines of the file:
@@
 $Descr A2 23386 16535
 encoding utf-8
-Sheet 59 101
+Sheet 52 75
 Title ""
 Date ""
@@
 	5450 5450 5525 5450
 $Comp
-L 74xx:74LS155 U197
+L 74xx:74LS155 U136
 U 1 1 81235F00
 P 3125 3475
-F 0 "U197" H 3125 4133 60  0000 C CNN
+F 0 "U136" H 3125 4133 60  0000 C CNN
 F 1 "74LS155" H 3125 4027 60  0000 C CNN
 F 2 "" H 3125 3475 60  0001 C CNN
@@
 $EndComp
 $Comp
-L power:VCC #PWR0400
+L power:VCC #PWR0150
 U 1 1 812B1ACA
 P 2900 4300
-F 0 "#PWR0400" H 2900 4400 30  0001 C CNN
+F 0 "#PWR0150" H 2900 4400 30  0001 C CNN
 F 1 "VCC" H 2904 4427 30  0000 C CNN
 F 2 "" H 2900 4300 60  0001 C CNN
@@
 $EndComp
 $Comp
-L power:GND #PWR0401
+L power:GND #PWR0151
 U 1 1 812B1AF6
 P 3400 4300
-F 0 "#PWR0401" H 3400 4300 30  0001 C CNN
+F 0 "#PWR0151" H 3400 4300 30  0001 C CNN
 F 1 "GND" H 3400 4230 30  0001 C CNN
 F 2 "" H 3400 4300 60  0001 C CNN
@@
 $EndComp
 $Comp
-L spice:C C233
+L spice:C C105
 U 1 1 812B1B42
 P 3150 4300
-F 0 "C233" V 2863 4300 60  0000 C CNN
+F 0 "C105" V 2863 4300 60  0000 C CNN
 F 1 "100nF" V 2969 4300 60  0000 C CNN
 F 2 "" H 3150 4300 60  0000 C CNN
@@
 	12125 6475 12475 6475
 $Comp
-L 74xx:74LS04 U196
+L 74xx:74LS04 U135
 U 1 1 5D22A95E
 P 1925 3250
-F 0 "U196" H 1925 3587 60  0000 C CNN
+F 0 "U135" H 1925 3587 60  0000 C CNN
 F 1 "74LS04" H 1925 3481 60  0000 C CNN
 F 2 "" H 1925 3250 60  0001 C CNN
@@
 ENABLE
 $Comp
-L power:VCC #PWR0398
+L power:VCC #PWR0148
 U 1 1 5D25ADDB
 P 1500 3600
-F 0 "#PWR0398" H 1500 3700 30  0001 C CNN
+F 0 "#PWR0148" H 1500 3700 30  0001 C CNN
 F 1 "VCC" H 1504 3727 30  0000 C CNN
 F 2 "" H 1500 3600 60  0001 C CNN
@@
 $EndComp
 $Comp
-L power:GND #PWR0399
+L power:GND #PWR0149
 U 1 1 5D25ADE1
 P 2000 3600
-F 0 "#PWR0399" H 2000 3600 30  0001 C CNN
+F 0 "#PWR0149" H 2000 3600 30  0001 C CNN
 F 1 "GND" H 2000 3530 30  0001 C CNN
 F 2 "" H 2000 3600 60  0001 C CNN
@@
 $EndComp
 $Comp
-L spice:C C232
+L spice:C C104
 U 1 1 5D25ADE7
 P 1750 3600
-F 0 "C232" V 1463 3600 60  0000 C CNN
+F 0 "C104" V 1463 3600 60  0000 C CNN
 F 1 "100nF" V 1569 3600 60  0000 C CNN
 F 2 "" H 1750 3600 60  0000 C CNN
