File: CALL_SELECTOR.sch (KiCad schematic (older format))
At the start: 4 parts, among them U244 74LS08, U245 4071

Commit message: message
Parts:
- renumbered C347 to C371, C348 to C372, U244 to U291, U244 to U292, U245 to U293, U245 to U294, U245 to U295
Changed lines of the file:
@@
 $Descr A4 11693 8268
 encoding utf-8
-Sheet 90 92
+Sheet 90 101
 Title ""
 Date ""
@@
 CARRY_S
 $Comp
-L 74xx:74LS08 U244
+L 74xx:74LS08 U292
 U 3 1 5B492A08
 P 1950 2025
-F 0 "U244" H 1950 2413 60  0000 C CNN
+F 0 "U292" H 1950 2413 60  0000 C CNN
 F 1 "74LS08" H 1950 2307 60  0000 C CNN
 F 2 "" H 1950 2025 60  0001 C CNN
@@
 $EndComp
 $Comp
-L 74xx:74LS08 U244
+L 74xx:74LS08 U292
 U 2 1 5B492A9A
 P 1925 2450
-F 0 "U244" H 1925 2838 60  0000 C CNN
+F 0 "U292" H 1925 2838 60  0000 C CNN
 F 1 "74LS08" H 1925 2732 60  0000 C CNN
 F 2 "" H 1925 2450 60  0001 C CNN
@@
 $EndComp
 $Comp
-L 74xx:74LS08 U244
+L 74xx:74LS08 U292
 U 4 1 5B492B0D
 P 5700 2325
-F 0 "U244" H 5700 2713 60  0000 C CNN
+F 0 "U292" H 5700 2713 60  0000 C CNN
 F 1 "74LS08" H 5700 2607 60  0000 C CNN
 F 2 "" H 5700 2325 60  0001 C CNN
@@
 $EndComp
 $Comp
-L 74xx:74LS08 U244
+L 74xx:74LS08 U291
 U 1 1 5B492B76
 P 1275 4275
-F 0 "U244" H 1275 4663 60  0000 C CNN
+F 0 "U291" H 1275 4663 60  0000 C CNN
 F 1 "74LS08" H 1275 4557 60  0000 C CNN
 F 2 "" H 1275 4275 60  0001 C CNN
@@
 	1350 1900 1350 1925
 $Comp
-L cmos4000:4071 U245
+L cmos4000:4071 U295
 U 4 1 5B492D06
 P 4500 2425
-F 0 "U245" H 4500 2813 60  0000 C CNN
+F 0 "U295" H 4500 2813 60  0000 C CNN
 F 1 "4071" H 4500 2707 60  0000 C CNN
 F 2 "" H 4500 2425 60  0001 C CNN
@@
 $EndComp
 $Comp
-L cmos4000:4071 U245
+L cmos4000:4071 U293
 U 1 1 5B492DBB
 P 3300 2325
-F 0 "U245" H 3300 2713 60  0000 C CNN
+F 0 "U293" H 3300 2713 60  0000 C CNN
 F 1 "4071" H 3300 2607 60  0000 C CNN
 F 2 "" H 3300 2325 60  0001 C CNN
@@
 	5100 1875 5100 2225
 $Comp
-L cmos4000:4071 U245
+L cmos4000:4071 U295
 U 3 1 5B4931E1
 P 3475 4400
-F 0 "U245" H 3475 4788 60  0000 C CNN
+F 0 "U295" H 3475 4788 60  0000 C CNN
 F 1 "4071" H 3475 4682 60  0000 C CNN
 F 2 "" H 3475 4400 60  0001 C CNN
@@
 $EndComp
 $Comp
-L cmos4000:4071 U245
+L cmos4000:4071 U294
 U 2 1 5B493251
 P 3375 5225
-F 0 "U245" H 3375 5613 60  0000 C CNN
+F 0 "U294" H 3375 5613 60  0000 C CNN
 F 1 "4071" H 3375 5507 60  0000 C CNN
 F 2 "" H 3375 5225 60  0001 C CNN
@@
 $EndComp
 $Comp
-L power:GND #PWR0638
+L power:GND #PWR0694
 U 1 1 5B4932E7
 P 1225 5125
-F 0 "#PWR0638" H 1225 5125 30  0001 C CNN
+F 0 "#PWR0694" H 1225 5125 30  0001 C CNN
 F 1 "GND" H 1225 5055 30  0001 C CNN
 F 2 "" H 1225 5125 60  0001 C CNN
@@
 $EndComp
 $Comp
-L myCpu-rescue:VCC #PWR0639
+L myCpu-rescue:VCC #PWR0695
 U 1 1 5B493336
 P 1725 5125
-F 0 "#PWR0639" H 1725 4975 50  0001 C CNN
+F 0 "#PWR0695" H 1725 4975 50  0001 C CNN
 F 1 "VCC" H 1742 5298 50  0000 C CNN
 F 2 "" H 1725 5125 50  0000 C CNN
@@
 $EndComp
 $Comp
-L pspice:C C347
+L pspice:C C371
 U 1 1 5B493385
 P 1475 5125
-F 0 "C347" V 1160 5125 50  0000 C CNN
+F 0 "C371" V 1160 5125 50  0000 C CNN
 F 1 "100nF" V 1251 5125 50  0000 C CNN
 F 2 "" H 1475 5125 60  0001 C CNN
@@
 $EndComp
 $Comp
-L power:GND #PWR0640
+L power:GND #PWR0696
 U 1 1 5B49352F
 P 3225 5800
-F 0 "#PWR0640" H 3225 5800 30  0001 C CNN
+F 0 "#PWR0696" H 3225 5800 30  0001 C CNN
 F 1 "GND" H 3225 5730 30  0001 C CNN
 F 2 "" H 3225 5800 60  0001 C CNN
@@
 $EndComp
 $Comp
-L myCpu-rescue:VCC #PWR0641
+L myCpu-rescue:VCC #PWR0697
 U 1 1 5B493535
 P 3725 5800
-F 0 "#PWR0641" H 3725 5650 50  0001 C CNN
+F 0 "#PWR0697" H 3725 5650 50  0001 C CNN
 F 1 "VCC" H 3742 5973 50  0000 C CNN
 F 2 "" H 3725 5800 50  0000 C CNN
@@
 $EndComp
 $Comp
-L pspice:C C348
+L pspice:C C372
 U 1 1 5B49353B
 P 3475 5800
-F 0 "C348" V 3160 5800 50  0000 C CNN
+F 0 "C372" V 3160 5800 50  0000 C CNN
 F 1 "100nF" V 3251 5800 50  0000 C CNN
 F 2 "" H 3475 5800 60  0001 C CNN

Commit message: .
Parts:
- renumbered C371 to C154, C372 to C155, U291 to U185, U292 to U186, U293 to U187, U294 to U188, U295 to U189
Connections:
- wire segments 29 -> 28
- no-connect marks 2 -> 3
Other:
- moved on the sheet: C154, U188B
Changed lines of the file:
@@
 $Descr A4 11693 8268
 encoding utf-8
-Sheet 90 101
+Sheet 98 75
 Title ""
 Date ""
@@
 CARRY_S
 $Comp
-L 74xx:74LS08 U292
+L 74xx:74LS08 U186
 U 3 1 5B492A08
 P 1950 2025
-F 0 "U292" H 1950 2413 60  0000 C CNN
+F 0 "U186" H 1950 2413 60  0000 C CNN
 F 1 "74LS08" H 1950 2307 60  0000 C CNN
 F 2 "" H 1950 2025 60  0001 C CNN
@@
 $EndComp
 $Comp
-L 74xx:74LS08 U292
+L 74xx:74LS08 U186
 U 2 1 5B492A9A
 P 1925 2450
-F 0 "U292" H 1925 2838 60  0000 C CNN
+F 0 "U186" H 1925 2838 60  0000 C CNN
 F 1 "74LS08" H 1925 2732 60  0000 C CNN
 F 2 "" H 1925 2450 60  0001 C CNN
@@
 $EndComp
 $Comp
-L 74xx:74LS08 U292
+L 74xx:74LS08 U186
 U 4 1 5B492B0D
 P 5700 2325
-F 0 "U292" H 5700 2713 60  0000 C CNN
+F 0 "U186" H 5700 2713 60  0000 C CNN
 F 1 "74LS08" H 5700 2607 60  0000 C CNN
 F 2 "" H 5700 2325 60  0001 C CNN
@@
 $EndComp
 $Comp
-L 74xx:74LS08 U291
+L 74xx:74LS08 U185
 U 1 1 5B492B76
 P 1275 4275
-F 0 "U291" H 1275 4663 60  0000 C CNN
+F 0 "U185" H 1275 4663 60  0000 C CNN
 F 1 "74LS08" H 1275 4557 60  0000 C CNN
 F 2 "" H 1275 4275 60  0001 C CNN
@@
 	1350 1900 1350 1925
 $Comp
-L cmos4000:4071 U295
+L cmos4000:4071 U189
 U 4 1 5B492D06
 P 4500 2425
-F 0 "U295" H 4500 2813 60  0000 C CNN
+F 0 "U189" H 4500 2813 60  0000 C CNN
 F 1 "4071" H 4500 2707 60  0000 C CNN
 F 2 "" H 4500 2425 60  0001 C CNN
@@
 $EndComp
 $Comp
-L cmos4000:4071 U293
+L cmos4000:4071 U187
 U 1 1 5B492DBB
 P 3300 2325
-F 0 "U293" H 3300 2713 60  0000 C CNN
+F 0 "U187" H 3300 2713 60  0000 C CNN
 F 1 "4071" H 3300 2607 60  0000 C CNN
 F 2 "" H 3300 2325 60  0001 C CNN
@@
 	5100 1875 5100 2225
 $Comp
-L cmos4000:4071 U295
+L cmos4000:4071 U189
 U 3 1 5B4931E1
 P 3475 4400
-F 0 "U295" H 3475 4788 60  0000 C CNN
+F 0 "U189" H 3475 4788 60  0000 C CNN
 F 1 "4071" H 3475 4682 60  0000 C CNN
 F 2 "" H 3475 4400 60  0001 C CNN
@@
 $EndComp
 $Comp
-L cmos4000:4071 U294
-U 2 1 5B493251
-P 3375 5225
-F 0 "U294" H 3375 5613 60  0000 C CNN
-F 1 "4071" H 3375 5507 60  0000 C CNN
-F 2 "" H 3375 5225 60  0001 C CNN
-F 3 "" H 3375 5225 60  0001 C CNN
-	2    3375 5225
-	1    0    0    -1
-$EndComp
-$Comp
-L power:GND #PWR0694
+L power:GND #PWR0266
 U 1 1 5B4932E7
-P 1225 5125
-F 0 "#PWR0694" H 1225 5125 30  0001 C CNN
-F 1 "GND" H 1225 5055 30  0001 C CNN
-F 2 "" H 1225 5125 60  0001 C CNN
-F 3 "" H 1225 5125 60  0001 C CNN
-	1    1225 5125
-	1    0    0    -1
-$EndComp
-$Comp
-L myCpu-rescue:VCC #PWR0695
+P 1250 5125
+F 0 "#PWR0266" H 1250 5125 30  0001 C CNN
+F 1 "GND" H 1250 5055 30  0001 C CNN
+F 2 "" H 1250 5125 60  0001 C CNN
+F 3 "" H 1250 5125 60  0001 C CNN
+	1    1250 5125
+	1    0    0    -1
+$EndComp
+$Comp
+L myCpu-rescue:VCC #PWR0267
 U 1 1 5B493336
-P 1725 5125
-F 0 "#PWR0695" H 1725 4975 50  0001 C CNN
-F 1 "VCC" H 1742 5298 50  0000 C CNN
-F 2 "" H 1725 5125 50  0000 C CNN
-F 3 "" H 1725 5125 50  0000 C CNN
-	1    1725 5125
-	1    0    0    -1
-$EndComp
-$Comp
-L pspice:C C371
+P 1750 5125
+F 0 "#PWR0267" H 1750 4975 50  0001 C CNN
+F 1 "VCC" H 1767 5298 50  0000 C CNN
+F 2 "" H 1750 5125 50  0000 C CNN
+F 3 "" H 1750 5125 50  0000 C CNN
+	1    1750 5125
+	1    0    0    -1
+$EndComp
+$Comp
+L pspice:C C154
 U 1 1 5B493385
-P 1475 5125
-F 0 "C371" V 1160 5125 50  0000 C CNN
-F 1 "100nF" V 1251 5125 50  0000 C CNN
-F 2 "" H 1475 5125 60  0001 C CNN
-F 3 "" H 1475 5125 60  0001 C CNN
-	1    1475 5125
+P 1500 5125
+F 0 "C154" V 1185 5125 50  0000 C CNN
+F 1 "100nF" V 1276 5125 50  0000 C CNN
+F 2 "" H 1500 5125 60  0001 C CNN
+F 3 "" H 1500 5125 60  0001 C CNN
+	1    1500 5125
 	0    1    1    0
 $EndComp
 $Comp
-L power:GND #PWR0696
+L power:GND #PWR0268
 U 1 1 5B49352F
 P 3225 5800
-F 0 "#PWR0696" H 3225 5800 30  0001 C CNN
+F 0 "#PWR0268" H 3225 5800 30  0001 C CNN
 F 1 "GND" H 3225 5730 30  0001 C CNN
 F 2 "" H 3225 5800 60  0001 C CNN
@@
 $EndComp
 $Comp
-L myCpu-rescue:VCC #PWR0697
+L myCpu-rescue:VCC #PWR0269
 U 1 1 5B493535
 P 3725 5800
-F 0 "#PWR0697" H 3725 5650 50  0001 C CNN
+F 0 "#PWR0269" H 3725 5650 50  0001 C CNN
 F 1 "VCC" H 3742 5973 50  0000 C CNN
 F 2 "" H 3725 5800 50  0000 C CNN
@@
 $EndComp
 $Comp
-L pspice:C C372
+L pspice:C C155
 U 1 1 5B49353B
 P 3475 5800
-F 0 "C372" V 3160 5800 50  0000 C CNN
+F 0 "C155" V 3160 5800 50  0000 C CNN
 F 1 "100nF" V 3251 5800 50  0000 C CNN
 F 2 "" H 3475 5800 60  0001 C CNN
@@
 	2875 4900 2775 4900
 Wire Wire Line
-	2775 4900 2775 5125
+	2775 4900 2750 5075
 Connection ~ 2875 4500
 Wire Wire Line
-	2800 5125 2775 5125
-Wire Wire Line
-	2775 5125 2775 5325
-Connection ~ 2775 5125
-Wire Wire Line
-	3250 5800 3250 5425
-Wire Wire Line
-	3250 5425 3975 5425
-Wire Wire Line
-	3975 5425 3975 5225
+	2750 5075 2750 5275
 NoConn ~ 4075 4400
 NoConn ~ 1875 4275
 Text HLabel 6300 2325 2    60   Output ~ 0
 CALL_ENABLE
+Connection ~ 2750 5075
+$Comp
+L cmos4000:4071 U188
+U 2 1 5B493251
+P 3350 5175
+F 0 "U188" H 3350 5563 60  0000 C CNN
+F 1 "4071" H 3350 5457 60  0000 C CNN
+F 2 "" H 3350 5175 60  0001 C CNN
+F 3 "" H 3350 5175 60  0001 C CNN
+	2    3350 5175
+	1    0    0    -1
+$EndComp
+NoConn ~ 3950 5175
+Wire Wire Line
+	3225 5800 3225 5625
+Wire Wire Line
+	3225 5625 2750 5625
+Wire Wire Line
+	2750 5625 2750 5275
+Connection ~ 3225 5800
+Connection ~ 2750 5275
+Connection ~ 1250 5125
 $EndSCHEMATC

Commit message: .
Parts:
- renumbered C154 to C167, C155 to C168, U186 to U1, U185 to U1, U189 to U199, U187 to U199, U188 to U199, U186 to U2
Changed lines of the file:
@@
 $Descr A4 11693 8268
 encoding utf-8
-Sheet 98 75
+Sheet 98 100
 Title ""
 Date ""
@@
 CARRY_S
 $Comp
-L 74xx:74LS08 U186
-U 3 1 5B492A08
+L 74xx:74LS08 U2
+U 1 1 5B492A08
 P 1950 2025
-F 0 "U186" H 1950 2413 60  0000 C CNN
+F 0 "U2" H 1950 2413 60  0000 C CNN
 F 1 "74LS08" H 1950 2307 60  0000 C CNN
 F 2 "" H 1950 2025 60  0001 C CNN
 F 3 "" H 1950 2025 60  0001 C CNN
-	3    1950 2025
-	1    0    0    -1
-$EndComp
-$Comp
-L 74xx:74LS08 U186
-U 2 1 5B492A9A
+	1    1950 2025
+	1    0    0    -1
+$EndComp
+$Comp
+L 74xx:74LS08 U1
+U 4 1 5B492A9A
 P 1925 2450
-F 0 "U186" H 1925 2838 60  0000 C CNN
+F 0 "U1" H 1925 2838 60  0000 C CNN
 F 1 "74LS08" H 1925 2732 60  0000 C CNN
 F 2 "" H 1925 2450 60  0001 C CNN
 F 3 "" H 1925 2450 60  0001 C CNN
-	2    1925 2450
-	1    0    0    -1
-$EndComp
-$Comp
-L 74xx:74LS08 U186
-U 4 1 5B492B0D
+	4    1925 2450
+	1    0    0    -1
+$EndComp
+$Comp
+L 74xx:74LS08 U2
+U 2 1 5B492B0D
 P 5700 2325
-F 0 "U186" H 5700 2713 60  0000 C CNN
+F 0 "U2" H 5700 2713 60  0000 C CNN
 F 1 "74LS08" H 5700 2607 60  0000 C CNN
 F 2 "" H 5700 2325 60  0001 C CNN
 F 3 "" H 5700 2325 60  0001 C CNN
-	4    5700 2325
-	1    0    0    -1
-$EndComp
-$Comp
-L 74xx:74LS08 U185
-U 1 1 5B492B76
+	2    5700 2325
+	1    0    0    -1
+$EndComp
+$Comp
+L 74xx:74LS08 U1
+U 3 1 5B492B76
 P 1275 4275
-F 0 "U185" H 1275 4663 60  0000 C CNN
+F 0 "U1" H 1275 4663 60  0000 C CNN
 F 1 "74LS08" H 1275 4557 60  0000 C CNN
 F 2 "" H 1275 4275 60  0001 C CNN
 F 3 "" H 1275 4275 60  0001 C CNN
-	1    1275 4275
+	3    1275 4275
 	1    0    0    -1
 $EndComp
@@
 	1350 1900 1350 1925
 $Comp
-L cmos4000:4071 U189
+L cmos4000:4071 U199
 U 4 1 5B492D06
 P 4500 2425
-F 0 "U189" H 4500 2813 60  0000 C CNN
+F 0 "U199" H 4500 2813 60  0000 C CNN
 F 1 "4071" H 4500 2707 60  0000 C CNN
 F 2 "" H 4500 2425 60  0001 C CNN
@@
 $EndComp
 $Comp
-L cmos4000:4071 U187
+L cmos4000:4071 U199
 U 1 1 5B492DBB
 P 3300 2325
-F 0 "U187" H 3300 2713 60  0000 C CNN
+F 0 "U199" H 3300 2713 60  0000 C CNN
 F 1 "4071" H 3300 2607 60  0000 C CNN
 F 2 "" H 3300 2325 60  0001 C CNN
@@
 	5100 1875 5100 2225
 $Comp
-L cmos4000:4071 U189
+L cmos4000:4071 U199
 U 3 1 5B4931E1
 P 3475 4400
-F 0 "U189" H 3475 4788 60  0000 C CNN
+F 0 "U199" H 3475 4788 60  0000 C CNN
 F 1 "4071" H 3475 4682 60  0000 C CNN
 F 2 "" H 3475 4400 60  0001 C CNN
@@
 $EndComp
 $Comp
-L power:GND #PWR0266
+L power:GND #PWR0292
 U 1 1 5B4932E7
 P 1250 5125
-F 0 "#PWR0266" H 1250 5125 30  0001 C CNN
+F 0 "#PWR0292" H 1250 5125 30  0001 C CNN
 F 1 "GND" H 1250 5055 30  0001 C CNN
 F 2 "" H 1250 5125 60  0001 C CNN
@@
 $EndComp
 $Comp
-L myCpu-rescue:VCC #PWR0267
+L myCpu-rescue:VCC #PWR0293
 U 1 1 5B493336
 P 1750 5125
-F 0 "#PWR0267" H 1750 4975 50  0001 C CNN
+F 0 "#PWR0293" H 1750 4975 50  0001 C CNN
 F 1 "VCC" H 1767 5298 50  0000 C CNN
 F 2 "" H 1750 5125 50  0000 C CNN
@@
 $EndComp
 $Comp
-L pspice:C C154
+L pspice:C C167
 U 1 1 5B493385
 P 1500 5125
-F 0 "C154" V 1185 5125 50  0000 C CNN
+F 0 "C167" V 1185 5125 50  0000 C CNN
 F 1 "100nF" V 1276 5125 50  0000 C CNN
 F 2 "" H 1500 5125 60  0001 C CNN
@@
 $EndComp
 $Comp
-L power:GND #PWR0268
+L power:GND #PWR0294
 U 1 1 5B49352F
 P 3225 5800
-F 0 "#PWR0268" H 3225 5800 30  0001 C CNN
+F 0 "#PWR0294" H 3225 5800 30  0001 C CNN
 F 1 "GND" H 3225 5730 30  0001 C CNN
 F 2 "" H 3225 5800 60  0001 C CNN
@@
 $EndComp
 $Comp
-L myCpu-rescue:VCC #PWR0269
+L myCpu-rescue:VCC #PWR0295
 U 1 1 5B493535
 P 3725 5800
-F 0 "#PWR0269" H 3725 5650 50  0001 C CNN
+F 0 "#PWR0295" H 3725 5650 50  0001 C CNN
 F 1 "VCC" H 3742 5973 50  0000 C CNN
 F 2 "" H 3725 5800 50  0000 C CNN
@@
 $EndComp
 $Comp
-L pspice:C C155
+L pspice:C C168
 U 1 1 5B49353B
 P 3475 5800
-F 0 "C155" V 3160 5800 50  0000 C CNN
+F 0 "C168" V 3160 5800 50  0000 C CNN
 F 1 "100nF" V 3251 5800 50  0000 C CNN
 F 2 "" H 3475 5800 60  0001 C CNN
@@
 Connection ~ 2750 5075
 $Comp
-L cmos4000:4071 U188
+L cmos4000:4071 U199
 U 2 1 5B493251
 P 3350 5175
-F 0 "U188" H 3350 5563 60  0000 C CNN
+F 0 "U199" H 3350 5563 60  0000 C CNN
 F 1 "4071" H 3350 5457 60  0000 C CNN
 F 2 "" H 3350 5175 60  0001 C CNN
