File: CarryShifter.sch (KiCad schematic (older format))
At the start: 3 parts

Commit message: .
Parts:
- gave numbers to parts that had none: 3
Changed lines of the file:
@@
 $Descr A4 11693 8268
 encoding utf-8
-Sheet 32 101
+Sheet 32 75
 Title ""
 Date ""
@@
 Z7
 $Comp
-L 74xx:74LS157 U?
+L 74xx:74LS157 U87
 U 1 1 5B1FC2A5
 P 3125 1425
-F 0 "U?" H 3125 2233 60  0000 C CNN
+F 0 "U87" H 3125 2233 60  0000 C CNN
 F 1 "74LS157" H 3125 2127 60  0000 C CNN
 F 2 "" H 3125 1425 60  0001 C CNN
@@
 $EndComp
 $Comp
-L 74xx:74LS157 U?
+L 74xx:74LS157 U88
 U 1 1 5B1FC316
 P 3125 2775
-F 0 "U?" H 3125 3583 60  0000 C CNN
+F 0 "U88" H 3125 3583 60  0000 C CNN
 F 1 "74LS157" H 3125 3477 60  0000 C CNN
 F 2 "" H 3125 2775 60  0001 C CNN
@@
 $EndComp
 $Comp
-L 74xx:74LS157 U?
+L 74xx:74LS157 U86
 U 1 1 5B1FC3B1
 P 3100 4200
-F 0 "U?" H 3100 5008 60  0000 C CNN
+F 0 "U86" H 3100 5008 60  0000 C CNN
 F 1 "74LS157" H 3100 4902 60  0000 C CNN
 F 2 "" H 3100 4200 60  0001 C CNN
@@
 S
 $Comp
-L power:GND #PWR?
+L power:GND #PWR0109
 U 1 1 5B20A36D
 P 2225 2075
-F 0 "#PWR?" H 2225 2075 30  0001 C CNN
+F 0 "#PWR0109" H 2225 2075 30  0001 C CNN
 F 1 "GND" H 2225 2005 30  0001 C CNN
 F 2 "" H 2225 2075 60  0001 C CNN
@@
 $EndComp
 $Comp
-L power:GND #PWR?
+L power:GND #PWR0108
 U 1 1 5B20A38D
 P 2200 3375
-F 0 "#PWR?" H 2200 3375 30  0001 C CNN
+F 0 "#PWR0108" H 2200 3375 30  0001 C CNN
 F 1 "GND" H 2200 3305 30  0001 C CNN
 F 2 "" H 2200 3375 60  0001 C CNN
@@
 $EndComp
 $Comp
-L power:GND #PWR?
+L power:GND #PWR0107
 U 1 1 5B20B7ED
 P 2125 4775
-F 0 "#PWR?" H 2125 4775 30  0001 C CNN
+F 0 "#PWR0107" H 2125 4775 30  0001 C CNN
 F 1 "GND" H 2125 4705 30  0001 C CNN
 F 2 "" H 2125 4775 60  0001 C CNN
