File: DEC.sch (KiCad schematic (older format))
At the start: 4 parts, among them U12 74LS283, U13 74LS283

Commit message: b
Parts:
- renumbered C10 to C12, C11 to C13, U12 to U14, U13 to U15
Changed lines of the file:
@@
 $Descr A4 11693 8268
 encoding utf-8
-Sheet 8 90
+Sheet 8 92
 Title ""
 Date ""
@@
 Z7
 $Comp
-L myCpu-rescue:74LS283 U12
+L myCpu-rescue:74LS283 U14
 U 1 1 5AE75C93
 P 3050 4250
-F 0 "U12" H 3050 4250 50  0000 C CNN
+F 0 "U14" H 3050 4250 50  0000 C CNN
 F 1 "74LS283" H 3100 3900 50  0000 C CNN
 F 2 "" H 3050 4250 50  0000 C CNN
@@
 $EndComp
 $Comp
-L myCpu-rescue:74LS283 U13
+L myCpu-rescue:74LS283 U15
 U 1 1 5AE75D41
 P 4625 4350
-F 0 "U13" H 4625 4350 50  0000 C CNN
+F 0 "U15" H 4625 4350 50  0000 C CNN
 F 1 "74LS283" H 4675 4000 50  0000 C CNN
 F 2 "" H 4625 4350 50  0000 C CNN
@@
 	4625 3100 4625 3650
 $Comp
-L myCpu-rescue:VCC #PWR015
+L myCpu-rescue:VCC #PWR022
 U 1 1 5AE760F6
 P 3375 5400
-F 0 "#PWR015" H 3375 5250 50  0001 C CNN
+F 0 "#PWR022" H 3375 5250 50  0001 C CNN
 F 1 "VCC" H 3375 5550 50  0000 C CNN
 F 2 "" H 3375 5400 50  0000 C CNN
@@
 $EndComp
 $Comp
-L myCpu-rescue:VCC #PWR016
+L myCpu-rescue:VCC #PWR023
 U 1 1 5AE7610E
 P 4925 5400
-F 0 "#PWR016" H 4925 5250 50  0001 C CNN
+F 0 "#PWR023" H 4925 5250 50  0001 C CNN
 F 1 "VCC" H 4925 5550 50  0000 C CNN
 F 2 "" H 4925 5400 50  0000 C CNN
@@
 	5075 5050 5025 5050
 $Comp
-L myCpu-rescue:VCC #PWR014
+L myCpu-rescue:VCC #PWR021
 U 1 1 5AE7639B
 P 2075 3750
-F 0 "#PWR014" H 2075 3600 50  0001 C CNN
+F 0 "#PWR021" H 2075 3600 50  0001 C CNN
 F 1 "VCC" H 2075 3900 50  0000 C CNN
 F 2 "" H 2075 3750 50  0000 C CNN
@@
 	2400 4950 2600 4950
 $Comp
-L spice:C C10
+L spice:C C12
 U 1 1 5AEBFB4F
 P 2075 4000
-F 0 "C10" V 1925 4000 60  0000 C CNN
+F 0 "C12" V 1925 4000 60  0000 C CNN
 F 1 "100nF" V 2225 4000 60  0000 C CNN
 F 2 "" H 2075 4000 60  0000 C CNN
@@
 $EndComp
 $Comp
-L spice:C C11
+L spice:C C13
 U 1 1 5AEBFBCE
 P 5475 5100
-F 0 "C11" V 5325 5100 60  0000 C CNN
+F 0 "C13" V 5325 5100 60  0000 C CNN
 F 1 "100nF" V 5625 5100 60  0000 C CNN
 F 2 "" H 5475 5100 60  0000 C CNN
@@
 $EndComp
 $Comp
-L spice:0 #GND17
+L spice:0 #GND14
 U 1 1 5AEBFC3B
 P 5500 4525
-F 0 "#GND17" H 5500 4425 60  0001 C CNN
+F 0 "#GND14" H 5500 4425 60  0001 C CNN
 F 1 "0" H 5500 4455 60  0000 C CNN
 F 2 "" H 5500 4525 60  0000 C CNN
@@
 $EndComp
 $Comp
-L spice:0 #GND16
+L spice:0 #GND13
 U 1 1 5AEBFC57
 P 2125 4525
-F 0 "#GND16" H 2125 4425 60  0001 C CNN
+F 0 "#GND13" H 2125 4425 60  0001 C CNN
 F 1 "0" H 2125 4455 60  0000 C CNN
 F 2 "" H 2125 4525 60  0000 C CNN

Commit message: message
Parts:
- renumbered U14 to U27, U15 to U28
Changed lines of the file:
@@
 $Descr A4 11693 8268
 encoding utf-8
-Sheet 8 92
+Sheet 8 101
 Title ""
 Date ""
@@
 Z7
 $Comp
-L myCpu-rescue:74LS283 U14
+L myCpu-rescue:74LS283 U27
 U 1 1 5AE75C93
 P 3050 4250
-F 0 "U14" H 3050 4250 50  0000 C CNN
+F 0 "U27" H 3050 4250 50  0000 C CNN
 F 1 "74LS283" H 3100 3900 50  0000 C CNN
 F 2 "" H 3050 4250 50  0000 C CNN
@@
 $EndComp
 $Comp
-L myCpu-rescue:74LS283 U15
+L myCpu-rescue:74LS283 U28
 U 1 1 5AE75D41
 P 4625 4350
-F 0 "U15" H 4625 4350 50  0000 C CNN
+F 0 "U28" H 4625 4350 50  0000 C CNN
 F 1 "74LS283" H 4675 4000 50  0000 C CNN
 F 2 "" H 4625 4350 50  0000 C CNN
@@
 	4625 3100 4625 3650
 $Comp
-L myCpu-rescue:VCC #PWR022
+L myCpu-rescue:VCC #PWR028
 U 1 1 5AE760F6
 P 3375 5400
-F 0 "#PWR022" H 3375 5250 50  0001 C CNN
+F 0 "#PWR028" H 3375 5250 50  0001 C CNN
 F 1 "VCC" H 3375 5550 50  0000 C CNN
 F 2 "" H 3375 5400 50  0000 C CNN
@@
 $EndComp
 $Comp
-L myCpu-rescue:VCC #PWR023
+L myCpu-rescue:VCC #PWR029
 U 1 1 5AE7610E
 P 4925 5400
-F 0 "#PWR023" H 4925 5250 50  0001 C CNN
+F 0 "#PWR029" H 4925 5250 50  0001 C CNN
 F 1 "VCC" H 4925 5550 50  0000 C CNN
 F 2 "" H 4925 5400 50  0000 C CNN
@@
 	5075 5050 5025 5050
 $Comp
-L myCpu-rescue:VCC #PWR021
+L myCpu-rescue:VCC #PWR027
 U 1 1 5AE7639B
 P 2075 3750
-F 0 "#PWR021" H 2075 3600 50  0001 C CNN
+F 0 "#PWR027" H 2075 3600 50  0001 C CNN
 F 1 "VCC" H 2075 3900 50  0000 C CNN
 F 2 "" H 2075 3750 50  0000 C CNN
@@
 $EndComp
 $Comp
-L spice:0 #GND14
+L spice:0 #GND9
 U 1 1 5AEBFC3B
 P 5500 4525
-F 0 "#GND14" H 5500 4425 60  0001 C CNN
+F 0 "#GND9" H 5500 4425 60  0001 C CNN
 F 1 "0" H 5500 4455 60  0000 C CNN
 F 2 "" H 5500 4525 60  0000 C CNN
@@
 $EndComp
 $Comp
-L spice:0 #GND13
+L spice:0 #GND8
 U 1 1 5AEBFC57
 P 2125 4525
-F 0 "#GND13" H 2125 4425 60  0001 C CNN
+F 0 "#GND8" H 2125 4425 60  0001 C CNN
 F 1 "0" H 2125 4455 60  0000 C CNN
 F 2 "" H 2125 4525 60  0000 C CNN
