File: DECODER.sch (KiCad schematic (older format))
At the start: 0 parts

Commit message: X
Parts:
- added C? (x9): 100nF, symbol pspice:C
- added U? (x4): 74LS32, symbol 74xx:74LS32
- added U? (x2): 4002, symbol cmos4000:4002
- added U? (x4): 74LS08, symbol 74xx:74LS08
- added U? (x28): 4071, symbol cmos4000:4071
Connections:
- net labels added: ADD, ADDC, ADDR_REG_ENABLE, ADDR_X_S0, ADDR_X_S1, ADDR_Z_S0, ADDR_Z_S1, ALU_S0, ALU_S0_W0, ALU_S0_W1, ALU_S0_W2, ALU_S1, ALU_S1_W0, ALU_S2, ALU_S2_W0, ALU_S3, AND, CALL, CALLC, CALLZ, CARRY, CARRY_S, DEC, GND, IM0, IM1, IM2, IM3, IM4, IM5, IM6, IM7, INC, INCADDR, IN_0, IN_1, JMP, JMPC, JMPZ, LADDR, LOAD, LSL, LSLC, LSR, LSRC, MOV, NOP, NOT, OR, PC-INC, PCSTACK, READ, REG_CLK_ENABLE, RET, RX_S0, RX_S1, RX_S2, RX_S3, RY_S0, RY_S1, RY_S2, RY_S3, RZ_S0, RZ_S1, RZ_S2, RZ_S3, SLL, SLLC, SLR, SLRC, SUB, SUBC, UNCOND, VCC, WRITE, XOR, ZFLAG_S
- net labels removed: ADDR16
- wire segments 0 -> 175

Commit message: b
Parts:
- removed U? (x4): 74LS08, symbol 74xx:74LS08
- added unit 2 of U255
- added unit 3 of U255
- added unit 3 of U256
- added unit 2 of U256
- gave numbers to parts that had none: 19
Connections:
- net labels added: CMP
- net labels removed: LSL, LSLC, LSR, LSRC, PC-INC, PCSTACK
- wire segments 175 -> 170
- no-connect marks 0 -> 5
Other:
- moved on the sheet: C355

Commit message: tst
Connections:
- net labels added: ALU_S3_W0
Changed lines of the file:
@@
 ALU_S3
 Text Label 6750 13525 2    59   ~ 0
-ALU_S3
+ALU_S3_W0
 Text Label 13700 6700 2    59   ~ 0
-ALU_S3
+ALU_S3_W0
 Text Label 4875 11225 2    59   ~ 0
 ALU_S0_W0

Commit message: fixed errors
Connections:
- net labels added: CALL_ANY, JMP_ANY
Changed lines of the file:
@@
 NoConn ~ 6475 7475
 Text HLabel 8950 8425 3    60   Output ~ 0
-CALL
+CALL_ANY
 Text HLabel 7650 6725 3    60   Output ~ 0
 RET
 Text HLabel 10525 8375 3    60   Output ~ 0
-JMP
+JMP_ANY
 $Comp
 L cmos4000:4071 U255

Commit message: message
Parts:
- added C?: 100nF, symbol pspice:C
- added U? (x4): 74LS32, symbol 74xx:74LS32
- renumbered C352 to C376, C353 to C377, C354 to C378, C355 to C379, C356 to C380, C357 to C381, C358 to C382, C359 to C383, C360 to C384, U249 to U304, U250 to U305, U249 to U306, U250 to U307, U251 to U308, U251 to U309, U252 to U310, U252 to U311, U253 to U312, U254 to U313, U254 to U314, U254 to U315, U255 to U316, U255 to U317, U256 to U318, U256 to U319, U256 to U320, U257 to U321, U257 to U322, U258 to U323, U258 to U324
Connections:
- wire segments 170 -> 194
- no-connect marks 5 -> 4
Other:
- moved on the sheet: C382

Commit message: .
Parts:
- gave numbers to parts that had none: 3
- renumbered C376 to C159, C377 to C160, C378 to C161, C379 to C162, C380 to C163, C381 to C164, C382 to C166, C383 to C167, C384 to C168, U304 to U198, U305 to U199, U306 to U200, U307 to U201, U308 to U202, U309 to U203, U310 to U204, U311 to U205, U312 to U206, U313 to U207, U314 to U208, U315 to U209, U316 to U210, U317 to U211, U318 to U214, U319 to U215, U320 to U216, U321 to U217, U322 to U218, U323 to U219, U324 to U220

Commit message: .
Parts:
- renumbered C159 to C154, C160 to C155, C161 to C159, C162 to C160, C163 to C161, C164 to C162, C165 to C163, C166 to C164, C167 to C165, C168 to C166, U199 to U11, U201 to U12, U202 to U13, U203 to U14, U206 to U185, U207 to U186, U208 to U186, U209 to U186, U211 to U187, U210 to U187, U216 to U188, U215 to U188, U214 to U188, U218 to U189, U217 to U189, U204 to U192, U205 to U192, U205 to U194, U219 to U198, U220 to U198, U198 to U3, U200 to U4, U212 to U5, U213 to U6
