File: NOT.sch (KiCad schematic (older format))
At the start: 2 parts, among them U6 4069, U7 4069

Commit message: b
Parts:
- renumbered U6 to U8, U7 to U9
Connections:
- net labels added: GND, VDD, VSS
- wire segments 50 -> 51
Changed lines of the file:
@@
 $Descr A4 11693 8268
 encoding utf-8
-Sheet 5 90
+Sheet 5 92
 Title ""
 Date ""
@@
 Z7
 $Comp
-L myCpu-rescue:4069 U6
+L myCpu-rescue:4069 U8
 U 1 1 5AE664B9
 P 1025 4250
-AR Path="/5AE62FB7/5AE6649D/5AE664B9" Ref="U6"  Part="1"
-AR Path="/5AE62FB7/5B1BA146/5AE664B9" Ref="U36"  Part="1"
-F 0 "U36" H 1220 4365 50  0000 C CNN
+AR Path="/5AE62FB7/5AE6649D/5AE664B9" Ref="U8"  Part="1"
+AR Path="/5AE62FB7/5B1BA146/5AE664B9" Ref="U38"  Part="1"
+F 0 "U38" H 1220 4365 50  0000 C CNN
 F 1 "4069" H 1215 4125 50  0000 C CNN
 F 2 "" H 1025 4250 60  0001 C CNN
@@
 $EndComp
 $Comp
-L myCpu-rescue:4069 U6
+L myCpu-rescue:4069 U8
 U 2 1 5AE6656E
 P 1450 4250
-AR Path="/5AE62FB7/5AE6649D/5AE6656E" Ref="U6"  Part="2"
-AR Path="/5AE62FB7/5B1BA146/5AE6656E" Ref="U36"  Part="2"
-F 0 "U36" H 1645 4365 50  0000 C CNN
+AR Path="/5AE62FB7/5AE6649D/5AE6656E" Ref="U8"  Part="2"
+AR Path="/5AE62FB7/5B1BA146/5AE6656E" Ref="U38"  Part="2"
+F 0 "U38" H 1645 4365 50  0000 C CNN
 F 1 "4069" H 1640 4125 50  0000 C CNN
 F 2 "" H 1450 4250 60  0001 C CNN
@@
 $EndComp
 $Comp
-L myCpu-rescue:4069 U6
+L myCpu-rescue:4069 U8
 U 3 1 5AE66605
 P 1925 4225
-AR Path="/5AE62FB7/5AE6649D/5AE66605" Ref="U6"  Part="3"
-AR Path="/5AE62FB7/5B1BA146/5AE66605" Ref="U36"  Part="3"
-F 0 "U36" H 2120 4340 50  0000 C CNN
+AR Path="/5AE62FB7/5AE6649D/5AE66605" Ref="U8"  Part="3"
+AR Path="/5AE62FB7/5B1BA146/5AE66605" Ref="U38"  Part="3"
+F 0 "U38" H 2120 4340 50  0000 C CNN
 F 1 "4069" H 2115 4100 50  0000 C CNN
 F 2 "" H 1925 4225 60  0001 C CNN
@@
 $EndComp
 $Comp
-L myCpu-rescue:4069 U6
+L myCpu-rescue:4069 U8
 U 4 1 5AE6667C
 P 2400 4225
-AR Path="/5AE62FB7/5AE6649D/5AE6667C" Ref="U6"  Part="4"
-AR Path="/5AE62FB7/5B1BA146/5AE6667C" Ref="U36"  Part="4"
-F 0 "U36" H 2595 4340 50  0000 C CNN
+AR Path="/5AE62FB7/5AE6649D/5AE6667C" Ref="U8"  Part="4"
+AR Path="/5AE62FB7/5B1BA146/5AE6667C" Ref="U38"  Part="4"
+F 0 "U38" H 2595 4340 50  0000 C CNN
 F 1 "4069" H 2590 4100 50  0000 C CNN
 F 2 "" H 2400 4225 60  0001 C CNN
@@
 $EndComp
 $Comp
-L myCpu-rescue:4069 U6
+L myCpu-rescue:4069 U8
 U 5 1 5AE66711
 P 2900 4225
-AR Path="/5AE62FB7/5AE6649D/5AE66711" Ref="U6"  Part="5"
-AR Path="/5AE62FB7/5B1BA146/5AE66711" Ref="U36"  Part="5"
-F 0 "U36" H 3095 4340 50  0000 C CNN
+AR Path="/5AE62FB7/5AE6649D/5AE66711" Ref="U8"  Part="5"
+AR Path="/5AE62FB7/5B1BA146/5AE66711" Ref="U38"  Part="5"
+F 0 "U38" H 3095 4340 50  0000 C CNN
 F 1 "4069" H 3090 4100 50  0000 C CNN
 F 2 "" H 2900 4225 60  0001 C CNN
@@
 $EndComp
 $Comp
-L myCpu-rescue:4069 U6
+L myCpu-rescue:4069 U8
 U 6 1 5AE667CA
 P 3400 4250
-AR Path="/5AE62FB7/5AE6649D/5AE667CA" Ref="U6"  Part="6"
-AR Path="/5AE62FB7/5B1BA146/5AE667CA" Ref="U36"  Part="6"
-F 0 "U36" H 3595 4365 50  0000 C CNN
+AR Path="/5AE62FB7/5AE6649D/5AE667CA" Ref="U8"  Part="6"
+AR Path="/5AE62FB7/5B1BA146/5AE667CA" Ref="U38"  Part="6"
+F 0 "U38" H 3595 4365 50  0000 C CNN
 F 1 "4069" H 3590 4125 50  0000 C CNN
 F 2 "" H 3400 4250 60  0001 C CNN
@@
 $EndComp
 $Comp
-L myCpu-rescue:4069 U7
+L myCpu-rescue:4069 U9
 U 1 1 5AE66867
 P 3875 4250
-AR Path="/5AE62FB7/5AE6649D/5AE66867" Ref="U7"  Part="1"
-AR Path="/5AE62FB7/5B1BA146/5AE66867" Ref="U37"  Part="1"
-F 0 "U37" H 4070 4365 50  0000 C CNN
+AR Path="/5AE62FB7/5AE6649D/5AE66867" Ref="U9"  Part="1"
+AR Path="/5AE62FB7/5B1BA146/5AE66867" Ref="U39"  Part="1"
+F 0 "U39" H 4070 4365 50  0000 C CNN
 F 1 "4069" H 4065 4125 50  0000 C CNN
 F 2 "" H 3875 4250 60  0001 C CNN
@@
 $EndComp
 $Comp
-L myCpu-rescue:4069 U7
+L myCpu-rescue:4069 U9
 U 2 1 5AE668EC
 P 4325 4225
-AR Path="/5AE62FB7/5AE6649D/5AE668EC" Ref="U7"  Part="2"
-AR Path="/5AE62FB7/5B1BA146/5AE668EC" Ref="U37"  Part="2"
-F 0 "U37" H 4520 4340 50  0000 C CNN
+AR Path="/5AE62FB7/5AE6649D/5AE668EC" Ref="U9"  Part="2"
+AR Path="/5AE62FB7/5B1BA146/5AE668EC" Ref="U39"  Part="2"
+F 0 "U39" H 4520 4340 50  0000 C CNN
 F 1 "4069" H 4515 4100 50  0000 C CNN
 F 2 "" H 4325 4225 60  0001 C CNN
@@
 $EndComp
 $Comp
-L myCpu-rescue:4069 U7
+L myCpu-rescue:4069 U9
 U 3 1 5AE66989
 P 4775 4225
-AR Path="/5AE62FB7/5AE6649D/5AE66989" Ref="U7"  Part="3"
-AR Path="/5AE62FB7/5B1BA146/5AE66989" Ref="U37"  Part="3"
-F 0 "U37" H 4970 4340 50  0000 C CNN
+AR Path="/5AE62FB7/5AE6649D/5AE66989" Ref="U9"  Part="3"
+AR Path="/5AE62FB7/5B1BA146/5AE66989" Ref="U39"  Part="3"
+F 0 "U39" H 4970 4340 50  0000 C CNN
 F 1 "4069" H 4965 4100 50  0000 C CNN
 F 2 "" H 4775 4225 60  0001 C CNN
@@
 $EndComp
 $Comp
-L myCpu-rescue:4069 U7
+L myCpu-rescue:4069 U9
 U 4 1 5AE66A24
 P 5250 4225
-AR Path="/5AE62FB7/5AE6649D/5AE66A24" Ref="U7"  Part="4"
-AR Path="/5AE62FB7/5B1BA146/5AE66A24" Ref="U37"  Part="4"
-F 0 "U37" H 5445 4340 50  0000 C CNN
+AR Path="/5AE62FB7/5AE6649D/5AE66A24" Ref="U9"  Part="4"
+AR Path="/5AE62FB7/5B1BA146/5AE66A24" Ref="U39"  Part="4"
+F 0 "U39" H 5445 4340 50  0000 C CNN
 F 1 "4069" H 5440 4100 50  0000 C CNN
 F 2 "" H 5250 4225 60  0001 C CNN
@@
 $EndComp
 $Comp
-L myCpu-rescue:4069 U7
+L myCpu-rescue:4069 U9
 U 5 1 5AE66A93
 P 5800 4250
-AR Path="/5AE62FB7/5AE6649D/5AE66A93" Ref="U7"  Part="5"
-AR Path="/5AE62FB7/5B1BA146/5AE66A93" Ref="U37"  Part="5"
-F 0 "U37" H 5995 4365 50  0000 C CNN
+AR Path="/5AE62FB7/5AE6649D/5AE66A93" Ref="U9"  Part="5"
+AR Path="/5AE62FB7/5B1BA146/5AE66A93" Ref="U39"  Part="5"
+F 0 "U39" H 5995 4365 50  0000 C CNN
 F 1 "4069" H 5990 4125 50  0000 C CNN
 F 2 "" H 5800 4250 60  0001 C CNN
@@
 $EndComp
 $Comp
-L myCpu-rescue:4069 U7
+L myCpu-rescue:4069 U9
 U 6 1 5AE66B26
 P 6375 4250
-AR Path="/5AE62FB7/5AE6649D/5AE66B26" Ref="U7"  Part="6"
-AR Path="/5AE62FB7/5B1BA146/5AE66B26" Ref="U37"  Part="6"
-F 0 "U37" H 6570 4365 50  0000 C CNN
+AR Path="/5AE62FB7/5AE6649D/5AE66B26" Ref="U9"  Part="6"
+AR Path="/5AE62FB7/5B1BA146/5AE66B26" Ref="U39"  Part="6"
+F 0 "U39" H 6570 4365 50  0000 C CNN
 F 1 "4069" H 6565 4125 50  0000 C CNN
 F 2 "" H 6375 4250 60  0001 C CNN
@@
 	5800 4700 6375 4700
 $Comp
-L myCpu-rescue:VCC #PWR09
+L myCpu-rescue:VCC #PWR012
 U 1 1 5AE66D66
 P 5600 5025
-AR Path="/5AE62FB7/5AE6649D/5AE66D66" Ref="#PWR09"  Part="1"
-AR Path="/5AE62FB7/5B1BA146/5AE66D66" Ref="#PWR039"  Part="1"
-F 0 "#PWR039" H 5600 4875 50  0001 C CNN
+AR Path="/5AE62FB7/5AE6649D/5AE66D66" Ref="#PWR012"  Part="1"
+AR Path="/5AE62FB7/5B1BA146/5AE66D66" Ref="#PWR046"  Part="1"
+F 0 "#PWR046" H 5600 4875 50  0001 C CNN
 F 1 "VCC" H 5600 5175 50  0000 C CNN
 F 2 "" H 5600 5025 50  0000 C CNN
@@
 NoConn ~ 6375 3800
 Wire Wire Line
-	5250 4675 5800 4675
+	5250 4675 5600 4675
+$Comp
+L myCpu-rescue:VCC #PWR015
+U 1 1 5C8F82BF
+P 7900 2250
+AR Path="/5AE62FB7/5AE6649D/5C8F82BF" Ref="#PWR015"  Part="1"
+AR Path="/5AE62FB7/5B1BA146/5C8F82BF" Ref="#PWR049"  Part="1"
+F 0 "#PWR049" H 7900 2100 50  0001 C CNN
+F 1 "VCC" H 7917 2423 50  0000 C CNN
+F 2 "" H 7900 2250 50  0000 C CNN
+F 3 "" H 7900 2250 50  0000 C CNN
+	1    7900 2250
+	1    0    0    -1
+$EndComp
+$Comp
+L power:VDD #PWR016
+U 1 1 5C8F8352
+P 7900 2250
+AR Path="/5AE62FB7/5AE6649D/5C8F8352" Ref="#PWR016"  Part="1"
+AR Path="/5AE62FB7/5B1BA146/5C8F8352" Ref="#PWR050"  Part="1"
+F 0 "#PWR050" H 7900 2350 30  0001 C CNN
+F 1 "VDD" H 7915 2387 30  0000 C CNN
+F 2 "" H 7900 2250 60  0001 C CNN
+F 3 "" H 7900 2250 60  0001 C CNN
+	1    7900 2250
+	-1   0    0    1
+$EndComp
+$Comp
+L power:GND #PWR013
+U 1 1 5C8FF848
+P 7250 4300
+AR Path="/5AE62FB7/5AE6649D/5C8FF848" Ref="#PWR013"  Part="1"
+AR Path="/5AE62FB7/5B1BA146/5C8FF848" Ref="#PWR047"  Part="1"
+F 0 "#PWR047" H 7250 4300 30  0001 C CNN
+F 1 "GND" H 7250 4230 30  0001 C CNN
+F 2 "" H 7250 4300 60  0001 C CNN
+F 3 "" H 7250 4300 60  0001 C CNN
+	1    7250 4300
+	1    0    0    -1
+$EndComp
+$Comp
+L power:VSS #PWR014
+U 1 1 5C8FF8DB
+P 7250 4300
+AR Path="/5AE62FB7/5AE6649D/5C8FF8DB" Ref="#PWR014"  Part="1"
+AR Path="/5AE62FB7/5B1BA146/5C8FF8DB" Ref="#PWR048"  Part="1"
+F 0 "#PWR048" H 7250 4300 30  0001 C CNN
+F 1 "VSS" H 7250 4358 30  0000 C CNN
+F 2 "" H 7250 4300 60  0001 C CNN
+F 3 "" H 7250 4300 60  0001 C CNN
+	1    7250 4300
+	-1   0    0    1
+$EndComp
+Connection ~ 5800 4700
+Connection ~ 5600 4675
+Wire Wire Line
+	5600 4675 5800 4675
 $EndSCHEMATC

Commit message: tst
Changed lines of the file:
@@
 AR Path="/5AE62FB7/5AE6649D/5AE664B9" Ref="U8"  Part="1"
 AR Path="/5AE62FB7/5B1BA146/5AE664B9" Ref="U38"  Part="1"
-F 0 "U38" H 1220 4365 50  0000 C CNN
+F 0 "U8" H 1220 4365 50  0000 C CNN
 F 1 "4069" H 1215 4125 50  0000 C CNN
 F 2 "" H 1025 4250 60  0001 C CNN
@@
 AR Path="/5AE62FB7/5AE6649D/5AE6656E" Ref="U8"  Part="2"
 AR Path="/5AE62FB7/5B1BA146/5AE6656E" Ref="U38"  Part="2"
-F 0 "U38" H 1645 4365 50  0000 C CNN
+F 0 "U8" H 1645 4365 50  0000 C CNN
 F 1 "4069" H 1640 4125 50  0000 C CNN
 F 2 "" H 1450 4250 60  0001 C CNN
@@
 AR Path="/5AE62FB7/5AE6649D/5AE66605" Ref="U8"  Part="3"
 AR Path="/5AE62FB7/5B1BA146/5AE66605" Ref="U38"  Part="3"
-F 0 "U38" H 2120 4340 50  0000 C CNN
+F 0 "U8" H 2120 4340 50  0000 C CNN
 F 1 "4069" H 2115 4100 50  0000 C CNN
 F 2 "" H 1925 4225 60  0001 C CNN
@@
 AR Path="/5AE62FB7/5AE6649D/5AE6667C" Ref="U8"  Part="4"
 AR Path="/5AE62FB7/5B1BA146/5AE6667C" Ref="U38"  Part="4"
-F 0 "U38" H 2595 4340 50  0000 C CNN
+F 0 "U8" H 2595 4340 50  0000 C CNN
 F 1 "4069" H 2590 4100 50  0000 C CNN
 F 2 "" H 2400 4225 60  0001 C CNN
@@
 AR Path="/5AE62FB7/5AE6649D/5AE66711" Ref="U8"  Part="5"
 AR Path="/5AE62FB7/5B1BA146/5AE66711" Ref="U38"  Part="5"
-F 0 "U38" H 3095 4340 50  0000 C CNN
+F 0 "U8" H 3095 4340 50  0000 C CNN
 F 1 "4069" H 3090 4100 50  0000 C CNN
 F 2 "" H 2900 4225 60  0001 C CNN
@@
 AR Path="/5AE62FB7/5AE6649D/5AE667CA" Ref="U8"  Part="6"
 AR Path="/5AE62FB7/5B1BA146/5AE667CA" Ref="U38"  Part="6"
-F 0 "U38" H 3595 4365 50  0000 C CNN
+F 0 "U8" H 3595 4365 50  0000 C CNN
 F 1 "4069" H 3590 4125 50  0000 C CNN
 F 2 "" H 3400 4250 60  0001 C CNN
@@
 AR Path="/5AE62FB7/5AE6649D/5AE66867" Ref="U9"  Part="1"
 AR Path="/5AE62FB7/5B1BA146/5AE66867" Ref="U39"  Part="1"
-F 0 "U39" H 4070 4365 50  0000 C CNN
+F 0 "U9" H 4070 4365 50  0000 C CNN
 F 1 "4069" H 4065 4125 50  0000 C CNN
 F 2 "" H 3875 4250 60  0001 C CNN
@@
 AR Path="/5AE62FB7/5AE6649D/5AE668EC" Ref="U9"  Part="2"
 AR Path="/5AE62FB7/5B1BA146/5AE668EC" Ref="U39"  Part="2"
-F 0 "U39" H 4520 4340 50  0000 C CNN
+F 0 "U9" H 4520 4340 50  0000 C CNN
 F 1 "4069" H 4515 4100 50  0000 C CNN
 F 2 "" H 4325 4225 60  0001 C CNN
@@
 AR Path="/5AE62FB7/5AE6649D/5AE66989" Ref="U9"  Part="3"
 AR Path="/5AE62FB7/5B1BA146/5AE66989" Ref="U39"  Part="3"
-F 0 "U39" H 4970 4340 50  0000 C CNN
+F 0 "U9" H 4970 4340 50  0000 C CNN
 F 1 "4069" H 4965 4100 50  0000 C CNN
 F 2 "" H 4775 4225 60  0001 C CNN
@@
 AR Path="/5AE62FB7/5AE6649D/5AE66A24" Ref="U9"  Part="4"
 AR Path="/5AE62FB7/5B1BA146/5AE66A24" Ref="U39"  Part="4"
-F 0 "U39" H 5445 4340 50  0000 C CNN
+F 0 "U9" H 5445 4340 50  0000 C CNN
 F 1 "4069" H 5440 4100 50  0000 C CNN
 F 2 "" H 5250 4225 60  0001 C CNN
@@
 AR Path="/5AE62FB7/5AE6649D/5AE66A93" Ref="U9"  Part="5"
 AR Path="/5AE62FB7/5B1BA146/5AE66A93" Ref="U39"  Part="5"
-F 0 "U39" H 5995 4365 50  0000 C CNN
+F 0 "U9" H 5995 4365 50  0000 C CNN
 F 1 "4069" H 5990 4125 50  0000 C CNN
 F 2 "" H 5800 4250 60  0001 C CNN
@@
 AR Path="/5AE62FB7/5AE6649D/5AE66B26" Ref="U9"  Part="6"
 AR Path="/5AE62FB7/5B1BA146/5AE66B26" Ref="U39"  Part="6"
-F 0 "U39" H 6570 4365 50  0000 C CNN
+F 0 "U9" H 6570 4365 50  0000 C CNN
 F 1 "4069" H 6565 4125 50  0000 C CNN
 F 2 "" H 6375 4250 60  0001 C CNN

Commit message: fixed errors
Changed lines of the file:
@@
 $Descr A4 11693 8268
 encoding utf-8
-Sheet 5 92
+Sheet 20 92
 Title ""
 Date ""
@@
 AR Path="/5AE62FB7/5AE6649D/5AE664B9" Ref="U8"  Part="1"
 AR Path="/5AE62FB7/5B1BA146/5AE664B9" Ref="U38"  Part="1"
-F 0 "U8" H 1220 4365 50  0000 C CNN
+F 0 "U38" H 1220 4365 50  0000 C CNN
 F 1 "4069" H 1215 4125 50  0000 C CNN
 F 2 "" H 1025 4250 60  0001 C CNN
@@
 AR Path="/5AE62FB7/5AE6649D/5AE6656E" Ref="U8"  Part="2"
 AR Path="/5AE62FB7/5B1BA146/5AE6656E" Ref="U38"  Part="2"
-F 0 "U8" H 1645 4365 50  0000 C CNN
+F 0 "U38" H 1645 4365 50  0000 C CNN
 F 1 "4069" H 1640 4125 50  0000 C CNN
 F 2 "" H 1450 4250 60  0001 C CNN
@@
 AR Path="/5AE62FB7/5AE6649D/5AE66605" Ref="U8"  Part="3"
 AR Path="/5AE62FB7/5B1BA146/5AE66605" Ref="U38"  Part="3"
-F 0 "U8" H 2120 4340 50  0000 C CNN
+F 0 "U38" H 2120 4340 50  0000 C CNN
 F 1 "4069" H 2115 4100 50  0000 C CNN
 F 2 "" H 1925 4225 60  0001 C CNN
@@
 AR Path="/5AE62FB7/5AE6649D/5AE6667C" Ref="U8"  Part="4"
 AR Path="/5AE62FB7/5B1BA146/5AE6667C" Ref="U38"  Part="4"
-F 0 "U8" H 2595 4340 50  0000 C CNN
+F 0 "U38" H 2595 4340 50  0000 C CNN
 F 1 "4069" H 2590 4100 50  0000 C CNN
 F 2 "" H 2400 4225 60  0001 C CNN
@@
 AR Path="/5AE62FB7/5AE6649D/5AE66711" Ref="U8"  Part="5"
 AR Path="/5AE62FB7/5B1BA146/5AE66711" Ref="U38"  Part="5"
-F 0 "U8" H 3095 4340 50  0000 C CNN
+F 0 "U38" H 3095 4340 50  0000 C CNN
 F 1 "4069" H 3090 4100 50  0000 C CNN
 F 2 "" H 2900 4225 60  0001 C CNN
@@
 AR Path="/5AE62FB7/5AE6649D/5AE667CA" Ref="U8"  Part="6"
 AR Path="/5AE62FB7/5B1BA146/5AE667CA" Ref="U38"  Part="6"
-F 0 "U8" H 3595 4365 50  0000 C CNN
+F 0 "U38" H 3595 4365 50  0000 C CNN
 F 1 "4069" H 3590 4125 50  0000 C CNN
 F 2 "" H 3400 4250 60  0001 C CNN
@@
 AR Path="/5AE62FB7/5AE6649D/5AE66867" Ref="U9"  Part="1"
 AR Path="/5AE62FB7/5B1BA146/5AE66867" Ref="U39"  Part="1"
-F 0 "U9" H 4070 4365 50  0000 C CNN
+F 0 "U39" H 4070 4365 50  0000 C CNN
 F 1 "4069" H 4065 4125 50  0000 C CNN
 F 2 "" H 3875 4250 60  0001 C CNN
@@
 AR Path="/5AE62FB7/5AE6649D/5AE668EC" Ref="U9"  Part="2"
 AR Path="/5AE62FB7/5B1BA146/5AE668EC" Ref="U39"  Part="2"
-F 0 "U9" H 4520 4340 50  0000 C CNN
+F 0 "U39" H 4520 4340 50  0000 C CNN
 F 1 "4069" H 4515 4100 50  0000 C CNN
 F 2 "" H 4325 4225 60  0001 C CNN
@@
 AR Path="/5AE62FB7/5AE6649D/5AE66989" Ref="U9"  Part="3"
 AR Path="/5AE62FB7/5B1BA146/5AE66989" Ref="U39"  Part="3"
-F 0 "U9" H 4970 4340 50  0000 C CNN
+F 0 "U39" H 4970 4340 50  0000 C CNN
 F 1 "4069" H 4965 4100 50  0000 C CNN
 F 2 "" H 4775 4225 60  0001 C CNN
@@
 AR Path="/5AE62FB7/5AE6649D/5AE66A24" Ref="U9"  Part="4"
 AR Path="/5AE62FB7/5B1BA146/5AE66A24" Ref="U39"  Part="4"
-F 0 "U9" H 5445 4340 50  0000 C CNN
+F 0 "U39" H 5445 4340 50  0000 C CNN
 F 1 "4069" H 5440 4100 50  0000 C CNN
 F 2 "" H 5250 4225 60  0001 C CNN
@@
 AR Path="/5AE62FB7/5AE6649D/5AE66A93" Ref="U9"  Part="5"
 AR Path="/5AE62FB7/5B1BA146/5AE66A93" Ref="U39"  Part="5"
-F 0 "U9" H 5995 4365 50  0000 C CNN
+F 0 "U39" H 5995 4365 50  0000 C CNN
 F 1 "4069" H 5990 4125 50  0000 C CNN
 F 2 "" H 5800 4250 60  0001 C CNN
@@
 AR Path="/5AE62FB7/5AE6649D/5AE66B26" Ref="U9"  Part="6"
 AR Path="/5AE62FB7/5B1BA146/5AE66B26" Ref="U39"  Part="6"
-F 0 "U9" H 6570 4365 50  0000 C CNN
+F 0 "U39" H 6570 4365 50  0000 C CNN
 F 1 "4069" H 6565 4125 50  0000 C CNN
 F 2 "" H 6375 4250 60  0001 C CNN
