File: NOT.sch (KiCad schematic (older format))
At the start: 2 parts, among them U8 4069, U9 4069

Commit message: message
Parts:
- renumbered U8 to U15, U8 to U16, U8 to U17, U9 to U18, U9 to U19, U9 to U20
Changed lines of the file:
@@
 $Descr A4 11693 8268
 encoding utf-8
-Sheet 20 92
+Sheet 20 101
 Title ""
 Date ""
@@
 Z7
 $Comp
-L myCpu-rescue:4069 U8
+L myCpu-rescue:4069 U15
 U 1 1 5AE664B9
 P 1025 4250
-AR Path="/5AE62FB7/5AE6649D/5AE664B9" Ref="U8"  Part="1"
-AR Path="/5AE62FB7/5B1BA146/5AE664B9" Ref="U38"  Part="1"
-F 0 "U38" H 1220 4365 50  0000 C CNN
+AR Path="/5AE62FB7/5AE6649D/5AE664B9" Ref="U15"  Part="1"
+AR Path="/5AE62FB7/5B1BA146/5AE664B9" Ref="U51"  Part="1"
+F 0 "U51" H 1220 4365 50  0000 C CNN
 F 1 "4069" H 1215 4125 50  0000 C CNN
 F 2 "" H 1025 4250 60  0001 C CNN
@@
 $EndComp
 $Comp
-L myCpu-rescue:4069 U8
+L myCpu-rescue:4069 U15
 U 2 1 5AE6656E
 P 1450 4250
-AR Path="/5AE62FB7/5AE6649D/5AE6656E" Ref="U8"  Part="2"
-AR Path="/5AE62FB7/5B1BA146/5AE6656E" Ref="U38"  Part="2"
-F 0 "U38" H 1645 4365 50  0000 C CNN
+AR Path="/5AE62FB7/5AE6649D/5AE6656E" Ref="U15"  Part="2"
+AR Path="/5AE62FB7/5B1BA146/5AE6656E" Ref="U51"  Part="2"
+F 0 "U51" H 1645 4365 50  0000 C CNN
 F 1 "4069" H 1640 4125 50  0000 C CNN
 F 2 "" H 1450 4250 60  0001 C CNN
@@
 $EndComp
 $Comp
-L myCpu-rescue:4069 U8
+L myCpu-rescue:4069 U16
 U 3 1 5AE66605
 P 1925 4225
-AR Path="/5AE62FB7/5AE6649D/5AE66605" Ref="U8"  Part="3"
-AR Path="/5AE62FB7/5B1BA146/5AE66605" Ref="U38"  Part="3"
-F 0 "U38" H 2120 4340 50  0000 C CNN
+AR Path="/5AE62FB7/5AE6649D/5AE66605" Ref="U16"  Part="3"
+AR Path="/5AE62FB7/5B1BA146/5AE66605" Ref="U52"  Part="3"
+F 0 "U52" H 2120 4340 50  0000 C CNN
 F 1 "4069" H 2115 4100 50  0000 C CNN
 F 2 "" H 1925 4225 60  0001 C CNN
@@
 $EndComp
 $Comp
-L myCpu-rescue:4069 U8
+L myCpu-rescue:4069 U16
 U 4 1 5AE6667C
 P 2400 4225
-AR Path="/5AE62FB7/5AE6649D/5AE6667C" Ref="U8"  Part="4"
-AR Path="/5AE62FB7/5B1BA146/5AE6667C" Ref="U38"  Part="4"
-F 0 "U38" H 2595 4340 50  0000 C CNN
+AR Path="/5AE62FB7/5AE6649D/5AE6667C" Ref="U16"  Part="4"
+AR Path="/5AE62FB7/5B1BA146/5AE6667C" Ref="U52"  Part="4"
+F 0 "U52" H 2595 4340 50  0000 C CNN
 F 1 "4069" H 2590 4100 50  0000 C CNN
 F 2 "" H 2400 4225 60  0001 C CNN
@@
 $EndComp
 $Comp
-L myCpu-rescue:4069 U8
+L myCpu-rescue:4069 U17
 U 5 1 5AE66711
 P 2900 4225
-AR Path="/5AE62FB7/5AE6649D/5AE66711" Ref="U8"  Part="5"
-AR Path="/5AE62FB7/5B1BA146/5AE66711" Ref="U38"  Part="5"
-F 0 "U38" H 3095 4340 50  0000 C CNN
+AR Path="/5AE62FB7/5AE6649D/5AE66711" Ref="U17"  Part="5"
+AR Path="/5AE62FB7/5B1BA146/5AE66711" Ref="U53"  Part="5"
+F 0 "U53" H 3095 4340 50  0000 C CNN
 F 1 "4069" H 3090 4100 50  0000 C CNN
 F 2 "" H 2900 4225 60  0001 C CNN
@@
 $EndComp
 $Comp
-L myCpu-rescue:4069 U8
+L myCpu-rescue:4069 U17
 U 6 1 5AE667CA
 P 3400 4250
-AR Path="/5AE62FB7/5AE6649D/5AE667CA" Ref="U8"  Part="6"
-AR Path="/5AE62FB7/5B1BA146/5AE667CA" Ref="U38"  Part="6"
-F 0 "U38" H 3595 4365 50  0000 C CNN
+AR Path="/5AE62FB7/5AE6649D/5AE667CA" Ref="U17"  Part="6"
+AR Path="/5AE62FB7/5B1BA146/5AE667CA" Ref="U53"  Part="6"
+F 0 "U53" H 3595 4365 50  0000 C CNN
 F 1 "4069" H 3590 4125 50  0000 C CNN
 F 2 "" H 3400 4250 60  0001 C CNN
@@
 $EndComp
 $Comp
-L myCpu-rescue:4069 U9
+L myCpu-rescue:4069 U18
 U 1 1 5AE66867
 P 3875 4250
-AR Path="/5AE62FB7/5AE6649D/5AE66867" Ref="U9"  Part="1"
-AR Path="/5AE62FB7/5B1BA146/5AE66867" Ref="U39"  Part="1"
-F 0 "U39" H 4070 4365 50  0000 C CNN
+AR Path="/5AE62FB7/5AE6649D/5AE66867" Ref="U18"  Part="1"
+AR Path="/5AE62FB7/5B1BA146/5AE66867" Ref="U54"  Part="1"
+F 0 "U54" H 4070 4365 50  0000 C CNN
 F 1 "4069" H 4065 4125 50  0000 C CNN
 F 2 "" H 3875 4250 60  0001 C CNN
@@
 $EndComp
 $Comp
-L myCpu-rescue:4069 U9
+L myCpu-rescue:4069 U18
 U 2 1 5AE668EC
 P 4325 4225
-AR Path="/5AE62FB7/5AE6649D/5AE668EC" Ref="U9"  Part="2"
-AR Path="/5AE62FB7/5B1BA146/5AE668EC" Ref="U39"  Part="2"
-F 0 "U39" H 4520 4340 50  0000 C CNN
+AR Path="/5AE62FB7/5AE6649D/5AE668EC" Ref="U18"  Part="2"
+AR Path="/5AE62FB7/5B1BA146/5AE668EC" Ref="U54"  Part="2"
+F 0 "U54" H 4520 4340 50  0000 C CNN
 F 1 "4069" H 4515 4100 50  0000 C CNN
 F 2 "" H 4325 4225 60  0001 C CNN
@@
 $EndComp
 $Comp
-L myCpu-rescue:4069 U9
+L myCpu-rescue:4069 U19
 U 3 1 5AE66989
 P 4775 4225
-AR Path="/5AE62FB7/5AE6649D/5AE66989" Ref="U9"  Part="3"
-AR Path="/5AE62FB7/5B1BA146/5AE66989" Ref="U39"  Part="3"
-F 0 "U39" H 4970 4340 50  0000 C CNN
+AR Path="/5AE62FB7/5AE6649D/5AE66989" Ref="U19"  Part="3"
+AR Path="/5AE62FB7/5B1BA146/5AE66989" Ref="U55"  Part="3"
+F 0 "U55" H 4970 4340 50  0000 C CNN
 F 1 "4069" H 4965 4100 50  0000 C CNN
 F 2 "" H 4775 4225 60  0001 C CNN
@@
 $EndComp
 $Comp
-L myCpu-rescue:4069 U9
+L myCpu-rescue:4069 U19
 U 4 1 5AE66A24
 P 5250 4225
-AR Path="/5AE62FB7/5AE6649D/5AE66A24" Ref="U9"  Part="4"
-AR Path="/5AE62FB7/5B1BA146/5AE66A24" Ref="U39"  Part="4"
-F 0 "U39" H 5445 4340 50  0000 C CNN
+AR Path="/5AE62FB7/5AE6649D/5AE66A24" Ref="U19"  Part="4"
+AR Path="/5AE62FB7/5B1BA146/5AE66A24" Ref="U55"  Part="4"
+F 0 "U55" H 5445 4340 50  0000 C CNN
 F 1 "4069" H 5440 4100 50  0000 C CNN
 F 2 "" H 5250 4225 60  0001 C CNN
@@
 $EndComp
 $Comp
-L myCpu-rescue:4069 U9
+L myCpu-rescue:4069 U20
 U 5 1 5AE66A93
 P 5800 4250
-AR Path="/5AE62FB7/5AE6649D/5AE66A93" Ref="U9"  Part="5"
-AR Path="/5AE62FB7/5B1BA146/5AE66A93" Ref="U39"  Part="5"
-F 0 "U39" H 5995 4365 50  0000 C CNN
+AR Path="/5AE62FB7/5AE6649D/5AE66A93" Ref="U20"  Part="5"
+AR Path="/5AE62FB7/5B1BA146/5AE66A93" Ref="U56"  Part="5"
+F 0 "U56" H 5995 4365 50  0000 C CNN
 F 1 "4069" H 5990 4125 50  0000 C CNN
 F 2 "" H 5800 4250 60  0001 C CNN
@@
 $EndComp
 $Comp
-L myCpu-rescue:4069 U9
+L myCpu-rescue:4069 U20
 U 6 1 5AE66B26
 P 6375 4250
-AR Path="/5AE62FB7/5AE6649D/5AE66B26" Ref="U9"  Part="6"
-AR Path="/5AE62FB7/5B1BA146/5AE66B26" Ref="U39"  Part="6"
-F 0 "U39" H 6570 4365 50  0000 C CNN
+AR Path="/5AE62FB7/5AE6649D/5AE66B26" Ref="U20"  Part="6"
+AR Path="/5AE62FB7/5B1BA146/5AE66B26" Ref="U56"  Part="6"
+F 0 "U56" H 6570 4365 50  0000 C CNN
 F 1 "4069" H 6565 4125 50  0000 C CNN
 F 2 "" H 6375 4250 60  0001 C CNN
@@
 	5800 4700 6375 4700
 $Comp
-L myCpu-rescue:VCC #PWR012
+L myCpu-rescue:VCC #PWR014
 U 1 1 5AE66D66
 P 5600 5025
-AR Path="/5AE62FB7/5AE6649D/5AE66D66" Ref="#PWR012"  Part="1"
-AR Path="/5AE62FB7/5B1BA146/5AE66D66" Ref="#PWR046"  Part="1"
-F 0 "#PWR046" H 5600 4875 50  0001 C CNN
+AR Path="/5AE62FB7/5AE6649D/5AE66D66" Ref="#PWR014"  Part="1"
+AR Path="/5AE62FB7/5B1BA146/5AE66D66" Ref="#PWR052"  Part="1"
+F 0 "#PWR052" H 5600 4875 50  0001 C CNN
 F 1 "VCC" H 5600 5175 50  0000 C CNN
 F 2 "" H 5600 5025 50  0000 C CNN
@@
 	5250 4675 5600 4675
 $Comp
-L myCpu-rescue:VCC #PWR015
+L myCpu-rescue:VCC #PWR017
 U 1 1 5C8F82BF
 P 7900 2250
-AR Path="/5AE62FB7/5AE6649D/5C8F82BF" Ref="#PWR015"  Part="1"
-AR Path="/5AE62FB7/5B1BA146/5C8F82BF" Ref="#PWR049"  Part="1"
-F 0 "#PWR049" H 7900 2100 50  0001 C CNN
+AR Path="/5AE62FB7/5AE6649D/5C8F82BF" Ref="#PWR017"  Part="1"
+AR Path="/5AE62FB7/5B1BA146/5C8F82BF" Ref="#PWR055"  Part="1"
+F 0 "#PWR055" H 7900 2100 50  0001 C CNN
 F 1 "VCC" H 7917 2423 50  0000 C CNN
 F 2 "" H 7900 2250 50  0000 C CNN
@@
 $EndComp
 $Comp
-L power:VDD #PWR016
+L power:VDD #PWR018
 U 1 1 5C8F8352
 P 7900 2250
-AR Path="/5AE62FB7/5AE6649D/5C8F8352" Ref="#PWR016"  Part="1"
-AR Path="/5AE62FB7/5B1BA146/5C8F8352" Ref="#PWR050"  Part="1"
-F 0 "#PWR050" H 7900 2350 30  0001 C CNN
+AR Path="/5AE62FB7/5AE6649D/5C8F8352" Ref="#PWR018"  Part="1"
+AR Path="/5AE62FB7/5B1BA146/5C8F8352" Ref="#PWR056"  Part="1"
+F 0 "#PWR056" H 7900 2350 30  0001 C CNN
 F 1 "VDD" H 7915 2387 30  0000 C CNN
 F 2 "" H 7900 2250 60  0001 C CNN
@@
 $EndComp
 $Comp
-L power:GND #PWR013
+L power:GND #PWR015
 U 1 1 5C8FF848
 P 7250 4300
-AR Path="/5AE62FB7/5AE6649D/5C8FF848" Ref="#PWR013"  Part="1"
-AR Path="/5AE62FB7/5B1BA146/5C8FF848" Ref="#PWR047"  Part="1"
-F 0 "#PWR047" H 7250 4300 30  0001 C CNN
+AR Path="/5AE62FB7/5AE6649D/5C8FF848" Ref="#PWR015"  Part="1"
+AR Path="/5AE62FB7/5B1BA146/5C8FF848" Ref="#PWR053"  Part="1"
+F 0 "#PWR053" H 7250 4300 30  0001 C CNN
 F 1 "GND" H 7250 4230 30  0001 C CNN
 F 2 "" H 7250 4300 60  0001 C CNN
@@
 $EndComp
 $Comp
-L power:VSS #PWR014
+L power:VSS #PWR016
 U 1 1 5C8FF8DB
 P 7250 4300
-AR Path="/5AE62FB7/5AE6649D/5C8FF8DB" Ref="#PWR014"  Part="1"
-AR Path="/5AE62FB7/5B1BA146/5C8FF8DB" Ref="#PWR048"  Part="1"
-F 0 "#PWR048" H 7250 4300 30  0001 C CNN
+AR Path="/5AE62FB7/5AE6649D/5C8FF8DB" Ref="#PWR016"  Part="1"
+AR Path="/5AE62FB7/5B1BA146/5C8FF8DB" Ref="#PWR054"  Part="1"
+F 0 "#PWR054" H 7250 4300 30  0001 C CNN
 F 1 "VSS" H 7250 4358 30  0000 C CNN
 F 2 "" H 7250 4300 60  0001 C CNN
