File: PC.sch (KiCad schematic (older format))
At the start: 0 parts

Commit message: .
Changed lines of the file:
@@
 $Descr A4 11693 8268
 encoding utf-8
-Sheet 73 101
+Sheet 58 75
 Title ""
 Date ""
@@
 Comment4 ""
 $EndDescr
-$Sheet
-S 3975 2450 850  1250
-U 82611AD7
-F0 "PCA" 60
-F1 "Register.sch" 60
-F2 "X0" I L 3975 2675 60
-F3 "X1" I L 3975 2800 60
-F4 "X2" I L 3975 2975 60
-F5 "X3" I L 3975 3075 60
-F6 "X4" I L 3975 3150 60
-F7 "X5" I L 3975 3225 60
-F8 "X6" I L 3975 3325 60
-F9 "X7" I L 3975 3425 60
-F10 "Z0" O R 4825 2650 60
-F11 "Z1" O R 4825 2750 60
-F12 "Z2" O R 4825 2850 60
-F13 "Z3" O R 4825 2950 60
-F14 "Z4" O R 4825 3050 60
-F15 "Z5" O R 4825 3150 60
-F16 "Z6" O R 4825 3250 60
-F17 "Z7" O R 4825 3325 60
-F18 "CLK" I L 3975 3575 60
-$EndSheet
-$Sheet
-S 4000 4200 900  1675
-U 82611ADA
-F0 "PCB" 60
-F1 "Register.sch" 60
-F2 "X0" I L 4000 4300 60
-F3 "X1" I L 4000 4450 60
-F4 "X2" I L 4000 4550 60
-F5 "X3" I L 4000 4675 60
-F6 "X4" I L 4000 4800 60
-F7 "X5" I L 4000 4925 60
-F8 "X6" I L 4000 5050 60
-F9 "X7" I L 4000 5175 60
-F10 "Z0" O R 4900 4400 60
-F11 "Z1" O R 4900 4525 60
-F12 "Z2" O R 4900 4625 60
-F13 "Z3" O R 4900 4775 60
-F14 "Z4" O R 4900 4900 60
-F15 "Z5" O R 4900 5000 60
-F16 "Z6" O R 4900 5100 60
-F17 "Z7" O R 4900 5225 60
-F18 "CLK" I L 4000 5525 60
-$EndSheet
 $Sheet
 S 6575 2475 1125 3050
@@
 Wire Wire Line
 	1825 6125 1825 6075
+$Sheet
+S 3975 2525 850  1325
+U 6464023A
+F0 "PCA" 60
+F1 "Register.sch" 60
+F2 "CLK" I L 3975 3575 60
+F3 "X0" I L 3975 2675 60
+F4 "X1" I L 3975 2800 60
+F5 "X2" I L 3975 2975 60
+F6 "X3" I L 3975 3075 60
+F7 "X4" I L 3975 3150 60
+F8 "X5" I L 3975 3225 60
+F9 "X6" I L 3975 3325 60
+F10 "X7" I L 3975 3425 60
+F11 "Z0" O R 4825 2650 60
+F12 "Z1" O R 4825 2750 60
+F13 "Z2" O R 4825 2850 60
+F14 "Z3" O R 4825 2950 60
+F15 "Z4" O R 4825 3050 60
+F16 "Z5" O R 4825 3150 60
+F17 "Z6" O R 4825 3250 60
+F18 "Z7" O R 4825 3325 60
+$EndSheet
+$Sheet
+S 4000 4175 900  1400
+U 64640400
+F0 "PCB" 60
+F1 "Register.sch" 60
+F2 "CLK" I L 4000 5525 60
+F3 "X0" I L 4000 4300 60
+F4 "X1" I L 4000 4450 60
+F5 "X2" I L 4000 4550 60
+F6 "X3" I L 4000 4675 60
+F7 "X4" I L 4000 4800 60
+F8 "X5" I L 4000 4925 60
+F9 "X6" I L 4000 5050 60
+F10 "X7" I L 4000 5175 60
+F11 "Z0" O R 4900 4400 60
+F12 "Z1" O R 4900 4525 60
+F13 "Z2" O R 4900 4625 60
+F14 "Z3" O R 4900 4775 60
+F15 "Z4" O R 4900 4900 60
+F16 "Z5" O R 4900 5000 60
+F17 "Z6" O R 4900 5100 60
+F18 "Z7" O R 4900 5225 60
+$EndSheet
 $EndSCHEMATC
