File: PC_INC_SELECTOR.sch (KiCad schematic (older format))
At the start: 7 parts, among them U149 74LS04, U246 74LS08, U247 4071, U248 74LS04

Commit message: fixed errors
Connections:
- wire segments 31 -> 37
- no-connect marks 2 -> 6
Changed lines of the file:
@@
 L 74xx:74LS04 U149
 U 2 1 5B70E3FE
-P 5925 5000
-F 0 "U149" H 5925 5337 60  0000 C CNN
-F 1 "74LS04" H 5925 5231 60  0000 C CNN
-F 2 "" H 5925 5000 60  0001 C CNN
-F 3 "" H 5925 5000 60  0001 C CNN
-	2    5925 5000
+P 6000 5400
+F 0 "U149" H 6000 5737 60  0000 C CNN
+F 1 "74LS04" H 6000 5631 60  0000 C CNN
+F 2 "" H 6000 5400 60  0001 C CNN
+F 3 "" H 6000 5400 60  0001 C CNN
+	2    6000 5400
 	1    0    0    -1
 $EndComp
@@
 L 74xx:74LS04 U149
 U 3 1 5B70E48E
-P 5925 5000
-F 0 "U149" H 5925 5337 60  0000 C CNN
-F 1 "74LS04" H 5925 5231 60  0000 C CNN
-F 2 "" H 5925 5000 60  0001 C CNN
-F 3 "" H 5925 5000 60  0001 C CNN
-	3    5925 5000
+P 6050 5800
+F 0 "U149" H 6050 6137 60  0000 C CNN
+F 1 "74LS04" H 6050 6031 60  0000 C CNN
+F 2 "" H 6050 5800 60  0001 C CNN
+F 3 "" H 6050 5800 60  0001 C CNN
+	3    6050 5800
 	1    0    0    -1
 $EndComp
@@
 L 74xx:74LS04 U149
 U 4 1 5B70E55D
-P 5925 5000
-F 0 "U149" H 5925 5337 60  0000 C CNN
-F 1 "74LS04" H 5925 5231 60  0000 C CNN
-F 2 "" H 5925 5000 60  0001 C CNN
-F 3 "" H 5925 5000 60  0001 C CNN
-	4    5925 5000
+P 6100 6250
+F 0 "U149" H 6100 6587 60  0000 C CNN
+F 1 "74LS04" H 6100 6481 60  0000 C CNN
+F 2 "" H 6100 6250 60  0001 C CNN
+F 3 "" H 6100 6250 60  0001 C CNN
+	4    6100 6250
 	1    0    0    -1
 $EndComp
-Connection ~ 6375 5000
 Connection ~ 5475 5000
-Connection ~ 5875 5100
-Connection ~ 5875 4900
 $Comp
 L 74xx:74LS04 U149
 U 5 1 5B70E605
-P 5925 5000
-F 0 "U149" H 5925 5337 60  0000 C CNN
-F 1 "74LS04" H 5925 5231 60  0000 C CNN
-F 2 "" H 5925 5000 60  0001 C CNN
-F 3 "" H 5925 5000 60  0001 C CNN
-	5    5925 5000
+P 6150 6650
+F 0 "U149" H 6150 6987 60  0000 C CNN
+F 1 "74LS04" H 6150 6881 60  0000 C CNN
+F 2 "" H 6150 6650 60  0001 C CNN
+F 3 "" H 6150 6650 60  0001 C CNN
+	5    6150 6650
 	1    0    0    -1
 $EndComp
@@
 Text HLabel 4225 2625 0    60   Input ~ 0
 RET
+Wire Wire Line
+	5475 5000 5475 5400
+Wire Wire Line
+	5475 5400 5550 5400
+Wire Wire Line
+	5550 5400 5550 5800
+Wire Wire Line
+	5550 5800 5600 5800
+Connection ~ 5550 5400
+Wire Wire Line
+	5550 5800 5550 6250
+Wire Wire Line
+	5550 6250 5650 6250
+Connection ~ 5550 5800
+NoConn ~ 6550 6250
+NoConn ~ 6500 5800
+NoConn ~ 6450 5400
+NoConn ~ 6375 5000
 $EndSCHEMATC

Commit message: message
Parts:
- renumbered C349 to C373, C350 to C374, C351 to C375, U246 to U296, U246 to U297, U247 to U298, U149 to U299, U247 to U300, U149 to U301, U149 to U302, U248 to U303
Changed lines of the file:
@@
 $Descr A4 11693 8268
 encoding utf-8
-Sheet 89 92
+Sheet 89 101
 Title ""
 Date ""
@@
 JMP
 $Comp
-L cmos4000:4071 U247
+L cmos4000:4071 U298
 U 2 1 5B6384EB
 P 5050 1450
-F 0 "U247" H 5050 1838 60  0000 C CNN
+F 0 "U298" H 5050 1838 60  0000 C CNN
 F 1 "4071" H 5050 1732 60  0000 C CNN
 F 2 "" H 5050 1450 60  0001 C CNN
@@
 $EndComp
 $Comp
-L cmos4000:4071 U247
+L cmos4000:4071 U300
 U 4 1 5B6385BA
 P 6250 1550
-F 0 "U247" H 6250 1938 60  0000 C CNN
+F 0 "U300" H 6250 1938 60  0000 C CNN
 F 1 "4071" H 6250 1832 60  0000 C CNN
 F 2 "" H 6250 1550 60  0001 C CNN
@@
 $EndComp
 $Comp
-L cmos4000:4071 U247
+L cmos4000:4071 U300
 U 3 1 5B638625
 P 6025 2625
-F 0 "U247" H 6025 3013 60  0000 C CNN
+F 0 "U300" H 6025 3013 60  0000 C CNN
 F 1 "4071" H 6025 2907 60  0000 C CNN
 F 2 "" H 6025 2625 60  0001 C CNN
@@
 $EndComp
 $Comp
-L cmos4000:4071 U247
+L cmos4000:4071 U298
 U 1 1 5B638687
 P 4825 2725
-F 0 "U247" H 4825 3113 60  0000 C CNN
+F 0 "U298" H 4825 3113 60  0000 C CNN
 F 1 "4071" H 4825 3007 60  0000 C CNN
 F 2 "" H 4825 2725 60  0001 C CNN
@@
 $EndComp
 $Comp
-L 74xx:74LS08 U246
+L 74xx:74LS08 U296
 U 1 1 5B6386F2
 P 3650 1275
-F 0 "U246" H 3650 1663 60  0000 C CNN
+F 0 "U296" H 3650 1663 60  0000 C CNN
 F 1 "74LS08" H 3650 1557 60  0000 C CNN
 F 2 "" H 3650 1275 60  0001 C CNN
@@
 $EndComp
 $Comp
-L 74xx:74LS08 U246
+L 74xx:74LS08 U296
 U 2 1 5B638778
 P 3675 1950
-F 0 "U246" H 3675 2338 60  0000 C CNN
+F 0 "U296" H 3675 2338 60  0000 C CNN
 F 1 "74LS08" H 3675 2232 60  0000 C CNN
 F 2 "" H 3675 1950 60  0001 C CNN
@@
 $EndComp
 $Comp
-L 74xx:74LS08 U246
+L 74xx:74LS08 U297
 U 4 1 5B6387ED
 P 7850 2100
-F 0 "U246" H 7850 2488 60  0000 C CNN
+F 0 "U297" H 7850 2488 60  0000 C CNN
 F 1 "74LS08" H 7850 2382 60  0000 C CNN
 F 2 "" H 7850 2100 60  0001 C CNN
@@
 $EndComp
 $Comp
-L 74xx:74LS08 U246
+L 74xx:74LS08 U297
 U 3 1 5B638869
 P 4175 6200
-F 0 "U246" H 4175 6588 60  0000 C CNN
+F 0 "U297" H 4175 6588 60  0000 C CNN
 F 1 "74LS08" H 4175 6482 60  0000 C CNN
 F 2 "" H 4175 6200 60  0001 C CNN
@@
 	7250 1550 7250 2000
 $Comp
-L myCpu-rescue:VCC #PWR0645
+L myCpu-rescue:VCC #PWR0701
 U 1 1 5B63A0B0
 P 4925 3625
-F 0 "#PWR0645" H 4925 3475 50  0001 C CNN
+F 0 "#PWR0701" H 4925 3475 50  0001 C CNN
 F 1 "VCC" H 4942 3798 50  0000 C CNN
 F 2 "" H 4925 3625 50  0000 C CNN
@@
 $EndComp
 $Comp
-L power:GND #PWR0643
+L power:GND #PWR0699
 U 1 1 5B63A0F1
 P 4425 3625
-F 0 "#PWR0643" H 4425 3625 30  0001 C CNN
+F 0 "#PWR0699" H 4425 3625 30  0001 C CNN
 F 1 "GND" H 4425 3555 30  0001 C CNN
 F 2 "" H 4425 3625 60  0001 C CNN
@@
 $EndComp
 $Comp
-L pspice:C C350
+L pspice:C C374
 U 1 1 5B63A150
 P 4675 3625
-F 0 "C350" V 4360 3625 50  0000 C CNN
+F 0 "C374" V 4360 3625 50  0000 C CNN
 F 1 "100nF" V 4451 3625 50  0000 C CNN
 F 2 "" H 4675 3625 60  0001 C CNN
@@
 $EndComp
 $Comp
-L myCpu-rescue:VCC #PWR0644
+L myCpu-rescue:VCC #PWR0700
 U 1 1 5B63A369
 P 4500 6850
-F 0 "#PWR0644" H 4500 6700 50  0001 C CNN
+F 0 "#PWR0700" H 4500 6700 50  0001 C CNN
 F 1 "VCC" H 4517 7023 50  0000 C CNN
 F 2 "" H 4500 6850 50  0000 C CNN
@@
 $EndComp
 $Comp
-L power:GND #PWR0642
+L power:GND #PWR0698
 U 1 1 5B63A36F
 P 4000 6850
-F 0 "#PWR0642" H 4000 6850 30  0001 C CNN
+F 0 "#PWR0698" H 4000 6850 30  0001 C CNN
 F 1 "GND" H 4000 6780 30  0001 C CNN
 F 2 "" H 4000 6850 60  0001 C CNN
@@
 $EndComp
 $Comp
-L pspice:C C349
+L pspice:C C373
 U 1 1 5B63A375
 P 4250 6850
-F 0 "C349" V 3935 6850 50  0000 C CNN
+F 0 "C373" V 3935 6850 50  0000 C CNN
 F 1 "100nF" V 4026 6850 50  0000 C CNN
 F 2 "" H 4250 6850 60  0001 C CNN
@@
 NoConn ~ 2950 6575
 $Comp
-L 74xx:74LS04 U248
+L 74xx:74LS04 U303
 U 1 1 5B70DE9D
 P 8900 2100
-F 0 "U248" H 8900 2437 60  0000 C CNN
+F 0 "U303" H 8900 2437 60  0000 C CNN
 F 1 "74LS04" H 8900 2331 60  0000 C CNN
 F 2 "" H 8900 2100 60  0001 C CNN
@@
 PC_INC
 $Comp
-L myCpu-rescue:VCC #PWR0646
+L myCpu-rescue:VCC #PWR0702
 U 1 1 5B70DFD2
 P 6075 4525
-F 0 "#PWR0646" H 6075 4375 50  0001 C CNN
+F 0 "#PWR0702" H 6075 4375 50  0001 C CNN
 F 1 "VCC" H 6092 4698 50  0000 C CNN
 F 2 "" H 6075 4525 50  0000 C CNN
@@
 $EndComp
 $Comp
-L pspice:C C351
+L pspice:C C375
 U 1 1 5B70DFD8
 P 5825 4525
-F 0 "C351" V 5510 4525 50  0000 C CNN
+F 0 "C375" V 5510 4525 50  0000 C CNN
 F 1 "100nF" V 5601 4525 50  0000 C CNN
 F 2 "" H 5825 4525 60  0001 C CNN
@@
 $EndComp
 $Comp
-L 74xx:74LS04 U149
+L 74xx:74LS04 U299
 U 2 1 5B70E3FE
 P 6000 5400
-F 0 "U149" H 6000 5737 60  0000 C CNN
+F 0 "U299" H 6000 5737 60  0000 C CNN
 F 1 "74LS04" H 6000 5631 60  0000 C CNN
 F 2 "" H 6000 5400 60  0001 C CNN
@@
 $EndComp
 $Comp
-L 74xx:74LS04 U149
+L 74xx:74LS04 U301
 U 3 1 5B70E48E
 P 6050 5800
-F 0 "U149" H 6050 6137 60  0000 C CNN
+F 0 "U301" H 6050 6137 60  0000 C CNN
 F 1 "74LS04" H 6050 6031 60  0000 C CNN
 F 2 "" H 6050 5800 60  0001 C CNN
@@
 $EndComp
 $Comp
-L 74xx:74LS04 U149
+L 74xx:74LS04 U301
 U 4 1 5B70E55D
 P 6100 6250
-F 0 "U149" H 6100 6587 60  0000 C CNN
+F 0 "U301" H 6100 6587 60  0000 C CNN
 F 1 "74LS04" H 6100 6481 60  0000 C CNN
 F 2 "" H 6100 6250 60  0001 C CNN
@@
 Connection ~ 5475 5000
 $Comp
-L 74xx:74LS04 U149
+L 74xx:74LS04 U302
 U 5 1 5B70E605
 P 6150 6650
-F 0 "U149" H 6150 6987 60  0000 C CNN
+F 0 "U302" H 6150 6987 60  0000 C CNN
 F 1 "74LS04" H 6150 6881 60  0000 C CNN
 F 2 "" H 6150 6650 60  0001 C CNN
@@
 $EndComp
 $Comp
-L 74xx:74LS04 U149
+L 74xx:74LS04 U299
 U 6 1 5B70E6B0
 P 5925 5000
-F 0 "U149" H 5925 5337 60  0000 C CNN
+F 0 "U299" H 5925 5337 60  0000 C CNN
 F 1 "74LS04" H 5925 5231 60  0000 C CNN
 F 2 "" H 5925 5000 60  0001 C CNN

Commit message: .
Parts:
- renumbered C373 to C156, C374 to C157, C375 to C158, U296 to U190, U297 to U191, U298 to U192, U299 to U193, U300 to U194, U301 to U195, U302 to U196, U303 to U197
Connections:
- wire segments 37 -> 39
- no-connect marks 6 -> 7
Changed lines of the file:
@@
 $Descr A4 11693 8268
 encoding utf-8
-Sheet 89 101
+Sheet 89 75
 Title ""
 Date ""
@@
 JMP
 $Comp
-L cmos4000:4071 U298
+L cmos4000:4071 U192
 U 2 1 5B6384EB
 P 5050 1450
-F 0 "U298" H 5050 1838 60  0000 C CNN
+F 0 "U192" H 5050 1838 60  0000 C CNN
 F 1 "4071" H 5050 1732 60  0000 C CNN
 F 2 "" H 5050 1450 60  0001 C CNN
@@
 $EndComp
 $Comp
-L cmos4000:4071 U300
+L cmos4000:4071 U194
 U 4 1 5B6385BA
 P 6250 1550
-F 0 "U300" H 6250 1938 60  0000 C CNN
+F 0 "U194" H 6250 1938 60  0000 C CNN
 F 1 "4071" H 6250 1832 60  0000 C CNN
 F 2 "" H 6250 1550 60  0001 C CNN
@@
 $EndComp
 $Comp
-L cmos4000:4071 U300
+L cmos4000:4071 U194
 U 3 1 5B638625
 P 6025 2625
-F 0 "U300" H 6025 3013 60  0000 C CNN
+F 0 "U194" H 6025 3013 60  0000 C CNN
 F 1 "4071" H 6025 2907 60  0000 C CNN
 F 2 "" H 6025 2625 60  0001 C CNN
@@
 $EndComp
 $Comp
-L cmos4000:4071 U298
+L cmos4000:4071 U192
 U 1 1 5B638687
 P 4825 2725
-F 0 "U298" H 4825 3113 60  0000 C CNN
+F 0 "U192" H 4825 3113 60  0000 C CNN
 F 1 "4071" H 4825 3007 60  0000 C CNN
 F 2 "" H 4825 2725 60  0001 C CNN
@@
 $EndComp
 $Comp
-L 74xx:74LS08 U296
+L 74xx:74LS08 U190
 U 1 1 5B6386F2
 P 3650 1275
-F 0 "U296" H 3650 1663 60  0000 C CNN
+F 0 "U190" H 3650 1663 60  0000 C CNN
 F 1 "74LS08" H 3650 1557 60  0000 C CNN
 F 2 "" H 3650 1275 60  0001 C CNN
@@
 $EndComp
 $Comp
-L 74xx:74LS08 U296
+L 74xx:74LS08 U190
 U 2 1 5B638778
 P 3675 1950
-F 0 "U296" H 3675 2338 60  0000 C CNN
+F 0 "U190" H 3675 2338 60  0000 C CNN
 F 1 "74LS08" H 3675 2232 60  0000 C CNN
 F 2 "" H 3675 1950 60  0001 C CNN
@@
 $EndComp
 $Comp
-L 74xx:74LS08 U297
+L 74xx:74LS08 U191
 U 4 1 5B6387ED
 P 7850 2100
-F 0 "U297" H 7850 2488 60  0000 C CNN
+F 0 "U191" H 7850 2488 60  0000 C CNN
 F 1 "74LS08" H 7850 2382 60  0000 C CNN
 F 2 "" H 7850 2100 60  0001 C CNN
@@
 $EndComp
 $Comp
-L 74xx:74LS08 U297
+L 74xx:74LS08 U191
 U 3 1 5B638869
 P 4175 6200
-F 0 "U297" H 4175 6588 60  0000 C CNN
+F 0 "U191" H 4175 6588 60  0000 C CNN
 F 1 "74LS08" H 4175 6482 60  0000 C CNN
 F 2 "" H 4175 6200 60  0001 C CNN
@@
 	7250 1550 7250 2000
 $Comp
-L myCpu-rescue:VCC #PWR0701
+L myCpu-rescue:VCC #PWR0273
 U 1 1 5B63A0B0
 P 4925 3625
-F 0 "#PWR0701" H 4925 3475 50  0001 C CNN
+F 0 "#PWR0273" H 4925 3475 50  0001 C CNN
 F 1 "VCC" H 4942 3798 50  0000 C CNN
 F 2 "" H 4925 3625 50  0000 C CNN
@@
 $EndComp
 $Comp
-L power:GND #PWR0699
+L power:GND #PWR0271
 U 1 1 5B63A0F1
 P 4425 3625
-F 0 "#PWR0699" H 4425 3625 30  0001 C CNN
+F 0 "#PWR0271" H 4425 3625 30  0001 C CNN
 F 1 "GND" H 4425 3555 30  0001 C CNN
 F 2 "" H 4425 3625 60  0001 C CNN
@@
 $EndComp
 $Comp
-L pspice:C C374
+L pspice:C C157
 U 1 1 5B63A150
 P 4675 3625
-F 0 "C374" V 4360 3625 50  0000 C CNN
+F 0 "C157" V 4360 3625 50  0000 C CNN
 F 1 "100nF" V 4451 3625 50  0000 C CNN
 F 2 "" H 4675 3625 60  0001 C CNN
@@
 $EndComp
 $Comp
-L myCpu-rescue:VCC #PWR0700
+L myCpu-rescue:VCC #PWR0272
 U 1 1 5B63A369
 P 4500 6850
-F 0 "#PWR0700" H 4500 6700 50  0001 C CNN
+F 0 "#PWR0272" H 4500 6700 50  0001 C CNN
 F 1 "VCC" H 4517 7023 50  0000 C CNN
 F 2 "" H 4500 6850 50  0000 C CNN
@@
 $EndComp
 $Comp
-L power:GND #PWR0698
+L power:GND #PWR0270
 U 1 1 5B63A36F
 P 4000 6850
-F 0 "#PWR0698" H 4000 6850 30  0001 C CNN
+F 0 "#PWR0270" H 4000 6850 30  0001 C CNN
 F 1 "GND" H 4000 6780 30  0001 C CNN
 F 2 "" H 4000 6850 60  0001 C CNN
@@
 $EndComp
 $Comp
-L pspice:C C373
+L pspice:C C156
 U 1 1 5B63A375
 P 4250 6850
-F 0 "C373" V 3935 6850 50  0000 C CNN
+F 0 "C156" V 3935 6850 50  0000 C CNN
 F 1 "100nF" V 4026 6850 50  0000 C CNN
 F 2 "" H 4250 6850 60  0001 C CNN
@@
 NoConn ~ 2950 6575
 $Comp
-L 74xx:74LS04 U303
+L 74xx:74LS04 U197
 U 1 1 5B70DE9D
 P 8900 2100
-F 0 "U303" H 8900 2437 60  0000 C CNN
+F 0 "U197" H 8900 2437 60  0000 C CNN
 F 1 "74LS04" H 8900 2331 60  0000 C CNN
 F 2 "" H 8900 2100 60  0001 C CNN
@@
 PC_INC
 $Comp
-L myCpu-rescue:VCC #PWR0702
+L myCpu-rescue:VCC #PWR0274
 U 1 1 5B70DFD2
 P 6075 4525
-F 0 "#PWR0702" H 6075 4375 50  0001 C CNN
+F 0 "#PWR0274" H 6075 4375 50  0001 C CNN
 F 1 "VCC" H 6092 4698 50  0000 C CNN
 F 2 "" H 6075 4525 50  0000 C CNN
@@
 $EndComp
 $Comp
-L pspice:C C375
+L pspice:C C158
 U 1 1 5B70DFD8
 P 5825 4525
-F 0 "C375" V 5510 4525 50  0000 C CNN
+F 0 "C158" V 5510 4525 50  0000 C CNN
 F 1 "100nF" V 5601 4525 50  0000 C CNN
 F 2 "" H 5825 4525 60  0001 C CNN
@@
 $EndComp
 $Comp
-L 74xx:74LS04 U299
+L 74xx:74LS04 U193
 U 2 1 5B70E3FE
 P 6000 5400
-F 0 "U299" H 6000 5737 60  0000 C CNN
+F 0 "U193" H 6000 5737 60  0000 C CNN
 F 1 "74LS04" H 6000 5631 60  0000 C CNN
 F 2 "" H 6000 5400 60  0001 C CNN
@@
 $EndComp
 $Comp
-L 74xx:74LS04 U301
+L 74xx:74LS04 U195
 U 3 1 5B70E48E
 P 6050 5800
-F 0 "U301" H 6050 6137 60  0000 C CNN
+F 0 "U195" H 6050 6137 60  0000 C CNN
 F 1 "74LS04" H 6050 6031 60  0000 C CNN
 F 2 "" H 6050 5800 60  0001 C CNN
@@
 $EndComp
 $Comp
-L 74xx:74LS04 U301
+L 74xx:74LS04 U195
 U 4 1 5B70E55D
 P 6100 6250
-F 0 "U301" H 6100 6587 60  0000 C CNN
+F 0 "U195" H 6100 6587 60  0000 C CNN
 F 1 "74LS04" H 6100 6481 60  0000 C CNN
 F 2 "" H 6100 6250 60  0001 C CNN
@@
 Connection ~ 5475 5000
 $Comp
-L 74xx:74LS04 U302
+L 74xx:74LS04 U196
 U 5 1 5B70E605
 P 6150 6650
-F 0 "U302" H 6150 6987 60  0000 C CNN
+F 0 "U196" H 6150 6987 60  0000 C CNN
 F 1 "74LS04" H 6150 6881 60  0000 C CNN
 F 2 "" H 6150 6650 60  0001 C CNN
@@
 $EndComp
 $Comp
-L 74xx:74LS04 U299
+L 74xx:74LS04 U193
 U 6 1 5B70E6B0
 P 5925 5000
-F 0 "U299" H 5925 5337 60  0000 C CNN
+F 0 "U193" H 5925 5337 60  0000 C CNN
 F 1 "74LS04" H 5925 5231 60  0000 C CNN
 F 2 "" H 5925 5000 60  0001 C CNN
@@
 NoConn ~ 6450 5400
 NoConn ~ 6375 5000
+Wire Wire Line
+	5550 6250 5550 6650
+Wire Wire Line
+	5550 6650 5700 6650
+Connection ~ 5550 6250
+NoConn ~ 6600 6650
 $EndSCHEMATC

Commit message: .
Changed lines of the file:
@@
 $Descr A4 11693 8268
 encoding utf-8
-Sheet 89 75
+Sheet 89 100
 Title ""
 Date ""
@@
 L 74xx:74LS08 U190
 U 1 1 5B6386F2
-P 3650 1275
-F 0 "U190" H 3650 1663 60  0000 C CNN
-F 1 "74LS08" H 3650 1557 60  0000 C CNN
-F 2 "" H 3650 1275 60  0001 C CNN
-F 3 "" H 3650 1275 60  0001 C CNN
-	1    3650 1275
+P 3600 1175
+F 0 "U190" H 3600 1563 60  0000 C CNN
+F 1 "74LS08" H 3600 1457 60  0000 C CNN
+F 2 "" H 3600 1175 60  0001 C CNN
+F 3 "" H 3600 1175 60  0001 C CNN
+	1    3600 1175
 	1    0    0    -1
 $EndComp
@@
 	2350 1475 2350 1175
 Wire Wire Line
-	2350 1175 3050 1175
+	2350 1175 3000 1075
 Wire Wire Line
 	950  1825 2500 1825
@@
 	2500 1825 2500 1375
 Wire Wire Line
-	2500 1375 3050 1375
+	2500 1375 3000 1275
 Wire Wire Line
 	900  2125 2500 2125
@@
 	2675 2375 2950 2375
 Wire Wire Line
-	4250 1275 4450 1275
+	4200 1175 4450 1275
 Wire Wire Line
 	4450 1275 4450 1350
