File: Reg16.sch (KiCad schematic (older format))
At the start: 0 parts

Commit message: .
Changed lines of the file:
@@
 $Descr A4 11693 8268
 encoding utf-8
-Sheet 59 101
+Sheet 54 75
 Title ""
 Date ""
@@
 Comment4 ""
 $EndDescr
-$Sheet
-S 3000 1975 1575 1375
-U 8116CFC7
-F0 "RegA" 60
-F1 "Register.sch" 60
-F2 "X0" I L 3000 2100 60
-F3 "X1" I L 3000 2200 60
-F4 "X2" I L 3000 2300 60
-F5 "X3" I L 3000 2400 60
-F6 "X4" I L 3000 2550 60
-F7 "X5" I L 3000 2650 60
-F8 "X6" I L 3000 2750 60
-F9 "X7" I L 3000 2875 60
-F10 "Z0" O R 4575 2075 60
-F11 "Z1" O R 4575 2175 60
-F12 "Z2" O R 4575 2300 60
-F13 "Z3" O R 4575 2425 60
-F14 "Z4" O R 4575 2575 60
-F15 "Z5" O R 4575 2750 60
-F16 "Z6" O R 4575 2875 60
-F17 "Z7" O R 4575 3000 60
-F18 "CLK" I L 3000 3050 60
-$EndSheet
-$Sheet
-S 3125 3725 1575 1375
-U 811D8C8B
-F0 "RegB" 60
-F1 "Register.sch" 60
-F2 "X0" I L 3125 3850 60
-F3 "X1" I L 3125 3950 60
-F4 "X2" I L 3125 4050 60
-F5 "X3" I L 3125 4150 60
-F6 "X4" I L 3125 4300 60
-F7 "X5" I L 3125 4400 60
-F8 "X6" I L 3125 4500 60
-F9 "X7" I L 3125 4625 60
-F10 "Z0" O R 4700 3825 60
-F11 "Z1" O R 4700 3925 60
-F12 "Z2" O R 4700 4050 60
-F13 "Z3" O R 4700 4175 60
-F14 "Z4" O R 4700 4325 60
-F15 "Z5" O R 4700 4500 60
-F16 "Z6" O R 4700 4625 60
-F17 "Z7" O R 4700 4750 60
-F18 "CLK" I L 3125 4800 60
-$EndSheet
 Text HLabel 2750 2150 0    60   Input ~ 0
 X0

Commit message: .
Changed lines of the file:
@@
 $Descr A4 11693 8268
 encoding utf-8
-Sheet 54 75
+Sheet 69 100
 Title ""
 Date ""
@@
 Wire Wire Line
 	2300 3050 2300 4800
+$Sheet
+S 3000 1925 1575 1275
+U 5BC2A5A4
+F0 "ADDRLOW" 60
+F1 "Register.sch" 60
+F2 "CLK" I L 3000 3050 60
+F3 "X0" I L 3000 2100 60
+F4 "X1" I L 3000 2200 60
+F5 "X2" I L 3000 2300 60
+F6 "X3" I L 3000 2400 60
+F7 "X4" I L 3000 2550 60
+F8 "X5" I L 3000 2650 60
+F9 "X6" I L 3000 2750 60
+F10 "X7" I L 3000 2875 60
+F11 "Z0" O R 4575 2075 60
+F12 "Z1" O R 4575 2175 60
+F13 "Z2" O R 4575 2300 60
+F14 "Z3" O R 4575 2425 60
+F15 "Z4" O R 4575 2575 60
+F16 "Z5" O R 4575 2750 60
+F17 "Z6" O R 4575 2875 60
+F18 "Z7" O R 4575 3000 60
+$EndSheet
+$Sheet
+S 3125 3650 1575 1325
+U 5BC2A640
+F0 "ADDRHIGH" 60
+F1 "Register.sch" 60
+F2 "CLK" I L 3125 4800 60
+F3 "X0" I L 3125 3850 60
+F4 "X1" I L 3125 3950 60
+F5 "X2" I L 3125 4050 60
+F6 "X3" I L 3125 4150 60
+F7 "X4" I L 3125 4300 60
+F8 "X5" I L 3125 4400 60
+F9 "X6" I L 3125 4500 60
+F10 "X7" I L 3125 4625 60
+F11 "Z0" O R 4700 3825 60
+F12 "Z1" O R 4700 3925 60
+F13 "Z2" O R 4700 4050 60
+F14 "Z3" O R 4700 4175 60
+F15 "Z4" O R 4700 4325 60
+F16 "Z5" O R 4700 4500 60
+F17 "Z6" O R 4700 4625 60
+F18 "Z7" O R 4700 4750 60
+$EndSheet
 $EndSCHEMATC
