File: Regisersatz.sch (KiCad schematic (older format))
At the start: 7 parts, among them U43 74HC04, U44 74LS154, U45 74HC04, U46 74HC04

Commit message: X
Connections:
- net labels added: ENABLE
- wire segments 1416 -> 1414
- no-connect marks 1 -> 0
Other:
- moved on the sheet: U43B
Changed lines of the file:
@@
 $Descr A0 33110 46811 portrait
 encoding utf-8
-Sheet 23 81
+Sheet 23 90
 Title ""
 Date ""
@@
 L 74xx:74HC04 U43
 U 2 1 5B592EC3
-P 5750 14775
-F 0 "U43" H 5750 15067 40  0000 C CNN
-F 1 "74HC04" H 5750 14991 40  0000 C CNN
-F 2 "" H 5750 14775 60  0001 C CNN
-F 3 "" H 5750 14775 60  0001 C CNN
-	2    5750 14775
+P 4175 13550
+F 0 "U43" H 4175 13842 40  0000 C CNN
+F 1 "74HC04" H 4175 13766 40  0000 C CNN
+F 2 "" H 4175 13550 60  0001 C CNN
+F 3 "" H 4175 13550 60  0001 C CNN
+	2    4175 13550
 	1    0    0    -1
 $EndComp
@@
 L power:VCC #PWR045
 U 1 1 5B592F64
-P 5150 14750
-F 0 "#PWR045" H 5150 14850 30  0001 C CNN
-F 1 "VCC" H 5154 14877 30  0000 C CNN
-F 2 "" H 5150 14750 60  0001 C CNN
-F 3 "" H 5150 14750 60  0001 C CNN
-	1    5150 14750
+P 5300 15125
+F 0 "#PWR045" H 5300 15225 30  0001 C CNN
+F 1 "VCC" H 5304 15252 30  0000 C CNN
+F 2 "" H 5300 15125 60  0001 C CNN
+F 3 "" H 5300 15125 60  0001 C CNN
+	1    5300 15125
 	1    0    0    -1
 $EndComp
@@
 	1    0    0    -1
 $EndComp
-NoConn ~ 6200 14775
 $Comp
 L spice:C C39
@@
 $EndComp
 Wire Wire Line
-	5150 14750 5300 14750
-Wire Wire Line
-	5300 14750 5300 14775
-Wire Wire Line
-	5300 14775 5300 15125
-Wire Wire Line
 	5300 15125 5550 15125
-Connection ~ 5300 14775
 Wire Wire Line
 	5550 15125 5600 15125
@@
 	4550 13175 5050 13175
 Wire Wire Line
-	5050 13275 5050 14250
-Wire Wire Line
-	5050 14250 5275 14250
-Wire Wire Line
-	5275 14250 5275 14375
-Wire Wire Line
-	5275 14375 6400 14375
-Wire Wire Line
-	6400 14375 6400 14875
-Connection ~ 6400 14875
-Wire Wire Line
 	4450 12675 5050 12675
 Wire Wire Line
@@
 Text HLabel 4450 12975 0    60   Input ~ 0
 RZ_S3
+Wire Wire Line
+	10200 13700 11175 13700
+Wire Wire Line
+	11175 13700 11175 13675
+Wire Wire Line
+	4650 13525 5050 13525
+Wire Wire Line
+	5050 13525 5050 13275
+Wire Wire Line
+	4625 13550 4650 13550
+Wire Wire Line
+	4650 13550 4650 13525
+Text HLabel 3725 13550 0    60   Output ~ 0
+ENABLE
 $EndSCHEMATC

Commit message: b
Parts:
- renumbered C39 to C41, C40 to C42, C41 to C43, U43 to U45, U44 to U46, U45 to U47, U46 to U48
Changed lines of the file:
@@
 $Descr A0 33110 46811 portrait
 encoding utf-8
-Sheet 23 90
+Sheet 24 92
 Title ""
 Date ""
@@
 	14450 44700 14450 44675
 $Comp
-L 74xx:74LS154 U44
+L 74xx:74LS154 U46
 U 1 1 5B57C04D
 P 5700 13475
-F 0 "U44" H 5725 14533 60  0000 C CNN
+F 0 "U46" H 5725 14533 60  0000 C CNN
 F 1 "74LS154" H 5725 14427 60  0000 C CNN
 F 2 "" H 5700 13475 60  0001 C CNN
@@
 	2950 13125 2950 13225
 $Comp
-L 74xx:74HC04 U43
+L 74xx:74HC04 U45
 U 1 1 5B5921C2
 P 3650 13100
-F 0 "U43" H 3650 13392 40  0000 C CNN
+F 0 "U45" H 3650 13392 40  0000 C CNN
 F 1 "74HC04" H 3650 13316 40  0000 C CNN
 F 2 "" H 3650 13100 60  0001 C CNN
@@
 $EndComp
 $Comp
-L 74xx:74HC04 U43
+L 74xx:74HC04 U45
 U 3 1 5B592285
 P 6850 12675
-F 0 "U43" H 6850 12967 40  0000 C CNN
+F 0 "U45" H 6850 12967 40  0000 C CNN
 F 1 "74HC04" H 6850 12891 40  0000 C CNN
 F 2 "" H 6850 12675 60  0001 C CNN
@@
 $EndComp
 $Comp
-L 74xx:74HC04 U43
+L 74xx:74HC04 U45
 U 4 1 5B5922ED
 P 6850 12775
-F 0 "U43" H 6850 13067 40  0000 C CNN
+F 0 "U45" H 6850 13067 40  0000 C CNN
 F 1 "74HC04" H 6850 12991 40  0000 C CNN
 F 2 "" H 6850 12775 60  0001 C CNN
@@
 $EndComp
 $Comp
-L 74xx:74HC04 U43
+L 74xx:74HC04 U45
 U 5 1 5B592386
 P 6850 12875
-F 0 "U43" H 6850 13167 40  0000 C CNN
+F 0 "U45" H 6850 13167 40  0000 C CNN
 F 1 "74HC04" H 6850 13091 40  0000 C CNN
 F 2 "" H 6850 12875 60  0001 C CNN
@@
 $EndComp
 $Comp
-L 74xx:74HC04 U43
+L 74xx:74HC04 U45
 U 6 1 5B5923F2
 P 6850 12975
-F 0 "U43" H 6850 13267 40  0000 C CNN
+F 0 "U45" H 6850 13267 40  0000 C CNN
 F 1 "74HC04" H 6850 13191 40  0000 C CNN
 F 2 "" H 6850 12975 60  0001 C CNN
@@
 $EndComp
 $Comp
-L 74xx:74HC04 U45
+L 74xx:74HC04 U47
 U 1 1 5B592493
 P 6850 13075
-F 0 "U45" H 6850 13367 40  0000 C CNN
+F 0 "U47" H 6850 13367 40  0000 C CNN
 F 1 "74HC04" H 6850 13291 40  0000 C CNN
 F 2 "" H 6850 13075 60  0001 C CNN
@@
 $EndComp
 $Comp
-L 74xx:74HC04 U45
+L 74xx:74HC04 U47
 U 2 1 5B59253B
 P 6850 13175
-F 0 "U45" H 6850 13467 40  0000 C CNN
+F 0 "U47" H 6850 13467 40  0000 C CNN
 F 1 "74HC04" H 6850 13391 40  0000 C CNN
 F 2 "" H 6850 13175 60  0001 C CNN
@@
 $EndComp
 $Comp
-L 74xx:74HC04 U45
+L 74xx:74HC04 U47
 U 3 1 5B5925EC
 P 6850 13275
-F 0 "U45" H 6850 13567 40  0000 C CNN
+F 0 "U47" H 6850 13567 40  0000 C CNN
 F 1 "74HC04" H 6850 13491 40  0000 C CNN
 F 2 "" H 6850 13275 60  0001 C CNN
@@
 $EndComp
 $Comp
-L 74xx:74HC04 U45
+L 74xx:74HC04 U47
 U 4 1 5B592674
 P 6850 13375
-F 0 "U45" H 6850 13667 40  0000 C CNN
+F 0 "U47" H 6850 13667 40  0000 C CNN
 F 1 "74HC04" H 6850 13591 40  0000 C CNN
 F 2 "" H 6850 13375 60  0001 C CNN
@@
 $EndComp
 $Comp
-L 74xx:74HC04 U45
+L 74xx:74HC04 U47
 U 5 1 5B592707
 P 6850 13475
-F 0 "U45" H 6850 13767 40  0000 C CNN
+F 0 "U47" H 6850 13767 40  0000 C CNN
 F 1 "74HC04" H 6850 13691 40  0000 C CNN
 F 2 "" H 6850 13475 60  0001 C CNN
@@
 $EndComp
 $Comp
-L 74xx:74HC04 U45
+L 74xx:74HC04 U47
 U 6 1 5B592787
 P 6850 13575
-F 0 "U45" H 6850 13867 40  0000 C CNN
+F 0 "U47" H 6850 13867 40  0000 C CNN
 F 1 "74HC04" H 6850 13791 40  0000 C CNN
 F 2 "" H 6850 13575 60  0001 C CNN
@@
 $EndComp
 $Comp
-L 74xx:74HC04 U46
+L 74xx:74HC04 U48
 U 1 1 5B5928BE
 P 6850 13675
-F 0 "U46" H 6850 13967 40  0000 C CNN
+F 0 "U48" H 6850 13967 40  0000 C CNN
 F 1 "74HC04" H 6850 13891 40  0000 C CNN
 F 2 "" H 6850 13675 60  0001 C CNN
@@
 $EndComp
 $Comp
-L 74xx:74HC04 U46
+L 74xx:74HC04 U48
 U 2 1 5B59298D
 P 6850 13775
-F 0 "U46" H 6850 14067 40  0000 C CNN
+F 0 "U48" H 6850 14067 40  0000 C CNN
 F 1 "74HC04" H 6850 13991 40  0000 C CNN
 F 2 "" H 6850 13775 60  0001 C CNN
@@
 $EndComp
 $Comp
-L 74xx:74HC04 U46
+L 74xx:74HC04 U48
 U 3 1 5B592A24
 P 6850 13875
-F 0 "U46" H 6850 14167 40  0000 C CNN
+F 0 "U48" H 6850 14167 40  0000 C CNN
 F 1 "74HC04" H 6850 14091 40  0000 C CNN
 F 2 "" H 6850 13875 60  0001 C CNN
@@
 $EndComp
 $Comp
-L 74xx:74HC04 U46
+L 74xx:74HC04 U48
 U 4 1 5B592ABA
 P 6850 13975
-F 0 "U46" H 6850 14267 40  0000 C CNN
+F 0 "U48" H 6850 14267 40  0000 C CNN
 F 1 "74HC04" H 6850 14191 40  0000 C CNN
 F 2 "" H 6850 13975 60  0001 C CNN
@@
 $EndComp
 $Comp
-L 74xx:74HC04 U46
+L 74xx:74HC04 U48
 U 5 1 5B592B5F
 P 6850 14075
-F 0 "U46" H 6850 14367 40  0000 C CNN
+F 0 "U48" H 6850 14367 40  0000 C CNN
 F 1 "74HC04" H 6850 14291 40  0000 C CNN
 F 2 "" H 6850 14075 60  0001 C CNN
@@
 $EndComp
 $Comp
-L 74xx:74HC04 U46
+L 74xx:74HC04 U48
 U 6 1 5B592C09
 P 6850 14175
-F 0 "U46" H 6850 14467 40  0000 C CNN
+F 0 "U48" H 6850 14467 40  0000 C CNN
 F 1 "74HC04" H 6850 14391 40  0000 C CNN
 F 2 "" H 6850 14175 60  0001 C CNN
@@
 $EndComp
 $Comp
-L 74xx:74HC04 U43
+L 74xx:74HC04 U45
 U 2 1 5B592EC3
 P 4175 13550
-F 0 "U43" H 4175 13842 40  0000 C CNN
+F 0 "U45" H 4175 13842 40  0000 C CNN
 F 1 "74HC04" H 4175 13766 40  0000 C CNN
 F 2 "" H 4175 13550 60  0001 C CNN
@@
 $EndComp
 $Comp
-L power:VCC #PWR045
+L power:VCC #PWR056
 U 1 1 5B592F64
 P 5300 15125
-F 0 "#PWR045" H 5300 15225 30  0001 C CNN
+F 0 "#PWR056" H 5300 15225 30  0001 C CNN
 F 1 "VCC" H 5304 15252 30  0000 C CNN
 F 2 "" H 5300 15125 60  0001 C CNN
@@
 $EndComp
 $Comp
-L power:GND #PWR046
+L power:GND #PWR057
 U 1 1 5B592FC6
 P 6400 14875
-F 0 "#PWR046" H 6400 14875 30  0001 C CNN
+F 0 "#PWR057" H 6400 14875 30  0001 C CNN
 F 1 "GND" H 6400 14805 30  0001 C CNN
 F 2 "" H 6400 14875 60  0001 C CNN
@@
 $EndComp
 $Comp
-L spice:C C39
+L spice:C C41
 U 1 1 5B5A8F5C
 P 5800 15125
-F 0 "C39" V 5513 15125 60  0000 C CNN
+F 0 "C41" V 5513 15125 60  0000 C CNN
 F 1 "100nF" V 5619 15125 60  0000 C CNN
 F 2 "" H 5800 15125 60  0000 C CNN
@@
 $EndComp
 $Comp
-L spice:C C40
+L spice:C C42
 U 1 1 5B5A902B
 P 5850 15450
-F 0 "C40" V 5563 15450 60  0000 C CNN
+F 0 "C42" V 5563 15450 60  0000 C CNN
 F 1 "100nF" V 5669 15450 60  0000 C CNN
 F 2 "" H 5850 15450 60  0000 C CNN
@@
 $EndComp
 $Comp
-L spice:C C41
+L spice:C C43
 U 1 1 5B5A90F6
 P 5875 15800
-F 0 "C41" V 5588 15800 60  0000 C CNN
+F 0 "C43" V 5588 15800 60  0000 C CNN
 F 1 "100nF" V 5694 15800 60  0000 C CNN
 F 2 "" H 5875 15800 60  0000 C CNN

Commit message: tst
Connections:
- wire segments 1414 -> 1512
Other:
- moved on the sheet: C41, C42, C43, U45A, U45B, U45C, U45D, U45E, U45F, U47A, U47B, U47C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

Commit message: message
Parts:
- renumbered C41 to C65, C42 to C66, C43 to C67, U45 to U86, U45 to U87, U46 to U88, U48 to U89, U48 to U90, U45 to U91, U47 to U92, U48 to U93, U47 to U94, U47 to U95
Changed lines of the file:
@@
 $Descr A0 33110 46811 portrait
 encoding utf-8
-Sheet 24 92
+Sheet 24 101
 Title ""
 Date ""
@@
 	14450 44700 14450 44675
 $Comp
-L 74xx:74LS154 U46
+L 74xx:74LS154 U88
 U 1 1 5B57C04D
 P 3475 13425
-F 0 "U46" H 3500 14483 60  0000 C CNN
+F 0 "U88" H 3500 14483 60  0000 C CNN
 F 1 "74LS154" H 3500 14377 60  0000 C CNN
 F 2 "" H 3475 13425 60  0001 C CNN
@@
 	725  13075 725  13175
 $Comp
-L 74xx:74HC04 U45
+L 74xx:74HC04 U86
 U 1 1 5B5921C2
 P 1425 13050
-F 0 "U45" H 1425 13342 40  0000 C CNN
+F 0 "U86" H 1425 13342 40  0000 C CNN
 F 1 "74HC04" H 1425 13266 40  0000 C CNN
 F 2 "" H 1425 13050 60  0001 C CNN
@@
 $EndComp
 $Comp
-L 74xx:74HC04 U45
+L 74xx:74HC04 U87
 U 3 1 5B592285
 P 5175 11700
-F 0 "U45" H 5175 11992 40  0000 C CNN
+F 0 "U87" H 5175 11992 40  0000 C CNN
 F 1 "74HC04" H 5175 11916 40  0000 C CNN
 F 2 "" H 5175 11700 60  0001 C CNN
@@
 $EndComp
 $Comp
-L 74xx:74HC04 U45
+L 74xx:74HC04 U91
 U 4 1 5B5922ED
 P 5200 12150
-F 0 "U45" H 5200 12442 40  0000 C CNN
+F 0 "U91" H 5200 12442 40  0000 C CNN
 F 1 "74HC04" H 5200 12366 40  0000 C CNN
 F 2 "" H 5200 12150 60  0001 C CNN
@@
 $EndComp
 $Comp
-L 74xx:74HC04 U45
+L 74xx:74HC04 U91
 U 6 1 5B5923F2
 P 6925 12050
-F 0 "U45" H 6925 12342 40  0000 C CNN
+F 0 "U91" H 6925 12342 40  0000 C CNN
 F 1 "74HC04" H 6925 12266 40  0000 C CNN
 F 2 "" H 6925 12050 60  0001 C CNN
@@
 $EndComp
 $Comp
-L 74xx:74HC04 U47
+L 74xx:74HC04 U92
 U 1 1 5B592493
 P 6850 12475
-F 0 "U47" H 6850 12767 40  0000 C CNN
+F 0 "U92" H 6850 12767 40  0000 C CNN
 F 1 "74HC04" H 6850 12691 40  0000 C CNN
 F 2 "" H 6850 12475 60  0001 C CNN
@@
 $EndComp
 $Comp
-L 74xx:74HC04 U47
+L 74xx:74HC04 U95
 U 2 1 5B59253B
 P 7025 14600
-F 0 "U47" H 7025 14892 40  0000 C CNN
+F 0 "U95" H 7025 14892 40  0000 C CNN
 F 1 "74HC04" H 7025 14816 40  0000 C CNN
 F 2 "" H 7025 14600 60  0001 C CNN
@@
 $EndComp
 $Comp
-L 74xx:74HC04 U47
+L 74xx:74HC04 U95
 U 3 1 5B5925EC
 P 6950 13375
-F 0 "U47" H 6950 13667 40  0000 C CNN
+F 0 "U95" H 6950 13667 40  0000 C CNN
 F 1 "74HC04" H 6950 13591 40  0000 C CNN
 F 2 "" H 6950 13375 60  0001 C CNN
@@
 $EndComp
 $Comp
-L 74xx:74HC04 U47
+L 74xx:74HC04 U94
 U 4 1 5B592674
 P 6925 12850
-F 0 "U47" H 6925 13142 40  0000 C CNN
+F 0 "U94" H 6925 13142 40  0000 C CNN
 F 1 "74HC04" H 6925 13066 40  0000 C CNN
 F 2 "" H 6925 12850 60  0001 C CNN
@@
 $EndComp
 $Comp
-L 74xx:74HC04 U47
+L 74xx:74HC04 U95
 U 5 1 5B592707
 P 7025 14025
-F 0 "U47" H 7025 14317 40  0000 C CNN
+F 0 "U95" H 7025 14317 40  0000 C CNN
 F 1 "74HC04" H 7025 14241 40  0000 C CNN
 F 2 "" H 7025 14025 60  0001 C CNN
@@
 $EndComp
 $Comp
-L 74xx:74HC04 U47
+L 74xx:74HC04 U92
 U 6 1 5B592787
 P 5200 12950
-F 0 "U47" H 5200 13242 40  0000 C CNN
+F 0 "U92" H 5200 13242 40  0000 C CNN
 F 1 "74HC04" H 5200 13166 40  0000 C CNN
 F 2 "" H 5200 12950 60  0001 C CNN
@@
 $EndComp
 $Comp
-L 74xx:74HC04 U48
+L 74xx:74HC04 U89
 U 1 1 5B5928BE
 P 5175 13325
-F 0 "U48" H 5175 13617 40  0000 C CNN
+F 0 "U89" H 5175 13617 40  0000 C CNN
 F 1 "74HC04" H 5175 13541 40  0000 C CNN
 F 2 "" H 5175 13325 60  0001 C CNN
@@
 $EndComp
 $Comp
-L 74xx:74HC04 U48
+L 74xx:74HC04 U90
 U 2 1 5B59298D
 P 5175 13900
-F 0 "U48" H 5175 14192 40  0000 C CNN
+F 0 "U90" H 5175 14192 40  0000 C CNN
 F 1 "74HC04" H 5175 14116 40  0000 C CNN
 F 2 "" H 5175 13900 60  0001 C CNN
@@
 $EndComp
 $Comp
-L 74xx:74HC04 U48
+L 74xx:74HC04 U89
 U 3 1 5B592A24
 P 5150 14325
-F 0 "U48" H 5150 14617 40  0000 C CNN
+F 0 "U89" H 5150 14617 40  0000 C CNN
 F 1 "74HC04" H 5150 14541 40  0000 C CNN
 F 2 "" H 5150 14325 60  0001 C CNN
@@
 $EndComp
 $Comp
-L 74xx:74HC04 U48
+L 74xx:74HC04 U90
 U 4 1 5B592ABA
 P 5200 14800
-F 0 "U48" H 5200 15092 40  0000 C CNN
+F 0 "U90" H 5200 15092 40  0000 C CNN
 F 1 "74HC04" H 5200 15016 40  0000 C CNN
 F 2 "" H 5200 14800 60  0001 C CNN
@@
 $EndComp
 $Comp
-L 74xx:74HC04 U48
+L 74xx:74HC04 U93
 U 5 1 5B592B5F
 P 5775 13675
-F 0 "U48" H 5775 13967 40  0000 C CNN
+F 0 "U93" H 5775 13967 40  0000 C CNN
 F 1 "74HC04" H 5775 13891 40  0000 C CNN
 F 2 "" H 5775 13675 60  0001 C CNN
@@
 $EndComp
 $Comp
-L 74xx:74HC04 U48
+L 74xx:74HC04 U93
 U 6 1 5B592C09
 P 7850 14425
-F 0 "U48" H 7850 14717 40  0000 C CNN
+F 0 "U93" H 7850 14717 40  0000 C CNN
 F 1 "74HC04" H 7850 14641 40  0000 C CNN
 F 2 "" H 7850 14425 60  0001 C CNN
@@
 $EndComp
 $Comp
-L 74xx:74HC04 U45
+L 74xx:74HC04 U87
 U 2 1 5B592EC3
 P 1950 13500
-F 0 "U45" H 1950 13792 40  0000 C CNN
+F 0 "U87" H 1950 13792 40  0000 C CNN
 F 1 "74HC04" H 1950 13716 40  0000 C CNN
 F 2 "" H 1950 13500 60  0001 C CNN
@@
 $EndComp
 $Comp
-L power:VCC #PWR056
+L power:VCC #PWR0104
 U 1 1 5B592F64
 P 3050 23300
-F 0 "#PWR056" H 3050 23400 30  0001 C CNN
+F 0 "#PWR0104" H 3050 23400 30  0001 C CNN
 F 1 "VCC" H 3054 23427 30  0000 C CNN
 F 2 "" H 3050 23300 60  0001 C CNN
@@
 $EndComp
 $Comp
-L power:GND #PWR057
+L power:GND #PWR0105
 U 1 1 5B592FC6
 P 4150 23050
-F 0 "#PWR057" H 4150 23050 30  0001 C CNN
+F 0 "#PWR0105" H 4150 23050 30  0001 C CNN
 F 1 "GND" H 4150 22980 30  0001 C CNN
 F 2 "" H 4150 23050 60  0001 C CNN
@@
 $EndComp
 $Comp
-L spice:C C41
+L spice:C C65
 U 1 1 5B5A8F5C
 P 3550 23300
-F 0 "C41" V 3263 23300 60  0000 C CNN
+F 0 "C65" V 3263 23300 60  0000 C CNN
 F 1 "100nF" V 3369 23300 60  0000 C CNN
 F 2 "" H 3550 23300 60  0000 C CNN
@@
 $EndComp
 $Comp
-L spice:C C42
+L spice:C C66
 U 1 1 5B5A902B
 P 3600 23625
-F 0 "C42" V 3313 23625 60  0000 C CNN
+F 0 "C66" V 3313 23625 60  0000 C CNN
 F 1 "100nF" V 3419 23625 60  0000 C CNN
 F 2 "" H 3600 23625 60  0000 C CNN
@@
 $EndComp
 $Comp
-L spice:C C43
+L spice:C C67
 U 1 1 5B5A90F6
 P 3625 23975
-F 0 "C43" V 3338 23975 60  0000 C CNN
+F 0 "C67" V 3338 23975 60  0000 C CNN
 F 1 "100nF" V 3444 23975 60  0000 C CNN
 F 2 "" H 3625 23975 60  0000 C CNN
@@
 ENABLE
 $Comp
-L 74xx:74HC04 U45
+L 74xx:74HC04 U87
 U 5 1 5B592386
 P 5250 12500
-F 0 "U45" H 5250 12792 40  0000 C CNN
+F 0 "U87" H 5250 12792 40  0000 C CNN
 F 1 "74HC04" H 5250 12716 40  0000 C CNN
 F 2 "" H 5250 12500 60  0001 C CNN

Commit message: .
Parts:
- renumbered U86 to U89, U87 to U90, U88 to U91, U89 to U92, U90 to U93, U91 to U94, U92 to U95, U93 to U96, U94 to U97, U95 to U98
Connections:
- wire segments 1512 -> 1514

Commit message: .
Connections:
- wire segments 1514 -> 1512
