File: Register.sch (KiCad schematic (older format))
At the start: 16 parts

Commit message: X
Connections:
- wire segments 148 -> 149
Changed lines of the file:
@@
 $Descr A3 11693 16535 portrait
 encoding utf-8
-Sheet 73 81
+Sheet 90 90
 Title ""
 Date ""
@@
 Wire Wire Line
 	2150 7475 2150 7525
-Wire Wire Line
-	2150 7975 2325 7975
 Wire Wire Line
 	2475 9400 2200 9400
@@
 Wire Wire Line
 	2150 7525 2150 7975
-Wire Wire Line
-	2325 7475 2150 7475
 Wire Wire Line
 	1500 9400 2200 9400
@@
 Wire Wire Line
 	2075 4125 2400 4125
+Wire Wire Line
+	2150 7975 2425 7975
+Wire Wire Line
+	2425 7725 2325 7725
+Wire Wire Line
+	2150 7475 2425 7475
 $EndSCHEMATC

Commit message: b
Parts:
- gave numbers to parts that had none: 12

Commit message: message
Parts:
- renumbered C44 to C68, C45 to C69, C46 to C70, C47 to C71, C48 to C72, C49 to C73, C50 to C74, C51 to C75, U49 to U96, U50 to U97, U51 to U98, U52 to U99

Commit message: .
Parts:
- renumbered C71 to C?, C70 to C?, C68 to C?, C69 to C?, C73 to C?, C74 to C?, C72 to C?, C75 to C?, U96 to U?, U97 to U?, U98 to U?, U99 to U?
Connections:
- wire segments 149 -> 146

Commit message: .
Parts:
- gave numbers to parts that had none: 12
