File: SREG.sch (KiCad schematic (older format))
At the start: 3 parts

Commit message: b
Parts:
- gave numbers to parts that had none: 2
Changed lines of the file:
@@
 $Descr A4 11693 8268
 encoding utf-8
-Sheet 89 90
+Sheet 89 92
 Title ""
 Date ""
@@
 CLK
 $Comp
-L 74xx:74LS109 U?
+L 74xx:74LS109 U239
 U 1 1 64EF87E3
 P 5125 3775
-F 0 "U?" H 5125 4675 60  0000 C CNN
+F 0 "U239" H 5125 4675 60  0000 C CNN
 F 1 "74LS109" H 5125 4569 60  0000 C CNN
 F 2 "" H 5125 3775 60  0001 C CNN
@@
 $EndComp
 $Comp
-L 74xx:74LS109 U?
+L 74xx:74LS109 U239
 U 2 1 64EF8A26
 P 5150 5750
-F 0 "U?" H 5150 6750 60  0000 C CNN
+F 0 "U239" H 5150 6750 60  0000 C CNN
 F 1 "74LS109" H 5150 6644 60  0000 C CNN
 F 2 "" H 5150 5750 60  0001 C CNN
@@
 $EndSheet
 $Comp
-L power:GND #PWR?
+L power:GND #PWR0620
 U 1 1 64F0B72B
 P 4600 2700
-F 0 "#PWR?" H 4600 2700 30  0001 C CNN
+F 0 "#PWR0620" H 4600 2700 30  0001 C CNN
 F 1 "GND" H 4600 2630 30  0001 C CNN
 F 2 "" H 4600 2700 59  0001 C CNN
@@
 $EndComp
 $Comp
-L power:VCC #PWR?
+L power:VCC #PWR0621
 U 1 1 64F0B75A
 P 5100 2700
-F 0 "#PWR?" H 5100 2800 30  0001 C CNN
+F 0 "#PWR0621" H 5100 2800 30  0001 C CNN
 F 1 "VCC" H 5104 2827 30  0000 C CNN
 F 2 "" H 5100 2700 59  0001 C CNN
@@
 $EndComp
 $Comp
-L pspice:C C?
+L pspice:C C338
 U 1 1 64F0B79E
 P 4850 2700
-F 0 "C?" V 4535 2700 50  0000 C CNN
+F 0 "C338" V 4535 2700 50  0000 C CNN
 F 1 "100nF" V 4626 2700 50  0000 C CNN
 F 2 "" H 4850 2700 59  0001 C CNN

Commit message: message
Parts:
- renumbered C338 to C362, U239 to U286
Changed lines of the file:
@@
 $Descr A4 11693 8268
 encoding utf-8
-Sheet 89 92
+Sheet 89 101
 Title ""
 Date ""
@@
 CLK
 $Comp
-L 74xx:74LS109 U239
+L 74xx:74LS109 U286
 U 1 1 64EF87E3
 P 5125 3775
-F 0 "U239" H 5125 4675 60  0000 C CNN
+F 0 "U286" H 5125 4675 60  0000 C CNN
 F 1 "74LS109" H 5125 4569 60  0000 C CNN
 F 2 "" H 5125 3775 60  0001 C CNN
@@
 $EndComp
 $Comp
-L 74xx:74LS109 U239
+L 74xx:74LS109 U286
 U 2 1 64EF8A26
 P 5150 5750
-F 0 "U239" H 5150 6750 60  0000 C CNN
+F 0 "U286" H 5150 6750 60  0000 C CNN
 F 1 "74LS109" H 5150 6644 60  0000 C CNN
 F 2 "" H 5150 5750 60  0001 C CNN
@@
 $EndSheet
 $Comp
-L power:GND #PWR0620
+L power:GND #PWR0676
 U 1 1 64F0B72B
 P 4600 2700
-F 0 "#PWR0620" H 4600 2700 30  0001 C CNN
+F 0 "#PWR0676" H 4600 2700 30  0001 C CNN
 F 1 "GND" H 4600 2630 30  0001 C CNN
 F 2 "" H 4600 2700 59  0001 C CNN
@@
 $EndComp
 $Comp
-L power:VCC #PWR0621
+L power:VCC #PWR0677
 U 1 1 64F0B75A
 P 5100 2700
-F 0 "#PWR0621" H 5100 2800 30  0001 C CNN
+F 0 "#PWR0677" H 5100 2800 30  0001 C CNN
 F 1 "VCC" H 5104 2827 30  0000 C CNN
 F 2 "" H 5100 2700 59  0001 C CNN
@@
 $EndComp
 $Comp
-L pspice:C C338
+L pspice:C C362
 U 1 1 64F0B79E
 P 4850 2700
-F 0 "C338" V 4535 2700 50  0000 C CNN
+F 0 "C362" V 4535 2700 50  0000 C CNN
 F 1 "100nF" V 4626 2700 50  0000 C CNN
 F 2 "" H 4850 2700 59  0001 C CNN

Commit message: .
Parts:
- renumbered C362 to C385, U286 to U347
Connections:
- wire segments 20 -> 27
Changed lines of the file:
@@
 $Descr A4 11693 8268
 encoding utf-8
-Sheet 89 87
+Sheet 100 100
 Title ""
 Date ""
@@
 CLK
 $Comp
-L 74xx:74LS109 U286
+L 74xx:74LS109 U347
 U 1 1 64EF87E3
 P 5125 3775
-F 0 "U286" H 5125 4675 60  0000 C CNN
+F 0 "U347" H 5125 4675 60  0000 C CNN
 F 1 "74LS109" H 5125 4569 60  0000 C CNN
 F 2 "" H 5125 3775 60  0001 C CNN
@@
 $EndComp
 $Comp
-L 74xx:74LS109 U286
+L 74xx:74LS109 U347
 U 2 1 64EF8A26
 P 5150 5750
-F 0 "U286" H 5150 6750 60  0000 C CNN
+F 0 "U347" H 5150 6750 60  0000 C CNN
 F 1 "74LS109" H 5150 6644 60  0000 C CNN
 F 2 "" H 5150 5750 60  0001 C CNN
@@
 	1    0    0    -1
 $EndComp
-$Sheet
-S 7575 4550 925  925
-U 64EF8B84
-F0 "Sheet64EF8B83" 59
-F1 "REGISTER.sch" 59
-$EndSheet
 $Comp
-L power:GND #PWR0676
+L power:GND #PWR0728
 U 1 1 64F0B72B
 P 4600 2700
-F 0 "#PWR0676" H 4600 2700 30  0001 C CNN
+F 0 "#PWR0728" H 4600 2700 30  0001 C CNN
 F 1 "GND" H 4600 2630 30  0001 C CNN
 F 2 "" H 4600 2700 59  0001 C CNN
@@
 $EndComp
 $Comp
-L power:VCC #PWR0677
+L power:VCC #PWR0729
 U 1 1 64F0B75A
 P 5100 2700
-F 0 "#PWR0677" H 5100 2800 30  0001 C CNN
+F 0 "#PWR0729" H 5100 2800 30  0001 C CNN
 F 1 "VCC" H 5104 2827 30  0000 C CNN
 F 2 "" H 5100 2700 59  0001 C CNN
@@
 $EndComp
 $Comp
-L pspice:C C362
+L pspice:C C385
 U 1 1 64F0B79E
 P 4850 2700
-F 0 "C362" V 4535 2700 50  0000 C CNN
+F 0 "C385" V 4535 2700 50  0000 C CNN
 F 1 "100nF" V 4626 2700 50  0000 C CNN
 F 2 "" H 4850 2700 59  0001 C CNN
@@
 Connection ~ 5125 3075
 Wire Wire Line
-	5125 4950 5150 4950
-Wire Wire Line
 	5125 3075 5125 4475
 Connection ~ 5125 4475
 Wire Wire Line
 	5125 4475 5125 4950
-Wire Wire Line
-	5150 4950 5150 6550
-Connection ~ 5150 4950
 Wire Wire Line
 	4000 3825 4475 3825
@@
 Text Label 4250 3825 0    59   ~ 0
 CLK
-Text Label 4400 5750 2    59   ~ 0
+Text Label 4325 5775 2    59   ~ 0
 CLK
-NoConn ~ 5900 6000
 NoConn ~ 5775 4025
 Text HLabel 3350 3725 0    59   Input ~ 0
@@
 	4150 5625 4150 5500
 Wire Wire Line
-	4150 5500 4400 5500
-Wire Wire Line
 	4125 5625 4125 6000
-Wire Wire Line
-	4125 6000 4400 6000
 Connection ~ 4125 5625
 Wire Wire Line
 	4125 5625 4150 5625
-Text HLabel 5900 5500 2    59   Output ~ 0
+Text HLabel 6275 5500 2    59   Output ~ 0
 Zout
 Text HLabel 5775 3525 2    59   Output ~ 0
 Cout
+Wire Wire Line
+	5275 5050 5225 5050
+Wire Wire Line
+	5225 4950 5225 5050
+NoConn ~ 5900 6000
+Wire Wire Line
+	4150 5500 4400 5500
+Wire Wire Line
+	4325 5775 4400 5775
+Wire Wire Line
+	4400 5775 4400 5750
+Wire Wire Line
+	4125 6000 4400 6000
+Wire Wire Line
+	5275 6550 5150 6550
+Wire Wire Line
+	5275 5050 5275 6550
+Wire Wire Line
+	5125 4950 5150 4950
+Wire Wire Line
+	5150 4950 5225 4950
+Connection ~ 5150 4950
+Wire Wire Line
+	5900 5500 6275 5500
 $EndSCHEMATC
