File: STACK.sch (KiCad schematic (older format))
At the start: 32 parts

Commit message: b
Parts:
- gave numbers to parts that had none: 32

Commit message: message
Parts:
- renumbered C306 to C330, C307 to C331, C308 to C332, C309 to C333, C310 to C334, C311 to C335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

Commit message: .
Parts:
- renumbered C330 to C122, C331 to C123, C332 to C124, C333 to C125, C334 to C126, C335 to C127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
