File: Schifter.sch (KiCad schematic (older format))
At the start: 0 parts

Commit message: message
Connections:
- net labels added: GND, Z0, Z1, Z2, Z3, Z4, Z5, Z6, Z7
- net labels removed: Cin
- wire segments 0 -> 293
