File: Alu/16-1MUX.sch (KiCad schematic (older format))
At the start: 6 parts, among them U10 74LS151, U8 74LS151, U9 74LS157

Commit message: footprints
Parts:
- C43, C44, C45: footprint (none) -> Capacitor_SMD:C_0805_2012Metric
Changed lines of the file:
@@
 $Descr A4 11693 8268
 encoding utf-8
-Sheet 108 156
+Sheet 139 191
 Title ""
 Date ""
@@
 AR Path="/5C1207F9/5B1EC381/5CEE5429" Ref="U29"  Part="1"
 AR Path="/5C1207F9/5B1EC399/5CEE5429" Ref="U32"  Part="1"
-F 0 "U11" V 2478 5398 60  0000 L CNN
+F 0 "U32" V 2478 5398 60  0000 L CNN
 F 1 "74LS151" V 2372 5398 60  0000 L CNN
 F 2 "" H 2425 4650 60  0001 C CNN
@@
 AR Path="/5C1207F9/5B1EC381/5CF16234" Ref="U30"  Part="1"
 AR Path="/5C1207F9/5B1EC399/5CF16234" Ref="U33"  Part="1"
-F 0 "U12" V 3053 1966 60  0000 R CNN
+F 0 "U33" V 3053 1966 60  0000 R CNN
 F 1 "74LS157" V 2947 1966 60  0000 R CNN
 F 2 "" H 3000 2625 60  0001 C CNN
 F 3 "" H 3000 2625 60  0001 C CNN
+F 4 "" H 0   0   50  0001 C CNN "Spice_Lib_File"
+F 5 "" H 0   0   50  0001 C CNN "Spice_Model"
+F 6 "" H 0   0   50  0001 C CNN "Spice_Netlist_Enabled"
+F 7 "" H 0   0   50  0001 C CNN "Spice_Primitive"
 	1    3000 2625
 	0    -1   -1   0
@@
 AR Path="/5C1207F9/5B1EC381/5CEE54B0" Ref="U31"  Part="1"
 AR Path="/5C1207F9/5B1EC399/5CEE54B0" Ref="U34"  Part="1"
-F 0 "U13" V 4353 5348 60  0000 L CNN
+F 0 "U34" V 4353 5348 60  0000 L CNN
 F 1 "74LS151" V 4247 5348 60  0000 L CNN
 F 2 "" H 4300 4600 60  0001 C CNN
 F 3 "" H 4300 4600 60  0001 C CNN
+F 4 "" H 0   0   50  0001 C CNN "Spice_Lib_File"
+F 5 "" H 0   0   50  0001 C CNN "Spice_Model"
+F 6 "" H 0   0   50  0001 C CNN "Spice_Netlist_Enabled"
+F 7 "" H 0   0   50  0001 C CNN "Spice_Primitive"
 	1    4300 4600
 	0    -1   -1   0
@@
 AR Path="/5C1207F9/5B1EC369/5F438084" Ref="#PWR0179"  Part="1"
 AR Path="/5C1207F9/5B1EC381/5F438084" Ref="#PWR0187"  Part="1"
-F 0 "#PWR0139" H 3375 4525 30  0001 C CNN
+F 0 "#PWR0195" H 3375 4525 30  0001 C CNN
 F 1 "VCC" H 3379 4552 30  0000 C CNN
 F 2 "" H 3375 4425 50  0001 C CNN
@@
 AR Path="/5C1207F9/5B1EC369/5F43824E" Ref="#PWR0177"  Part="1"
 AR Path="/5C1207F9/5B1EC381/5F43824E" Ref="#PWR0185"  Part="1"
-F 0 "#PWR0137" H 2100 2600 30  0001 C CNN
+F 0 "#PWR0193" H 2100 2600 30  0001 C CNN
 F 1 "VCC" H 2104 2627 30  0000 C CNN
 F 2 "" H 2100 2500 50  0001 C CNN
@@
 AR Path="/5C1207F9/5B1EC369/5F43846F" Ref="#PWR0181"  Part="1"
 AR Path="/5C1207F9/5B1EC381/5F43846F" Ref="#PWR0189"  Part="1"
-F 0 "#PWR0141" H 5325 4850 30  0001 C CNN
+F 0 "#PWR0197" H 5325 4850 30  0001 C CNN
 F 1 "GND" H 5325 4780 30  0001 C CNN
 F 2 "" H 5325 4850 50  0001 C CNN
@@
 AR Path="/5C1207F9/5B1EC369/64FCAAB3" Ref="#PWR0180"  Part="1"
 AR Path="/5C1207F9/5B1EC381/64FCAAB3" Ref="#PWR0188"  Part="1"
-F 0 "#PWR0140" H 3775 3475 30  0001 C CNN
+F 0 "#PWR0196" H 3775 3475 30  0001 C CNN
 F 1 "GND-power" H 3775 3405 30  0001 C CNN
 F 2 "" H 3775 3475 50  0001 C CNN
@@
 AR Path="/5C1207F9/5B1EC369/65020F3D" Ref="#PWR0178"  Part="1"
 AR Path="/5C1207F9/5B1EC381/65020F3D" Ref="#PWR0186"  Part="1"
-F 0 "#PWR0138" H 3350 4900 30  0001 C CNN
+F 0 "#PWR0194" H 3350 4900 30  0001 C CNN
 F 1 "GND-power" H 3350 4830 30  0001 C CNN
 F 2 "" H 3350 4900 50  0001 C CNN
@@
 AR Path="/5C1207F9/5B1EC369/6502C1A5" Ref="#PWR0176"  Part="1"
 AR Path="/5C1207F9/5B1EC381/6502C1A5" Ref="#PWR0184"  Part="1"
-F 0 "#PWR0136" H 1325 4400 50  0001 C CNN
+F 0 "#PWR0192" H 1325 4400 50  0001 C CNN
 F 1 "VCC" H 1342 4723 50  0000 C CNN
 F 2 "" H 1325 4550 50  0001 C CNN
@@
 AR Path="/5C1207F9/5B1EC369/650FDD6F" Ref="C58"  Part="1"
 AR Path="/5C1207F9/5B1EC381/650FDD6F" Ref="C61"  Part="1"
-F 0 "C43" H 5742 2746 50  0000 L CNN
+F 0 "C64" H 5742 2746 50  0000 L CNN
 F 1 "100nF" H 5742 2655 50  0000 L CNN
-F 2 "" H 5650 2700 50  0001 C CNN
+F 2 "Capacitor_SMD:C_0805_2012Metric" H 5650 2700 50  0001 C CNN
 F 3 "~" H 5650 2700 50  0001 C CNN
+F 4 "" H 0   0   50  0001 C CNN "Spice_Lib_File"
+F 5 "" H 0   0   50  0001 C CNN "Spice_Model"
+F 6 "" H 0   0   50  0001 C CNN "Spice_Netlist_Enabled"
+F 7 "" H 0   0   50  0001 C CNN "Spice_Primitive"
 	1    5650 2700
 	1    0    0    -1
@@
 AR Path="/5C1207F9/5B1EC369/650FDF0B" Ref="C59"  Part="1"
 AR Path="/5C1207F9/5B1EC381/650FDF0B" Ref="C62"  Part="1"
-F 0 "C44" H 6342 2746 50  0000 L CNN
+F 0 "C65" H 6342 2746 50  0000 L CNN
 F 1 "100nF" H 6342 2655 50  0000 L CNN
-F 2 "" H 6250 2700 50  0001 C CNN
+F 2 "Capacitor_SMD:C_0805_2012Metric" H 6250 2700 50  0001 C CNN
 F 3 "~" H 6250 2700 50  0001 C CNN
+F 4 "" H 0   0   50  0001 C CNN "Spice_Lib_File"
+F 5 "" H 0   0   50  0001 C CNN "Spice_Model"
+F 6 "" H 0   0   50  0001 C CNN "Spice_Netlist_Enabled"
+F 7 "" H 0   0   50  0001 C CNN "Spice_Primitive"
 	1    6250 2700
 	1    0    0    -1
@@
 AR Path="/5C1207F9/5B1EC369/650FDFCC" Ref="C60"  Part="1"
 AR Path="/5C1207F9/5B1EC381/650FDFCC" Ref="C63"  Part="1"
-F 0 "C45" H 7017 2771 50  0000 L CNN
+F 0 "C66" H 7017 2771 50  0000 L CNN
 F 1 "100nF" H 7017 2680 50  0000 L CNN
-F 2 "" H 6925 2725 50  0001 C CNN
+F 2 "Capacitor_SMD:C_0805_2012Metric" H 6925 2725 50  0001 C CNN
 F 3 "~" H 6925 2725 50  0001 C CNN
+F 4 "" H 0   0   50  0001 C CNN "Spice_Lib_File"
+F 5 "" H 0   0   50  0001 C CNN "Spice_Model"
+F 6 "" H 0   0   50  0001 C CNN "Spice_Netlist_Enabled"
+F 7 "" H 0   0   50  0001 C CNN "Spice_Primitive"
 	1    6925 2725
 	1    0    0    -1
@@
 AR Path="/5C1207F9/5B1EC369/650FE0D2" Ref="#PWR0182"  Part="1"
 AR Path="/5C1207F9/5B1EC381/650FE0D2" Ref="#PWR0190"  Part="1"
-F 0 "#PWR0142" H 6275 1825 50  0001 C CNN
+F 0 "#PWR0198" H 6275 1825 50  0001 C CNN
 F 1 "VCC" H 6292 2148 50  0000 C CNN
 F 2 "" H 6275 1975 50  0001 C CNN
@@
 AR Path="/5C1207F9/5B1EC369/650FE10D" Ref="#PWR0183"  Part="1"
 AR Path="/5C1207F9/5B1EC381/650FE10D" Ref="#PWR0191"  Part="1"
-F 0 "#PWR0143" H 6300 3150 30  0001 C CNN
+F 0 "#PWR0199" H 6300 3150 30  0001 C CNN
 F 1 "GND-power" H 6300 3080 30  0001 C CNN
 F 2 "" H 6300 3150 50  0001 C CNN

Commit message: started routing
Parts:
- U10, U8, U9: footprint (none) -> Package_SO:SOIC-16_3.9x9.9mm_P1.27mm
Changed lines of the file:
@@
 $Descr A4 11693 8268
 encoding utf-8
-Sheet 139 191
+Sheet 130 191
 Title ""
 Date ""
@@
 F 0 "U32" V 2478 5398 60  0000 L CNN
 F 1 "74LS151" V 2372 5398 60  0000 L CNN
-F 2 "" H 2425 4650 60  0001 C CNN
+F 2 "Package_SO:SOIC-16_3.9x9.9mm_P1.27mm" H 2425 4650 60  0001 C CNN
 F 3 "" H 2425 4650 60  0001 C CNN
 F 4 "X" H 2425 4650 50  0001 C CNN "Spice_Primitive"
@@
 F 0 "U33" V 3053 1966 60  0000 R CNN
 F 1 "74LS157" V 2947 1966 60  0000 R CNN
-F 2 "" H 3000 2625 60  0001 C CNN
+F 2 "Package_SO:SOIC-16_3.9x9.9mm_P1.27mm" H 3000 2625 60  0001 C CNN
 F 3 "" H 3000 2625 60  0001 C CNN
 F 4 "" H 0   0   50  0001 C CNN "Spice_Lib_File"
@@
 F 0 "U34" V 4353 5348 60  0000 L CNN
 F 1 "74LS151" V 4247 5348 60  0000 L CNN
-F 2 "" H 4300 4600 60  0001 C CNN
+F 2 "Package_SO:SOIC-16_3.9x9.9mm_P1.27mm" H 4300 4600 60  0001 C CNN
 F 3 "" H 4300 4600 60  0001 C CNN
 F 4 "" H 0   0   50  0001 C CNN "Spice_Lib_File"
