File: Alu/OR.sch (KiCad schematic (older format))
At the start: 4 parts, among them U38 74HC02, U7 74HC02

Commit message: footprints
Parts:
- removed U38, U7: 74HC02, symbol 74xx:74HC02
- added U4, U7: 74LS32, Package_SO:SOIC-14_3.9x8.7mm_P1.27mm, symbol 74xx:74LS32
- C4, C5: footprint (none) -> Capacitor_SMD:C_0805_2012Metric
Changed lines of the file:
@@
 $Descr A4 11693 8268
 encoding utf-8
-Sheet 11 156
+Sheet 11 191
 Title ""
 Date ""
@@
 Text HLabel 4525 2075 1    60   Output ~ 0
 Z7
-$Comp
-L 74xx:74HC02 U7
-U 1 1 64F60C6D
-P 1125 6325
-F 0 "U7" V 1171 6145 50  0000 R CNN
-F 1 "74HC02" V 1080 6145 50  0000 R CNN
-F 2 "" H 1125 6325 50  0001 C CNN
-F 3 "http://www.ti.com/lit/gpn/sn74hc02" H 1125 6325 50  0001 C CNN
-	1    1125 6325
-	0    -1   -1   0
-$EndComp
-$Comp
-L 74xx:74HC02 U7
-U 2 1 64F60E01
-P 1775 6325
-F 0 "U7" V 1821 6145 50  0000 R CNN
-F 1 "74HC02" V 1730 6145 50  0000 R CNN
-F 2 "" H 1775 6325 50  0001 C CNN
-F 3 "http://www.ti.com/lit/gpn/sn74hc02" H 1775 6325 50  0001 C CNN
-	2    1775 6325
-	0    -1   -1   0
-$EndComp
-$Comp
-L 74xx:74HC02 U7
-U 3 1 64F60EF5
-P 2450 6325
-F 0 "U7" V 2496 6145 50  0000 R CNN
-F 1 "74HC02" V 2405 6145 50  0000 R CNN
-F 2 "" H 2450 6325 50  0001 C CNN
-F 3 "http://www.ti.com/lit/gpn/sn74hc02" H 2450 6325 50  0001 C CNN
-	3    2450 6325
-	0    -1   -1   0
-$EndComp
-$Comp
-L 74xx:74HC02 U7
-U 4 1 64F60FB1
-P 3125 6325
-F 0 "U7" V 3171 6145 50  0000 R CNN
-F 1 "74HC02" V 3080 6145 50  0000 R CNN
-F 2 "" H 3125 6325 50  0001 C CNN
-F 3 "http://www.ti.com/lit/gpn/sn74hc02" H 3125 6325 50  0001 C CNN
-	4    3125 6325
-	0    -1   -1   0
-$EndComp
-$Comp
-L 74xx:74HC02 U7
-U 5 1 64F61101
-P 7400 4525
-F 0 "U7" H 7630 4571 50  0000 L CNN
-F 1 "74HC02" H 7630 4480 50  0000 L CNN
-F 2 "" H 7400 4525 50  0001 C CNN
-F 3 "http://www.ti.com/lit/gpn/sn74hc02" H 7400 4525 50  0001 C CNN
-	5    7400 4525
-	1    0    0    -1
-$EndComp
-$Comp
-L 74xx:74HC02 U38
-U 1 1 64F611CB
-P 3775 6375
-F 0 "U38" V 3821 6195 50  0000 R CNN
-F 1 "74HC02" V 3730 6195 50  0000 R CNN
-F 2 "" H 3775 6375 50  0001 C CNN
-F 3 "http://www.ti.com/lit/gpn/sn74hc02" H 3775 6375 50  0001 C CNN
-	1    3775 6375
-	0    -1   -1   0
-$EndComp
-$Comp
-L 74xx:74HC02 U38
-U 2 1 64F612B3
-P 4450 6400
-F 0 "U38" V 4496 6220 50  0000 R CNN
-F 1 "74HC02" V 4405 6220 50  0000 R CNN
-F 2 "" H 4450 6400 50  0001 C CNN
-F 3 "http://www.ti.com/lit/gpn/sn74hc02" H 4450 6400 50  0001 C CNN
-	2    4450 6400
-	0    -1   -1   0
-$EndComp
-$Comp
-L 74xx:74HC02 U38
-U 3 1 64F61401
-P 5150 6450
-F 0 "U38" V 5196 6270 50  0000 R CNN
-F 1 "74HC02" V 5105 6270 50  0000 R CNN
-F 2 "" H 5150 6450 50  0001 C CNN
-F 3 "http://www.ti.com/lit/gpn/sn74hc02" H 5150 6450 50  0001 C CNN
-	3    5150 6450
-	0    -1   -1   0
-$EndComp
-$Comp
-L 74xx:74HC02 U38
-U 4 1 64F615A4
-P 5900 6450
-F 0 "U38" V 5946 6270 50  0000 R CNN
-F 1 "74HC02" V 5855 6270 50  0000 R CNN
-F 2 "" H 5900 6450 50  0001 C CNN
-F 3 "http://www.ti.com/lit/gpn/sn74hc02" H 5900 6450 50  0001 C CNN
-	4    5900 6450
-	0    -1   -1   0
-$EndComp
-$Comp
-L 74xx:74HC02 U38
-U 5 1 64F61E46
-P 8025 4525
-F 0 "U38" H 8255 4571 50  0000 L CNN
-F 1 "74HC02" H 8255 4480 50  0000 L CNN
-F 2 "" H 8025 4525 50  0001 C CNN
-F 3 "http://www.ti.com/lit/gpn/sn74hc02" H 8025 4525 50  0001 C CNN
-	5    8025 4525
-	1    0    0    -1
-$EndComp
-$Sheet
-S 975  2975 5225 1200
-U 64F62017
-F0 "OR_NOT" 50
-F1 "NOT.sch" 50
-F2 "X0" I B 6075 4175 50
-F3 "X1" I B 5175 4175 50
-F4 "X2" I B 4575 4175 50
-F5 "X3" I B 3925 4175 50
-F6 "X4" I B 3100 4175 50
-F7 "X5" I B 2400 4175 50
-F8 "X6" I B 1800 4175 50
-F9 "X7" I B 1175 4175 50
-F10 "Z0" O T 4625 2975 50
-F11 "Z2" O T 3750 2975 50
-F12 "Z1" O T 4150 2975 50
-F13 "Z3" O T 2925 2975 50
-F14 "Z4" O T 2275 2975 50
-F15 "Z5" O T 2000 2975 50
-F16 "Z6" O T 1700 2975 50
-F17 "Z7" O T 1275 2975 50
-$EndSheet
 Wire Wire Line
 	1025 7050 1025 6625
@@
 F 0 "C5" H 9117 4571 50  0000 L CNN
 F 1 "100nF" H 9117 4480 50  0000 L CNN
-F 2 "" H 9025 4525 50  0001 C CNN
+F 2 "Capacitor_SMD:C_0805_2012Metric" H 9025 4525 50  0001 C CNN
 F 3 "~" H 9025 4525 50  0001 C CNN
+F 4 "" H 0   0   50  0001 C CNN "Spice_Lib_File"
+F 5 "" H 0   0   50  0001 C CNN "Spice_Model"
+F 6 "" H 0   0   50  0001 C CNN "Spice_Netlist_Enabled"
+F 7 "" H 0   0   50  0001 C CNN "Spice_Primitive"
 	1    9025 4525
 	1    0    0    -1
@@
 F 0 "C4" H 6967 4546 50  0000 L CNN
 F 1 "100nF" H 6967 4455 50  0000 L CNN
-F 2 "" H 6875 4500 50  0001 C CNN
+F 2 "Capacitor_SMD:C_0805_2012Metric" H 6875 4500 50  0001 C CNN
 F 3 "~" H 6875 4500 50  0001 C CNN
+F 4 "" H 0   0   50  0001 C CNN "Spice_Lib_File"
+F 5 "" H 0   0   50  0001 C CNN "Spice_Model"
+F 6 "" H 0   0   50  0001 C CNN "Spice_Netlist_Enabled"
+F 7 "" H 0   0   50  0001 C CNN "Spice_Primitive"
 	1    6875 4500
 	1    0    0    -1
@@
 F2 "X" I B 6075 5075 50
 $EndSheet
+$Comp
+L 74xx:74LS32 U4
+U 1 1 5BF22B06
+P 1125 6325
+F 0 "U4" V 1171 6145 50  0000 R CNN
+F 1 "74LS32" V 1080 6145 50  0000 R CNN
+F 2 "Package_SO:SOIC-14_3.9x8.7mm_P1.27mm" H 1125 6325 50  0001 C CNN
+F 3 "http://www.ti.com/lit/gpn/sn74LS32" H 1125 6325 50  0001 C CNN
+F 4 "" H 0   0   50  0001 C CNN "Spice_Lib_File"
+F 5 "" H 0   0   50  0001 C CNN "Spice_Model"
+F 6 "" H 0   0   50  0001 C CNN "Spice_Netlist_Enabled"
+F 7 "" H 0   0   50  0001 C CNN "Spice_Primitive"
+	1    1125 6325
+	0    -1   -1   0
+$EndComp
+$Comp
+L 74xx:74LS32 U4
+U 2 1 5BF22C6E
+P 1775 6325
+F 0 "U4" V 1821 6145 50  0000 R CNN
+F 1 "74LS32" V 1730 6145 50  0000 R CNN
+F 2 "Package_SO:SOIC-14_3.9x8.7mm_P1.27mm" H 1775 6325 50  0001 C CNN
+F 3 "http://www.ti.com/lit/gpn/sn74LS32" H 1775 6325 50  0001 C CNN
+F 4 "" H 0   0   50  0001 C CNN "Spice_Lib_File"
+F 5 "" H 0   0   50  0001 C CNN "Spice_Model"
+F 6 "" H 0   0   50  0001 C CNN "Spice_Netlist_Enabled"
+F 7 "" H 0   0   50  0001 C CNN "Spice_Primitive"
+	2    1775 6325
+	0    -1   -1   0
+$EndComp
+$Comp
+L 74xx:74LS32 U4
+U 3 1 5BF22D02
+P 2450 6325
+F 0 "U4" V 2496 6145 50  0000 R CNN
+F 1 "74LS32" V 2405 6145 50  0000 R CNN
+F 2 "Package_SO:SOIC-14_3.9x8.7mm_P1.27mm" H 2450 6325 50  0001 C CNN
+F 3 "http://www.ti.com/lit/gpn/sn74LS32" H 2450 6325 50  0001 C CNN
+F 4 "" H 0   0   50  0001 C CNN "Spice_Lib_File"
+F 5 "" H 0   0   50  0001 C CNN "Spice_Model"
+F 6 "" H 0   0   50  0001 C CNN "Spice_Netlist_Enabled"
+F 7 "" H 0   0   50  0001 C CNN "Spice_Primitive"
+	3    2450 6325
+	0    -1   -1   0
+$EndComp
+$Comp
+L 74xx:74LS32 U4
+U 4 1 5BF22DB2
+P 3125 6325
+F 0 "U4" V 3171 6145 50  0000 R CNN
+F 1 "74LS32" V 3080 6145 50  0000 R CNN
+F 2 "Package_SO:SOIC-14_3.9x8.7mm_P1.27mm" H 3125 6325 50  0001 C CNN
+F 3 "http://www.ti.com/lit/gpn/sn74LS32" H 3125 6325 50  0001 C CNN
+F 4 "" H 0   0   50  0001 C CNN "Spice_Lib_File"
+F 5 "" H 0   0   50  0001 C CNN "Spice_Model"
+F 6 "" H 0   0   50  0001 C CNN "Spice_Netlist_Enabled"
+F 7 "" H 0   0   50  0001 C CNN "Spice_Primitive"
+	4    3125 6325
+	0    -1   -1   0
+$EndComp
+$Comp
+L 74xx:74LS32 U4
+U 5 1 5BF22E94
+P 7400 4525
+F 0 "U4" H 7630 4571 50  0000 L CNN
+F 1 "74LS32" H 7630 4480 50  0000 L CNN
+F 2 "Package_SO:SOIC-14_3.9x8.7mm_P1.27mm" H 7400 4525 50  0001 C CNN
+F 3 "http://www.ti.com/lit/gpn/sn74LS32" H 7400 4525 50  0001 C CNN
+F 4 "" H 0   0   50  0001 C CNN "Spice_Lib_File"
+F 5 "" H 0   0   50  0001 C CNN "Spice_Model"
+F 6 "" H 0   0   50  0001 C CNN "Spice_Netlist_Enabled"
+F 7 "" H 0   0   50  0001 C CNN "Spice_Primitive"
+	5    7400 4525
+	1    0    0    -1
+$EndComp
+$Comp
+L 74xx:74LS32 U7
+U 1 1 5BF2308B
+P 3775 6375
+F 0 "U7" V 3821 6195 50  0000 R CNN
+F 1 "74LS32" V 3730 6195 50  0000 R CNN
+F 2 "Package_SO:SOIC-14_3.9x8.7mm_P1.27mm" H 3775 6375 50  0001 C CNN
+F 3 "http://www.ti.com/lit/gpn/sn74LS32" H 3775 6375 50  0001 C CNN
+F 4 "" H 0   0   50  0001 C CNN "Spice_Lib_File"
+F 5 "" H 0   0   50  0001 C CNN "Spice_Model"
+F 6 "" H 0   0   50  0001 C CNN "Spice_Netlist_Enabled"
+F 7 "" H 0   0   50  0001 C CNN "Spice_Primitive"
+	1    3775 6375
+	0    -1   -1   0
+$EndComp
+$Comp
+L 74xx:74LS32 U7
+U 2 1 5BF2314D
+P 4450 6400
+F 0 "U7" V 4496 6220 50  0000 R CNN
+F 1 "74LS32" V 4405 6220 50  0000 R CNN
+F 2 "Package_SO:SOIC-14_3.9x8.7mm_P1.27mm" H 4450 6400 50  0001 C CNN
+F 3 "http://www.ti.com/lit/gpn/sn74LS32" H 4450 6400 50  0001 C CNN
+F 4 "" H 0   0   50  0001 C CNN "Spice_Lib_File"
+F 5 "" H 0   0   50  0001 C CNN "Spice_Model"
+F 6 "" H 0   0   50  0001 C CNN "Spice_Netlist_Enabled"
+F 7 "" H 0   0   50  0001 C CNN "Spice_Primitive"
+	2    4450 6400
+	0    -1   -1   0
+$EndComp
+$Comp
+L 74xx:74LS32 U7
+U 3 1 5BF231E9
+P 5150 6450
+F 0 "U7" V 5196 6270 50  0000 R CNN
+F 1 "74LS32" V 5105 6270 50  0000 R CNN
+F 2 "Package_SO:SOIC-14_3.9x8.7mm_P1.27mm" H 5150 6450 50  0001 C CNN
+F 3 "http://www.ti.com/lit/gpn/sn74LS32" H 5150 6450 50  0001 C CNN
+F 4 "" H 0   0   50  0001 C CNN "Spice_Lib_File"
+F 5 "" H 0   0   50  0001 C CNN "Spice_Model"
+F 6 "" H 0   0   50  0001 C CNN "Spice_Netlist_Enabled"
+F 7 "" H 0   0   50  0001 C CNN "Spice_Primitive"
+	3    5150 6450
+	0    -1   -1   0
+$EndComp
+$Comp
+L 74xx:74LS32 U7
+U 4 1 5BF2329B
+P 5900 6450
+F 0 "U7" V 5946 6270 50  0000 R CNN
+F 1 "74LS32" V 5855 6270 50  0000 R CNN
+F 2 "Package_SO:SOIC-14_3.9x8.7mm_P1.27mm" H 5900 6450 50  0001 C CNN
+F 3 "http://www.ti.com/lit/gpn/sn74LS32" H 5900 6450 50  0001 C CNN
+F 4 "" H 0   0   50  0001 C CNN "Spice_Lib_File"
+F 5 "" H 0   0   50  0001 C CNN "Spice_Model"
+F 6 "" H 0   0   50  0001 C CNN "Spice_Netlist_Enabled"
+F 7 "" H 0   0   50  0001 C CNN "Spice_Primitive"
+	4    5900 6450
+	0    -1   -1   0
+$EndComp
+$Comp
+L 74xx:74LS32 U7
+U 5 1 5BF23426
+P 8025 4525
+F 0 "U7" H 8255 4571 50  0000 L CNN
+F 1 "74LS32" H 8255 4480 50  0000 L CNN
+F 2 "Package_SO:SOIC-14_3.9x8.7mm_P1.27mm" H 8025 4525 50  0001 C CNN
+F 3 "http://www.ti.com/lit/gpn/sn74LS32" H 8025 4525 50  0001 C CNN
+F 4 "" H 0   0   50  0001 C CNN "Spice_Lib_File"
+F 5 "" H 0   0   50  0001 C CNN "Spice_Model"
+F 6 "" H 0   0   50  0001 C CNN "Spice_Netlist_Enabled"
+F 7 "" H 0   0   50  0001 C CNN "Spice_Primitive"
+	5    8025 4525
+	1    0    0    -1
+$EndComp
 $EndSCHEMATC

Commit message: started routing
Connections:
- wire segments 87 -> 125
Changed lines of the file:
@@
 	6050 6750 6000 6750
 Wire Wire Line
-	1125 6025 1125 4250
+	1125 6025 1125 5300
 Wire Wire Line
 	1125 4250 1175 4250
 Wire Wire Line
-	1175 4250 1175 4175
-Wire Wire Line
-	1800 4175 1800 6025
+	1800 4175 1800 5375
 Wire Wire Line
 	1800 6025 1775 6025
 Wire Wire Line
-	2400 4175 2400 6025
-Wire Wire Line
 	2400 6025 2450 6025
 Wire Wire Line
-	3100 4175 3100 6025
+	3100 4175 3100 5200
 Wire Wire Line
 	3100 6025 3125 6025
 Wire Wire Line
-	3925 4175 3925 6075
-Wire Wire Line
 	3925 6075 3775 6075
 Wire Wire Line
-	4575 4175 4575 6100
-Wire Wire Line
 	4575 6100 4450 6100
 Wire Wire Line
-	5175 4175 5175 6025
-Wire Wire Line
 	5175 6025 5150 6025
 Wire Wire Line
 	5150 6025 5150 6150
 Wire Wire Line
-	6075 4175 6075 6150
-Wire Wire Line
 	6075 6150 5900 6150
 Wire Wire Line
@@
 	1600 2875 1700 2875
 Wire Wire Line
-	1700 2875 1700 2975
-Wire Wire Line
-	2000 2975 2000 2725
-Wire Wire Line
 	2000 2725 1825 2725
 Wire Wire Line
@@
 	2000 2450 2275 2450
 Wire Wire Line
-	2275 2450 2275 2975
-Wire Wire Line
 	2900 2025 2900 2875
 Wire Wire Line
@@
 Wire Wire Line
 	2925 2875 2925 2975
-Wire Wire Line
-	3750 2975 3750 2150
 Wire Wire Line
 	3750 2150 3725 2150
@@
 	6875 5225 7750 5225
 $Sheet
-S 1050 4575 150  500
+S 1225 4600 150  500
 U 5C40E172
 F0 "Sheet5C40E171" 50
 F1 "LED_RED.sch" 50
-F2 "X" I B 1125 5075 50
-$EndSheet
-$Sheet
-S 1725 4700 150  500
+F2 "X" I B 1300 5100 50
+$EndSheet
+$Sheet
+S 1925 4650 150  500
 U 5C40E25E
 F0 "sheet5C40E25B" 50
 F1 "LED_RED.sch" 50
-F2 "X" I B 1800 5200 50
-$EndSheet
-$Sheet
-S 2325 4575 150  500
+F2 "X" I B 2000 5150 50
+$EndSheet
+$Sheet
+S 2525 4550 150  500
 U 5C40FEDF
 F0 "sheet5C40FEDB" 50
 F1 "LED_RED.sch" 50
-F2 "X" I B 2400 5075 50
-$EndSheet
-$Sheet
-S 3025 4600 150  500
+F2 "X" I B 2600 5050 50
+$EndSheet
+$Sheet
+S 3175 4575 150  500
 U 5C40FEE2
 F0 "sheet5C40FEDC" 50
 F1 "LED_RED.sch" 50
-F2 "X" I B 3100 5100 50
-$EndSheet
-$Sheet
-S 3850 4675 150  500
+F2 "X" I B 3250 5075 50
+$EndSheet
+$Sheet
+S 3950 4650 150  500
 U 5C411B69
 F0 "sheet5C411B63" 50
 F1 "LED_RED.sch" 50
-F2 "X" I B 3925 5175 50
-$EndSheet
-$Sheet
-S 4500 4700 150  500
+F2 "X" I B 4025 5150 50
+$EndSheet
+$Sheet
+S 4625 4650 150  500
 U 5C411B6C
 F0 "sheet5C411B64" 50
 F1 "LED_RED.sch" 50
-F2 "X" I B 4575 5200 50
-$EndSheet
-$Sheet
-S 5100 4625 150  500
+F2 "X" I B 4700 5150 50
+$EndSheet
+$Sheet
+S 5225 4600 150  500
 U 5C411B6F
 F0 "sheet5C411B65" 50
 F1 "LED_RED.sch" 50
-F2 "X" I B 5175 5125 50
-$EndSheet
-$Sheet
-S 6000 4575 150  500
+F2 "X" I B 5300 5100 50
+$EndSheet
+$Sheet
+S 5725 4550 150  500
 U 5C411B72
 F0 "sheet5C411B66" 50
 F1 "LED_RED.sch" 50
-F2 "X" I B 6075 5075 50
+F2 "X" I B 5800 5050 50
 $EndSheet
 $Comp
@@
 	1    0    0    -1
 $EndComp
+Wire Wire Line
+	1175 2975 1275 2975
+Wire Wire Line
+	1175 2975 1175 4250
+Wire Wire Line
+	1700 4175 1800 4175
+Wire Wire Line
+	1700 2875 1700 4175
+Wire Wire Line
+	2400 3575 2000 3575
+Wire Wire Line
+	2400 3575 2400 5250
+Wire Wire Line
+	2000 2725 2000 3575
+Wire Wire Line
+	2275 3275 2900 3275
+Wire Wire Line
+	2900 3275 2900 4175
+Wire Wire Line
+	2900 4175 3100 4175
+Wire Wire Line
+	2275 2450 2275 3275
+Wire Wire Line
+	2925 2975 3225 2975
+Wire Wire Line
+	3225 2975 3225 3900
+Wire Wire Line
+	3225 3900 3925 3900
+Wire Wire Line
+	3925 3900 3925 5275
+Wire Wire Line
+	3750 3600 4575 3600
+Wire Wire Line
+	4575 3600 4575 5250
+Wire Wire Line
+	3750 2150 3750 3600
+Wire Wire Line
+	4625 2975 6075 2975
+Wire Wire Line
+	6075 2975 6075 5275
+Wire Wire Line
+	4175 2975 4175 3275
+Wire Wire Line
+	4175 3275 5175 3275
+Wire Wire Line
+	5175 3275 5175 5225
+Wire Wire Line
+	4150 2975 4175 2975
+Wire Wire Line
+	1125 5300 1300 5300
+Wire Wire Line
+	1300 5300 1300 5100
+Connection ~ 1125 5300
+Wire Wire Line
+	1125 5300 1125 4250
+Wire Wire Line
+	1800 5375 2000 5375
+Wire Wire Line
+	2000 5375 2000 5150
+Connection ~ 1800 5375
+Wire Wire Line
+	1800 5375 1800 6025
+Wire Wire Line
+	2400 5250 2600 5250
+Wire Wire Line
+	2600 5250 2600 5050
+Connection ~ 2400 5250
+Wire Wire Line
+	2400 5250 2400 6025
+Wire Wire Line
+	3100 5200 3250 5200
+Wire Wire Line
+	3250 5200 3250 5075
+Connection ~ 3100 5200
+Wire Wire Line
+	3100 5200 3100 6025
+Wire Wire Line
+	3925 5275 4025 5275
+Wire Wire Line
+	4025 5275 4025 5150
+Connection ~ 3925 5275
+Wire Wire Line
+	3925 5275 3925 6075
+Wire Wire Line
+	4575 5250 4700 5250
+Wire Wire Line
+	4700 5250 4700 5150
+Connection ~ 4575 5250
+Wire Wire Line
+	4575 5250 4575 6100
+Wire Wire Line
+	5175 5225 5300 5225
+Wire Wire Line
+	5300 5225 5300 5100
+Connection ~ 5175 5225
+Wire Wire Line
+	5175 5225 5175 6025
+Wire Wire Line
+	6075 5275 5800 5275
+Wire Wire Line
+	5800 5275 5800 5050
+Connection ~ 6075 5275
+Wire Wire Line
+	6075 5275 6075 6150
 $EndSCHEMATC
