File: Alu/INC8.sch (KiCad schematic (older format))
At the start: 4 parts, among them U45 74LS283, U46 74LS283

Commit message: footprints
Parts:
- C12, C13: footprint (none) -> Capacitor_SMD:C_0805_2012Metric
Changed lines of the file:
@@
 $Descr A4 11693 8268
 encoding utf-8
-Sheet 96 156
+Sheet 38 191
 Title ""
 Date ""
@@
 AR Path="/5AE74AF7/5CF197AB" Ref="#PWR020"  Part="1"
 AR Path="/5AF84E03/5CF197AB" Ref="#PWR029"  Part="1"
-F 0 "#PWR029" H 4125 5650 30  0001 C CNN
+F 0 "#PWR020" H 4125 5650 30  0001 C CNN
 F 1 "GND" H 4125 5580 30  0001 C CNN
 F 2 "" H 4125 5650 60  0001 C CNN
@@
 AR Path="/5AE74AF7/5CF198E5" Ref="#PWR018"  Part="1"
 AR Path="/5AF84E03/5CF198E5" Ref="#PWR027"  Part="1"
-F 0 "#PWR027" H 1975 5575 30  0001 C CNN
+F 0 "#PWR018" H 1975 5575 30  0001 C CNN
 F 1 "GND" H 1975 5505 30  0001 C CNN
 F 2 "" H 1975 5575 60  0001 C CNN
@@
 AR Path="/5AE74AF7/5CF199DA" Ref="#PWR019"  Part="1"
 AR Path="/5AF84E03/5CF199DA" Ref="#PWR028"  Part="1"
-F 0 "#PWR028" H 2850 4300 30  0001 C CNN
+F 0 "#PWR019" H 2850 4300 30  0001 C CNN
 F 1 "GND" H 2850 4230 30  0001 C CNN
 F 2 "" H 2850 4300 60  0001 C CNN
@@
 AR Path="/5AE74AF7/5CF19D18" Ref="#PWR017"  Part="1"
 AR Path="/5AF84E03/5CF19D18" Ref="#PWR026"  Part="1"
-F 0 "#PWR026" H 700 4200 30  0001 C CNN
+F 0 "#PWR017" H 700 4200 30  0001 C CNN
 F 1 "GND" H 700 4130 30  0001 C CNN
 F 2 "" H 700 4200 60  0001 C CNN
@@
 AR Path="/5AE74AF7/5F3A2E1C" Ref="#PWR061"  Part="1"
 AR Path="/5AF84E03/5F3A2E1C" Ref="#PWR0127"  Part="1"
-F 0 "#PWR0127" H 2525 5100 30  0001 C CNN
+F 0 "#PWR061" H 2525 5100 30  0001 C CNN
 F 1 "VCC" H 2529 5127 30  0000 C CNN
 F 2 "" H 2525 5000 50  0001 C CNN
@@
 AR Path="/5AE74AF7/5F3A2E46" Ref="#PWR060"  Part="1"
 AR Path="/5AF84E03/5F3A2E46" Ref="#PWR0126"  Part="1"
-F 0 "#PWR0126" H 875 5000 30  0001 C CNN
+F 0 "#PWR060" H 875 5000 30  0001 C CNN
 F 1 "VCC" H 879 5027 30  0000 C CNN
 F 2 "" H 875 4900 50  0001 C CNN
@@
 AR Path="/5AE74AF7/5F3A2F2F" Ref="U45"  Part="1"
 AR Path="/5AF84E03/5F3A2F2F" Ref="U73"  Part="1"
-F 0 "U73" V 1603 4031 60  0000 R CNN
+F 0 "U45" V 1603 4031 60  0000 R CNN
 F 1 "74LS283" V 1497 4031 60  0000 R CNN
 F 2 "" H 1550 4575 60  0001 C CNN
 F 3 "" H 1550 4575 60  0001 C CNN
+F 4 "" H 0   0   50  0001 C CNN "Spice_Lib_File"
+F 5 "" H 0   0   50  0001 C CNN "Spice_Model"
+F 6 "" H 0   0   50  0001 C CNN "Spice_Netlist_Enabled"
+F 7 "" H 0   0   50  0001 C CNN "Spice_Primitive"
 	1    1550 4575
 	0    -1   -1   0
@@
 AR Path="/5AE74AF7/5F3A5CFF" Ref="U46"  Part="1"
 AR Path="/5AF84E03/5F3A5CFF" Ref="U74"  Part="1"
-F 0 "U74" V 3628 4156 60  0000 R CNN
+F 0 "U46" V 3628 4156 60  0000 R CNN
 F 1 "74LS283" V 3522 4156 60  0000 R CNN
 F 2 "" H 3575 4700 60  0001 C CNN
 F 3 "" H 3575 4700 60  0001 C CNN
+F 4 "" H 0   0   50  0001 C CNN "Spice_Lib_File"
+F 5 "" H 0   0   50  0001 C CNN "Spice_Model"
+F 6 "" H 0   0   50  0001 C CNN "Spice_Netlist_Enabled"
+F 7 "" H 0   0   50  0001 C CNN "Spice_Primitive"
 	1    3575 4700
 	0    -1   -1   0
@@
 AR Path="/5AE74AF7/64F2C9E1" Ref="C12"  Part="1"
 AR Path="/5AF84E03/64F2C9E1" Ref="C38"  Part="1"
-F 0 "C38" H 667 4646 50  0000 L CNN
+F 0 "C12" H 667 4646 50  0000 L CNN
 F 1 "100nF" H 667 4555 50  0000 L CNN
-F 2 "" H 575 4600 50  0001 C CNN
+F 2 "Capacitor_SMD:C_0805_2012Metric" H 575 4600 50  0001 C CNN
 F 3 "~" H 575 4600 50  0001 C CNN
+F 4 "" H 0   0   50  0001 C CNN "Spice_Lib_File"
+F 5 "" H 0   0   50  0001 C CNN "Spice_Model"
+F 6 "" H 0   0   50  0001 C CNN "Spice_Netlist_Enabled"
+F 7 "" H 0   0   50  0001 C CNN "Spice_Primitive"
 	1    575  4600
 	1    0    0    -1
@@
 AR Path="/5AE74AF7/64F33B67" Ref="C13"  Part="1"
 AR Path="/5AF84E03/64F33B67" Ref="C39"  Part="1"
-F 0 "C39" H 2692 4771 50  0000 L CNN
+F 0 "C13" H 2692 4771 50  0000 L CNN
 F 1 "100nF" H 2692 4680 50  0000 L CNN
-F 2 "" H 2600 4725 50  0001 C CNN
+F 2 "Capacitor_SMD:C_0805_2012Metric" H 2600 4725 50  0001 C CNN
 F 3 "~" H 2600 4725 50  0001 C CNN
+F 4 "" H 0   0   50  0001 C CNN "Spice_Lib_File"
+F 5 "" H 0   0   50  0001 C CNN "Spice_Model"
+F 6 "" H 0   0   50  0001 C CNN "Spice_Netlist_Enabled"
+F 7 "" H 0   0   50  0001 C CNN "Spice_Primitive"
 	1    2600 4725
 	1    0    0    -1

Commit message: started routing
Parts:
- U45, U46: footprint (none) -> Package_SO:SOIC-16_3.9x9.9mm_P1.27mm
Changed lines of the file:
@@
 AR Path="/5AE74AF7/5CF197AB" Ref="#PWR020"  Part="1"
 AR Path="/5AF84E03/5CF197AB" Ref="#PWR029"  Part="1"
-F 0 "#PWR020" H 4125 5650 30  0001 C CNN
+F 0 "#PWR029" H 4125 5650 30  0001 C CNN
 F 1 "GND" H 4125 5580 30  0001 C CNN
 F 2 "" H 4125 5650 60  0001 C CNN
@@
 AR Path="/5AE74AF7/5CF198E5" Ref="#PWR018"  Part="1"
 AR Path="/5AF84E03/5CF198E5" Ref="#PWR027"  Part="1"
-F 0 "#PWR018" H 1975 5575 30  0001 C CNN
+F 0 "#PWR027" H 1975 5575 30  0001 C CNN
 F 1 "GND" H 1975 5505 30  0001 C CNN
 F 2 "" H 1975 5575 60  0001 C CNN
@@
 AR Path="/5AE74AF7/5CF199DA" Ref="#PWR019"  Part="1"
 AR Path="/5AF84E03/5CF199DA" Ref="#PWR028"  Part="1"
-F 0 "#PWR019" H 2850 4300 30  0001 C CNN
+F 0 "#PWR028" H 2850 4300 30  0001 C CNN
 F 1 "GND" H 2850 4230 30  0001 C CNN
 F 2 "" H 2850 4300 60  0001 C CNN
@@
 AR Path="/5AE74AF7/5CF19D18" Ref="#PWR017"  Part="1"
 AR Path="/5AF84E03/5CF19D18" Ref="#PWR026"  Part="1"
-F 0 "#PWR017" H 700 4200 30  0001 C CNN
+F 0 "#PWR026" H 700 4200 30  0001 C CNN
 F 1 "GND" H 700 4130 30  0001 C CNN
 F 2 "" H 700 4200 60  0001 C CNN
@@
 AR Path="/5AE74AF7/5F3A2E1C" Ref="#PWR061"  Part="1"
 AR Path="/5AF84E03/5F3A2E1C" Ref="#PWR0127"  Part="1"
-F 0 "#PWR061" H 2525 5100 30  0001 C CNN
+F 0 "#PWR0127" H 2525 5100 30  0001 C CNN
 F 1 "VCC" H 2529 5127 30  0000 C CNN
 F 2 "" H 2525 5000 50  0001 C CNN
@@
 AR Path="/5AE74AF7/5F3A2E46" Ref="#PWR060"  Part="1"
 AR Path="/5AF84E03/5F3A2E46" Ref="#PWR0126"  Part="1"
-F 0 "#PWR060" H 875 5000 30  0001 C CNN
+F 0 "#PWR0126" H 875 5000 30  0001 C CNN
 F 1 "VCC" H 879 5027 30  0000 C CNN
 F 2 "" H 875 4900 50  0001 C CNN
@@
 AR Path="/5AE74AF7/5F3A2F2F" Ref="U45"  Part="1"
 AR Path="/5AF84E03/5F3A2F2F" Ref="U73"  Part="1"
-F 0 "U45" V 1603 4031 60  0000 R CNN
+F 0 "U73" V 1603 4031 60  0000 R CNN
 F 1 "74LS283" V 1497 4031 60  0000 R CNN
-F 2 "" H 1550 4575 60  0001 C CNN
+F 2 "Package_SO:SOIC-16_3.9x9.9mm_P1.27mm" H 1550 4575 60  0001 C CNN
 F 3 "" H 1550 4575 60  0001 C CNN
 F 4 "" H 0   0   50  0001 C CNN "Spice_Lib_File"
@@
 AR Path="/5AE74AF7/5F3A5CFF" Ref="U46"  Part="1"
 AR Path="/5AF84E03/5F3A5CFF" Ref="U74"  Part="1"
-F 0 "U46" V 3628 4156 60  0000 R CNN
+F 0 "U74" V 3628 4156 60  0000 R CNN
 F 1 "74LS283" V 3522 4156 60  0000 R CNN
-F 2 "" H 3575 4700 60  0001 C CNN
+F 2 "Package_SO:SOIC-16_3.9x9.9mm_P1.27mm" H 3575 4700 60  0001 C CNN
 F 3 "" H 3575 4700 60  0001 C CNN
 F 4 "" H 0   0   50  0001 C CNN "Spice_Lib_File"
@@
 AR Path="/5AE74AF7/64F2C9E1" Ref="C12"  Part="1"
 AR Path="/5AF84E03/64F2C9E1" Ref="C38"  Part="1"
-F 0 "C12" H 667 4646 50  0000 L CNN
+F 0 "C38" H 667 4646 50  0000 L CNN
 F 1 "100nF" H 667 4555 50  0000 L CNN
 F 2 "Capacitor_SMD:C_0805_2012Metric" H 575 4600 50  0001 C CNN
@@
 AR Path="/5AE74AF7/64F33B67" Ref="C13"  Part="1"
 AR Path="/5AF84E03/64F33B67" Ref="C39"  Part="1"
-F 0 "C13" H 2692 4771 50  0000 L CNN
+F 0 "C39" H 2692 4771 50  0000 L CNN
 F 1 "100nF" H 2692 4680 50  0000 L CNN
 F 2 "Capacitor_SMD:C_0805_2012Metric" H 2600 4725 50  0001 C CNN

Commit message: coniued layouting
Changed lines of the file:
@@
 $Descr A4 11693 8268
 encoding utf-8
-Sheet 38 191
+Sheet 120 191
 Title ""
 Date ""
@@
 	2850 4300 2675 4300
 Wire Wire Line
-	2675 4300 2675 4375
-Wire Wire Line
 	2675 5000 2525 5000
 Wire Wire Line
@@
 Wire Wire Line
 	750  4575 750  4925
-Wire Wire Line
-	2775 4700 2775 4375
-Wire Wire Line
-	2775 4375 2675 4375
-Connection ~ 2675 4375
-Wire Wire Line
-	2675 4375 2675 4500
 $Comp
 L Device:C_Small C12
@@
 	2600 4900 2675 4900
 Wire Wire Line
-	2675 4900 2675 5000
+	2675 4900 2675 4925
 Wire Wire Line
 	2600 4625 2600 4500
@@
 Wire Wire Line
 	4375 2225 4375 4000
+Wire Wire Line
+	2675 4300 2675 4500
+Wire Wire Line
+	2775 4700 2775 4925
+Wire Wire Line
+	2775 4925 2675 4925
+Connection ~ 2675 4925
+Wire Wire Line
+	2675 4925 2675 5000
 $EndSCHEMATC
