File: Alu/NOT.sch (KiCad schematic (older format))
At the start: 4 parts, among them U41 74HC04, U42 74HC04

Commit message: footprints
Parts:
- C36, C37: footprint (none) -> Capacitor_SMD:C_0805_2012Metric
- U41, U42: footprint (none) -> Package_SO:SOIC-14_3.9x8.7mm_P1.27mm

Commit message: started routing
Parts:
- added R155: 0, Resistor_SMD:R_1206_3216Metric_Pad1.39x1.80mm_HandSolder, symbol Device:R
- U41, U42: footprint (none) -> Package_SO:SOIC-14_3.9x8.7mm_P1.27mm
Connections:
- wire segments 79 -> 82
Changed lines of the file:
@@
 AR Path="/5AE655FE/64F62017/5C8F8352" Ref="#PWR050"  Part="1"
 AR Path="/5AE6649D/5C8F8352" Ref="#PWR057"  Part="1"
-F 0 "#PWR057" H 7900 2425 30  0001 C CNN
+F 0 "#PWR0125" H 7900 2425 30  0001 C CNN
 F 1 "VDD" H 7915 2462 30  0000 C CNN
 F 2 "" H 7900 2325 60  0001 C CNN
@@
 AR Path="/5AE655FE/64F62017/5C8FF848" Ref="#PWR048"  Part="1"
 AR Path="/5AE6649D/5C8FF848" Ref="#PWR055"  Part="1"
-F 0 "#PWR055" H 7375 4250 30  0001 C CNN
+F 0 "#PWR0123" H 7375 4250 30  0001 C CNN
 F 1 "GND" H 7375 4180 30  0001 C CNN
 F 2 "" H 7375 4250 60  0001 C CNN
@@
 AR Path="/5AE655FE/64F62017/5C8FF8DB" Ref="#PWR047"  Part="1"
 AR Path="/5AE6649D/5C8FF8DB" Ref="#PWR054"  Part="1"
-F 0 "#PWR054" H 7250 4300 30  0001 C CNN
+F 0 "#PWR0122" H 7250 4300 30  0001 C CNN
 F 1 "VSS" H 7250 4358 30  0000 C CNN
 F 2 "" H 7250 4300 60  0001 C CNN
@@
 AR Path="/5AE655FE/64F62017/5F2354CD" Ref="#PWR025"  Part="1"
 AR Path="/5AE6649D/5F2354CD" Ref="#PWR053"  Part="1"
-F 0 "#PWR053" H 5600 5125 30  0001 C CNN
+F 0 "#PWR0121" H 5600 5125 30  0001 C CNN
 F 1 "VCC" H 5604 5152 30  0000 C CNN
 F 2 "" H 5600 5025 50  0001 C CNN
@@
 AR Path="/5AE655FE/64F62017/5F235506" Ref="#PWR049"  Part="1"
 AR Path="/5AE6649D/5F235506" Ref="#PWR056"  Part="1"
-F 0 "#PWR056" H 7900 2350 30  0001 C CNN
+F 0 "#PWR0124" H 7900 2350 30  0001 C CNN
 F 1 "VCC" H 7904 2377 30  0000 C CNN
 F 2 "" H 7900 2250 50  0001 C CNN
@@
 F 0 "U41" V 2963 2772 40  0000 R CNN
 F 1 "74HC04" V 2887 2772 40  0000 R CNN
-F 2 "" H 2925 2950 60  0001 C CNN
+F 2 "Package_SO:SOIC-14_3.9x8.7mm_P1.27mm" H 2925 2950 60  0001 C CNN
 F 3 "" H 2925 2950 60  0001 C CNN
 F 4 "" H 0   0   50  0001 C CNN "Spice_Lib_File"
@@
 F 0 "U41" V 3638 2772 40  0000 R CNN
 F 1 "74HC04" V 3562 2772 40  0000 R CNN
-F 2 "" H 3600 2950 60  0001 C CNN
+F 2 "Package_SO:SOIC-14_3.9x8.7mm_P1.27mm" H 3600 2950 60  0001 C CNN
 F 3 "" H 3600 2950 60  0001 C CNN
 F 4 "" H 0   0   50  0001 C CNN "Spice_Lib_File"
@@
 F 0 "U41" V 4163 2772 40  0000 R CNN
 F 1 "74HC04" V 4087 2772 40  0000 R CNN
-F 2 "" H 4125 2950 60  0001 C CNN
+F 2 "Package_SO:SOIC-14_3.9x8.7mm_P1.27mm" H 4125 2950 60  0001 C CNN
 F 3 "" H 4125 2950 60  0001 C CNN
 F 4 "" H 0   0   50  0001 C CNN "Spice_Lib_File"
@@
 F 0 "U42" V 5413 2822 40  0000 R CNN
 F 1 "74HC04" V 5337 2822 40  0000 R CNN
-F 2 "" H 5375 3000 60  0001 C CNN
+F 2 "Package_SO:SOIC-14_3.9x8.7mm_P1.27mm" H 5375 3000 60  0001 C CNN
 F 3 "" H 5375 3000 60  0001 C CNN
 F 4 "" H 0   0   50  0001 C CNN "Spice_Lib_File"
@@
 F 0 "U42" H 7175 5317 40  0000 C CNN
 F 1 "74HC04" H 7175 5241 40  0000 C CNN
-F 2 "" H 7175 5025 60  0001 C CNN
+F 2 "Package_SO:SOIC-14_3.9x8.7mm_P1.27mm" H 7175 5025 60  0001 C CNN
 F 3 "" H 7175 5025 60  0001 C CNN
 F 4 "" H 0   0   50  0001 C CNN "Spice_Lib_File"
@@
 F 0 "U42" H 7375 5892 40  0000 C CNN
 F 1 "74HC04" H 7375 5816 40  0000 C CNN
-F 2 "" H 7375 5600 60  0001 C CNN
+F 2 "Package_SO:SOIC-14_3.9x8.7mm_P1.27mm" H 7375 5600 60  0001 C CNN
 F 3 "" H 7375 5600 60  0001 C CNN
 F 4 "" H 0   0   50  0001 C CNN "Spice_Lib_File"
@@
 F 0 "U42" H 7350 6442 40  0000 C CNN
 F 1 "74HC04" H 7350 6366 40  0000 C CNN
-F 2 "" H 7350 6150 60  0001 C CNN
+F 2 "Package_SO:SOIC-14_3.9x8.7mm_P1.27mm" H 7350 6150 60  0001 C CNN
 F 3 "" H 7350 6150 60  0001 C CNN
 F 4 "" H 0   0   50  0001 C CNN "Spice_Lib_File"
@@
 F 0 "U42" H 7375 6842 40  0000 C CNN
 F 1 "74HC04" H 7375 6766 40  0000 C CNN
-F 2 "" H 7375 6550 60  0001 C CNN
+F 2 "Package_SO:SOIC-14_3.9x8.7mm_P1.27mm" H 7375 6550 60  0001 C CNN
 F 3 "" H 7375 6550 60  0001 C CNN
 F 4 "" H 0   0   50  0001 C CNN "Spice_Lib_File"
@@
 F 0 "U41" H 3530 4946 50  0000 L CNN
 F 1 "74HC04" H 3530 4855 50  0000 L CNN
-F 2 "" H 3300 4900 50  0001 C CNN
+F 2 "Package_SO:SOIC-14_3.9x8.7mm_P1.27mm" H 3300 4900 50  0001 C CNN
 F 3 "http://www.nxp.com/documents/data_sheet/74HC_HCT04.pdf" H 3300 4900 50  0001 C CNN
 F 4 "" H 0   0   50  0001 C CNN "Spice_Lib_File"
@@
 F 0 "U42" H 4455 4971 50  0000 L CNN
 F 1 "74HC04" H 4455 4880 50  0000 L CNN
-F 2 "" H 4225 4925 50  0001 C CNN
+F 2 "Package_SO:SOIC-14_3.9x8.7mm_P1.27mm" H 4225 4925 50  0001 C CNN
 F 3 "http://www.nxp.com/documents/data_sheet/74HC_HCT04.pdf" H 4225 4925 50  0001 C CNN
 F 4 "" H 0   0   50  0001 C CNN "Spice_Lib_File"
@@
 AR Path="/5AE655FE/64F62017/5FB88813" Ref="#PWR023"  Part="1"
 AR Path="/5AE6649D/5FB88813" Ref="#PWR051"  Part="1"
-F 0 "#PWR051" H 3675 5550 30  0001 C CNN
+F 0 "#PWR0119" H 3675 5550 30  0001 C CNN
 F 1 "GND-power" H 3675 5480 30  0001 C CNN
 F 2 "" H 3675 5550 50  0001 C CNN
@@
 AR Path="/5AE655FE/64F62017/5FB8886C" Ref="#PWR024"  Part="1"
 AR Path="/5AE6649D/5FB8886C" Ref="#PWR052"  Part="1"
-F 0 "#PWR052" H 3750 3950 50  0001 C CNN
+F 0 "#PWR0120" H 3750 3950 50  0001 C CNN
 F 1 "VCC" H 3767 4273 50  0000 C CNN
 F 2 "" H 3750 4100 50  0001 C CNN
@@
 	1600 1425 1600 2675
 Wire Wire Line
-	2225 1375 2225 2225
-Wire Wire Line
 	2225 2225 2275 2225
-Connection ~ 2275 2225
-Wire Wire Line
-	2275 2225 2275 2650
 Wire Wire Line
 	2900 1375 2825 1375
@@
 Wire Wire Line
 	5325 2550 5375 2550
+$Comp
+L Device:R R155
+U 1 1 5B650DAB
+P 1900 2400
+AR Path="/5AE6649D/5B650DAB" Ref="R155"  Part="1"
+AR Path="/5B1BA146/5B650DAB" Ref="R156"  Part="1"
+F 0 "R155" H 1970 2446 50  0000 L CNN
+F 1 "0" H 1970 2355 50  0000 L CNN
+F 2 "Resistor_SMD:R_1206_3216Metric_Pad1.39x1.80mm_HandSolder" V 1830 2400 50  0001 C CNN
+F 3 "~" H 1900 2400 50  0001 C CNN
+	1    1900 2400
+	1    0    0    -1
+$EndComp
+Wire Wire Line
+	2275 2650 1900 2650
+Wire Wire Line
+	1900 2650 1900 2550
+Wire Wire Line
+	1900 2250 2225 2250
+Wire Wire Line
+	2225 1375 2225 2225
+Connection ~ 2225 2225
+Wire Wire Line
+	2225 2225 2225 2250
 $EndSCHEMATC

Commit message: coniued layouting
Parts:
- added R157, R158: 0, Resistor_SMD:R_1806_4516Metric, symbol Device:R
Connections:
- wire segments 82 -> 95
Changed lines of the file:
@@
 $Descr A4 11693 8268
 encoding utf-8
-Sheet 20 191
+Sheet 111 191
 Title ""
 Date ""
@@
 AR Path="/5B1BA146/5F235FE9" Ref="U71"  Part="1"
 AR Path="/5AE655FE/64F62017/5F235FE9" Ref="U39"  Part="1"
-F 0 "U41" V 1038 2747 40  0000 R CNN
+F 0 "U71" V 1038 2747 40  0000 R CNN
 F 1 "74HC04" V 962 2747 40  0000 R CNN
 F 2 "Package_SO:SOIC-14_3.9x8.7mm_P1.27mm" H 1000 2925 60  0001 C CNN
@@
 AR Path="/5B1BA146/5F2360F5" Ref="U71"  Part="2"
 AR Path="/5AE655FE/64F62017/5F2360F5" Ref="U39"  Part="2"
-F 0 "U41" V 1638 2797 40  0000 R CNN
+F 0 "U71" V 1638 2797 40  0000 R CNN
 F 1 "74HC04" V 1562 2797 40  0000 R CNN
 F 2 "Package_SO:SOIC-14_3.9x8.7mm_P1.27mm" H 1600 2975 60  0001 C CNN
@@
 AR Path="/5B1BA146/5F2361D5" Ref="U71"  Part="3"
 AR Path="/5AE655FE/64F62017/5F2361D5" Ref="U39"  Part="3"
-F 0 "U41" V 2313 2772 40  0000 R CNN
+F 0 "U71" V 2313 2772 40  0000 R CNN
 F 1 "74HC04" V 2237 2772 40  0000 R CNN
 F 2 "Package_SO:SOIC-14_3.9x8.7mm_P1.27mm" H 2275 2950 60  0001 C CNN
@@
 AR Path="/5B1BA146/5F236273" Ref="U71"  Part="4"
 AR Path="/5AE655FE/64F62017/5F236273" Ref="U39"  Part="4"
-F 0 "U41" V 2963 2772 40  0000 R CNN
+F 0 "U71" V 2963 2772 40  0000 R CNN
 F 1 "74HC04" V 2887 2772 40  0000 R CNN
 F 2 "Package_SO:SOIC-14_3.9x8.7mm_P1.27mm" H 2925 2950 60  0001 C CNN
@@
 AR Path="/5B1BA146/5F236307" Ref="U71"  Part="5"
 AR Path="/5AE655FE/64F62017/5F236307" Ref="U39"  Part="5"
-F 0 "U41" V 3638 2772 40  0000 R CNN
+F 0 "U71" V 3638 2772 40  0000 R CNN
 F 1 "74HC04" V 3562 2772 40  0000 R CNN
 F 2 "Package_SO:SOIC-14_3.9x8.7mm_P1.27mm" H 3600 2950 60  0001 C CNN
@@
 AR Path="/5B1BA146/5F23638F" Ref="U71"  Part="6"
 AR Path="/5AE655FE/64F62017/5F23638F" Ref="U39"  Part="6"
-F 0 "U41" V 4163 2772 40  0000 R CNN
+F 0 "U71" V 4163 2772 40  0000 R CNN
 F 1 "74HC04" V 4087 2772 40  0000 R CNN
 F 2 "Package_SO:SOIC-14_3.9x8.7mm_P1.27mm" H 4125 2950 60  0001 C CNN
@@
 AR Path="/5B1BA146/5F23644B" Ref="U72"  Part="1"
 AR Path="/5AE655FE/64F62017/5F23644B" Ref="U40"  Part="1"
-F 0 "U42" V 4813 2797 40  0000 R CNN
+F 0 "U72" V 4813 2797 40  0000 R CNN
 F 1 "74HC04" V 4737 2797 40  0000 R CNN
 F 2 "Package_SO:SOIC-14_3.9x8.7mm_P1.27mm" H 4775 2975 60  0001 C CNN
@@
 AR Path="/5B1BA146/5F236521" Ref="U72"  Part="2"
 AR Path="/5AE655FE/64F62017/5F236521" Ref="U40"  Part="2"
-F 0 "U42" V 5413 2822 40  0000 R CNN
+F 0 "U72" V 5413 2822 40  0000 R CNN
 F 1 "74HC04" V 5337 2822 40  0000 R CNN
 F 2 "Package_SO:SOIC-14_3.9x8.7mm_P1.27mm" H 5375 3000 60  0001 C CNN
@@
 AR Path="/5B1BA146/5F2365E7" Ref="U72"  Part="3"
 AR Path="/5AE655FE/64F62017/5F2365E7" Ref="U40"  Part="3"
-F 0 "U42" H 7175 5317 40  0000 C CNN
+F 0 "U72" H 7175 5317 40  0000 C CNN
 F 1 "74HC04" H 7175 5241 40  0000 C CNN
 F 2 "Package_SO:SOIC-14_3.9x8.7mm_P1.27mm" H 7175 5025 60  0001 C CNN
@@
 AR Path="/5B1BA146/5F236679" Ref="U72"  Part="5"
 AR Path="/5AE655FE/64F62017/5F236679" Ref="U40"  Part="5"
-F 0 "U42" H 7375 5892 40  0000 C CNN
+F 0 "U72" H 7375 5892 40  0000 C CNN
 F 1 "74HC04" H 7375 5816 40  0000 C CNN
 F 2 "Package_SO:SOIC-14_3.9x8.7mm_P1.27mm" H 7375 5600 60  0001 C CNN
@@
 AR Path="/5B1BA146/5F236716" Ref="U72"  Part="4"
 AR Path="/5AE655FE/64F62017/5F236716" Ref="U40"  Part="4"
-F 0 "U42" H 7350 6442 40  0000 C CNN
+F 0 "U72" H 7350 6442 40  0000 C CNN
 F 1 "74HC04" H 7350 6366 40  0000 C CNN
 F 2 "Package_SO:SOIC-14_3.9x8.7mm_P1.27mm" H 7350 6150 60  0001 C CNN
@@
 AR Path="/5B1BA146/5F2367A4" Ref="U72"  Part="6"
 AR Path="/5AE655FE/64F62017/5F2367A4" Ref="U40"  Part="6"
-F 0 "U42" H 7375 6842 40  0000 C CNN
+F 0 "U72" H 7375 6842 40  0000 C CNN
 F 1 "74HC04" H 7375 6766 40  0000 C CNN
 F 2 "Package_SO:SOIC-14_3.9x8.7mm_P1.27mm" H 7375 6550 60  0001 C CNN
@@
 AR Path="/5B1BA146/5FB83B89" Ref="U71"  Part="7"
 AR Path="/5AE655FE/64F62017/5FB83B89" Ref="U39"  Part="7"
-F 0 "U41" H 3530 4946 50  0000 L CNN
+F 0 "U71" H 3530 4946 50  0000 L CNN
 F 1 "74HC04" H 3530 4855 50  0000 L CNN
 F 2 "Package_SO:SOIC-14_3.9x8.7mm_P1.27mm" H 3300 4900 50  0001 C CNN
@@
 AR Path="/5B1BA146/5FB83CAA" Ref="U72"  Part="7"
 AR Path="/5AE655FE/64F62017/5FB83CAA" Ref="U40"  Part="7"
-F 0 "U42" H 4455 4971 50  0000 L CNN
+F 0 "U72" H 4455 4971 50  0000 L CNN
 F 1 "74HC04" H 4455 4880 50  0000 L CNN
 F 2 "Package_SO:SOIC-14_3.9x8.7mm_P1.27mm" H 4225 4925 50  0001 C CNN
@@
 AR Path="/5AE655FE/64F62017/5FB83DC0" Ref="C6"  Part="1"
 AR Path="/5AE6649D/5FB83DC0" Ref="C8"  Part="1"
-F 0 "C8" H 2792 4921 50  0000 L CNN
+F 0 "C36" H 2792 4921 50  0000 L CNN
 F 1 "100nF" H 2792 4830 50  0000 L CNN
 F 2 "Capacitor_SMD:C_0805_2012Metric" H 2700 4875 50  0001 C CNN
@@
 AR Path="/5AE655FE/64F62017/5FB83F1E" Ref="C7"  Part="1"
 AR Path="/5AE6649D/5FB83F1E" Ref="C9"  Part="1"
-F 0 "C9" H 4942 4921 50  0000 L CNN
+F 0 "C37" H 4942 4921 50  0000 L CNN
 F 1 "100nF" H 4942 4830 50  0000 L CNN
 F 2 "Capacitor_SMD:C_0805_2012Metric" H 4850 4875 50  0001 C CNN
@@
 $EndSheet
 Wire Wire Line
-	1000 1425 1000 2625
-Wire Wire Line
-	1600 1425 1600 2675
-Wire Wire Line
 	2225 2225 2275 2225
 Wire Wire Line
@@
 AR Path="/5AE6649D/5B650DAB" Ref="R155"  Part="1"
 AR Path="/5B1BA146/5B650DAB" Ref="R156"  Part="1"
-F 0 "R155" H 1970 2446 50  0000 L CNN
+F 0 "R156" H 1970 2446 50  0000 L CNN
 F 1 "0" H 1970 2355 50  0000 L CNN
 F 2 "Resistor_SMD:R_1206_3216Metric_Pad1.39x1.80mm_HandSolder" V 1830 2400 50  0001 C CNN
@@
 Wire Wire Line
 	2225 2225 2225 2250
+$Comp
+L Device:R R157
+U 1 1 5B654B5A
+P 700 2450
+AR Path="/5AE6649D/5B654B5A" Ref="R157"  Part="1"
+AR Path="/5B1BA146/5B654B5A" Ref="R159"  Part="1"
+F 0 "R159" H 770 2496 50  0000 L CNN
+F 1 "0" H 770 2405 50  0000 L CNN
+F 2 "Resistor_SMD:R_1806_4516Metric" V 630 2450 50  0001 C CNN
+F 3 "~" H 700 2450 50  0001 C CNN
+	1    700  2450
+	1    0    0    -1
+$EndComp
+$Comp
+L Device:R R158
+U 1 1 5B656920
+P 1325 2450
+AR Path="/5AE6649D/5B656920" Ref="R158"  Part="1"
+AR Path="/5B1BA146/5B656920" Ref="R160"  Part="1"
+F 0 "R160" H 1395 2496 50  0000 L CNN
+F 1 "0" H 1395 2405 50  0000 L CNN
+F 2 "Resistor_SMD:R_1806_4516Metric" V 1255 2450 50  0001 C CNN
+F 3 "~" H 1325 2450 50  0001 C CNN
+	1    1325 2450
+	1    0    0    -1
+$EndComp
+Wire Wire Line
+	1000 2625 700  2625
+Wire Wire Line
+	700  2625 700  2600
+Wire Wire Line
+	700  2300 700  1975
+Wire Wire Line
+	700  1975 825  1975
+Wire Wire Line
+	825  1975 825  1675
+Wire Wire Line
+	825  1675 1000 1675
+Wire Wire Line
+	1000 1675 1000 1425
+Connection ~ 825  1975
+Wire Wire Line
+	825  1975 1000 1975
+Wire Wire Line
+	1600 1425 1325 1425
+Wire Wire Line
+	1325 1425 1325 2125
+Wire Wire Line
+	1325 2125 1600 2125
+Wire Wire Line
+	1600 2125 1600 2050
+Connection ~ 1325 2125
+Wire Wire Line
+	1325 2125 1325 2300
+Wire Wire Line
+	1325 2600 1600 2600
+Wire Wire Line
+	1600 2600 1600 2675
 $EndSCHEMATC
