File: Alu/16-2MUX.sch (KiCad schematic (older format))
At the start: 4 parts, among them U55 74LS251, U56 74LS251

Commit message: footprints
Parts:
- C20, C21: footprint (none) -> Capacitor_SMD:C_0805_2012Metric
Connections:
- wire segments 90 -> 97
Changed lines of the file:
@@
 $Descr A4 11693 8268
 encoding utf-8
-Sheet 12 156
+Sheet 79 191
 Title ""
 Date ""
@@
 Z1
 Wire Wire Line
-	2150 3700 2150 4525
-Wire Wire Line
-	2250 3700 3700 3700
+	2150 3700 2150 3800
+Wire Wire Line
+	2250 3700 2550 3700
 Wire Wire Line
 	3700 3700 3700 4575
@@
 AR Path="/5AE9DF6E/5AEC72A2/66184586" Ref="U67"  Part="1"
 AR Path="/5AE9DF6E/5AEC72B9/66184586" Ref="U69"  Part="1"
-F 0 "U69" V 2621 4384 50  0000 R CNN
+F 0 "U55" V 2621 4384 50  0000 R CNN
 F 1 "74LS251" V 2530 4384 50  0000 R CNN
 F 2 "" H 2575 5425 50  0001 C CNN
 F 3 "http://www.ti.com/lit/gpn/sn74LS251" H 2575 5425 50  0001 C CNN
+F 4 "" H 0   0   50  0001 C CNN "Spice_Lib_File"
+F 5 "" H 0   0   50  0001 C CNN "Spice_Model"
+F 6 "" H 0   0   50  0001 C CNN "Spice_Netlist_Enabled"
+F 7 "" H 0   0   50  0001 C CNN "Spice_Primitive"
 	1    2575 5425
 	0    -1   -1   0
@@
 AR Path="/5AE9DF6E/5AEC72A2/66189CD4" Ref="U68"  Part="1"
 AR Path="/5AE9DF6E/5AEC72B9/66189CD4" Ref="U70"  Part="1"
-F 0 "U70" V 5821 4334 50  0000 R CNN
+F 0 "U56" V 5821 4334 50  0000 R CNN
 F 1 "74LS251" V 5730 4334 50  0000 R CNN
 F 2 "" H 5775 5375 50  0001 C CNN
 F 3 "http://www.ti.com/lit/gpn/sn74LS251" H 5775 5375 50  0001 C CNN
+F 4 "" H 0   0   50  0001 C CNN "Spice_Lib_File"
+F 5 "" H 0   0   50  0001 C CNN "Spice_Model"
+F 6 "" H 0   0   50  0001 C CNN "Spice_Netlist_Enabled"
+F 7 "" H 0   0   50  0001 C CNN "Spice_Primitive"
 	1    5775 5375
 	0    -1   -1   0
@@
 AR Path="/5AE9DF6E/5AEC72A2/6618B226" Ref="C32"  Part="1"
 AR Path="/5AE9DF6E/5AEC72B9/6618B226" Ref="C34"  Part="1"
-F 0 "C34" H 4067 5771 50  0000 L CNN
+F 0 "C20" H 4067 5771 50  0000 L CNN
 F 1 "100nF" H 4067 5680 50  0000 L CNN
-F 2 "" H 3975 5725 50  0001 C CNN
+F 2 "Capacitor_SMD:C_0805_2012Metric" H 3975 5725 50  0001 C CNN
 F 3 "~" H 3975 5725 50  0001 C CNN
+F 4 "" H 0   0   50  0001 C CNN "Spice_Lib_File"
+F 5 "" H 0   0   50  0001 C CNN "Spice_Model"
+F 6 "" H 0   0   50  0001 C CNN "Spice_Netlist_Enabled"
+F 7 "" H 0   0   50  0001 C CNN "Spice_Primitive"
 	1    3975 5725
 	1    0    0    -1
@@
 AR Path="/5AE9DF6E/5AEC72A2/6618B289" Ref="C33"  Part="1"
 AR Path="/5AE9DF6E/5AEC72B9/6618B289" Ref="C35"  Part="1"
-F 0 "C35" H 4467 5796 50  0000 L CNN
+F 0 "C21" H 4467 5796 50  0000 L CNN
 F 1 "100nF" H 4467 5705 50  0000 L CNN
-F 2 "" H 4375 5750 50  0001 C CNN
+F 2 "Capacitor_SMD:C_0805_2012Metric" H 4375 5750 50  0001 C CNN
 F 3 "~" H 4375 5750 50  0001 C CNN
+F 4 "" H 0   0   50  0001 C CNN "Spice_Lib_File"
+F 5 "" H 0   0   50  0001 C CNN "Spice_Model"
+F 6 "" H 0   0   50  0001 C CNN "Spice_Netlist_Enabled"
+F 7 "" H 0   0   50  0001 C CNN "Spice_Primitive"
 	1    4375 5750
 	1    0    0    -1
@@
 AR Path="/5AE9DF6E/5AEC72A2/6618B361" Ref="#PWR0113"  Part="1"
 AR Path="/5AE9DF6E/5AEC72B9/6618B361" Ref="#PWR0117"  Part="1"
-F 0 "#PWR0117" H 4375 5175 50  0001 C CNN
+F 0 "#PWR089" H 4375 5175 50  0001 C CNN
 F 1 "VCC" H 4392 5498 50  0000 C CNN
 F 2 "" H 4375 5325 50  0001 C CNN
@@
 AR Path="/5AE9DF6E/5AEC72A2/6618B396" Ref="#PWR0112"  Part="1"
 AR Path="/5AE9DF6E/5AEC72B9/6618B396" Ref="#PWR0116"  Part="1"
-F 0 "#PWR0116" H 3700 5950 30  0001 C CNN
+F 0 "#PWR088" H 3700 5950 30  0001 C CNN
 F 1 "GND-power" H 3700 5880 30  0001 C CNN
 F 2 "" H 3700 5950 50  0001 C CNN
@@
 AR Path="/5AE9DF6E/5AEC72A2/66197FCF" Ref="#PWR0114"  Part="1"
 AR Path="/5AE9DF6E/5AEC72B9/66197FCF" Ref="#PWR0118"  Part="1"
-F 0 "#PWR0118" H 6800 6100 30  0001 C CNN
+F 0 "#PWR090" H 6800 6100 30  0001 C CNN
 F 1 "GND-power" H 6800 6030 30  0001 C CNN
 F 2 "" H 6800 6100 50  0001 C CNN
@@
 AR Path="/5AE9DF6E/5AEC72A2/66199FC5" Ref="#PWR0111"  Part="1"
 AR Path="/5AE9DF6E/5AEC72B9/66199FC5" Ref="#PWR0115"  Part="1"
-F 0 "#PWR0115" H 1325 5250 50  0001 C CNN
+F 0 "#PWR087" H 1325 5250 50  0001 C CNN
 F 1 "VCC" H 1342 5573 50  0000 C CNN
 F 2 "" H 1325 5400 50  0001 C CNN
@@
 Wire Wire Line
 	1675 5400 1675 5425
+$Sheet
+S 2025 2900 500  150
+U 5B83E62A
+F0 "Sheet5B83E629" 50
+F1 "LED_RED.sch" 50
+F2 "X" I L 2025 2975 50
+$EndSheet
+$Sheet
+S 3000 3250 500  150
+U 5B83E648
+F0 "sheet5B83E645" 50
+F1 "LED_RED.sch" 50
+F2 "X" I L 3000 3325 50
+$EndSheet
+Wire Wire Line
+	2150 3800 1550 3800
+Wire Wire Line
+	1550 3800 1550 2975
+Wire Wire Line
+	1550 2975 2025 2975
+Connection ~ 2150 3800
+Wire Wire Line
+	2150 3800 2150 4525
+Wire Wire Line
+	3000 3325 2550 3325
+Wire Wire Line
+	2550 3325 2550 3700
+Connection ~ 2550 3700
+Wire Wire Line
+	2550 3700 3700 3700
 $EndSCHEMATC

Commit message: started routing
Parts:
- U55, U56: footprint (none) -> Package_SO:SOIC-16_3.9x9.9mm_P1.27mm
Changed lines of the file:
@@
 AR Path="/5AE9DF6E/5AEC72A2/66184586" Ref="U67"  Part="1"
 AR Path="/5AE9DF6E/5AEC72B9/66184586" Ref="U69"  Part="1"
-F 0 "U55" V 2621 4384 50  0000 R CNN
+F 0 "U69" V 2621 4384 50  0000 R CNN
 F 1 "74LS251" V 2530 4384 50  0000 R CNN
-F 2 "" H 2575 5425 50  0001 C CNN
+F 2 "Package_SO:SOIC-16_3.9x9.9mm_P1.27mm" H 2575 5425 50  0001 C CNN
 F 3 "http://www.ti.com/lit/gpn/sn74LS251" H 2575 5425 50  0001 C CNN
 F 4 "" H 0   0   50  0001 C CNN "Spice_Lib_File"
@@
 AR Path="/5AE9DF6E/5AEC72A2/66189CD4" Ref="U68"  Part="1"
 AR Path="/5AE9DF6E/5AEC72B9/66189CD4" Ref="U70"  Part="1"
-F 0 "U56" V 5821 4334 50  0000 R CNN
+F 0 "U70" V 5821 4334 50  0000 R CNN
 F 1 "74LS251" V 5730 4334 50  0000 R CNN
-F 2 "" H 5775 5375 50  0001 C CNN
+F 2 "Package_SO:SOIC-16_3.9x9.9mm_P1.27mm" H 5775 5375 50  0001 C CNN
 F 3 "http://www.ti.com/lit/gpn/sn74LS251" H 5775 5375 50  0001 C CNN
 F 4 "" H 0   0   50  0001 C CNN "Spice_Lib_File"
@@
 AR Path="/5AE9DF6E/5AEC72A2/6618B226" Ref="C32"  Part="1"
 AR Path="/5AE9DF6E/5AEC72B9/6618B226" Ref="C34"  Part="1"
-F 0 "C20" H 4067 5771 50  0000 L CNN
+F 0 "C34" H 4067 5771 50  0000 L CNN
 F 1 "100nF" H 4067 5680 50  0000 L CNN
 F 2 "Capacitor_SMD:C_0805_2012Metric" H 3975 5725 50  0001 C CNN
@@
 AR Path="/5AE9DF6E/5AEC72A2/6618B289" Ref="C33"  Part="1"
 AR Path="/5AE9DF6E/5AEC72B9/6618B289" Ref="C35"  Part="1"
-F 0 "C21" H 4467 5796 50  0000 L CNN
+F 0 "C35" H 4467 5796 50  0000 L CNN
 F 1 "100nF" H 4467 5705 50  0000 L CNN
 F 2 "Capacitor_SMD:C_0805_2012Metric" H 4375 5750 50  0001 C CNN
@@
 AR Path="/5AE9DF6E/5AEC72A2/6618B361" Ref="#PWR0113"  Part="1"
 AR Path="/5AE9DF6E/5AEC72B9/6618B361" Ref="#PWR0117"  Part="1"
-F 0 "#PWR089" H 4375 5175 50  0001 C CNN
+F 0 "#PWR0117" H 4375 5175 50  0001 C CNN
 F 1 "VCC" H 4392 5498 50  0000 C CNN
 F 2 "" H 4375 5325 50  0001 C CNN
@@
 AR Path="/5AE9DF6E/5AEC72A2/6618B396" Ref="#PWR0112"  Part="1"
 AR Path="/5AE9DF6E/5AEC72B9/6618B396" Ref="#PWR0116"  Part="1"
-F 0 "#PWR088" H 3700 5950 30  0001 C CNN
+F 0 "#PWR0116" H 3700 5950 30  0001 C CNN
 F 1 "GND-power" H 3700 5880 30  0001 C CNN
 F 2 "" H 3700 5950 50  0001 C CNN
@@
 AR Path="/5AE9DF6E/5AEC72A2/66197FCF" Ref="#PWR0114"  Part="1"
 AR Path="/5AE9DF6E/5AEC72B9/66197FCF" Ref="#PWR0118"  Part="1"
-F 0 "#PWR090" H 6800 6100 30  0001 C CNN
+F 0 "#PWR0118" H 6800 6100 30  0001 C CNN
 F 1 "GND-power" H 6800 6030 30  0001 C CNN
 F 2 "" H 6800 6100 50  0001 C CNN
@@
 AR Path="/5AE9DF6E/5AEC72A2/66199FC5" Ref="#PWR0111"  Part="1"
 AR Path="/5AE9DF6E/5AEC72B9/66199FC5" Ref="#PWR0115"  Part="1"
-F 0 "#PWR087" H 1325 5250 50  0001 C CNN
+F 0 "#PWR0115" H 1325 5250 50  0001 C CNN
 F 1 "VCC" H 1342 5573 50  0000 C CNN
 F 2 "" H 1325 5400 50  0001 C CNN
