File: Alu/ADD.sch (KiCad schematic (older format))
At the start: 4 parts, among them U51 74LS283, U52 74LS283

Commit message: footprints
Parts:
- C16, C17: footprint (none) -> Capacitor_SMD:C_0805_2012Metric
Changed lines of the file:
@@
 $Descr A4 11693 8268
 encoding utf-8
-Sheet 58 156
+Sheet 67 191
 Title ""
 Date ""
@@
 AR Path="/5AE93FA0/5F3AAAB6" Ref="#PWR079"  Part="1"
 AR Path="/5AEA44C6/5F3AAAB6" Ref="#PWR073"  Part="1"
-F 0 "#PWR073" H 5275 5025 30  0001 C CNN
+F 0 "#PWR079" H 5275 5025 30  0001 C CNN
 F 1 "VCC" H 5279 5052 30  0000 C CNN
 F 2 "" H 5275 4925 50  0001 C CNN
@@
 AR Path="/5AE93FA0/5F3AAAF3" Ref="#PWR075"  Part="1"
 AR Path="/5AEA44C6/5F3AAAF3" Ref="#PWR069"  Part="1"
-F 0 "#PWR069" H 2050 4925 30  0001 C CNN
+F 0 "#PWR075" H 2050 4925 30  0001 C CNN
 F 1 "VCC" H 2054 4952 30  0000 C CNN
 F 2 "" H 2050 4825 50  0001 C CNN
@@
 AR Path="/5AE93FA0/5F3AAB22" Ref="#PWR076"  Part="1"
 AR Path="/5AEA44C6/5F3AAB22" Ref="#PWR070"  Part="1"
-F 0 "#PWR070" H 2300 4000 30  0001 C CNN
+F 0 "#PWR076" H 2300 4000 30  0001 C CNN
 F 1 "GND" H 2300 3930 30  0001 C CNN
 F 2 "" H 2300 4000 50  0001 C CNN
@@
 AR Path="/5AE93FA0/5F3AAB5F" Ref="#PWR080"  Part="1"
 AR Path="/5AEA44C6/5F3AAB5F" Ref="#PWR074"  Part="1"
-F 0 "#PWR074" H 5850 4125 30  0001 C CNN
+F 0 "#PWR080" H 5850 4125 30  0001 C CNN
 F 1 "GND" H 5850 4055 30  0001 C CNN
 F 2 "" H 5850 4125 50  0001 C CNN
@@
 AR Path="/5AE93FA0/5F3AAB90" Ref="U51"  Part="1"
 AR Path="/5AEA44C6/5F3AAB90" Ref="U49"  Part="1"
-F 0 "U49" V 3128 3956 60  0000 R CNN
+F 0 "U51" V 3128 3956 60  0000 R CNN
 F 1 "74LS283" V 3022 3956 60  0000 R CNN
 F 2 "" H 3075 4500 60  0001 C CNN
 F 3 "" H 3075 4500 60  0001 C CNN
+F 4 "" H 0   0   50  0001 C CNN "Spice_Lib_File"
+F 5 "" H 0   0   50  0001 C CNN "Spice_Model"
+F 6 "" H 0   0   50  0001 C CNN "Spice_Netlist_Enabled"
+F 7 "" H 0   0   50  0001 C CNN "Spice_Primitive"
 	1    3075 4500
 	0    -1   -1   0
@@
 AR Path="/5AE93FA0/5F3AAC37" Ref="U52"  Part="1"
 AR Path="/5AEA44C6/5F3AAC37" Ref="U50"  Part="1"
-F 0 "U50" V 4628 4131 60  0000 R CNN
+F 0 "U52" V 4628 4131 60  0000 R CNN
 F 1 "74LS283" V 4522 4131 60  0000 R CNN
 F 2 "" H 4575 4675 60  0001 C CNN
 F 3 "" H 4575 4675 60  0001 C CNN
+F 4 "" H 0   0   50  0001 C CNN "Spice_Lib_File"
+F 5 "" H 0   0   50  0001 C CNN "Spice_Model"
+F 6 "" H 0   0   50  0001 C CNN "Spice_Netlist_Enabled"
+F 7 "" H 0   0   50  0001 C CNN "Spice_Primitive"
 	1    4575 4675
 	0    -1   -1   0
@@
 AR Path="/5AE93FA0/64F3B924" Ref="C17"  Part="1"
 AR Path="/5AEA44C6/64F3B924" Ref="C15"  Part="1"
-F 0 "C15" H 5692 4521 50  0000 L CNN
+F 0 "C17" H 5692 4521 50  0000 L CNN
 F 1 "100nF" H 5692 4430 50  0000 L CNN
-F 2 "" H 5600 4475 50  0001 C CNN
+F 2 "Capacitor_SMD:C_0805_2012Metric" H 5600 4475 50  0001 C CNN
 F 3 "~" H 5600 4475 50  0001 C CNN
+F 4 "" H 0   0   50  0001 C CNN "Spice_Lib_File"
+F 5 "" H 0   0   50  0001 C CNN "Spice_Model"
+F 6 "" H 0   0   50  0001 C CNN "Spice_Netlist_Enabled"
+F 7 "" H 0   0   50  0001 C CNN "Spice_Primitive"
 	1    5600 4475
 	1    0    0    -1
@@
 AR Path="/5AE93FA0/64F3BAE9" Ref="C16"  Part="1"
 AR Path="/5AEA44C6/64F3BAE9" Ref="C14"  Part="1"
-F 0 "C14" H 2092 4471 50  0000 L CNN
+F 0 "C16" H 2092 4471 50  0000 L CNN
 F 1 "100nF" H 2092 4380 50  0000 L CNN
-F 2 "" H 2000 4425 50  0001 C CNN
+F 2 "Capacitor_SMD:C_0805_2012Metric" H 2000 4425 50  0001 C CNN
 F 3 "~" H 2000 4425 50  0001 C CNN
+F 4 "" H 0   0   50  0001 C CNN "Spice_Lib_File"
+F 5 "" H 0   0   50  0001 C CNN "Spice_Model"
+F 6 "" H 0   0   50  0001 C CNN "Spice_Netlist_Enabled"
+F 7 "" H 0   0   50  0001 C CNN "Spice_Primitive"
 	1    2000 4425
 	1    0    0    -1
@@
 AR Path="/5AE93FA0/64F4E2BB" Ref="#PWR077"  Part="1"
 AR Path="/5AEA44C6/64F4E2BB" Ref="#PWR071"  Part="1"
-F 0 "#PWR071" H 3825 4325 30  0001 C CNN
+F 0 "#PWR077" H 3825 4325 30  0001 C CNN
 F 1 "GND-power" H 3825 4255 30  0001 C CNN
 F 2 "" H 3825 4325 50  0001 C CNN
@@
 AR Path="/5AE93FA0/64F4E2F8" Ref="#PWR078"  Part="1"
 AR Path="/5AEA44C6/64F4E2F8" Ref="#PWR072"  Part="1"
-F 0 "#PWR072" H 3875 4725 50  0001 C CNN
+F 0 "#PWR078" H 3875 4725 50  0001 C CNN
 F 1 "VCC" H 3892 5048 50  0000 C CNN
 F 2 "" H 3875 4875 50  0001 C CNN

Commit message: started routing
Parts:
- U51, U52: footprint (none) -> Package_SO:SOIC-16_3.9x9.9mm_P1.27mm
Changed lines of the file:
@@
 F 0 "U51" V 3128 3956 60  0000 R CNN
 F 1 "74LS283" V 3022 3956 60  0000 R CNN
-F 2 "" H 3075 4500 60  0001 C CNN
+F 2 "Package_SO:SOIC-16_3.9x9.9mm_P1.27mm" H 3075 4500 60  0001 C CNN
 F 3 "" H 3075 4500 60  0001 C CNN
 F 4 "" H 0   0   50  0001 C CNN "Spice_Lib_File"
@@
 F 0 "U52" V 4628 4131 60  0000 R CNN
 F 1 "74LS283" V 4522 4131 60  0000 R CNN
-F 2 "" H 4575 4675 60  0001 C CNN
+F 2 "Package_SO:SOIC-16_3.9x9.9mm_P1.27mm" H 4575 4675 60  0001 C CNN
 F 3 "" H 4575 4675 60  0001 C CNN
 F 4 "" H 0   0   50  0001 C CNN "Spice_Lib_File"
