File: Alu/Alu.kicad_pcb (KiCad board)
At the start: 2 copper layers, 628 parts, among them J1 Conn_01x34, J2 Barrel_Jack, Q1 2N7002, Q10 2N7002, Q100 2N7002, Q101 2N7002, Q102 2N7002, Q103 2N7002, Q104 2N7002, Q105 2N7002, Q106 2N7002, Q107 2N7002, Q108 2N7002, Q109 2N7002, Q11 2N7002, Q110 2N7002, Q111 2N7002, Q112 2N7002, Q113 2N7002, Q114 2N7002, Q115 2N7002, Q116 2N7002, Q117 2N7002, Q118 2N7002, Q119 2N7002, Q12 2N7002, Q120 2N7002, Q121 2N7002, Q122 2N7002, Q123 2N7002, Q124 2N7002, Q125 2N7002, Q126 2N7002, Q127 2N7002, Q128 2N7002, Q129 2N7002, Q13 2N7002, Q130 2N7002, Q131 2N7002, Q132 2N7002, Q133 2N7002, Q134 2N7002, Q135 2N7002, Q136 2N7002, Q137 2N7002, Q138 2N7002, Q139 2N7002, Q14 2N7002, Q140 2N7002, Q141 2N7002, Q142 2N7002, Q143 2N7002, Q144 2N7002, Q145 2N7002, Q146 2N7002, Q147 2N7002, Q148 2N7002, Q149 2N7002, Q15 2N7002, Q150 2N7002, Q151 2N7002, Q152 2N7002, Q153 2N7002, Q154 2N7002, Q16 2N7002, Q163 2N7002, Q164 2N7002, Q165 2N7002, Q166 2N7002, Q167 2N7002, Q168 2N7002, Q17 2N7002, Q18 2N7002, Q19 2N7002, Q2 2N7002, Q20 2N7002, Q21 2N7002, Q22 2N7002, Q23 2N7002, Q24 2N7002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

Commit message: coniued layouting
Parts:
- added C6: 100nF, Capacitor_SMD:C_0805_2012Metric_Pad1.29x1.40mm_HandSolder, F.Cu at (34.3, 247.0)
- added C7: 100nF, Capacitor_SMD:C_0805_2012Metric_Pad1.29x1.40mm_HandSolder, F.Cu at (33.7, 268.6)
- moved Q96 615.1 mm to (55.3, 449.9)
- moved R96 610.5 mm to (67.1, 448.9), turned to 180 degrees
- moved D96 604.3 mm to (80.4, 449.0)
- moved Q94 549.0 mm to (55.2, 432.4)
- moved Q98 543.3 mm to (55.0, 460.3)
- moved R98 540.5 mm to (67.9, 460.4), turned to 180 degrees
- moved D98 527.0 mm to (80.0, 459.7)
- moved Q53 517.8 mm to (45.7, 378.5)
- moved R53 517.1 mm to (56.5, 378.5), turned to 180 degrees
- moved C36 512.2 mm to (31.5, 462.3), turned to 180 degrees
- moved D53 507.8 mm to (65.8, 378.5)
- moved Q50 504.2 mm to (45.7, 360.0)
- moved U72 499.6 mm to (31.8, 455.3)
- moved C37 499.2 mm to (31.8, 441.3), turned to 180 degrees
- moved Q58 489.2 mm to (45.3, 403.9)
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Connections:
- U46 pad 16: GND -> VCC
- U74 pad 16: GND -> VCC

Commit message: started routing :)
Parts:
- added J10: Conn_01x08, Connector_PinHeader_2.54mm:PinHeader_1x08_P2.54mm_Vertical_SMD_Pin1Right, F.Cu at (-865.0, -19.9)
- added J11: Conn_01x08, Connector_PinHeader_2.54mm:PinHeader_1x08_P2.54mm_Vertical_SMD_Pin1Right, F.Cu at (-894.5, -19.9)
- added J12: Conn_01x08, Connector_PinHeader_2.54mm:PinHeader_1x08_P2.54mm_Vertical_SMD_Pin1Right, F.Cu at (-855.2, -19.9)
- added J13: Conn_01x08, Connector_PinHeader_2.54mm:PinHeader_1x08_P2.54mm_Vertical_SMD_Pin1Right, F.Cu at (-884.7, -19.9)
- added J14: Conn_01x08, Connector_PinHeader_2.54mm:PinHeader_1x08_P2.54mm_Vertical_SMD_Pin1Right, F.Cu at (31.8, 76.8)
- added J3: Conn_01x08, Connector_PinHeader_2.54mm:PinHeader_1x08_P2.54mm_Vertical_SMD_Pin1Right, F.Cu at (-894.1, -43.2)
- added J4: Conn_01x18, Connector_PinHeader_2.54mm:PinHeader_1x18_P2.54mm_Vertical_SMD_Pin1Left, F.Cu at (-892.8, 101.0)
- added J5: Conn_01x08, Connector_PinHeader_2.54mm:PinHeader_1x08_P2.54mm_Vertical_SMD_Pin1Right, F.Cu at (-882.5, -43.4)
- added J6: Conn_01x08, Connector_PinHeader_2.54mm:PinHeader_1x08_P2.54mm_Vertical_SMD_Pin1Right, F.Cu at (-872.6, -43.4)
- added J7: Conn_01x08, Connector_PinHeader_2.54mm:PinHeader_1x08_P2.54mm_Vertical_SMD_Pin1Right, F.Cu at (-862.8, -43.4)
- added J8: Conn_01x18, Connector_PinHeader_2.54mm:PinHeader_1x18_P2.54mm_Vertical_SMD_Pin1Left, F.Cu at (-839.5, -30.5)
- added J9: Conn_01x08, Connector_PinHeader_2.54mm:PinHeader_1x08_P2.54mm_Vertical_SMD_Pin1Right, F.Cu at (-874.9, -19.9)
- J1: value Conn_01x34 -> Conn_01x08; footprint Connector_PinHeader_2.54mm:PinHeader_1x34_P2.54mm_Vertical_SMD_Pin1Right -> Connector_PinHeader_2.54mm:PinHeader_1x08_P2.54mm_Vertical_SMD_Pin1Right
- R135, R136, R137, R138, R166: footprint Resistor_SMD:R_0815_2038Metric_Pad1.64x4.00mm_HandSolder -> Resistor_SMD:R_0805_2012Metric_Pad1.29x1.40mm_HandSolder
- moved Q151 1305.5 mm to (-802.3, -54.7)
- moved R151 1301.3 mm to (-792.9, -54.6), turned to 180 degrees
- moved D151 1296.2 mm to (-783.3, -54.6)
- moved Q148 1265.2 mm to (-803.0, -69.6)
- moved R148 1260.2 mm to (-792.5, -70.5), turned to 180 degrees
- moved Q133 1257.7 mm to (-788.0, 11.4)
- moved Q147 1256.9 mm to (-802.4, -74.7)
- moved R147 1256.7 mm to (-792.5, -74.9), turned to 180 degrees
- moved D148 1255.3 mm to (-783.2, -69.8)
- moved Q127 1251.5 mm to (-787.1, -24.0)
- moved R133 1251.1 mm to (-776.0, 10.2), turned to 180 degrees
- moved D133 1246.6 mm to (-767.1, 9.95)
- moved R127 1246.2 mm to (-776.4, -24.8), turned to 180 degrees
- moved D147 1243.6 mm to (-783.8, -73.7)
- moved D127 1239.7 mm to (-765.6, -24.1)
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Connections:
- J1 pad 1: GND -> /Bit7_X10
- J1 pad 2: VCC -> /Bit6_X10
- J1 pad 3: /Z7 -> /Bit5_X10
- J1 pad 4: /Z6 -> /Bit4_X10
- J1 pad 5: /Z5 -> /Bit3_X10
- J1 pad 6: /Z4 -> /Bit2_X10
- J1 pad 7: /Z3 -> /Bit1_X10
- J1 pad 8: /Z2 -> /Bit0_X10
Routing:
- net VCC: track 129.6 -> 363.1 mm, vias 2 -> 4
- net GND: track 147.0 -> 336.9 mm
- net /Bit3_X10: track 0.00 -> 138.2 mm, vias 0 -> 2
- net /Bit2_X10: track 0.00 -> 134.4 mm, vias 0 -> 2
- net /Bit6_X10: track 0.00 -> 124.5 mm, vias 0 -> 2
- net /Bit1_X10: track 0.00 -> 123.7 mm
- net /Bit5_X10: track 0.00 -> 119.9 mm
- net /Bit0_X10: track 0.00 -> 119.5 mm
- net /Bit4_X10: track 0.00 -> 114.7 mm
- net /Bit7_X10: track 0.00 -> 94.2 mm
- net /Y7: track 37.8 -> 119.8 mm
- net /Y6: track 34.9 -> 115.5 mm
- net /Y5: track 40.3 -> 117.8 mm
- net /Y4: track 38.7 -> 111.1 mm
- net /Y3: track 42.0 -> 113.9 mm
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Other:
- copper layers 2 -> 4
- board text added: "CARRY-MUX"
