File: Alu/LED_BLUE.sch (KiCad schematic (older format))
At the start: 3 parts

Commit message: footprints
Parts:
- D49: renamed from D?; footprint (none) -> LED_SMD:LED_0805_2012Metric_Pad1.12x1.40mm_HandSolder
- R49: renamed from R?; footprint (none) -> Resistor_SMD:R_0805_2012Metric_Pad1.29x1.40mm_HandSolder
- gave numbers to parts that had none: 1
Changed lines of the file:
@@
 $Descr A4 11693 8268
 encoding utf-8
-Sheet 69 156
+Sheet 187 191
 Title ""
 Date ""
@@
 $EndDescr
 $Comp
-L Device:R R?
+L Device:R R49
 U 1 1 6AD31404
 P 5675 3800
-F 0 "R?" V 5468 3800 50  0000 C CNN
+AR Path="/5AE74AF7/5C384037/6AD31404" Ref="R49"  Part="1"
+AR Path="/5AE75BF4/5B58AD87/6AD31404" Ref="R57"  Part="1"
+AR Path="/5AEA44C6/5C3E9C32/6AD31404" Ref="R67"  Part="1"
+AR Path="/5AE93FA0/5C3E9C32/6AD31404" Ref="R76"  Part="1"
+AR Path="/5AF84E03/5C384037/6AD31404" Ref="R117"  Part="1"
+AR Path="/5B1FBE47/5B7ED1CC/6AD31404" Ref="R134"  Part="1"
+AR Path="/5B51FFE4/6AD31404" Ref="R163"  Part="1"
+AR Path="/5B6E14C2/6AD31404" Ref="R164"  Part="1"
+AR Path="/5B35E95A/6AD31404" Ref="R165"  Part="1"
+AR Path="/5BB8E174/6AD31404" Ref="R167"  Part="1"
+AR Path="/5BD55BA2/6AD31404" Ref="R168"  Part="1"
+F 0 "R164" V 5468 3800 50  0000 C CNN
 F 1 "820R" V 5559 3800 50  0000 C CNN
-F 2 "" V 5605 3800 50  0001 C CNN
+F 2 "Resistor_SMD:R_0805_2012Metric_Pad1.29x1.40mm_HandSolder" V 5605 3800 50  0001 C CNN
 F 3 "~" H 5675 3800 50  0001 C CNN
+F 4 "" H 0   0   50  0001 C CNN "Spice_Lib_File"
+F 5 "" H 0   0   50  0001 C CNN "Spice_Model"
+F 6 "" H 0   0   50  0001 C CNN "Spice_Netlist_Enabled"
+F 7 "" H 0   0   50  0001 C CNN "Spice_Primitive"
 	1    5675 3800
 	0    1    1    0
 $EndComp
 $Comp
-L Transistor_FET:2N7002 Q?
+L Transistor_FET:2N7002 Q49
 U 1 1 6AD31405
 P 5100 3725
-F 0 "Q?" V 5350 3725 50  0000 C CNN
+AR Path="/5AE74AF7/5C384037/6AD31405" Ref="Q49"  Part="1"
+AR Path="/5AE75BF4/5B58AD87/6AD31405" Ref="Q57"  Part="1"
+AR Path="/5AEA44C6/5C3E9C32/6AD31405" Ref="Q67"  Part="1"
+AR Path="/5AE93FA0/5C3E9C32/6AD31405" Ref="Q76"  Part="1"
+AR Path="/5AF84E03/5C384037/6AD31405" Ref="Q117"  Part="1"
+AR Path="/5B1FBE47/5B7ED1CC/6AD31405" Ref="Q134"  Part="1"
+AR Path="/5B51FFE4/6AD31405" Ref="Q163"  Part="1"
+AR Path="/5B6E14C2/6AD31405" Ref="Q164"  Part="1"
+AR Path="/5B35E95A/6AD31405" Ref="Q165"  Part="1"
+AR Path="/5BB8E174/6AD31405" Ref="Q167"  Part="1"
+AR Path="/5BD55BA2/6AD31405" Ref="Q168"  Part="1"
+F 0 "Q164" V 5350 3725 50  0000 C CNN
 F 1 "2N7002" V 5441 3725 50  0000 C CNN
 F 2 "Package_TO_SOT_SMD:SOT-23" H 5300 3650 50  0001 L CIN
 F 3 "https://www.fairchildsemi.com/datasheets/2N/2N7002.pdf" H 5100 3725 50  0001 L CNN
+F 4 "" H 0   0   50  0001 C CNN "Spice_Lib_File"
+F 5 "" H 0   0   50  0001 C CNN "Spice_Model"
+F 6 "" H 0   0   50  0001 C CNN "Spice_Netlist_Enabled"
+F 7 "" H 0   0   50  0001 C CNN "Spice_Primitive"
 	1    5100 3725
 	0    1    1    0
 $EndComp
 $Comp
-L Alu-rescue:GND-power #PWR?
+L Alu-rescue:GND-power #PWR0301
 U 1 1 6AD31406
 P 4450 3850
-F 0 "#PWR?" H 4450 3850 30  0001 C CNN
+AR Path="/5AE74AF7/5C384037/6AD31406" Ref="#PWR0301"  Part="1"
+AR Path="/5AE75BF4/5B58AD87/6AD31406" Ref="#PWR0317"  Part="1"
+AR Path="/5AEA44C6/5C3E9C32/6AD31406" Ref="#PWR0337"  Part="1"
+AR Path="/5AE93FA0/5C3E9C32/6AD31406" Ref="#PWR0355"  Part="1"
+AR Path="/5AF84E03/5C384037/6AD31406" Ref="#PWR0437"  Part="1"
+AR Path="/5B1FBE47/5B7ED1CC/6AD31406" Ref="#PWR0471"  Part="1"
+AR Path="/5B51FFE4/6AD31406" Ref="#PWR0529"  Part="1"
+AR Path="/5B6E14C2/6AD31406" Ref="#PWR0531"  Part="1"
+AR Path="/5B35E95A/6AD31406" Ref="#PWR0533"  Part="1"
+AR Path="/5BB8E174/6AD31406" Ref="#PWR0537"  Part="1"
+AR Path="/5BD55BA2/6AD31406" Ref="#PWR0539"  Part="1"
+F 0 "#PWR0531" H 4450 3850 30  0001 C CNN
 F 1 "GND-power" H 4450 3780 30  0001 C CNN
 F 2 "" H 4450 3850 50  0001 C CNN
@@
 	4900 3850 4900 3825
 $Comp
-L Device:LED D?
+L Device:LED D49
 U 1 1 6AD31407
 P 6200 3800
-F 0 "D?" H 6191 3545 50  0000 C CNN
+AR Path="/5AE74AF7/5C384037/6AD31407" Ref="D49"  Part="1"
+AR Path="/5AE75BF4/5B58AD87/6AD31407" Ref="D57"  Part="1"
+AR Path="/5AEA44C6/5C3E9C32/6AD31407" Ref="D67"  Part="1"
+AR Path="/5AE93FA0/5C3E9C32/6AD31407" Ref="D76"  Part="1"
+AR Path="/5AF84E03/5C384037/6AD31407" Ref="D117"  Part="1"
+AR Path="/5B1FBE47/5B7ED1CC/6AD31407" Ref="D134"  Part="1"
+AR Path="/5B51FFE4/6AD31407" Ref="D163"  Part="1"
+AR Path="/5B6E14C2/6AD31407" Ref="D164"  Part="1"
+AR Path="/5B35E95A/6AD31407" Ref="D165"  Part="1"
+AR Path="/5BB8E174/6AD31407" Ref="D167"  Part="1"
+AR Path="/5BD55BA2/6AD31407" Ref="D168"  Part="1"
+F 0 "D164" H 6191 3545 50  0000 C CNN
 F 1 "BLUE" H 6191 3636 50  0000 C CNN
-F 2 "" H 6200 3800 50  0001 C CNN
+F 2 "LED_SMD:LED_0805_2012Metric_Pad1.12x1.40mm_HandSolder" H 6200 3800 50  0001 C CNN
 F 3 "~" H 6200 3800 50  0001 C CNN
+F 4 "" H 0   0   50  0001 C CNN "Spice_Lib_File"
+F 5 "" H 0   0   50  0001 C CNN "Spice_Model"
+F 6 "" H 0   0   50  0001 C CNN "Spice_Netlist_Enabled"
+F 7 "" H 0   0   50  0001 C CNN "Spice_Primitive"
 	1    6200 3800
 	1    0    0    1
@@
 	5825 3800 6050 3800
 $Comp
-L power:VCC #PWR?
+L power:VCC #PWR0302
 U 1 1 6AD31408
 P 6525 3800
-F 0 "#PWR?" H 6525 3650 50  0001 C CNN
+AR Path="/5AE74AF7/5C384037/6AD31408" Ref="#PWR0302"  Part="1"
+AR Path="/5AE75BF4/5B58AD87/6AD31408" Ref="#PWR0318"  Part="1"
+AR Path="/5AEA44C6/5C3E9C32/6AD31408" Ref="#PWR0338"  Part="1"
+AR Path="/5AE93FA0/5C3E9C32/6AD31408" Ref="#PWR0356"  Part="1"
+AR Path="/5AF84E03/5C384037/6AD31408" Ref="#PWR0438"  Part="1"
+AR Path="/5B1FBE47/5B7ED1CC/6AD31408" Ref="#PWR0472"  Part="1"
+AR Path="/5B51FFE4/6AD31408" Ref="#PWR0530"  Part="1"
+AR Path="/5B6E14C2/6AD31408" Ref="#PWR0532"  Part="1"
+AR Path="/5B35E95A/6AD31408" Ref="#PWR0534"  Part="1"
+AR Path="/5BB8E174/6AD31408" Ref="#PWR0538"  Part="1"
+AR Path="/5BD55BA2/6AD31408" Ref="#PWR0540"  Part="1"
+F 0 "#PWR0532" H 6525 3650 50  0001 C CNN
 F 1 "VCC" H 6542 3973 50  0000 C CNN
 F 2 "" H 6525 3800 50  0001 C CNN

Commit message: started routing
Changed lines of the file:
@@
 AR Path="/5BB8E174/6AD31404" Ref="R167"  Part="1"
 AR Path="/5BD55BA2/6AD31404" Ref="R168"  Part="1"
-F 0 "R164" V 5468 3800 50  0000 C CNN
+F 0 "R168" V 5468 3800 50  0000 C CNN
 F 1 "820R" V 5559 3800 50  0000 C CNN
 F 2 "Resistor_SMD:R_0805_2012Metric_Pad1.29x1.40mm_HandSolder" V 5605 3800 50  0001 C CNN
@@
 AR Path="/5BB8E174/6AD31405" Ref="Q167"  Part="1"
 AR Path="/5BD55BA2/6AD31405" Ref="Q168"  Part="1"
-F 0 "Q164" V 5350 3725 50  0000 C CNN
+F 0 "Q168" V 5350 3725 50  0000 C CNN
 F 1 "2N7002" V 5441 3725 50  0000 C CNN
 F 2 "Package_TO_SOT_SMD:SOT-23" H 5300 3650 50  0001 L CIN
@@
 AR Path="/5BB8E174/6AD31406" Ref="#PWR0537"  Part="1"
 AR Path="/5BD55BA2/6AD31406" Ref="#PWR0539"  Part="1"
-F 0 "#PWR0531" H 4450 3850 30  0001 C CNN
+F 0 "#PWR0539" H 4450 3850 30  0001 C CNN
 F 1 "GND-power" H 4450 3780 30  0001 C CNN
 F 2 "" H 4450 3850 50  0001 C CNN
@@
 AR Path="/5BB8E174/6AD31407" Ref="D167"  Part="1"
 AR Path="/5BD55BA2/6AD31407" Ref="D168"  Part="1"
-F 0 "D164" H 6191 3545 50  0000 C CNN
+F 0 "D168" H 6191 3545 50  0000 C CNN
 F 1 "BLUE" H 6191 3636 50  0000 C CNN
 F 2 "LED_SMD:LED_0805_2012Metric_Pad1.12x1.40mm_HandSolder" H 6200 3800 50  0001 C CNN
@@
 AR Path="/5BB8E174/6AD31408" Ref="#PWR0538"  Part="1"
 AR Path="/5BD55BA2/6AD31408" Ref="#PWR0540"  Part="1"
-F 0 "#PWR0532" H 6525 3650 50  0001 C CNN
+F 0 "#PWR0540" H 6525 3650 50  0001 C CNN
 F 1 "VCC" H 6542 3973 50  0000 C CNN
 F 2 "" H 6525 3800 50  0001 C CNN

Commit message: coniued layouting
Changed lines of the file:
@@
 $Descr A4 11693 8268
 encoding utf-8
-Sheet 187 191
+Sheet 56 191
 Title ""
 Date ""
@@
 AR Path="/5BB8E174/6AD31404" Ref="R167"  Part="1"
 AR Path="/5BD55BA2/6AD31404" Ref="R168"  Part="1"
-F 0 "R168" V 5468 3800 50  0000 C CNN
+F 0 "R57" V 5468 3800 50  0000 C CNN
 F 1 "820R" V 5559 3800 50  0000 C CNN
 F 2 "Resistor_SMD:R_0805_2012Metric_Pad1.29x1.40mm_HandSolder" V 5605 3800 50  0001 C CNN
@@
 AR Path="/5BB8E174/6AD31405" Ref="Q167"  Part="1"
 AR Path="/5BD55BA2/6AD31405" Ref="Q168"  Part="1"
-F 0 "Q168" V 5350 3725 50  0000 C CNN
+F 0 "Q57" V 5350 3725 50  0000 C CNN
 F 1 "2N7002" V 5441 3725 50  0000 C CNN
 F 2 "Package_TO_SOT_SMD:SOT-23" H 5300 3650 50  0001 L CIN
@@
 AR Path="/5BB8E174/6AD31406" Ref="#PWR0537"  Part="1"
 AR Path="/5BD55BA2/6AD31406" Ref="#PWR0539"  Part="1"
-F 0 "#PWR0539" H 4450 3850 30  0001 C CNN
+F 0 "#PWR0317" H 4450 3850 30  0001 C CNN
 F 1 "GND-power" H 4450 3780 30  0001 C CNN
 F 2 "" H 4450 3850 50  0001 C CNN
@@
 AR Path="/5BB8E174/6AD31407" Ref="D167"  Part="1"
 AR Path="/5BD55BA2/6AD31407" Ref="D168"  Part="1"
-F 0 "D168" H 6191 3545 50  0000 C CNN
+F 0 "D57" H 6191 3545 50  0000 C CNN
 F 1 "BLUE" H 6191 3636 50  0000 C CNN
 F 2 "LED_SMD:LED_0805_2012Metric_Pad1.12x1.40mm_HandSolder" H 6200 3800 50  0001 C CNN
@@
 AR Path="/5BB8E174/6AD31408" Ref="#PWR0538"  Part="1"
 AR Path="/5BD55BA2/6AD31408" Ref="#PWR0540"  Part="1"
-F 0 "#PWR0540" H 6525 3650 50  0001 C CNN
+F 0 "#PWR0318" H 6525 3650 50  0001 C CNN
 F 1 "VCC" H 6542 3973 50  0000 C CNN
 F 2 "" H 6525 3800 50  0001 C CNN

Commit message: started routing :)
Changed lines of the file:
@@
 $Descr A4 11693 8268
 encoding utf-8
-Sheet 56 191
+Sheet 187 191
 Title ""
 Date ""
@@
 AR Path="/5BB8E174/6AD31404" Ref="R167"  Part="1"
 AR Path="/5BD55BA2/6AD31404" Ref="R168"  Part="1"
-F 0 "R57" V 5468 3800 50  0000 C CNN
+F 0 "R168" V 5468 3800 50  0000 C CNN
 F 1 "820R" V 5559 3800 50  0000 C CNN
 F 2 "Resistor_SMD:R_0805_2012Metric_Pad1.29x1.40mm_HandSolder" V 5605 3800 50  0001 C CNN
@@
 AR Path="/5BB8E174/6AD31405" Ref="Q167"  Part="1"
 AR Path="/5BD55BA2/6AD31405" Ref="Q168"  Part="1"
-F 0 "Q57" V 5350 3725 50  0000 C CNN
+F 0 "Q168" V 5350 3725 50  0000 C CNN
 F 1 "2N7002" V 5441 3725 50  0000 C CNN
 F 2 "Package_TO_SOT_SMD:SOT-23" H 5300 3650 50  0001 L CIN
@@
 AR Path="/5BB8E174/6AD31406" Ref="#PWR0537"  Part="1"
 AR Path="/5BD55BA2/6AD31406" Ref="#PWR0539"  Part="1"
-F 0 "#PWR0317" H 4450 3850 30  0001 C CNN
+F 0 "#PWR0539" H 4450 3850 30  0001 C CNN
 F 1 "GND-power" H 4450 3780 30  0001 C CNN
 F 2 "" H 4450 3850 50  0001 C CNN
@@
 AR Path="/5BB8E174/6AD31407" Ref="D167"  Part="1"
 AR Path="/5BD55BA2/6AD31407" Ref="D168"  Part="1"
-F 0 "D57" H 6191 3545 50  0000 C CNN
+F 0 "D168" H 6191 3545 50  0000 C CNN
 F 1 "BLUE" H 6191 3636 50  0000 C CNN
 F 2 "LED_SMD:LED_0805_2012Metric_Pad1.12x1.40mm_HandSolder" H 6200 3800 50  0001 C CNN
@@
 AR Path="/5BB8E174/6AD31408" Ref="#PWR0538"  Part="1"
 AR Path="/5BD55BA2/6AD31408" Ref="#PWR0540"  Part="1"
-F 0 "#PWR0318" H 6525 3650 50  0001 C CNN
+F 0 "#PWR0540" H 6525 3650 50  0001 C CNN
 F 1 "VCC" H 6542 3973 50  0000 C CNN
 F 2 "" H 6525 3800 50  0001 C CNN
