File: Alu/Alu.sch (KiCad schematic (older format))
At the start: 9 parts, among them J1 Conn_01x34, J2 Barrel_Jack, U1 74LS08, U2 74LS32, U3 74LS32, U4 74LS32

Commit message: footprints
Parts:
- removed U2, U3, U4: 74LS32, symbol 74xx:74LS32
- added U2, U3: 74HC02, Package_SO:SOIC-14_3.9x8.7mm_P1.27mm, symbol 74xx:74HC02
- C1, C70, C71: footprint (none) -> Capacitor_SMD:C_0805_2012Metric
Connections:
- wire segments 1262 -> 1272

Commit message: started routing
Parts:
- J1: footprint (none) -> Connector_PinHeader_2.54mm:PinHeader_1x34_P2.54mm_Vertical_SMD_Pin1Right
- J2: footprint (none) -> Connector_BarrelJack:BarrelJack_Horizontal
- U1: footprint (none) -> Package_SO:SOIC-14_3.9x8.7mm_P1.27mm
Connections:
- net labels removed: Zflag
- wire segments 1272 -> 1271
- no-connect marks 5 -> 4
Changed lines of the file:
@@
 F 0 "U1" H 3100 19163 60  0000 C CNN
 F 1 "74LS08" H 3100 19057 60  0000 C CNN
-F 2 "" H 3100 18775 60  0001 C CNN
+F 2 "Package_SO:SOIC-14_3.9x8.7mm_P1.27mm" H 3100 18775 60  0001 C CNN
 F 3 "" H 3100 18775 60  0001 C CNN
 F 4 "" H 0   0   50  0001 C CNN "Spice_Lib_File"
@@
 F 0 "U1" H 3125 19913 60  0000 C CNN
 F 1 "74LS08" H 3125 19807 60  0000 C CNN
-F 2 "" H 3125 19525 60  0001 C CNN
+F 2 "Package_SO:SOIC-14_3.9x8.7mm_P1.27mm" H 3125 19525 60  0001 C CNN
 F 3 "" H 3125 19525 60  0001 C CNN
 F 4 "" H 0   0   50  0001 C CNN "Spice_Lib_File"
@@
 F 0 "U1" H 3250 20538 60  0000 C CNN
 F 1 "74LS08" H 3250 20432 60  0000 C CNN
-F 2 "" H 3250 20150 60  0001 C CNN
+F 2 "Package_SO:SOIC-14_3.9x8.7mm_P1.27mm" H 3250 20150 60  0001 C CNN
 F 3 "" H 3250 20150 60  0001 C CNN
 F 4 "" H 0   0   50  0001 C CNN "Spice_Lib_File"
@@
 F 0 "U1" H 3225 21188 60  0000 C CNN
 F 1 "74LS08" H 3225 21082 60  0000 C CNN
-F 2 "" H 3225 20800 60  0001 C CNN
+F 2 "Package_SO:SOIC-14_3.9x8.7mm_P1.27mm" H 3225 20800 60  0001 C CNN
 F 3 "" H 3225 20800 60  0001 C CNN
 F 4 "" H 0   0   50  0001 C CNN "Spice_Lib_File"
@@
 Wire Wire Line
 	26350 11900 26350 11925
-NoConn ~ 11000 8325
 Wire Wire Line
 	21200 5900 21200 5750
@@
 F 0 "U1" V 3492 22025 50  0000 C CNN
 F 1 "74LS08" V 3401 22025 50  0000 C CNN
-F 2 "" H 3125 22025 50  0001 C CNN
+F 2 "Package_SO:SOIC-14_3.9x8.7mm_P1.27mm" H 3125 22025 50  0001 C CNN
 F 3 "http://www.ti.com/lit/gpn/sn74LS08" H 3125 22025 50  0001 C CNN
 F 4 "" H 0   0   50  0001 C CNN "Spice_Lib_File"
@@
 	24650 8325 24650 8675
 Connection ~ 24500 8075
-Wire Wire Line
-	24500 8075 24625 8075
 Wire Wire Line
 	23175 8725 23250 8725
@@
 F 0 "J1" H 1995 4975 50  0000 C CNN
 F 1 "Conn_01x34" H 1995 5066 50  0000 C CNN
-F 2 "" H 2075 6900 50  0001 C CNN
+F 2 "Connector_PinHeader_2.54mm:PinHeader_1x34_P2.54mm_Vertical_SMD_Pin1Right" H 2075 6900 50  0001 C CNN
 F 3 "~" H 2075 6900 50  0001 C CNN
 F 4 "" H 0   0   50  0001 C CNN "Spice_Lib_File"
@@
 F 0 "J2" H 29365 11277 50  0000 R CNN
 F 1 "Barrel_Jack" H 29365 11368 50  0000 R CNN
-F 2 "" H 29600 11260 50  0001 C CNN
+F 2 "Connector_BarrelJack:BarrelJack_Horizontal" H 29600 11260 50  0001 C CNN
 F 3 "~" H 29600 11260 50  0001 C CNN
 F 4 "" H 0   0   50  0001 C CNN "Spice_Lib_File"
@@
 	975  14025 975  14050
 Text Label 800  14400 2    50   ~ 0
-Zflag
+ZFlag
 Wire Wire Line
 	800  14400 975  14400
@@
 $EndComp
 Wire Wire Line
-	24625 8075 24675 8075
-Wire Wire Line
 	24675 8075 24675 7875
-Connection ~ 24625 8075
-Wire Wire Line
-	24625 8075 24675 8075
 Connection ~ 24675 8075
 $Comp
@@
 	0    1    1    0
 $EndComp
+Wire Wire Line
+	24625 8075 24675 8075
+Wire Wire Line
+	24500 8075 24675 8075
 $EndSCHEMATC

Commit message: started routing :)
Parts:
- removed J1: Conn_01x34, Connector_PinHeader_2.54mm:PinHeader_1x34_P2.54mm_Vertical_SMD_Pin1Right, symbol Connector_Generic:Conn_01x34
- added J1, J10, J11, J12, J13, J3, J5, J6, J7, J9, J?: Conn_01x08, Connector_PinHeader_2.54mm:PinHeader_1x08_P2.54mm_Vertical_SMD_Pin1Right, symbol Connector_Generic:Conn_01x08
- added J4, J8: Conn_01x18, Connector_PinHeader_2.54mm:PinHeader_1x18_P2.54mm_Vertical_SMD_Pin1Left, symbol Connector_Generic:Conn_01x18
Connections:
- wire segments 1271 -> 1435

Commit message: split pcbs
Parts:
- added J15, J18: Conn_01x02_Male, Connector_PinHeader_2.54mm:PinHeader_1x02_P2.54mm_Vertical, symbol Connector:Conn_01x02_Male
- added J16, J17, J19, J20: Conn_01x08, Connector_PinHeader_2.54mm:PinHeader_1x08_P2.54mm_Vertical, symbol Connector_Generic:Conn_01x08
- added R169, R170: 0, Resistor_SMD:R_1206_3216Metric, symbol Device:R
- J1, J10, J11, J12, J13, J3, J5, J6, J7, J9: footprint Connector_PinHeader_2.54mm:PinHeader_1x08_P2.54mm_Vertical_SMD_Pin1Right -> Connector_PinHeader_2.54mm:PinHeader_1x08_P2.54mm_Vertical
- J14: renamed from J?; footprint Connector_PinHeader_2.54mm:PinHeader_1x08_P2.54mm_Vertical_SMD_Pin1Right -> Connector_PinHeader_2.54mm:PinHeader_1x08_P2.54mm_Vertical
- J4, J8: footprint Connector_PinHeader_2.54mm:PinHeader_1x18_P2.54mm_Vertical_SMD_Pin1Left -> Connector_PinHeader_2.54mm:PinHeader_1x18_P2.54mm_Vertical
Connections:
- wire segments 1435 -> 1514
