File: Alu/LED_RED.sch (KiCad schematic (older format))
At the start: 3 parts

Commit message: footprints
Parts:
- removed D?: RED, symbol Device:LED
- removed Q?: 2N7002, Package_TO_SOT_SMD:SOT-23, symbol Transistor_FET:2N7002
- removed R?: 1k, symbol Device:R
- added D1: RED, LED_SMD:LED_0805_2012Metric_Pad1.12x1.40mm_HandSolder, symbol Device:LED
- added Q1: 2N7002, Package_TO_SOT_SMD:SOT-23, symbol Transistor_FET:2N7002
- added R1: 1k, Resistor_SMD:R_0805_2012Metric, symbol Device:R

Commit message: coniued layouting
Changed lines of the file:
@@
 $Descr A4 11693 8268
 encoding utf-8
-Sheet 26 191
+Sheet 57 191
 Title ""
 Date ""
@@
 AR Path="/6823D887/5BF1FBAA" Ref="R153"  Part="1"
 AR Path="/6823D88A/5BF1FBAA" Ref="R154"  Part="1"
-F 0 "R154" V 5468 3800 50  0000 C CNN
+F 0 "R48" V 5468 3800 50  0000 C CNN
 F 1 "1k" V 5559 3800 50  0000 C CNN
 F 2 "Resistor_SMD:R_0805_2012Metric" V 5605 3800 50  0001 C CNN
@@
 AR Path="/6823D887/5BF1FBAB" Ref="Q153"  Part="1"
 AR Path="/6823D88A/5BF1FBAB" Ref="Q154"  Part="1"
-F 0 "Q154" V 5350 3725 50  0000 C CNN
+F 0 "Q48" V 5350 3725 50  0000 C CNN
 F 1 "2N7002" V 5441 3725 50  0000 C CNN
 F 2 "Package_TO_SOT_SMD:SOT-23" H 5300 3650 50  0001 L CIN
@@
 AR Path="/6823D887/5BF1FBAC" Ref="#PWR0509"  Part="1"
 AR Path="/6823D88A/5BF1FBAC" Ref="#PWR0511"  Part="1"
-F 0 "#PWR0511" H 4450 3850 30  0001 C CNN
+F 0 "#PWR0299" H 4450 3850 30  0001 C CNN
 F 1 "GND-power" H 4450 3780 30  0001 C CNN
 F 2 "" H 4450 3850 50  0001 C CNN
@@
 AR Path="/6823D887/5BF1FBAD" Ref="D153"  Part="1"
 AR Path="/6823D88A/5BF1FBAD" Ref="D154"  Part="1"
-F 0 "D154" H 6191 3545 50  0000 C CNN
+F 0 "D48" H 6191 3545 50  0000 C CNN
 F 1 "RED" H 6191 3636 50  0000 C CNN
 F 2 "LED_SMD:LED_0805_2012Metric_Pad1.12x1.40mm_HandSolder" H 6200 3800 50  0001 C CNN
@@
 AR Path="/6823D887/5BF1FBAE" Ref="#PWR0510"  Part="1"
 AR Path="/6823D88A/5BF1FBAE" Ref="#PWR0512"  Part="1"
-F 0 "#PWR0512" H 6525 3650 50  0001 C CNN
+F 0 "#PWR0300" H 6525 3650 50  0001 C CNN
 F 1 "VCC" H 6542 3973 50  0000 C CNN
 F 2 "" H 6525 3800 50  0001 C CNN

Commit message: started routing :)
Changed lines of the file:
@@
 $Descr A4 11693 8268
 encoding utf-8
-Sheet 57 191
+Sheet 177 191
 Title ""
 Date ""
@@
 AR Path="/6823D887/5BF1FBAA" Ref="R153"  Part="1"
 AR Path="/6823D88A/5BF1FBAA" Ref="R154"  Part="1"
-F 0 "R48" V 5468 3800 50  0000 C CNN
+F 0 "R152" V 5468 3800 50  0000 C CNN
 F 1 "1k" V 5559 3800 50  0000 C CNN
 F 2 "Resistor_SMD:R_0805_2012Metric" V 5605 3800 50  0001 C CNN
@@
 AR Path="/6823D887/5BF1FBAB" Ref="Q153"  Part="1"
 AR Path="/6823D88A/5BF1FBAB" Ref="Q154"  Part="1"
-F 0 "Q48" V 5350 3725 50  0000 C CNN
+F 0 "Q152" V 5350 3725 50  0000 C CNN
 F 1 "2N7002" V 5441 3725 50  0000 C CNN
 F 2 "Package_TO_SOT_SMD:SOT-23" H 5300 3650 50  0001 L CIN
@@
 AR Path="/6823D887/5BF1FBAC" Ref="#PWR0509"  Part="1"
 AR Path="/6823D88A/5BF1FBAC" Ref="#PWR0511"  Part="1"
-F 0 "#PWR0299" H 4450 3850 30  0001 C CNN
+F 0 "#PWR0507" H 4450 3850 30  0001 C CNN
 F 1 "GND-power" H 4450 3780 30  0001 C CNN
 F 2 "" H 4450 3850 50  0001 C CNN
@@
 AR Path="/6823D887/5BF1FBAD" Ref="D153"  Part="1"
 AR Path="/6823D88A/5BF1FBAD" Ref="D154"  Part="1"
-F 0 "D48" H 6191 3545 50  0000 C CNN
+F 0 "D152" H 6191 3545 50  0000 C CNN
 F 1 "RED" H 6191 3636 50  0000 C CNN
 F 2 "LED_SMD:LED_0805_2012Metric_Pad1.12x1.40mm_HandSolder" H 6200 3800 50  0001 C CNN
@@
 AR Path="/6823D887/5BF1FBAE" Ref="#PWR0510"  Part="1"
 AR Path="/6823D88A/5BF1FBAE" Ref="#PWR0512"  Part="1"
-F 0 "#PWR0300" H 6525 3650 50  0001 C CNN
+F 0 "#PWR0508" H 6525 3650 50  0001 C CNN
 F 1 "VCC" H 6542 3973 50  0000 C CNN
 F 2 "" H 6525 3800 50  0001 C CNN
