File: Alu/NOT_0.sch (KiCad schematic (older format))
At the start: 7 parts, among them U38 74HC04, U39 74HC04

Commit message: split pcbs
Parts:
- removed R96: 0, Resistor_SMD:R_1806_4516Metric, symbol Device:R
- removed unit 1 of U38
- removed unit 2 of U38
- removed unit 3 of U38
- removed unit 5 of U38
- removed unit 6 of U38
- removed unit 1 of U39
- removed unit 3 of U39
- removed unit 4 of U39
- removed unit 7 of U39
- added R157: 0, Resistor_SMD:R_1806_4516Metric, symbol Device:R
- added unit 1 of U41
- added unit 2 of U41
- added unit 3 of U41
- added unit 5 of U41
- added unit 6 of U41
- added unit 1 of U42
- added unit 3 of U42
- added unit 4 of U42
- added unit 7 of U42
- renumbered R98 to R155, R97 to R158, U38 to U41, U39 to U42
