File: Alu/XOR.sch (KiCad schematic (older format))
At the start: 4 parts, among them U43 74HC86, U44 74HC86

Commit message: footprints
Parts:
- C10, C11: footprint (none) -> Capacitor_SMD:C_0805_2012Metric
- U43, U44: footprint (none) -> Package_SO:SOIC-14_3.9x8.7mm_P1.27mm
Connections:
- wire segments 91 -> 89
Changed lines of the file:
@@
 $Descr A4 11693 8268
 encoding utf-8
-Sheet 38 156
+Sheet 29 191
 Title ""
 Date ""
@@
 F 0 "U43" V 2446 2595 50  0000 R CNN
 F 1 "74HC86" V 2355 2595 50  0000 R CNN
-F 2 "" H 2400 2775 50  0001 C CNN
+F 2 "Package_SO:SOIC-14_3.9x8.7mm_P1.27mm" H 2400 2775 50  0001 C CNN
 F 3 "http://www.ti.com/lit/gpn/sn74HC86" H 2400 2775 50  0001 C CNN
+F 4 "" H 0   0   50  0001 C CNN "Spice_Lib_File"
+F 5 "" H 0   0   50  0001 C CNN "Spice_Model"
+F 6 "" H 0   0   50  0001 C CNN "Spice_Netlist_Enabled"
+F 7 "" H 0   0   50  0001 C CNN "Spice_Primitive"
 	1    2400 2775
 	0    -1   -1   0
@@
 F 0 "U43" V 3146 2595 50  0000 R CNN
 F 1 "74HC86" V 3055 2595 50  0000 R CNN
-F 2 "" H 3100 2775 50  0001 C CNN
+F 2 "Package_SO:SOIC-14_3.9x8.7mm_P1.27mm" H 3100 2775 50  0001 C CNN
 F 3 "http://www.ti.com/lit/gpn/sn74HC86" H 3100 2775 50  0001 C CNN
+F 4 "" H 0   0   50  0001 C CNN "Spice_Lib_File"
+F 5 "" H 0   0   50  0001 C CNN "Spice_Model"
+F 6 "" H 0   0   50  0001 C CNN "Spice_Netlist_Enabled"
+F 7 "" H 0   0   50  0001 C CNN "Spice_Primitive"
 	2    3100 2775
 	0    -1   -1   0
@@
 F 0 "U43" V 3896 2595 50  0000 R CNN
 F 1 "74HC86" V 3805 2595 50  0000 R CNN
-F 2 "" H 3850 2775 50  0001 C CNN
+F 2 "Package_SO:SOIC-14_3.9x8.7mm_P1.27mm" H 3850 2775 50  0001 C CNN
 F 3 "http://www.ti.com/lit/gpn/sn74HC86" H 3850 2775 50  0001 C CNN
+F 4 "" H 0   0   50  0001 C CNN "Spice_Lib_File"
+F 5 "" H 0   0   50  0001 C CNN "Spice_Model"
+F 6 "" H 0   0   50  0001 C CNN "Spice_Netlist_Enabled"
+F 7 "" H 0   0   50  0001 C CNN "Spice_Primitive"
 	3    3850 2775
 	0    -1   -1   0
@@
 F 0 "U43" V 4671 2595 50  0000 R CNN
 F 1 "74HC86" V 4580 2595 50  0000 R CNN
-F 2 "" H 4625 2775 50  0001 C CNN
+F 2 "Package_SO:SOIC-14_3.9x8.7mm_P1.27mm" H 4625 2775 50  0001 C CNN
 F 3 "http://www.ti.com/lit/gpn/sn74HC86" H 4625 2775 50  0001 C CNN
+F 4 "" H 0   0   50  0001 C CNN "Spice_Lib_File"
+F 5 "" H 0   0   50  0001 C CNN "Spice_Model"
+F 6 "" H 0   0   50  0001 C CNN "Spice_Netlist_Enabled"
+F 7 "" H 0   0   50  0001 C CNN "Spice_Primitive"
 	4    4625 2775
 	0    -1   -1   0
@@
 F 0 "U43" H 9330 3771 50  0000 L CNN
 F 1 "74HC86" H 9330 3680 50  0000 L CNN
-F 2 "" H 9100 3725 50  0001 C CNN
+F 2 "Package_SO:SOIC-14_3.9x8.7mm_P1.27mm" H 9100 3725 50  0001 C CNN
 F 3 "http://www.ti.com/lit/gpn/sn74HC86" H 9100 3725 50  0001 C CNN
+F 4 "" H 0   0   50  0001 C CNN "Spice_Lib_File"
+F 5 "" H 0   0   50  0001 C CNN "Spice_Model"
+F 6 "" H 0   0   50  0001 C CNN "Spice_Netlist_Enabled"
+F 7 "" H 0   0   50  0001 C CNN "Spice_Primitive"
 	5    9100 3725
 	1    0    0    -1
@@
 F 0 "U44" V 5546 2570 50  0000 R CNN
 F 1 "74HC86" V 5455 2570 50  0000 R CNN
-F 2 "" H 5500 2750 50  0001 C CNN
-F 3 "http://www.ti.com/lit/gpn/sn74HC86" H 5500 2750 50  0001 C CNN
+F 2 "Package_SO:SOIC-14_3.9x8.7mm_P1.27mm" H 5500 2750 50  0001 C CNN
+F 3 "" H 5500 2750 50  0001 C CNN
+F 4 "" H 0   0   50  0001 C CNN "Spice_Lib_File"
+F 5 "" H 0   0   50  0001 C CNN "Spice_Model"
+F 6 "" H 0   0   50  0001 C CNN "Spice_Netlist_Enabled"
+F 7 "" H 0   0   50  0001 C CNN "Spice_Primitive"
 	1    5500 2750
 	0    -1   -1   0
@@
 F 0 "U44" V 6246 2570 50  0000 R CNN
 F 1 "74HC86" V 6155 2570 50  0000 R CNN
-F 2 "" H 6200 2750 50  0001 C CNN
+F 2 "Package_SO:SOIC-14_3.9x8.7mm_P1.27mm" H 6200 2750 50  0001 C CNN
 F 3 "http://www.ti.com/lit/gpn/sn74HC86" H 6200 2750 50  0001 C CNN
+F 4 "" H 0   0   50  0001 C CNN "Spice_Lib_File"
+F 5 "" H 0   0   50  0001 C CNN "Spice_Model"
+F 6 "" H 0   0   50  0001 C CNN "Spice_Netlist_Enabled"
+F 7 "" H 0   0   50  0001 C CNN "Spice_Primitive"
 	2    6200 2750
 	0    -1   -1   0
@@
 F 0 "U44" V 6996 2570 50  0000 R CNN
 F 1 "74HC86" V 6905 2570 50  0000 R CNN
-F 2 "" H 6950 2750 50  0001 C CNN
+F 2 "Package_SO:SOIC-14_3.9x8.7mm_P1.27mm" H 6950 2750 50  0001 C CNN
 F 3 "http://www.ti.com/lit/gpn/sn74HC86" H 6950 2750 50  0001 C CNN
+F 4 "" H 0   0   50  0001 C CNN "Spice_Lib_File"
+F 5 "" H 0   0   50  0001 C CNN "Spice_Model"
+F 6 "" H 0   0   50  0001 C CNN "Spice_Netlist_Enabled"
+F 7 "" H 0   0   50  0001 C CNN "Spice_Primitive"
 	3    6950 2750
 	0    -1   -1   0
@@
 F 0 "U44" V 7721 2595 50  0000 R CNN
 F 1 "74HC86" V 7630 2595 50  0000 R CNN
-F 2 "" H 7675 2775 50  0001 C CNN
+F 2 "Package_SO:SOIC-14_3.9x8.7mm_P1.27mm" H 7675 2775 50  0001 C CNN
 F 3 "http://www.ti.com/lit/gpn/sn74HC86" H 7675 2775 50  0001 C CNN
+F 4 "" H 0   0   50  0001 C CNN "Spice_Lib_File"
+F 5 "" H 0   0   50  0001 C CNN "Spice_Model"
+F 6 "" H 0   0   50  0001 C CNN "Spice_Netlist_Enabled"
+F 7 "" H 0   0   50  0001 C CNN "Spice_Primitive"
 	4    7675 2775
 	0    -1   -1   0
@@
 F 0 "U44" H 10580 3771 50  0000 L CNN
 F 1 "74HC86" H 10580 3680 50  0000 L CNN
-F 2 "" H 10350 3725 50  0001 C CNN
+F 2 "Package_SO:SOIC-14_3.9x8.7mm_P1.27mm" H 10350 3725 50  0001 C CNN
 F 3 "http://www.ti.com/lit/gpn/sn74HC86" H 10350 3725 50  0001 C CNN
+F 4 "" H 0   0   50  0001 C CNN "Spice_Lib_File"
+F 5 "" H 0   0   50  0001 C CNN "Spice_Model"
+F 6 "" H 0   0   50  0001 C CNN "Spice_Netlist_Enabled"
+F 7 "" H 0   0   50  0001 C CNN "Spice_Primitive"
 	5    10350 3725
 	1    0    0    -1
@@
 Wire Wire Line
 	7675 2475 7675 2225
-Wire Wire Line
-	7675 2225 7575 2225
 Wire Wire Line
 	7425 2225 7425 2050
@@
 F 0 "C10" H 8642 3796 50  0000 L CNN
 F 1 "100nF" H 8642 3705 50  0000 L CNN
-F 2 "" H 8550 3750 50  0001 C CNN
+F 2 "Capacitor_SMD:C_0805_2012Metric" H 8550 3750 50  0001 C CNN
 F 3 "~" H 8550 3750 50  0001 C CNN
+F 4 "" H 0   0   50  0001 C CNN "Spice_Lib_File"
+F 5 "" H 0   0   50  0001 C CNN "Spice_Model"
+F 6 "" H 0   0   50  0001 C CNN "Spice_Netlist_Enabled"
+F 7 "" H 0   0   50  0001 C CNN "Spice_Primitive"
 	1    8550 3750
 	1    0    0    -1
@@
 F 0 "C11" H 11017 3771 50  0000 L CNN
 F 1 "100nF" H 11017 3680 50  0000 L CNN
-F 2 "" H 10925 3725 50  0001 C CNN
+F 2 "Capacitor_SMD:C_0805_2012Metric" H 10925 3725 50  0001 C CNN
 F 3 "~" H 10925 3725 50  0001 C CNN
+F 4 "" H 0   0   50  0001 C CNN "Spice_Lib_File"
+F 5 "" H 0   0   50  0001 C CNN "Spice_Model"
+F 6 "" H 0   0   50  0001 C CNN "Spice_Netlist_Enabled"
+F 7 "" H 0   0   50  0001 C CNN "Spice_Primitive"
 	1    10925 3725
 	1    0    0    -1
@@
 Wire Wire Line
 	7675 1625 7675 2225
-Wire Wire Line
-	7675 2225 7575 2225
 Connection ~ 7675 2225
-Connection ~ 7575 2225
-Wire Wire Line
-	7575 2225 7425 2225
+Wire Wire Line
+	7425 2225 7675 2225
 $EndSCHEMATC

Commit message: split pcbs
Parts:
- added R161: 0, Resistor_SMD:R_1206_3216Metric, symbol Device:R
Connections:
- wire segments 89 -> 92
Changed lines of the file:
@@
 Wire Wire Line
 	3075 2250 3075 2475
-Wire Wire Line
-	3650 1550 3650 2225
-Wire Wire Line
-	3650 2225 4000 2225
 Connection ~ 4000 2225
 Wire Wire Line
@@
 Wire Wire Line
 	7425 2225 7675 2225
+$Comp
+L Device:R R161
+U 1 1 5FBC962A
+P 3625 1875
+F 0 "R161" H 3695 1921 50  0000 L CNN
+F 1 "0" H 3695 1830 50  0000 L CNN
+F 2 "Resistor_SMD:R_1206_3216Metric" V 3555 1875 50  0001 C CNN
+F 3 "~" H 3625 1875 50  0001 C CNN
+	1    3625 1875
+	1    0    0    -1
+$EndComp
+Wire Wire Line
+	3625 1725 3625 1625
+Wire Wire Line
+	3625 1625 3650 1625
+Wire Wire Line
+	3650 1625 3650 1550
+Wire Wire Line
+	3625 2025 3625 2225
+Wire Wire Line
+	3625 2225 4000 2225
 $EndSCHEMATC
