File: Alu/DEC/DEC.sch (KiCad schematic (older format))
At the start: 4 parts, among them U47 74LS283, U48 74LS283

Commit message: split pcbs
Parts:
- added J1: Conn_01x08, Connector_PinHeader_2.54mm:PinHeader_1x08_P2.54mm_Vertical, symbol Connector_Generic:Conn_01x08
- added J2: Conn_01x09, Connector_PinHeader_2.54mm:PinHeader_1x09_P2.54mm_Vertical, symbol Connector_Generic:Conn_01x09
- added J3: Conn_01x02, Connector_PinHeader_2.54mm:PinHeader_1x02_P2.54mm_Vertical, symbol Connector_Generic:Conn_01x02
- added R10, R11, R12: 0, Resistor_SMD:R_1206_3216Metric_Pad1.39x1.80mm_HandSolder, symbol Device:R
- renumbered C6 to C1, C7 to C2, U47 to U1, U48 to U2
Connections:
- net labels added: GND
- net labels removed: GND-power
- wire segments 103 -> 128
