File: Alu/OR/OR.sch (KiCad schematic (older format))
At the start: 7 parts, among them U4 74LS32, U7 74LS32

Commit message: split pcbs
Parts:
- removed R162, R171, R172: 0, Resistor_SMD:R_1206_3216Metric, symbol Device:R
- added J1, J2, J4: Conn_01x08, Connector_PinHeader_2.54mm:PinHeader_1x08_P2.54mm_Vertical, symbol Connector_Generic:Conn_01x08
- added J3: Conn_01x02_Male, Connector_PinHeader_2.54mm:PinHeader_1x02_P2.54mm_Vertical, symbol Connector:Conn_01x02_Male
- added R1, R2, R3: 0, Resistor_SMD:R_1206_3216Metric_Pad1.39x1.80mm_HandSolder, symbol Device:R
- renumbered C4 to C1, C5 to C2, U4 to U1, U7 to U2
Connections:
- net labels added: GND
- net labels removed: GND-power
- wire segments 132 -> 169
